File: hw/krecek-0.9/krecek-0.9.kicad_sch (KiCad schematic)
At the start: 3 parts, among them J1 USB_C_Receptacle_USB2.0, U1 RP2040, U2 W25Q128JVS

Commit message: Expert hardware design *dab*
Parts:
- added C1, C2: 27p, symbol Device:C_Small
- added C3: 100n, symbol Device:C_Small
- added R1, R3: 1k, symbol Device:R_Small
- added R2: 33k, symbol Device:R_Small
- added X1: X322512MSB4SI, LCSC:OSC-SMD_4P-L3.2-W2.5-BL, symbol LCSC:X322512MSB4SI
- J1: footprint (none) -> LCSC:USB-C-SMD_TYPEC-304J-BCP16; LCSC Part (none) -> C2835315
- U1: LCSC Part (none) -> C2040
- U2: LCSC Part (none) -> C97521
Connections:
- net XIN: now reaches U1.20 (XIN)
- net XIN: now also C2.1, X1.1 (OSC1)
- net QSPI_SD3: now reaches U1.51 (QSPI_SD3)
- net QSPI_SD3: now also U2.7 (IO3)
- net QSPI_SCLK: now reaches U1.52 (QSPI_SCLK)
- net QSPI_SCLK: now also U2.6 (CLK)
- net QSPI_SD0: now reaches U1.53 (QSPI_SD0)
- net QSPI_SD0: now also U2.5 (DI(IO0))
- net QSPI_SD2: now reaches U1.54 (QSPI_SD2)
- net QSPI_SD2: now also U2.3 (IO2)
- net QSPI_SD1: now reaches U1.55 (QSPI_SD1)
- net QSPI_SD1: now also U2.2 (DO(IO1))
- net QSPI_SS: now reaches U1.56 (QSPI_SS)
- net QSPI_SS: now also U2.1 (~{CS}), R2.2, R3.1
- net GND: now reaches U2.4 (GND)
- net GND: now also C1.2, C2.2, C3.2, X1.2 (GND), X1.4 (GND)
- net +3.3V: now reaches U2.8 (VCC)
- net +3.3V: now also C3.1, R2.1
- new net: C1.1, R1.2, X1.3 (OSC2)
- new net XOUT: R1.1
Other:
- moved on the sheet: U2

Commit message: expand design
Parts:
- added U3: BQ24045DSQR, LCSC:WSON-10_L2.0-W2.0-P0.40-BL-EP, symbol LCSC:BQ24045DSQR
Connections:
- new net: U3.11 (VSS), U3.3 (VSS)
Other:
- moved on the sheet: C3, J1, R2, R3, U1, U2

Commit message: assign GPIO pins
Parts:
- removed C1, C2: 27p, symbol Device:C_Small
- removed C3: 100n, symbol Device:C_Small
- removed R1, R3: 1k, symbol Device:R_Small
- removed R2: 33k, symbol Device:R_Small
- removed U1: RP2040, Package_DFN_QFN:QFN-56-1EP_7x7mm_P0.4mm_EP3.2x3.2mm, symbol MCU_RaspberryPi:RP2040
- removed U2: W25Q128JVS, Package_SO:SOIC-8_5.23x5.23mm_P1.27mm, symbol Memory_Flash:W25Q128JVS
- removed U3: BQ24045DSQR, LCSC:WSON-10_L2.0-W2.0-P0.40-BL-EP, symbol LCSC:BQ24045DSQR
- removed X1: X322512MSB4SI, LCSC:OSC-SMD_4P-L3.2-W2.5-BL, symbol LCSC:X322512MSB4SI
Other:
- added sheet Power (power.kicad_sch)
- added sheet RP2040 (rp2040.kicad_sch)

Commit message: More work on power supply section
Parts:
- removed J1: USB_C_Receptacle_USB2.0, LCSC:USB-C-SMD_TYPEC-304J-BCP16, symbol Connector:USB_C_Receptacle_USB2.0
Other:
- sheet Power ports: added ISET2; removed none
- sheet RP2040 ports: added CHG_{ISET2}; removed none
Changed lines of the file:
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@@
     (title "Křeček")
   )
-  (symbol (lib_id "Connector:USB_C_Receptacle_USB2.0") (at 269.24 38.1 0) (mirror y) (unit 1)
-    (in_bom yes) (on_board yes) (dnp no)
-    (property "Reference" "J1" (at 256.54 15.24 0)
-      (effects (font (size 1.27 1.27)) (justify right))
-    )
-    (property "Value" "USB_C_Receptacle_USB2.0" (at 256.54 17.78 0)
-      (effects (font (size 1.27 1.27)) (justify right))
-    )
-    (property "Footprint" "LCSC:USB-C-SMD_TYPEC-304J-BCP16" (at 265.43 38.1 0)
-      (effects (font (size 1.27 1.27)) hide)
-    )
-    (property "Datasheet" "https://www.usb.org/sites/default/files/documents/usb_type-c.zip" (at 265.43 38.1 0)
-      (effects (font (size 1.27 1.27)) hide)
-    )
-    (property "LCSC Part" "C2835315" (at 269.24 38.1 0)
-      (effects (font (size 1.27 1.27)) hide)
-    )
-    (pin "A1")
-    (pin "A12")
-    (pin "A4")
-    (pin "A5")
-    (pin "A6")
-    (pin "A7")
-    (pin "A8")
-    (pin "A9")
-    (pin "B1")
-    (pin "B12")
-    (pin "B4")
-    (pin "B5")
-    (pin "B6")
-    (pin "B7")
-    (pin "B8")
-    (pin "B9")
-    (pin "S1")
-    (instances
-      (project "krecek-0.9"
-        (path "/8888f37b-ecc2-47df-8824-4b4e1e726451"
-          (reference "J1") (unit 1)
-        )
-      )
-    )
+  (wire (pts (xy 63.5 40.64) (xy 88.9 40.64))
+    (stroke (width 0) (type default))
+  )
+  (hierarchical_label "OUT" (shape input) (at 88.9 43.18 0) (fields_autoplaced)
+    (effects (font (size 1.27 1.27)) (justify left))
   )
   (sheet (at 38.1 38.1) (size 25.4 38.1) (fields_autoplaced)
@@
       (effects (font (size 1.27 1.27)) (justify left top))
     )
+    (pin "CHG_{ISET2}" output (at 63.5 40.64 0)
+      (effects (font (size 1.27 1.27)) (justify right))
+    )
     (instances
       (project "krecek-0.9"
@@
     )
   )
-  (sheet (at 114.3 38.1) (size 25.4 38.1) (fields_autoplaced)
+  (sheet (at 88.9 38.1) (size 25.4 38.1) (fields_autoplaced)
     (stroke (width 0.1524) (type solid))
     (fill (color 0 0 0 0.0000))
-    (property "Sheetname" "Power" (at 114.3 37.3884 0)
+    (property "Sheetname" "Power" (at 88.9 37.3884 0)
       (effects (font (size 1.27 1.27)) (justify left bottom))
     )
-    (property "Sheetfile" "power.kicad_sch" (at 114.3 76.7846 0)
+    (property "Sheetfile" "power.kicad_sch" (at 88.9 76.7846 0)
       (effects (font (size 1.27 1.27)) (justify left top))
     )
+    (pin "ISET2" input (at 88.9 40.64 180)
+      (effects (font (size 1.27 1.27)) (justify left))
+    )
     (instances

Commit message: Expand hardware design to cover more areas
Signed-off-by: Jan Hamal Dvořák <mordae@anilinux.org>
Parts:
- added U13: Display, Krecek:TftDisplay, symbol Krecek:TftDisplay
Connections:
- new net +3.3V: U13.1 (VCC)
- new net GND: U13.2 (GND)
- new net RP2040/TFT_{CS}: U13.3 (CS)
- new net RP2040/TFT_{LED}: U13.8 (LED)
- new net RP2040/TFT_{MISO}: U13.9 (MISO)
- new net RP2040/TFT_{MOSI}: U13.6 (MOSI)
- new net RP2040/TFT_{RST}: U13.4 (RST)
- new net RP2040/TFT_{RS}: U13.5 (DC)
- new net RP2040/TFT_{SCK}: U13.7 (SCK)
- no-connect marks 0 -> 9
Other:
- added sheet Audio (audio.kicad_sch)
- added sheet Inputs (inputs.kicad_sch)
- added sheet Radio (radio.kicad_sch)
- sheet Power ports: added OFF, USB_{CC1}, USB_{CC2}, USB_{D+}, USB_{D-}; removed none
- sheet RP2040 ports: added BTN_{A}, BTN_{B}, BTN_{SELECT}, BTN_{START}, BTN_{X}, BTN_{Y}, JOY_{SW}, JOY_{X}, JOY_{Y}, OFF, RF_{CS}, TFT_{CS}, TFT_{LED}, TFT_{MISO}, TFT_{MOSI}, TFT_{RST}, TFT_{RS}, TFT_{SCK}; removed none

Commit message: Update schematic
Signed-off-by: Jan Hamal Dvořák <mordae@anilinux.org>
Other:
- sheet RP2040 ports: added USB_{D+}, USB_{D-}; removed none
Changed lines of the file:
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@@
+    (stroke (width 0) (type default))
+  )
+  (wire (pts (xy 139.7 60.96) (xy 165.1 60.96))
     (stroke (width 0) (type default))
   )
@@
   )
   (wire (pts (xy 149.86 137.16) (xy 149.86 101.6))
+    (stroke (width 0) (type default))
+  )
+  (wire (pts (xy 139.7 58.42) (xy 165.1 58.42))
     (stroke (width 0) (type default))
   )
@@
       (effects (font (size 1.27 1.27)) (justify left))
     )
-    (instances
+    (pin "USB_{D+}" bidirectional (at 139.7 58.42 0)
+      (effects (font (size 1.27 1.27)) (justify right))
+    )
+    (pin "USB_{D-}" bidirectional (at 139.7 60.96 0)
+      (effects (font (size 1.27 1.27)) (justify right))
+    )
+    (instances

Commit message: Further tweaks and improvements
- Use a nicer schematic template
- Tie START button with power on
- Add ferrite to USB shield
- Add CC1/CC2 makeshift ADC
- Tidy up schematics a little bit

Signed-off-by: Jan Hamal Dvořák <mordae@anilinux.org>
Other:
- sheet RP2040 ports: added USB_{CC1}, USB_{CC2}; removed none
- company: (none) -> DDM Spirála
Changed lines of the file:
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@@
   (title_block
     (title "Křeček")
+    (date "2023-12-20")
+    (rev "v0.9-wip")
+    (company "DDM Spirála")
   )
   (junction (at 147.32 109.22) (diameter 0) (color 0 0 0 0)
@@
     (stroke (width 0) (type default))
   )
+  (wire (pts (xy 139.7 63.5) (xy 165.1 63.5))
+    (stroke (width 0) (type default))
+  )
   (wire (pts (xy 147.32 134.62) (xy 147.32 109.22))
     (stroke (width 0) (type default))
@@
   )
   (wire (pts (xy 139.7 111.76) (xy 142.24 111.76))
+    (stroke (width 0) (type default))
+  )
+  (wire (pts (xy 139.7 66.04) (xy 165.1 66.04))
     (stroke (width 0) (type default))
   )
@@
       (effects (font (size 1.27 1.27)) (justify right))
     )
+    (pin "USB_{CC1}" input (at 139.7 63.5 0)
+      (effects (font (size 1.27 1.27)) (justify right))
+    )
+    (pin "USB_{CC2}" input (at 139.7 66.04 0)
+      (effects (font (size 1.27 1.27)) (justify right))
+    )

Commit message: Complete most of the design, except for RF
Signed-off-by: Jan Hamal Dvořák <mordae@anilinux.org>
Parts:
- renumbered U13 to U1
Connections:
- net RP2040/T_{SCK}: now reaches U1.10 (T_CLK)
- net RP2040/T_{CS}: now reaches U1.11 (T_CS)
- net RP2040/T_{MOSI}: now reaches U1.12 (T_DIN)
- net RP2040/T_{MISO}: now reaches U1.13 (T_DO)
- net RP2040/T_{IRQ}: now reaches U1.14 (T_IRQ)
- no-connect marks 9 -> 4
Other:
- added sheet MicroSD Card (sdcard.kicad_sch)
- sheet Audio ports: added ADC, AMP_{EN}, CCLK, CDATA, DAC, HP_{SENSE}, IR_{TX}, LRCK, SCLK; removed none
- sheet Inputs ports: added BRACK_{L}, BRACK_{R}, VOL_{DOWN}, VOL_{SW}, VOL_{UP}; removed BTN_{START}
- sheet Power ports: added BAT_{Vsense}, ON; removed none
- sheet RP2040 ports: added AMP_{EN}, BAT_{Vsense}, BRACK_{L}, BRACK_{R}, DSP_{ASDIN}, DSP_{ASDOUT}, DSP_{CCLK}, DSP_{CDATA}, DSP_{LRCK}, DSP_{SCLK}, HP_{SENSE}, IR_{TX}, SD_{CS}, SD_{MISO}, SD_{MOSI}, SD_{SCLK}, T_{CS}, T_{IRQ}, T_{MISO}, T_{MOSI}, T_{SCK}, VOL_{DOWN}, VOL_{SW}, VOL_{UP}; removed none
- moved on the sheet: U1
