File: hw/krecek-0.9/krecek-0.9.kicad_sch (KiCad schematic)
At the start: 1 part, among them U1 Display

Commit message: Complete the RF section
Connections:
- net RP2040/TFT_{SCK} is gone; now on net RP2040/TFT_{MISO}: U1.7 (SCK)
Other:
- sheet RP2040 ports: added RF_{CLK}; removed none
- sheet Radio ports: added RF_{CLK}; removed none
Changed lines of the file:
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@@
   (junction (at 172.72 109.22) (diameter 0) (color 0 0 0 0)
   )
-  (junction (at 170.18 104.14) (diameter 0) (color 0 0 0 0)
-  )
-  (junction (at 175.26 101.6) (diameter 0) (color 0 0 0 0)
+  (junction (at 177.8 101.6) (diameter 0) (color 0 0 0 0)
+  )
+  (junction (at 175.26 109.22) (diameter 0) (color 0 0 0 0)
+  )
+  (junction (at 172.72 104.14) (diameter 0) (color 0 0 0 0)
   )
   (no_connect (at 215.9 96.52))
@@
     (stroke (width 0) (type default))
   )
-  (wire (pts (xy 170.18 104.14) (xy 190.5 104.14))
+  (wire (pts (xy 165.1 104.14) (xy 172.72 104.14))
+    (stroke (width 0) (type default))
+  )
+  (wire (pts (xy 175.26 109.22) (xy 172.72 109.22))
+    (stroke (width 0) (type default))
+  )
+  (wire (pts (xy 165.1 114.3) (xy 167.64 114.3))
+    (stroke (width 0) (type default))
+  )
+  (wire (pts (xy 172.72 109.22) (xy 172.72 104.14))
     (stroke (width 0) (type default))
   )
@@
     (stroke (width 0) (type default))
   )
-  (wire (pts (xy 190.5 137.16) (xy 175.26 137.16))
-    (stroke (width 0) (type default))
-  )
-  (wire (pts (xy 167.64 129.54) (xy 190.5 129.54))
+  (wire (pts (xy 190.5 134.62) (xy 177.8 134.62))
+    (stroke (width 0) (type default))
+  )
+  (wire (pts (xy 170.18 127) (xy 190.5 127))
     (stroke (width 0) (type default))
   )
@@
     (stroke (width 0) (type default))
   )
-  (wire (pts (xy 172.72 134.62) (xy 172.72 109.22))
+  (wire (pts (xy 175.26 132.08) (xy 175.26 109.22))
     (stroke (width 0) (type default))
   )
@@
     (stroke (width 0) (type default))
   )
+  (wire (pts (xy 190.5 137.16) (xy 167.64 137.16))
+    (stroke (width 0) (type default))
+  )
   (wire (pts (xy 114.3 58.42) (xy 139.7 58.42))
     (stroke (width 0) (type default))
@@
     (stroke (width 0) (type default))
   )
+  (wire (pts (xy 175.26 109.22) (xy 190.5 109.22))
+    (stroke (width 0) (type default))
+  )
   (wire (pts (xy 165.1 58.42) (xy 190.5 58.42))
     (stroke (width 0) (type default))
@@
     (stroke (width 0) (type default))
   )
-  (wire (pts (xy 175.26 101.6) (xy 190.5 101.6))
+  (wire (pts (xy 165.1 101.6) (xy 177.8 101.6))
     (stroke (width 0) (type default))
   )
@@
     (stroke (width 0) (type default))
   )
+  (wire (pts (xy 172.72 104.14) (xy 190.5 104.14))
+    (stroke (width 0) (type default))
+  )
   (wire (pts (xy 114.3 96.52) (xy 139.7 96.52))
     (stroke (width 0) (type default))
@@
     (stroke (width 0) (type default))
   )
-  (wire (pts (xy 172.72 109.22) (xy 190.5 109.22))
-    (stroke (width 0) (type default))
-  )
   (wire (pts (xy 165.1 96.52) (xy 190.5 96.52))
     (stroke (width 0) (type default))
@@
     (stroke (width 0) (type default))
   )
-  (wire (pts (xy 170.18 132.08) (xy 170.18 104.14))
+  (wire (pts (xy 172.72 129.54) (xy 172.72 109.22))
     (stroke (width 0) (type default))
   )
@@
     (stroke (width 0) (type default))
   )
-  (wire (pts (xy 165.1 104.14) (xy 170.18 104.14))
+  (wire (pts (xy 167.64 137.16) (xy 167.64 114.3))
     (stroke (width 0) (type default))
   )
@@
     (stroke (width 0) (type default))
   )
-  (wire (pts (xy 165.1 101.6) (xy 175.26 101.6))
-    (stroke (width 0) (type default))
-  )
   (wire (pts (xy 165.1 73.66) (xy 227.33 73.66))
     (stroke (width 0) (type default))
@@
     (stroke (width 0) (type default))
   )
-  (wire (pts (xy 167.64 111.76) (xy 167.64 129.54))
-    (stroke (width 0) (type default))
-  )
-  (wire (pts (xy 165.1 111.76) (xy 167.64 111.76))
+  (wire (pts (xy 170.18 111.76) (xy 170.18 127))
+    (stroke (width 0) (type default))
+  )
+  (wire (pts (xy 165.1 111.76) (xy 170.18 111.76))
     (stroke (width 0) (type default))
   )
@@
     (stroke (width 0) (type default))
   )
-  (wire (pts (xy 175.26 137.16) (xy 175.26 101.6))
+  (wire (pts (xy 177.8 134.62) (xy 177.8 101.6))
     (stroke (width 0) (type default))
   )
@@
     (stroke (width 0) (type default))
   )
+  (wire (pts (xy 177.8 101.6) (xy 190.5 101.6))
+    (stroke (width 0) (type default))
+  )
   (wire (pts (xy 215.9 111.76) (xy 229.87 111.76))
     (stroke (width 0) (type default))
@@
     (stroke (width 0) (type default))
   )
-  (wire (pts (xy 190.5 132.08) (xy 170.18 132.08))
+  (wire (pts (xy 190.5 129.54) (xy 172.72 129.54))
     (stroke (width 0) (type default))
   )
@@
     (stroke (width 0) (type default))
   )
-  (wire (pts (xy 190.5 134.62) (xy 172.72 134.62))
+  (wire (pts (xy 190.5 132.08) (xy 175.26 132.08))
     (stroke (width 0) (type default))
   )
@@
     )
   )
-  (sheet (at 190.5 127) (size 25.4 12.7) (fields_autoplaced)
+  (sheet (at 190.5 124.46) (size 25.4 15.24) (fields_autoplaced)
     (stroke (width 0.1524) (type solid))
     (fill (color 0 0 0 0.0000))
-    (property "Sheetname" "Radio" (at 190.5 126.2884 0)
+    (property "Sheetname" "Radio" (at 190.5 123.7484 0)
       (effects (font (size 1.27 1.27)) (justify left bottom))
     )
@@
       (effects (font (size 1.27 1.27)) (justify left top))
     )
-    (pin "RF_{CS}" input (at 190.5 129.54 180)
-      (effects (font (size 1.27 1.27)) (justify left))
-    )
-    (pin "RF_{SCLK}" input (at 190.5 132.08 180)
-      (effects (font (size 1.27 1.27)) (justify left))
-    )
-    (pin "RF_{MISO}" output (at 190.5 134.62 180)
-      (effects (font (size 1.27 1.27)) (justify left))
-    )
-    (pin "RF_{MOSI}" input (at 190.5 137.16 180)
+    (pin "RF_{CS}" input (at 190.5 127 180)
+      (effects (font (size 1.27 1.27)) (justify left))
+    )
+    (pin "RF_{SCLK}" input (at 190.5 129.54 180)
+      (effects (font (size 1.27 1.27)) (justify left))
+    )
+    (pin "RF_{MISO}" output (at 190.5 132.08 180)
+      (effects (font (size 1.27 1.27)) (justify left))
+    )
+    (pin "RF_{MOSI}" input (at 190.5 134.62 180)
+      (effects (font (size 1.27 1.27)) (justify left))
+    )
+    (pin "RF_{CLK}" input (at 190.5 137.16 180)
       (effects (font (size 1.27 1.27)) (justify left))
     )
@@
       (effects (font (size 1.27 1.27)) (justify left))
     )
+    (pin "RF_{CLK}" output (at 165.1 114.3 0)
+      (effects (font (size 1.27 1.27)) (justify right))
+    )
     (instances

Commit message: Further progress with the PCB layout
Signed-off-by: Jan Hamal Dvořák <mordae@anilinux.org>
Other:
- sheet Power ports: added USB+, USB-; removed USB_{D+}, USB_{D-}
- sheet RP2040 ports: added USB+, USB-; removed USB_{D+}, USB_{D-}
Changed lines of the file:
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@@
       (effects (font (size 1.27 1.27)) (justify left))
     )
-    (pin "USB_{D+}" bidirectional (at 165.1 45.72 0)
+    (pin "USB+" bidirectional (at 165.1 45.72 0)
       (effects (font (size 1.27 1.27)) (justify right))
     )
-    (pin "USB_{D-}" bidirectional (at 165.1 48.26 0)
+    (pin "USB-" bidirectional (at 165.1 48.26 0)
       (effects (font (size 1.27 1.27)) (justify right))
     )
@@
       (effects (font (size 1.27 1.27)) (justify left))
     )
-    (pin "USB_{D+}" bidirectional (at 190.5 45.72 180)
+    (pin "USB+" bidirectional (at 190.5 45.72 180)
       (effects (font (size 1.27 1.27)) (justify left))
     )
-    (pin "USB_{D-}" bidirectional (at 190.5 48.26 180)
+    (pin "USB-" bidirectional (at 190.5 48.26 180)
       (effects (font (size 1.27 1.27)) (justify left))
     )

Commit message: Progress on PCB
Signed-off-by: Jan Hamal Dvořák <mordae@anilinux.org>
Connections:
- net RP2040/TFT_{MISO}: no longer U1.7 (SCK)
- new net RP2040/TFT_{SCK}: U1.7 (SCK)
Changed lines of the file:
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@@
     (company "DDM Spirála")
-  )
-  (junction (at 172.72 109.22) (diameter 0) (color 0 0 0 0)
   )
   (junction (at 177.8 101.6) (diameter 0) (color 0 0 0 0)
@@
     (stroke (width 0) (type default))
   )
-  (wire (pts (xy 175.26 109.22) (xy 172.72 109.22))
+  (wire (pts (xy 165.1 109.22) (xy 175.26 109.22))
     (stroke (width 0) (type default))
   )
@@
     (stroke (width 0) (type default))
   )
-  (wire (pts (xy 172.72 109.22) (xy 172.72 104.14))
+  (wire (pts (xy 172.72 104.14) (xy 172.72 129.54))
     (stroke (width 0) (type default))
   )
@@
   )
   (wire (pts (xy 114.3 137.16) (xy 139.7 137.16))
-    (stroke (width 0) (type default))
-  )
-  (wire (pts (xy 165.1 109.22) (xy 172.72 109.22))
     (stroke (width 0) (type default))
   )
@@
     (stroke (width 0) (type default))
   )
-  (wire (pts (xy 172.72 129.54) (xy 172.72 109.22))
-    (stroke (width 0) (type default))
-  )

Commit message: Hardware as sent for manufacturing
Parts:
- added H1, H2, H3, H4: MountingHole, MountingHole:MountingHole_2.2mm_M2, symbol Mechanical:MountingHole
- added H5, H6, H7, H8: ToolingHole, Krecek:ToolingHole, symbol Mechanical:MountingHole
Changed lines of the file:
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@@
     (stroke (width 0) (type default))
   )
+  (symbol (lib_id "Mechanical:MountingHole") (at 50.8 177.8 0) (unit 1)
+    (in_bom yes) (on_board yes) (dnp no) (fields_autoplaced)
+    (property "Reference" "H7" (at 53.34 176.53 0)
+      (effects (font (size 1.27 1.27)) (justify left))
+    )
+    (property "Value" "ToolingHole" (at 53.34 179.07 0)
+      (effects (font (size 1.27 1.27)) (justify left))
+    )
+    (property "Footprint" "Krecek:ToolingHole" (at 50.8 177.8 0)
+      (effects (font (size 1.27 1.27)) hide)
+    )
+    (property "Datasheet" "~" (at 50.8 177.8 0)
+      (effects (font (size 1.27 1.27)) hide)
+    )
+    (instances
+      (project "krecek-0.9"
+        (path "/8888f37b-ecc2-47df-8824-4b4e1e726451"
+          (reference "H7") (unit 1)
+        )
+      )
+    )
+  )
+  (symbol (lib_id "Mechanical:MountingHole") (at 50.8 152.4 0) (unit 1)
+    (in_bom yes) (on_board yes) (dnp no) (fields_autoplaced)
+    (property "Reference" "H5" (at 53.34 151.13 0)
+      (effects (font (size 1.27 1.27)) (justify left))
+    )
+    (property "Value" "ToolingHole" (at 53.34 153.67 0)
+      (effects (font (size 1.27 1.27)) (justify left))
+    )
+    (property "Footprint" "Krecek:ToolingHole" (at 50.8 152.4 0)
+      (effects (font (size 1.27 1.27)) hide)
+    )
+    (property "Datasheet" "~" (at 50.8 152.4 0)
+      (effects (font (size 1.27 1.27)) hide)
+    )
+    (instances
+      (project "krecek-0.9"
+        (path "/8888f37b-ecc2-47df-8824-4b4e1e726451"
+          (reference "H5") (unit 1)
+        )
+      )
+    )
+  )
   (symbol (lib_id "power:+3.3V") (at 190.5 91.44 90) (unit 1)
     (in_bom yes) (on_board yes) (dnp no) (fields_autoplaced)
@@
         (path "/8888f37b-ecc2-47df-8824-4b4e1e726451"
           (reference "#PWR01") (unit 1)
+        )
+      )
+    )
+  )
+  (symbol (lib_id "Mechanical:MountingHole") (at 25.4 152.4 0) (unit 1)
+    (in_bom yes) (on_board yes) (dnp no) (fields_autoplaced)
+    (property "Reference" "H1" (at 27.94 151.13 0)
+      (effects (font (size 1.27 1.27)) (justify left))
+    )
+    (property "Value" "MountingHole" (at 27.94 153.67 0)
+      (effects (font (size 1.27 1.27)) (justify left))
+    )
+    (property "Footprint" "MountingHole:MountingHole_2.2mm_M2" (at 25.4 152.4 0)
+      (effects (font (size 1.27 1.27)) hide)
+    )
+    (property "Datasheet" "~" (at 25.4 152.4 0)
+      (effects (font (size 1.27 1.27)) hide)
+    )
+    (instances
+      (project "krecek-0.9"
+        (path "/8888f37b-ecc2-47df-8824-4b4e1e726451"
+          (reference "H1") (unit 1)
         )
       )
@@
         (path "/8888f37b-ecc2-47df-8824-4b4e1e726451"
           (reference "#PWR02") (unit 1)
+        )
+      )
+    )
+  )
+  (symbol (lib_id "Mechanical:MountingHole") (at 25.4 190.5 0) (unit 1)
+    (in_bom yes) (on_board yes) (dnp no) (fields_autoplaced)
+    (property "Reference" "H4" (at 27.94 189.23 0)
+      (effects (font (size 1.27 1.27)) (justify left))
+    )
+    (property "Value" "MountingHole" (at 27.94 191.77 0)
+      (effects (font (size 1.27 1.27)) (justify left))
+    )
+    (property "Footprint" "MountingHole:MountingHole_2.2mm_M2" (at 25.4 190.5 0)
+      (effects (font (size 1.27 1.27)) hide)
+    )
+    (property "Datasheet" "~" (at 25.4 190.5 0)
+      (effects (font (size 1.27 1.27)) hide)
+    )
+    (instances
+      (project "krecek-0.9"
+        (path "/8888f37b-ecc2-47df-8824-4b4e1e726451"
+          (reference "H4") (unit 1)
+        )
+      )
+    )
+  )
+  (symbol (lib_id "Mechanical:MountingHole") (at 50.8 165.1 0) (unit 1)
+    (in_bom yes) (on_board yes) (dnp no) (fields_autoplaced)
+    (property "Reference" "H6" (at 53.34 163.83 0)
+      (effects (font (size 1.27 1.27)) (justify left))
+    )
+    (property "Value" "ToolingHole" (at 53.34 166.37 0)
+      (effects (font (size 1.27 1.27)) (justify left))
+    )
+    (property "Footprint" "Krecek:ToolingHole" (at 50.8 165.1 0)
+      (effects (font (size 1.27 1.27)) hide)
+    )
+    (property "Datasheet" "~" (at 50.8 165.1 0)
+      (effects (font (size 1.27 1.27)) hide)
+    )
+    (instances
+      (project "krecek-0.9"
+        (path "/8888f37b-ecc2-47df-8824-4b4e1e726451"
+          (reference "H6") (unit 1)
         )
       )
@@
         )
       )
+    )
+  )
+  (symbol (lib_id "Mechanical:MountingHole") (at 25.4 165.1 0) (unit 1)
+    (in_bom yes) (on_board yes) (dnp no) (fields_autoplaced)
+    (property "Reference" "H2" (at 27.94 163.83 0)
+      (effects (font (size 1.27 1.27)) (justify left))
+    )
+    (property "Value" "MountingHole" (at 27.94 166.37 0)
+      (effects (font (size 1.27 1.27)) (justify left))
+    )
+    (property "Footprint" "MountingHole:MountingHole_2.2mm_M2" (at 25.4 165.1 0)
+      (effects (font (size 1.27 1.27)) hide)
+    )
+    (property "Datasheet" "~" (at 25.4 165.1 0)
+      (effects (font (size 1.27 1.27)) hide)
+    )
+    (instances
+      (project "krecek-0.9"
+        (path "/8888f37b-ecc2-47df-8824-4b4e1e726451"
+          (reference "H2") (unit 1)
+        )
+      )
+    )
+  )
+  (symbol (lib_id "Mechanical:MountingHole") (at 25.4 177.8 0) (unit 1)
+    (in_bom yes) (on_board yes) (dnp no) (fields_autoplaced)
+    (property "Reference" "H3" (at 27.94 176.53 0)
+      (effects (font (size 1.27 1.27)) (justify left))
+    )
+    (property "Value" "MountingHole" (at 27.94 179.07 0)
+      (effects (font (size 1.27 1.27)) (justify left))
+    )
+    (property "Footprint" "MountingHole:MountingHole_2.2mm_M2" (at 25.4 177.8 0)
+      (effects (font (size 1.27 1.27)) hide)
+    )
+    (property "Datasheet" "~" (at 25.4 177.8 0)
+      (effects (font (size 1.27 1.27)) hide)
+    )
+    (instances
+      (project "krecek-0.9"
+        (path "/8888f37b-ecc2-47df-8824-4b4e1e726451"
+          (reference "H3") (unit 1)
+        )
+      )
+    )
+  )
+  (symbol (lib_id "Mechanical:MountingHole") (at 50.8 190.5 0) (unit 1)
+    (in_bom yes) (on_board yes) (dnp no) (fields_autoplaced)
+    (property "Reference" "H8" (at 53.34 189.23 0)
+      (effects (font (size 1.27 1.27)) (justify left))
+    )
+    (property "Value" "ToolingHole" (at 53.34 191.77 0)
+      (effects (font (size 1.27 1.27)) (justify left))
+    )
+    (property "Footprint" "Krecek:ToolingHole" (at 50.8 190.5 0)
+      (effects (font (size 1.27 1.27)) hide)
+    )
+    (property "Datasheet" "~" (at 50.8 190.5 0)
+      (effects (font (size 1.27 1.27)) hide)
+    )
+    (instances
+      (project "krecek-0.9"
+        (path "/8888f37b-ecc2-47df-8824-4b4e1e726451"
+          (reference "H8") (unit 1)
+        )
+      )

Commit message: Fix input PMOS orientation (again)
Parts:
- renumbered H5 to H2, H2 to H3, H6 to H4, H3 to H5, H7 to H6, H4 to H7
Changed lines of the file:
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@@
   (symbol (lib_id "Mechanical:MountingHole") (at 50.8 177.8 0) (unit 1)
     (in_bom yes) (on_board yes) (dnp no) (fields_autoplaced)
-    (property "Reference" "H7" (at 53.34 176.53 0)
+    (property "Reference" "H6" (at 53.34 176.53 0)
       (effects (font (size 1.27 1.27)) (justify left))
     )
@@
       (project "krecek-0.9"
         (path "/8888f37b-ecc2-47df-8824-4b4e1e726451"
-          (reference "H7") (unit 1)
+          (reference "H6") (unit 1)
         )
       )
@@
   (symbol (lib_id "Mechanical:MountingHole") (at 50.8 152.4 0) (unit 1)
     (in_bom yes) (on_board yes) (dnp no) (fields_autoplaced)
-    (property "Reference" "H5" (at 53.34 151.13 0)
+    (property "Reference" "H2" (at 53.34 151.13 0)
       (effects (font (size 1.27 1.27)) (justify left))
     )
@@
       (project "krecek-0.9"
         (path "/8888f37b-ecc2-47df-8824-4b4e1e726451"
-          (reference "H5") (unit 1)
+          (reference "H2") (unit 1)
         )
       )
@@
   (symbol (lib_id "Mechanical:MountingHole") (at 25.4 190.5 0) (unit 1)
     (in_bom yes) (on_board yes) (dnp no) (fields_autoplaced)
-    (property "Reference" "H4" (at 27.94 189.23 0)
+    (property "Reference" "H7" (at 27.94 189.23 0)
       (effects (font (size 1.27 1.27)) (justify left))
     )
@@
       (project "krecek-0.9"
         (path "/8888f37b-ecc2-47df-8824-4b4e1e726451"
+          (reference "H7") (unit 1)
+        )
+      )
+    )
+  )
+  (symbol (lib_id "Mechanical:MountingHole") (at 50.8 165.1 0) (unit 1)
+    (in_bom yes) (on_board yes) (dnp no) (fields_autoplaced)
+    (property "Reference" "H4" (at 53.34 163.83 0)
+      (effects (font (size 1.27 1.27)) (justify left))
+    )
+    (property "Value" "ToolingHole" (at 53.34 166.37 0)
+      (effects (font (size 1.27 1.27)) (justify left))
+    )
+    (property "Footprint" "Krecek:ToolingHole" (at 50.8 165.1 0)
+      (effects (font (size 1.27 1.27)) hide)
+    )
+    (property "Datasheet" "~" (at 50.8 165.1 0)
+      (effects (font (size 1.27 1.27)) hide)
+    )
+    (instances
+      (project "krecek-0.9"
+        (path "/8888f37b-ecc2-47df-8824-4b4e1e726451"
           (reference "H4") (unit 1)
-        )
-      )
-    )
-  )
-  (symbol (lib_id "Mechanical:MountingHole") (at 50.8 165.1 0) (unit 1)
-    (in_bom yes) (on_board yes) (dnp no) (fields_autoplaced)
-    (property "Reference" "H6" (at 53.34 163.83 0)
-      (effects (font (size 1.27 1.27)) (justify left))
-    )
-    (property "Value" "ToolingHole" (at 53.34 166.37 0)
-      (effects (font (size 1.27 1.27)) (justify left))
-    )
-    (property "Footprint" "Krecek:ToolingHole" (at 50.8 165.1 0)
-      (effects (font (size 1.27 1.27)) hide)
-    )
-    (property "Datasheet" "~" (at 50.8 165.1 0)
-      (effects (font (size 1.27 1.27)) hide)
-    )
-    (instances
-      (project "krecek-0.9"
-        (path "/8888f37b-ecc2-47df-8824-4b4e1e726451"
-          (reference "H6") (unit 1)
         )
       )
@@
   (symbol (lib_id "Mechanical:MountingHole") (at 25.4 165.1 0) (unit 1)
     (in_bom yes) (on_board yes) (dnp no) (fields_autoplaced)
-    (property "Reference" "H2" (at 27.94 163.83 0)
+    (property "Reference" "H3" (at 27.94 163.83 0)
       (effects (font (size 1.27 1.27)) (justify left))
     )
@@
       (project "krecek-0.9"
         (path "/8888f37b-ecc2-47df-8824-4b4e1e726451"
-          (reference "H2") (unit 1)
+          (reference "H3") (unit 1)
         )
       )
@@
   (symbol (lib_id "Mechanical:MountingHole") (at 25.4 177.8 0) (unit 1)
     (in_bom yes) (on_board yes) (dnp no) (fields_autoplaced)
-    (property "Reference" "H3" (at 27.94 176.53 0)
+    (property "Reference" "H5" (at 27.94 176.53 0)
       (effects (font (size 1.27 1.27)) (justify left))
     )
@@
       (project "krecek-0.9"
         (path "/8888f37b-ecc2-47df-8824-4b4e1e726451"
-          (reference "H3") (unit 1)
-        )
-      )
+          (reference "H5") (unit 1)
+        )
+      )
