File: hw/krecek-0.9/krecek-0.9.kicad_sch (KiCad schematic)
At the start: 9 parts, among them U1 Display

Commit message: Add display components to library
Also move CC1101 communication to second chip.
Resolves #13.
Other:
- sheet RP2040 ports: added RF_{XOSC}; removed RF_{CLK}
- sheet Radio ports: added RF_{XOSC}; removed RF_{CLK}
Changed lines of the file:
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@@
     (company "DDM Spirála")
   )
-  (junction (at 177.8 101.6) (diameter 0) (color 0 0 0 0)
-  )
-  (junction (at 175.26 109.22) (diameter 0) (color 0 0 0 0)
-  )
-  (junction (at 172.72 104.14) (diameter 0) (color 0 0 0 0)
+  (junction (at 222.25 104.14) (diameter 0) (color 0 0 0 0)
+  )
+  (junction (at 229.87 111.76) (diameter 0) (color 0 0 0 0)
+  )
+  (junction (at 224.79 106.68) (diameter 0) (color 0 0 0 0)
   )
   (no_connect (at 215.9 96.52))
@@
     (stroke (width 0) (type default))
   )
-  (wire (pts (xy 165.1 104.14) (xy 172.72 104.14))
-    (stroke (width 0) (type default))
-  )
-  (wire (pts (xy 165.1 109.22) (xy 175.26 109.22))
-    (stroke (width 0) (type default))
-  )
-  (wire (pts (xy 165.1 114.3) (xy 167.64 114.3))
-    (stroke (width 0) (type default))
-  )
-  (wire (pts (xy 172.72 104.14) (xy 172.72 129.54))
+  (wire (pts (xy 165.1 109.22) (xy 190.5 109.22))
+    (stroke (width 0) (type default))
+  )
+  (wire (pts (xy 180.34 111.76) (xy 180.34 127))
     (stroke (width 0) (type default))
   )
@@
     (stroke (width 0) (type default))
   )
+  (wire (pts (xy 224.79 106.68) (xy 224.79 129.54))
+    (stroke (width 0) (type default))
+  )
   (wire (pts (xy 224.79 76.2) (xy 165.1 76.2))
     (stroke (width 0) (type default))
   )
-  (wire (pts (xy 190.5 134.62) (xy 177.8 134.62))
-    (stroke (width 0) (type default))
-  )
-  (wire (pts (xy 170.18 127) (xy 190.5 127))
+  (wire (pts (xy 165.1 114.3) (xy 177.8 114.3))
     (stroke (width 0) (type default))
   )
@@
     (stroke (width 0) (type default))
   )
-  (wire (pts (xy 175.26 132.08) (xy 175.26 109.22))
-    (stroke (width 0) (type default))
-  )
   (wire (pts (xy 114.3 45.72) (xy 139.7 45.72))
     (stroke (width 0) (type default))
@@
     (stroke (width 0) (type default))
   )
-  (wire (pts (xy 190.5 137.16) (xy 167.64 137.16))
+  (wire (pts (xy 224.79 129.54) (xy 215.9 129.54))
     (stroke (width 0) (type default))
   )
@@
     (stroke (width 0) (type default))
   )
-  (wire (pts (xy 175.26 109.22) (xy 190.5 109.22))
-    (stroke (width 0) (type default))
-  )
   (wire (pts (xy 165.1 58.42) (xy 190.5 58.42))
     (stroke (width 0) (type default))
@@
     (stroke (width 0) (type default))
   )
+  (wire (pts (xy 222.25 104.14) (xy 222.25 127))
+    (stroke (width 0) (type default))
+  )
   (wire (pts (xy 114.3 81.28) (xy 139.7 81.28))
     (stroke (width 0) (type default))
@@
     (stroke (width 0) (type default))
   )
-  (wire (pts (xy 165.1 101.6) (xy 177.8 101.6))
-    (stroke (width 0) (type default))
-  )
   (wire (pts (xy 114.3 63.5) (xy 139.7 63.5))
     (stroke (width 0) (type default))
   )
-  (wire (pts (xy 172.72 104.14) (xy 190.5 104.14))
+  (wire (pts (xy 165.1 104.14) (xy 190.5 104.14))
     (stroke (width 0) (type default))
   )
@@
     (stroke (width 0) (type default))
   )
+  (wire (pts (xy 215.9 132.08) (xy 229.87 132.08))
+    (stroke (width 0) (type default))
+  )
   (wire (pts (xy 165.1 96.52) (xy 190.5 96.52))
     (stroke (width 0) (type default))
@@
     (stroke (width 0) (type default))
   )
-  (wire (pts (xy 167.64 137.16) (xy 167.64 114.3))
-    (stroke (width 0) (type default))
-  )
   (wire (pts (xy 224.79 106.68) (xy 224.79 76.2))
     (stroke (width 0) (type default))
   )
+  (wire (pts (xy 180.34 127) (xy 190.5 127))
+    (stroke (width 0) (type default))
+  )
   (wire (pts (xy 114.3 132.08) (xy 139.7 132.08))
     (stroke (width 0) (type default))
@@
     (stroke (width 0) (type default))
   )
+  (wire (pts (xy 229.87 132.08) (xy 229.87 111.76))
+    (stroke (width 0) (type default))
+  )
   (wire (pts (xy 165.1 106.68) (xy 190.5 106.68))
     (stroke (width 0) (type default))
   )
-  (wire (pts (xy 170.18 111.76) (xy 170.18 127))
-    (stroke (width 0) (type default))
-  )
-  (wire (pts (xy 165.1 111.76) (xy 170.18 111.76))
+  (wire (pts (xy 177.8 129.54) (xy 190.5 129.54))
     (stroke (width 0) (type default))
   )
@@
     (stroke (width 0) (type default))
   )
-  (wire (pts (xy 177.8 134.62) (xy 177.8 101.6))
-    (stroke (width 0) (type default))
-  )
   (wire (pts (xy 219.71 101.6) (xy 219.71 81.28))
     (stroke (width 0) (type default))
@@
     (stroke (width 0) (type default))
   )
-  (wire (pts (xy 177.8 101.6) (xy 190.5 101.6))
+  (wire (pts (xy 165.1 101.6) (xy 190.5 101.6))
     (stroke (width 0) (type default))
   )
@@
     (stroke (width 0) (type default))
   )
-  (wire (pts (xy 190.5 129.54) (xy 172.72 129.54))
-    (stroke (width 0) (type default))
-  )
   (wire (pts (xy 114.3 68.58) (xy 139.7 68.58))
     (stroke (width 0) (type default))
@@
     (stroke (width 0) (type default))
   )
-  (wire (pts (xy 190.5 132.08) (xy 175.26 132.08))
-    (stroke (width 0) (type default))
-  )
   (wire (pts (xy 114.3 106.68) (xy 139.7 106.68))
     (stroke (width 0) (type default))
   )
+  (wire (pts (xy 177.8 114.3) (xy 177.8 129.54))
+    (stroke (width 0) (type default))
+  )
   (wire (pts (xy 114.3 78.74) (xy 139.7 78.74))
     (stroke (width 0) (type default))
   )
   (wire (pts (xy 165.1 43.18) (xy 190.5 43.18))
+    (stroke (width 0) (type default))
+  )
+  (wire (pts (xy 165.1 111.76) (xy 180.34 111.76))
+    (stroke (width 0) (type default))
+  )
+  (wire (pts (xy 222.25 127) (xy 215.9 127))
     (stroke (width 0) (type default))
   )
@@
       (effects (font (size 1.27 1.27)) (justify left))
     )
-    (pin "RF_{SCLK}" input (at 190.5 129.54 180)
-      (effects (font (size 1.27 1.27)) (justify left))
-    )
-    (pin "RF_{MISO}" output (at 190.5 132.08 180)
-      (effects (font (size 1.27 1.27)) (justify left))
-    )
-    (pin "RF_{MOSI}" input (at 190.5 134.62 180)
-      (effects (font (size 1.27 1.27)) (justify left))
-    )
-    (pin "RF_{CLK}" input (at 190.5 137.16 180)
+    (pin "RF_{SCLK}" input (at 215.9 132.08 0)
+      (effects (font (size 1.27 1.27)) (justify right))
+    )
+    (pin "RF_{MISO}" output (at 215.9 127 0)
+      (effects (font (size 1.27 1.27)) (justify right))
+    )
+    (pin "RF_{MOSI}" input (at 215.9 129.54 0)
+      (effects (font (size 1.27 1.27)) (justify right))
+    )
+    (pin "RF_{XOSC}" input (at 190.5 129.54 180)
       (effects (font (size 1.27 1.27)) (justify left))
     )
@@
       (effects (font (size 1.27 1.27)) (justify left))
     )
-    (pin "RF_{CLK}" output (at 165.1 114.3 0)
-      (effects (font (size 1.27 1.27)) (justify right))
-    )
+    (pin "RF_{XOSC}" output (at 165.1 114.3 0)
+      (effects (font (size 1.27 1.27)) (justify right))
+    )

Commit message: hw: use non-PCB screen with touch ADC
Parts:
- removed U1: Display, Krecek:TftDisplay, symbol Krecek:TftDisplay
Connections:
- no-connect marks 4 -> 0
Other:
- added sheet Display (display.kicad_sch)
- sheet RP2040 ports: added none; removed T_{IRQ}
Changed lines of the file:
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@@
   (junction (at 224.79 106.68) (diameter 0) (color 0 0 0 0)
   )
-  (no_connect (at 215.9 96.52))
-  (no_connect (at 215.9 99.06))
-  (no_connect (at 215.9 93.98))
-  (no_connect (at 215.9 91.44))
   (wire (pts (xy 114.3 114.3) (xy 139.7 114.3))
     (stroke (width 0) (type default))
@@
     (stroke (width 0) (type default))
   )
-  (wire (pts (xy 219.71 101.6) (xy 219.71 81.28))
-    (stroke (width 0) (type default))
-  )
   (wire (pts (xy 165.1 45.72) (xy 190.5 45.72))
     (stroke (width 0) (type default))
@@
     (stroke (width 0) (type default))
   )
-  (wire (pts (xy 219.71 81.28) (xy 165.1 81.28))
-    (stroke (width 0) (type default))
-  )
   (wire (pts (xy 114.3 129.54) (xy 139.7 129.54))
     (stroke (width 0) (type default))
   )
-  (wire (pts (xy 215.9 101.6) (xy 219.71 101.6))
-    (stroke (width 0) (type default))
-  )
   (wire (pts (xy 114.3 99.06) (xy 139.7 99.06))
     (stroke (width 0) (type default))
@@
     )
   )
-  (symbol (lib_id "power:+3.3V") (at 190.5 91.44 90) (unit 1)
-    (in_bom yes) (on_board yes) (dnp no) (fields_autoplaced)
-    (property "Reference" "#PWR01" (at 194.31 91.44 0)
-      (effects (font (size 1.27 1.27)) hide)
-    )
-    (property "Value" "+3.3V" (at 186.69 91.44 90)
-      (effects (font (size 1.27 1.27)) (justify left))
-    )
-    (property "Footprint" "" (at 190.5 91.44 0)
-      (effects (font (size 1.27 1.27)) hide)
-    )
-    (property "Datasheet" "" (at 190.5 91.44 0)
-      (effects (font (size 1.27 1.27)) hide)
-    )
-    (pin "1")
-    (instances
-      (project "krecek-0.9"
-        (path "/8888f37b-ecc2-47df-8824-4b4e1e726451"
-          (reference "#PWR01") (unit 1)
-        )
-      )
-    )
-  )
   (symbol (lib_id "Mechanical:MountingHole") (at 25.4 152.4 0) (unit 1)
     (in_bom yes) (on_board yes) (dnp no) (fields_autoplaced)
@@
     )
   )
-  (symbol (lib_id "power:GND") (at 190.5 111.76 270) (unit 1)
-    (in_bom yes) (on_board yes) (dnp no) (fields_autoplaced)
-    (property "Reference" "#PWR02" (at 184.15 111.76 0)
-      (effects (font (size 1.27 1.27)) hide)
-    )
-    (property "Value" "GND" (at 186.69 111.76 90)
-      (effects (font (size 1.27 1.27)) (justify right))
-    )
-    (property "Footprint" "" (at 190.5 111.76 0)
-      (effects (font (size 1.27 1.27)) hide)
-    )
-    (property "Datasheet" "" (at 190.5 111.76 0)
-      (effects (font (size 1.27 1.27)) hide)
-    )
-    (pin "1")
-    (instances
-      (project "krecek-0.9"
-        (path "/8888f37b-ecc2-47df-8824-4b4e1e726451"
-          (reference "#PWR02") (unit 1)
-        )
-      )
-    )
-  )
   (symbol (lib_id "Mechanical:MountingHole") (at 25.4 190.5 0) (unit 1)
     (in_bom yes) (on_board yes) (dnp no) (fields_autoplaced)
@@
         (path "/8888f37b-ecc2-47df-8824-4b4e1e726451"
           (reference "H4") (unit 1)
-        )
-      )
-    )
-  )
-  (symbol (lib_id "Krecek:TftDisplay") (at 203.2 101.6 0) (unit 1)
-    (in_bom yes) (on_board yes) (dnp no) (fields_autoplaced)
-    (property "Reference" "U1" (at 203.2 83.82 0)
-      (effects (font (size 1.27 1.27)))
-    )
-    (property "Value" "Display" (at 203.2 86.36 0)
-      (effects (font (size 1.27 1.27)))
-    )
-    (property "Footprint" "Krecek:TftDisplay" (at 203.2 118.11 0)
-      (effects (font (size 1.27 1.27)) hide)
-    )
-    (property "Datasheet" "" (at 182.88 96.52 0)
-      (effects (font (size 1.27 1.27)) hide)
-    )
-    (pin "1")
-    (pin "10")
-    (pin "11")
-    (pin "12")
-    (pin "13")
-    (pin "14")
-    (pin "15")
-    (pin "16")
-    (pin "17")
-    (pin "18")
-    (pin "2")
-    (pin "3")
-    (pin "4")
-    (pin "5")
-    (pin "6")
-    (pin "7")
-    (pin "8")
-    (pin "9")
-    (instances
-      (project "krecek-0.9"
-        (path "/8888f37b-ecc2-47df-8824-4b4e1e726451"
-          (reference "U1") (unit 1)
         )
       )
@@
     )
   )
+  (sheet (at 190.5 88.9) (size 25.4 25.4) (fields_autoplaced)
+    (stroke (width 0.1524) (type solid))
+    (fill (color 0 0 0 0.0000))
+    (property "Sheetname" "Display" (at 190.5 88.1884 0)
+      (effects (font (size 1.27 1.27)) (justify left bottom))
+    )
+    (property "Sheetfile" "display.kicad_sch" (at 190.5 114.8846 0)
+      (effects (font (size 1.27 1.27)) (justify left top))
+    )
+    (pin "TFT_{RST}" input (at 190.5 96.52 180)
+      (effects (font (size 1.27 1.27)) (justify left))
+    )
+    (pin "TFT_{SCLK}" input (at 190.5 104.14 180)
+      (effects (font (size 1.27 1.27)) (justify left))
+    )
+    (pin "TFT_{DC}" input (at 190.5 99.06 180)
+      (effects (font (size 1.27 1.27)) (justify left))
+    )
+    (pin "TFT_{MOSI}" input (at 190.5 101.6 180)
+      (effects (font (size 1.27 1.27)) (justify left))
+    )
+    (pin "TFT_{CS}" input (at 190.5 93.98 180)
+      (effects (font (size 1.27 1.27)) (justify left))
+    )
+    (pin "TFT_{MISO}" input (at 190.5 109.22 180)
+      (effects (font (size 1.27 1.27)) (justify left))
+    )
+    (pin "TOUCH_{MISO}" input (at 215.9 104.14 0)
+      (effects (font (size 1.27 1.27)) (justify right))
+    )
+    (pin "TOUCH_{SCLK}" input (at 215.9 111.76 0)
+      (effects (font (size 1.27 1.27)) (justify right))
+    )
+    (pin "TOUCH_{CS}" input (at 215.9 109.22 0)
+      (effects (font (size 1.27 1.27)) (justify right))
+    )
+    (pin "TOUCH_{MOSI}" input (at 215.9 106.68 0)
+      (effects (font (size 1.27 1.27)) (justify right))
+    )
+    (pin "TFT_{LED}" input (at 190.5 106.68 180)
+      (effects (font (size 1.27 1.27)) (justify left))
+    )
+    (instances
+      (project "krecek-0.9"
+        (path "/8888f37b-ecc2-47df-8824-4b4e1e726451" (page "8"))
+      )
+    )
+  )
   (sheet (at 190.5 124.46) (size 25.4 15.24) (fields_autoplaced)
     (stroke (width 0.1524) (type solid))
@@
       (effects (font (size 1.27 1.27)) (justify right))
     )
-    (pin "T_{IRQ}" input (at 165.1 81.28 0)
-      (effects (font (size 1.27 1.27)) (justify right))
-    )
