File: hw/krecek-0.9/krecek-0.9.kicad_sch (KiCad schematic)
At the start: 8 parts

Commit message: Replace Joystick with flat JoyCon
Other:
- sheet Inputs ports: added none; removed JOY_{SW}
- sheet RP2040 ports: added none; removed JOY_{SW}
Changed lines of the file:
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@@
-	(wire
-		(pts
-			(xy 114.3 58.42) (xy 139.7 58.42)
-		)
-		(stroke
-			(width 0)
-			(type default)
-		)
-	)
 	(wire
 		(pts
@@
 			)
 		)
-		(pin "JOY_{SW}" output
-			(at 114.3 58.42 0)
-			(effects
-				(font
-					(size 1.27 1.27)
-				)
-				(justify right)
-			)
-		)
 		(pin "BTN_{SELECT}" output
 			(at 114.3 63.5 0)
@@
 			(effects
 				(font
-					(size 1.27 1.27)
-				)
-				(justify left)
-			)
-		)
-		(pin "JOY_{SW}" input
-			(at 139.7 58.42 180)
-			(effects
-				(font

Commit message: Progress on HW design
Parts:
- added TFT1: Panel, Krecek:Panel, symbol Mechanical:MountingHole
- renumbered H1 to H2, H2 to H3, H3 to H4, H4 to H5, H5 to H6, H6 to H7, H7 to H8, H8 to H9
Other:
- sheet Audio ports: added none; removed AMP_{EN}
- sheet RP2040 ports: added none; removed AMP_{EN}
Changed lines of the file:
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@@
-	(wire
-		(pts
-			(xy 114.3 93.98) (xy 139.7 93.98)
-		)
-		(stroke
-			(width 0)
-			(type default)
-		)
-	)
 	(wire
 		(pts
@@
 		(dnp no)
 		(fields_autoplaced yes)
-		(property "Reference" "H6"
+		(property "Reference" "H7"
 			(at 53.34 176.53 0)
 			(effects
@@
 			(project "krecek-0.9"
 				(path "/8888f37b-ecc2-47df-8824-4b4e1e726451"
-					(reference "H6")
+					(reference "H7")
 					(unit 1)
 				)
@@
 		(dnp no)
 		(fields_autoplaced yes)
-		(property "Reference" "H2"
+		(property "Reference" "H3"
 			(at 53.34 151.13 0)
 			(effects
@@
 			(project "krecek-0.9"
 				(path "/8888f37b-ecc2-47df-8824-4b4e1e726451"
-					(reference "H2")
+					(reference "H3")
 					(unit 1)
 				)
@@
 		(dnp no)
 		(fields_autoplaced yes)
-		(property "Reference" "H1"
+		(property "Reference" "H2"
 			(at 27.94 151.13 0)
 			(effects
@@
 			(project "krecek-0.9"
 				(path "/8888f37b-ecc2-47df-8824-4b4e1e726451"
-					(reference "H1")
+					(reference "H2")
+					(unit 1)
+				)
+			)
+		)
+	)
+	(symbol
+		(lib_id "Mechanical:MountingHole")
+		(at 25.4 127 0)
+		(unit 1)
+		(exclude_from_sim no)
+		(in_bom yes)
+		(on_board yes)
+		(dnp no)
+		(fields_autoplaced yes)
+		(property "Reference" "TFT1"
+			(at 27.94 125.73 0)
+			(effects
+				(font
+					(size 1.27 1.27)
+				)
+				(justify left)
+			)
+		)
+		(property "Value" "Panel"
+			(at 27.94 128.27 0)
+			(effects
+				(font
+					(size 1.27 1.27)
+				)
+				(justify left)
+			)
+		)
+		(property "Footprint" "Krecek:Panel"
+			(at 25.4 127 0)
+			(effects
+				(font
+					(size 1.27 1.27)
+				)
+				(hide yes)
+			)
+		)
+		(property "Datasheet" "~"
+			(at 25.4 127 0)
+			(effects
+				(font
+					(size 1.27 1.27)
+				)
+				(hide yes)
+			)
+		)
+		(property "Description" ""
+			(at 25.4 127 0)
+			(effects
+				(font
+					(size 1.27 1.27)
+				)
+				(hide yes)
+			)
+		)
+		(instances
+			(project "krecek-0.9"
+				(path "/8888f37b-ecc2-47df-8824-4b4e1e726451"
+					(reference "TFT1")
 					(unit 1)
 				)
@@
 		(dnp no)
 		(fields_autoplaced yes)
-		(property "Reference" "H7"
+		(property "Reference" "H8"
 			(at 27.94 189.23 0)
 			(effects
@@
 			(project "krecek-0.9"
 				(path "/8888f37b-ecc2-47df-8824-4b4e1e726451"
-					(reference "H7")
+					(reference "H8")
 					(unit 1)
 				)
@@
 		(dnp no)
 		(fields_autoplaced yes)
-		(property "Reference" "H4"
+		(property "Reference" "H5"
 			(at 53.34 163.83 0)
 			(effects
@@
 			(project "krecek-0.9"
 				(path "/8888f37b-ecc2-47df-8824-4b4e1e726451"
-					(reference "H4")
+					(reference "H5")
 					(unit 1)
 				)
@@
 		(dnp no)
 		(fields_autoplaced yes)
-		(property "Reference" "H3"
+		(property "Reference" "H4"
 			(at 27.94 163.83 0)
 			(effects
@@
 			(project "krecek-0.9"
 				(path "/8888f37b-ecc2-47df-8824-4b4e1e726451"
-					(reference "H3")
+					(reference "H4")
 					(unit 1)
 				)
@@
 		(dnp no)
 		(fields_autoplaced yes)
-		(property "Reference" "H5"
+		(property "Reference" "H6"
 			(at 27.94 176.53 0)
 			(effects
@@
 			(project "krecek-0.9"
 				(path "/8888f37b-ecc2-47df-8824-4b4e1e726451"
-					(reference "H5")
+					(reference "H6")
 					(unit 1)
 				)
@@
 		(dnp no)
 		(fields_autoplaced yes)
-		(property "Reference" "H8"
+		(property "Reference" "H9"
 			(at 53.34 189.23 0)
 			(effects
@@
 			(project "krecek-0.9"
 				(path "/8888f37b-ecc2-47df-8824-4b4e1e726451"
-					(reference "H8")
+					(reference "H9")
 					(unit 1)
 				)
@@
 			)
 		)
-		(pin "AMP_{EN}" output
-			(at 139.7 93.98 180)
-			(effects
-				(font
-					(size 1.27 1.27)
-				)
-				(justify left)
-			)
-		)
 		(pin "RF_{XOSC}" output
 			(at 165.1 114.3 0)
@@
 			(effects
 				(font
-					(size 1.27 1.27)
-				)
-				(justify right)
-			)
-		)
-		(pin "AMP_{EN}" input
-			(at 114.3 93.98 0)
-			(effects
-				(font

Commit message: Work on board layout
Parts:
- renumbered H2 to H1, H3 to H2, H4 to H3, H5 to H4, H6 to H5, H7 to H6, H8 to H7, H9 to H8
Changed lines of the file:
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@@
 		(dnp no)
 		(fields_autoplaced yes)
-		(property "Reference" "H7"
+		(property "Reference" "H6"
 			(at 53.34 176.53 0)
 			(effects
@@
 			(project "krecek-0.9"
 				(path "/8888f37b-ecc2-47df-8824-4b4e1e726451"
-					(reference "H7")
+					(reference "H6")
 					(unit 1)
 				)
@@
 		(dnp no)
 		(fields_autoplaced yes)
-		(property "Reference" "H3"
+		(property "Reference" "H2"
 			(at 53.34 151.13 0)
 			(effects
@@
 			(project "krecek-0.9"
 				(path "/8888f37b-ecc2-47df-8824-4b4e1e726451"
-					(reference "H3")
+					(reference "H2")
 					(unit 1)
 				)
@@
 		(dnp no)
 		(fields_autoplaced yes)
-		(property "Reference" "H2"
+		(property "Reference" "H1"
 			(at 27.94 151.13 0)
 			(effects
@@
 			(project "krecek-0.9"
 				(path "/8888f37b-ecc2-47df-8824-4b4e1e726451"
-					(reference "H2")
+					(reference "H1")
 					(unit 1)
 				)
@@
 		(dnp no)
 		(fields_autoplaced yes)
-		(property "Reference" "H8"
+		(property "Reference" "H7"
 			(at 27.94 189.23 0)
 			(effects
@@
 			(project "krecek-0.9"
 				(path "/8888f37b-ecc2-47df-8824-4b4e1e726451"
-					(reference "H8")
+					(reference "H7")
 					(unit 1)
 				)
@@
 		(dnp no)
 		(fields_autoplaced yes)
-		(property "Reference" "H5"
+		(property "Reference" "H4"
 			(at 53.34 163.83 0)
 			(effects
@@
 			(project "krecek-0.9"
 				(path "/8888f37b-ecc2-47df-8824-4b4e1e726451"
-					(reference "H5")
+					(reference "H4")
 					(unit 1)
 				)
@@
 		(dnp no)
 		(fields_autoplaced yes)
-		(property "Reference" "H4"
+		(property "Reference" "H3"
 			(at 27.94 163.83 0)
 			(effects
@@
 			(project "krecek-0.9"
 				(path "/8888f37b-ecc2-47df-8824-4b4e1e726451"
-					(reference "H4")
+					(reference "H3")
 					(unit 1)
 				)
@@
 		(dnp no)
 		(fields_autoplaced yes)
-		(property "Reference" "H6"
+		(property "Reference" "H5"
 			(at 27.94 176.53 0)
 			(effects
@@
 			(project "krecek-0.9"
 				(path "/8888f37b-ecc2-47df-8824-4b4e1e726451"
-					(reference "H6")
+					(reference "H5")
 					(unit 1)
 				)
@@
 		(dnp no)
 		(fields_autoplaced yes)
-		(property "Reference" "H9"
+		(property "Reference" "H8"
 			(at 53.34 189.23 0)
 			(effects
@@
 			(project "krecek-0.9"
 				(path "/8888f37b-ecc2-47df-8824-4b4e1e726451"
-					(reference "H9")
-					(unit 1)
-				)
+					(reference "H8")
+					(unit 1)
+				)

Commit message: Route more parts of the board
Other:
- sheet Display ports: added none; removed TFT_{LED}
- sheet RP2040 ports: added none; removed TFT_{LED}
Changed lines of the file:
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@@
 	(wire
 		(pts
-			(xy 165.1 109.22) (xy 190.5 109.22)
+			(xy 165.1 106.68) (xy 190.5 106.68)
 		)
 		(stroke
@@
 		(pts
 			(xy 229.87 132.08) (xy 229.87 111.76)
-		)
-		(stroke
-			(width 0)
-			(type default)
-		)
-	)
-	(wire
-		(pts
-			(xy 165.1 106.68) (xy 190.5 106.68)
 		)
 		(stroke
@@
 		)
 		(pin "TFT_{MISO}" input
-			(at 190.5 109.22 180)
+			(at 190.5 106.68 180)
 			(effects
 				(font
@@
 				)
 				(justify right)
-			)
-		)
-		(pin "TFT_{LED}" input
-			(at 190.5 106.68 180)
-			(effects
-				(font
-					(size 1.27 1.27)
-				)
-				(justify left)
 			)
 		)
@@
 			)
 		)
-		(pin "TFT_{LED}" output
-			(at 165.1 106.68 0)
-			(effects
-				(font
-					(size 1.27 1.27)
-				)
-				(justify right)
-			)
-		)
 		(pin "TFT_{SCK}" output
 			(at 165.1 104.14 0)
@@
 		)
 		(pin "TFT_{MISO}" input
-			(at 165.1 109.22 0)
-			(effects
-				(font
+			(at 165.1 106.68 0)
+			(effects
+				(font
