File: hw/krecek-0.9/rp2040.kicad_sch (KiCad schematic)
At the start: 10 parts, among them U1 RP2040, U2 W25Q128JVS, U4 XL9555, X1 X322512MSB4SI

Commit message: More work on power supply section
Connections:
- net CHGR_{ISET2} renamed CHG_{ISET2}
Changed lines of the file:
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@@
-    (effects (font (size 1.27 1.27)) (justify right bottom))
-  )
-  (label "CHGR_{ISET2}" (at 185.42 63.5 180) (fields_autoplaced)
     (effects (font (size 1.27 1.27)) (justify right bottom))
   )
@@
     (effects (font (size 1.27 1.27)) (justify left bottom))
   )
+  (hierarchical_label "CHG_{ISET2}" (shape output) (at 185.42 63.5 0) (fields_autoplaced)
+    (effects (font (size 1.27 1.27)) (justify left))
+  )
   (symbol (lib_id "Device:R_Small") (at 161.29 167.64 90) (unit 1)

Commit message: Expand hardware design to cover more areas
Signed-off-by: Jan Hamal Dvořák <mordae@anilinux.org>
Connections:
- net XOUT: now also U1.21 (XOUT)
- net OFF: now reaches U4.15 (IO1_2)
- net JOY_{BTN} renamed JOY_{SW}
- no-connect marks 7 -> 6
Changed lines of the file:
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@@
   )
   (no_connect (at 175.26 76.2))
-  (no_connect (at 175.26 68.58))
   (no_connect (at 175.26 73.66))
   (no_connect (at 175.26 78.74))
@@
     (stroke (width 0) (type default))
   )
+  (wire (pts (xy 175.26 68.58) (xy 185.42 68.58))
+    (stroke (width 0) (type default))
+  )
   (wire (pts (xy 85.09 49.53) (xy 95.25 49.53))
     (stroke (width 0) (type default))
@@
     (stroke (width 0) (type default))
   )
+  (wire (pts (xy 25.4 97.79) (xy 34.29 97.79))
+    (stroke (width 0) (type default))
+  )
   (wire (pts (xy 109.22 157.48) (xy 109.22 162.56))
     (stroke (width 0) (type default))
@@
     (stroke (width 0) (type default))
   )
-  (label "BTN_{B}" (at 95.25 97.79 180) (fields_autoplaced)
-    (effects (font (size 1.27 1.27)) (justify right bottom))
-  )
   (label "QSPI_SS" (at 25.4 59.69 0) (fields_autoplaced)
     (effects (font (size 1.27 1.27)) (justify left bottom))
@@
     (effects (font (size 1.27 1.27)) (justify right bottom))
   )
-  (label "TFT_{SCK}" (at 95.25 46.99 180) (fields_autoplaced)
-    (effects (font (size 1.27 1.27)) (justify right bottom))
-  )
   (label "IR_{TX}" (at 95.25 87.63 180) (fields_autoplaced)
     (effects (font (size 1.27 1.27)) (justify right bottom))
@@
     (effects (font (size 1.27 1.27)) (justify right bottom))
   )
-  (label "TFT_{RST}" (at 185.42 40.64 180) (fields_autoplaced)
-    (effects (font (size 1.27 1.27)) (justify right bottom))
-  )
   (label "SD_{MISO}" (at 95.25 62.23 180) (fields_autoplaced)
     (effects (font (size 1.27 1.27)) (justify right bottom))
@@
     (effects (font (size 1.27 1.27)) (justify right bottom))
   )
-  (label "TFT_{MISO}" (at 95.25 41.91 180) (fields_autoplaced)
-    (effects (font (size 1.27 1.27)) (justify right bottom))
-  )
   (label "AMP_{SHDN}" (at 185.42 50.8 180) (fields_autoplaced)
     (effects (font (size 1.27 1.27)) (justify right bottom))
@@
     (effects (font (size 1.27 1.27)) (justify right bottom))
   )
+  (label "XOUT" (at 25.4 97.79 0) (fields_autoplaced)
+    (effects (font (size 1.27 1.27)) (justify left bottom))
+  )
   (label "SD_{SCLK}" (at 95.25 67.31 180) (fields_autoplaced)
     (effects (font (size 1.27 1.27)) (justify right bottom))
@@
     (effects (font (size 1.27 1.27)) (justify right bottom))
   )
-  (label "TFT_{LED}" (at 95.25 105.41 180) (fields_autoplaced)
-    (effects (font (size 1.27 1.27)) (justify right bottom))
-  )
   (label "VOL_{DOWN}" (at 185.42 55.88 180) (fields_autoplaced)
     (effects (font (size 1.27 1.27)) (justify right bottom))
   )
-  (label "BTN_{SELECT}" (at 185.42 48.26 180) (fields_autoplaced)
-    (effects (font (size 1.27 1.27)) (justify right bottom))
-  )
   (label "XIN" (at 26.67 172.72 0) (fields_autoplaced)
     (effects (font (size 1.27 1.27)) (justify left bottom))
@@
     (effects (font (size 1.27 1.27)) (justify right bottom))
   )
-  (label "BTN_{A}" (at 95.25 95.25 180) (fields_autoplaced)
-    (effects (font (size 1.27 1.27)) (justify right bottom))
-  )
   (label "VOL_{UP}" (at 185.42 53.34 180) (fields_autoplaced)
     (effects (font (size 1.27 1.27)) (justify right bottom))
   )
-  (label "JOY_{BTN}" (at 185.42 43.18 180) (fields_autoplaced)
-    (effects (font (size 1.27 1.27)) (justify right bottom))
-  )
-  (label "TFT_{CS}" (at 95.25 44.45 180) (fields_autoplaced)
-    (effects (font (size 1.27 1.27)) (justify right bottom))
-  )
   (label "QSPI_SD3" (at 129.54 180.34 0) (fields_autoplaced)
     (effects (font (size 1.27 1.27)) (justify left bottom))
@@
     (effects (font (size 1.27 1.27)) (justify left bottom))
   )
-  (label "RF_{CS}" (at 95.25 54.61 180) (fields_autoplaced)
-    (effects (font (size 1.27 1.27)) (justify right bottom))
-  )
-  (label "BTN_{Y}" (at 95.25 59.69 180) (fields_autoplaced)
-    (effects (font (size 1.27 1.27)) (justify right bottom))
-  )
-  (label "TFT_{RS}" (at 95.25 52.07 180) (fields_autoplaced)
-    (effects (font (size 1.27 1.27)) (justify right bottom))
-  )
   (label "DSP_{ASDOUT}" (at 95.25 77.47 180) (fields_autoplaced)
     (effects (font (size 1.27 1.27)) (justify right bottom))
@@
     (effects (font (size 1.27 1.27)) (justify right bottom))
   )
-  (label "TFT_{MOSI}" (at 95.25 49.53 180) (fields_autoplaced)
-    (effects (font (size 1.27 1.27)) (justify right bottom))
-  )
-  (label "JOY_{Y}" (at 95.25 113.03 180) (fields_autoplaced)
-    (effects (font (size 1.27 1.27)) (justify right bottom))
-  )
   (label "QSPI_SD2" (at 129.54 177.8 0) (fields_autoplaced)
     (effects (font (size 1.27 1.27)) (justify left bottom))
@@
     (effects (font (size 1.27 1.27)) (justify right bottom))
   )
-  (label "BTN_{START}" (at 185.42 45.72 180) (fields_autoplaced)
-    (effects (font (size 1.27 1.27)) (justify right bottom))
-  )
-  (label "BTN_{X}" (at 95.25 57.15 180) (fields_autoplaced)
-    (effects (font (size 1.27 1.27)) (justify right bottom))
-  )
   (label "DSP_{DSDIN}" (at 95.25 80.01 180) (fields_autoplaced)
     (effects (font (size 1.27 1.27)) (justify right bottom))
@@
     (effects (font (size 1.27 1.27)) (justify left bottom))
   )
-  (label "JOY_{X}" (at 95.25 110.49 180) (fields_autoplaced)
-    (effects (font (size 1.27 1.27)) (justify right bottom))
-  )
   (label "QSPI_SD1" (at 25.4 67.31 0) (fields_autoplaced)
     (effects (font (size 1.27 1.27)) (justify left bottom))
@@
     (effects (font (size 1.27 1.27)) (justify left bottom))
   )
+  (hierarchical_label "TFT_{LED}" (shape output) (at 95.25 105.41 0) (fields_autoplaced)
+    (effects (font (size 1.27 1.27)) (justify left))
+  )
+  (hierarchical_label "JOY_{Y}" (shape input) (at 95.25 113.03 0) (fields_autoplaced)
+    (effects (font (size 1.27 1.27)) (justify left))
+  )
+  (hierarchical_label "BTN_{SELECT}" (shape input) (at 185.42 48.26 0) (fields_autoplaced)
+    (effects (font (size 1.27 1.27)) (justify left))
+  )
+  (hierarchical_label "BTN_{Y}" (shape input) (at 95.25 59.69 0) (fields_autoplaced)
+    (effects (font (size 1.27 1.27)) (justify left))
+  )
+  (hierarchical_label "JOY_{X}" (shape input) (at 95.25 110.49 0) (fields_autoplaced)
+    (effects (font (size 1.27 1.27)) (justify left))
+  )
+  (hierarchical_label "BTN_{A}" (shape input) (at 95.25 95.25 0) (fields_autoplaced)
+    (effects (font (size 1.27 1.27)) (justify left))
+  )
+  (hierarchical_label "BTN_{START}" (shape input) (at 185.42 45.72 0) (fields_autoplaced)
+    (effects (font (size 1.27 1.27)) (justify left))
+  )
   (hierarchical_label "CHG_{ISET2}" (shape output) (at 185.42 63.5 0) (fields_autoplaced)
     (effects (font (size 1.27 1.27)) (justify left))
   )
+  (hierarchical_label "OFF" (shape output) (at 185.42 68.58 0) (fields_autoplaced)
+    (effects (font (size 1.27 1.27)) (justify left))
+  )
+  (hierarchical_label "TFT_{RST}" (shape output) (at 185.42 40.64 0) (fields_autoplaced)
+    (effects (font (size 1.27 1.27)) (justify left))
+  )
+  (hierarchical_label "TFT_{CS}" (shape output) (at 95.25 44.45 0) (fields_autoplaced)
+    (effects (font (size 1.27 1.27)) (justify left))
+  )
+  (hierarchical_label "BTN_{X}" (shape input) (at 95.25 57.15 0) (fields_autoplaced)
+    (effects (font (size 1.27 1.27)) (justify left))
+  )
+  (hierarchical_label "TFT_{MISO}" (shape input) (at 95.25 41.91 0) (fields_autoplaced)
+    (effects (font (size 1.27 1.27)) (justify left))
+  )
+  (hierarchical_label "TFT_{MOSI}" (shape output) (at 95.25 49.53 0) (fields_autoplaced)
+    (effects (font (size 1.27 1.27)) (justify left))
+  )
+  (hierarchical_label "TFT_{SCK}" (shape output) (at 95.25 46.99 0) (fields_autoplaced)
+    (effects (font (size 1.27 1.27)) (justify left))
+  )
+  (hierarchical_label "BTN_{B}" (shape input) (at 95.25 97.79 0) (fields_autoplaced)
+    (effects (font (size 1.27 1.27)) (justify left))
+  )
+  (hierarchical_label "JOY_{SW}" (shape input) (at 185.42 43.18 0) (fields_autoplaced)
+    (effects (font (size 1.27 1.27)) (justify left))
+  )
+  (hierarchical_label "TFT_{RS}" (shape output) (at 95.25 52.07 0) (fields_autoplaced)
+    (effects (font (size 1.27 1.27)) (justify left))
+  )
+  (hierarchical_label "RF_{CS}" (shape output) (at 95.25 54.61 0) (fields_autoplaced)
+    (effects (font (size 1.27 1.27)) (justify left))
+  )

Commit message: Update schematic
Signed-off-by: Jan Hamal Dvořák <mordae@anilinux.org>
Parts:
- added C3: 100n, Capacitor_SMD:C_0402_1005Metric, symbol Device:C_Small
- added R25, R26: 27, Resistor_SMD:R_0603_1608Metric, symbol Device:R_Small
- added SW5: SW_Push, LCSC:SW-SMD_4P-L5.1-W5.1-P3.70-LS6.5-TL-2, symbol Switch:SW_Push
- C1, C2: value 27p -> 33p; footprint (none) -> Capacitor_SMD:C_0402_1005Metric; LCSC Part (none) -> C1562
- C3: footprint (none) -> Capacitor_SMD:C_0402_1005Metric; LCSC Part (none) -> C307331
- R1, R3: footprint (none) -> Resistor_SMD:R_0402_1005Metric; LCSC Part (none) -> C11702
- R2: footprint (none) -> Capacitor_SMD:C_0402_1005Metric; LCSC Part (none) -> C25779
Connections:
- net +3V3: now also C3.1
- net GND: now also U1.19 (TESTEN), U1.57 (GND), C3.2, SW5.2
- net at R3.2: now also SW5.1
- net at U1.46 (USB_DM): now also R26.2
- net at U1.47 (USB_DP): now also R25.2
- new net USB_{D+}: R25.1
- new net USB_{D-}: R26.1
Other:
- moved on the sheet: C1, C2, C3, R1, R2, R3, U1, U2, U4

Commit message: Further tweaks and improvements
- Use a nicer schematic template
- Tie START button with power on
- Add ferrite to USB shield
- Add CC1/CC2 makeshift ADC
- Tidy up schematics a little bit

Signed-off-by: Jan Hamal Dvořák <mordae@anilinux.org>
Parts:
- removed C2: 33p, Capacitor_SMD:C_0402_1005Metric, symbol Device:C_Small
- added C1: 33p, Capacitor_SMD:C_0402_1005Metric, symbol Device:C_Small
Connections:
- net GND: now also C1.1, C1.2; no longer C1.2
- net XIN: now also C1.1
- net XOUT: now also R1.2; no longer R1.1
- new net: C1.2, R1.1, X1.3 (OSC2)
Other:
- company: (none) -> DDM Spirála
- title: (none) -> Křeček
- moved on the sheet: C1, C3, R1, R2, R25, R26, R3, SW5, U1, U2, U4

Commit message: TRRS audio connector
Signed-off-by: Jan Hamal Dvořák <mordae@anilinux.org>
Connections:
- net BRACK_{L}: no longer U1.35 (GPIO23)
- net BRACK_{R}: no longer U1.36 (GPIO24)
- net BTN_{A}: no longer U1.32 (GPIO21)
- net BTN_{B}: no longer U1.34 (GPIO22)
- net BTN_{X}: no longer U1.8 (GPIO6)
- net BTN_{Y}: no longer U1.9 (GPIO7)
- net USB_{CC1}: no longer U1.30 (GPIO19)
- net USB_{CC2}: no longer U1.31 (GPIO20)
Changed lines of the file:
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@@
     (stroke (width 0) (type default))
   )
-  (wire (pts (xy 95.25 118.11) (xy 105.41 118.11))
+  (wire (pts (xy 144.78 118.11) (xy 154.94 118.11))
     (stroke (width 0) (type default))
   )
@@
     (stroke (width 0) (type default))
   )
-  (wire (pts (xy 95.25 120.65) (xy 105.41 120.65))
+  (wire (pts (xy 144.78 120.65) (xy 154.94 120.65))
     (stroke (width 0) (type default))
   )
@@
     (stroke (width 0) (type default))
   )
-  (wire (pts (xy 95.25 107.95) (xy 105.41 107.95))
+  (wire (pts (xy 144.78 107.95) (xy 154.94 107.95))
     (stroke (width 0) (type default))
   )
@@
     (stroke (width 0) (type default))
   )
-  (wire (pts (xy 95.25 110.49) (xy 105.41 110.49))
+  (wire (pts (xy 144.78 110.49) (xy 154.94 110.49))
     (stroke (width 0) (type default))
   )
@@
     (stroke (width 0) (type default))
   )
-  (wire (pts (xy 95.25 115.57) (xy 105.41 115.57))
+  (wire (pts (xy 144.78 100.33) (xy 154.94 100.33))
     (stroke (width 0) (type default))
   )
@@
     (stroke (width 0) (type default))
   )
-  (wire (pts (xy 95.25 113.03) (xy 105.41 113.03))
+  (wire (pts (xy 144.78 97.79) (xy 154.94 97.79))
     (stroke (width 0) (type default))
   )
@@
     (stroke (width 0) (type default))
   )
-  (wire (pts (xy 95.25 74.93) (xy 105.41 74.93))
+  (wire (pts (xy 144.78 102.87) (xy 154.94 102.87))
     (stroke (width 0) (type default))
   )
@@
     (stroke (width 0) (type default))
   )
-  (wire (pts (xy 95.25 77.47) (xy 105.41 77.47))
+  (wire (pts (xy 144.78 105.41) (xy 154.94 105.41))
     (stroke (width 0) (type default))
   )
@@
     (effects (font (size 1.27 1.27)) (justify left bottom))
   )
-  (label "BRACK_{R}" (at 105.41 120.65 180) (fields_autoplaced)
+  (label "BRACK_{R}" (at 154.94 120.65 180) (fields_autoplaced)
     (effects (font (size 1.27 1.27)) (justify right bottom))
   )
@@
     (effects (font (size 1.27 1.27)) (justify right bottom))
   )
-  (label "BRACK_{L}" (at 105.41 118.11 180) (fields_autoplaced)
+  (label "BRACK_{L}" (at 154.94 118.11 180) (fields_autoplaced)
     (effects (font (size 1.27 1.27)) (justify right bottom))
   )
@@
     (effects (font (size 1.27 1.27)) (justify left))
   )
-  (hierarchical_label "BTN_{Y}" (shape input) (at 105.41 77.47 0) (fields_autoplaced)
+  (hierarchical_label "BTN_{Y}" (shape input) (at 154.94 105.41 0) (fields_autoplaced)
     (effects (font (size 1.27 1.27)) (justify left))
   )
@@
     (effects (font (size 1.27 1.27)) (justify left))
   )
-  (hierarchical_label "BTN_{A}" (shape input) (at 105.41 113.03 0) (fields_autoplaced)
-    (effects (font (size 1.27 1.27)) (justify left))
-  )
-  (hierarchical_label "USB_{CC1}" (shape input) (at 105.41 107.95 0) (fields_autoplaced)
+  (hierarchical_label "BTN_{A}" (shape input) (at 154.94 97.79 0) (fields_autoplaced)
+    (effects (font (size 1.27 1.27)) (justify left))
+  )
+  (hierarchical_label "USB_{CC1}" (shape input) (at 154.94 107.95 0) (fields_autoplaced)
     (effects (font (size 1.27 1.27)) (justify left))
   )
@@
     (effects (font (size 1.27 1.27)) (justify left))
   )
-  (hierarchical_label "BTN_{X}" (shape input) (at 105.41 74.93 0) (fields_autoplaced)
-    (effects (font (size 1.27 1.27)) (justify left))
-  )
-  (hierarchical_label "USB_{CC2}" (shape input) (at 105.41 110.49 0) (fields_autoplaced)
+  (hierarchical_label "BTN_{X}" (shape input) (at 154.94 102.87 0) (fields_autoplaced)
+    (effects (font (size 1.27 1.27)) (justify left))
+  )
+  (hierarchical_label "USB_{CC2}" (shape input) (at 154.94 110.49 0) (fields_autoplaced)
     (effects (font (size 1.27 1.27)) (justify left))
   )
@@
     (effects (font (size 1.27 1.27)) (justify left))
   )
-  (hierarchical_label "BTN_{B}" (shape input) (at 105.41 115.57 0) (fields_autoplaced)
-    (effects (font (size 1.27 1.27)) (justify left))
-  )
+  (hierarchical_label "BTN_{B}" (shape input) (at 154.94 100.33 0) (fields_autoplaced)
+    (effects (font (size 1.27 1.27)) (justify left))
+  )

Commit message: Complete most of the design, except for RF
Signed-off-by: Jan Hamal Dvořák <mordae@anilinux.org>
Parts:
- removed C3: 100n, Capacitor_SMD:C_0402_1005Metric, symbol Device:C_Small
- removed U4: XL9555, LCSC:TSSOP-24_L7.8-W4.4-P0.65-LS6.4-BL, symbol LCSC:XL9555
- removed X1: X322512MSB4SI, LCSC:OSC-SMD_4P-L3.2-W2.5-BL, symbol LCSC:X322512MSB4SI
- added C6 (x22): 10u, Capacitor_SMD:C_0402_1005Metric, symbol Device:C_Small
- added J1: DAP, Connector_PinHeader_2.54mm:PinHeader_1x03_P2.54mm_Vertical, symbol Connector:Conn_01x03_Pin
- added J2: AUX, Connector_PinHeader_2.54mm:PinHeader_2x08_P2.54mm_Vertical, symbol Connector_Generic:Conn_02x08_Odd_Even
- added U1: RP2040, Package_DFN_QFN:QFN-56-1EP_7x7mm_P0.4mm_EP3.2x3.2mm, symbol MCU_RaspberryPi:RP2040
- added Y1: 12MHz, LCSC:OSC-SMD_4P-L3.2-W2.5-BL, symbol Device:Crystal_GND24
- renumbered R25 to R1, R26 to R2, SW5 to SW1
Connections:
- net DSP_{DSDIN} is gone; now on net DSP_{ASDOUT}: U1.18 (GPIO15)
- net +3.3V: now also U1.1 (IOVDD), U1.10 (IOVDD), U1.22 (IOVDD), U1.33 (IOVDD), U1.42 (IOVDD), U1.43 (ADC_AVDD), U1.44 (VREG_IN), U1.48 (USB_VDD), U1.49 (IOVDD), C6.1, C6.1, C6.1, C6.1, C6.1, C6.1, C6.1, C6.1, C6.1, C6.1, C6.1, C6.1, C6.1, C6.1, C6.1, C6.1, J2.2 (Pin_2), U1.1 (IOVDD), U1.10 (IOVDD), U1.22 (IOVDD), U1.33 (IOVDD), U1.42 (IOVDD), U1.43 (ADC_AVDD), U1.44 (VREG_IN), U1.48 (USB_VDD), U1.49 (IOVDD)
- net BRACK_{L}: now also U1.40 (GPIO28_ADC2)
- net BRACK_{R}: now also U1.41 (GPIO29_ADC3)
- net BTN_{A}: now also U1.34 (GPIO22)
- net BTN_{B}: now also U1.35 (GPIO23)
- net BTN_{SELECT}: now also U1.32 (GPIO21)
- net BTN_{START}: now also U1.31 (GPIO20)
- net BTN_{X}: now also U1.36 (GPIO24)
- net BTN_{Y}: now also U1.37 (GPIO25)
- net CHG_{ISET2}: now also U1.9 (GPIO7)
- net DSP_{ASDOUT}: no longer U1.17 (GPIO14)
- net GND: now also C1.1, C6.2, C6.2, C6.2, C6.2, C6.2, C6.2, C6.2, C6.2, C6.2, C6.2, C6.2, C6.2, C6.2, C6.2, C6.2, C6.2, C6.2, C6.2, C6.2, C6.2, C6.2, C6.2, J1.2 (Pin_2), J2.10 (Pin_10), J2.15 (Pin_15), J2.16 (Pin_16), J2.3 (Pin_3), J2.4 (Pin_4), J2.9 (Pin_9), U1.19 (TESTEN), U1.57 (GND), Y1.2, Y1.4; no longer C1.2
- net JOY_{SW}: now also U1.30 (GPIO19)
- net JOY_{X}: now also U1.38 (GPIO26_ADC0); no longer U1.38 (GPIO26_ADC0)
- net JOY_{Y}: now also U1.39 (GPIO27_ADC1); no longer U1.39 (GPIO27_ADC1)
- net OFF: now also U1.16 (GPIO13)
- net TFT_{LED}: now also U1.17 (GPIO14); no longer U1.37 (GPIO25)
- net TFT_{RST}: now also U1.8 (GPIO6)
- net USB_{CC1}: now also U1.38 (GPIO26_ADC0)
- net USB_{CC2}: now also U1.39 (GPIO27_ADC1)
- net VOL_{DOWN}: now also U1.28 (GPIO17)
- net VOL_{UP}: now also U1.27 (GPIO16)
- net XIN: now also C1.2, Y1.1; no longer C1.1
- net at C1.2, R1.1: now also Y1.3
- net at U1.23 (DVDD), U1.50 (DVDD): now also U1.45 (VREG_VOUT), C6.1, C6.1, C6.1
- net at U1.24 (SWCLK): now also J1.3 (Pin_3)
- net at U1.25 (SWD): now also J1.1 (Pin_1)
- net BUS0: now reaches U1.30 (GPIO19)
- net BUS0: now also U1.7 (GPIO5)
- net BUS1: now reaches U1.31 (GPIO20)
- net BUS1: now also U1.8 (GPIO6)
- net BUS2: now reaches U1.32 (GPIO21)
- net BUS2: now also U1.9 (GPIO7)
- net BUS3: now reaches U1.34 (GPIO22)
- net BUS3: now also U1.11 (GPIO8)
- net at U1.35 (GPIO23): now also U1.20 (XIN)
- net at U1.36 (GPIO24): now also U1.24 (SWCLK)
- net HP_{ctrl} renamed HP_{SENSE}
- net SCL renamed DSP_{CCLK}
- net SDA renamed DSP_{CDATA}
- new net: C6.1, C6.1, C6.1, U1.23 (DVDD), U1.45 (VREG_VOUT), U1.50 (DVDD)
- new net: U1.25 (SWD), U1.37 (GPIO25)
- new net +5V: J2.1 (Pin_1)
- new net AMP_{EN}: U1.18 (GPIO15)
- new net AUX0: J2.6 (Pin_6), U1.12 (GPIO9)
- new net AUX1: J2.8 (Pin_8), U1.13 (GPIO10)
- new net AUX2: J2.12 (Pin_12), U1.14 (GPIO11)
- new net AUX3: J2.14 (Pin_14), U1.15 (GPIO12)
- new net AUX4: J2.5 (Pin_5), U1.53 (QSPI_SD0)
- new net AUX5: J2.7 (Pin_7), U1.55 (QSPI_SD1)
- new net AUX6: J2.11 (Pin_11), U1.54 (QSPI_SD2)
- new net AUX7: J2.13 (Pin_13), U1.51 (QSPI_SD3)
- new net DSP_{ASDIN}: U1.17 (GPIO14)
- new net T_{CS}: U1.3 (GPIO1)
- new net T_{IRQ}: U1.6 (GPIO4)
- new net T_{MISO}: U1.2 (GPIO0)
- new net T_{MOSI}: U1.5 (GPIO3)
- new net T_{SCK}: U1.4 (GPIO2)
- new net VOL_{SW}: U1.29 (GPIO18)
- no-connect marks 6 -> 7
Other:
- moved on the sheet: C1, C3, R1, R2, R3, SW1, U1, U2

Commit message: Complete the RF section
Connections:
- net AMP_{EN}: now also U1.17 (GPIO14); no longer U1.18 (GPIO15)
- net BTN_{SELECT}: now also U1.31 (GPIO20); no longer U1.32 (GPIO21)
- net BTN_{START}: now also U1.30 (GPIO19); no longer U1.31 (GPIO20)
- net JOY_{SW}: now also U1.29 (GPIO18); no longer U1.30 (GPIO19)
- net OFF: now also U1.52 (QSPI_SCLK); no longer U1.16 (GPIO13)
- net TFT_{LED}: now also U1.16 (GPIO13); no longer U1.17 (GPIO14)
- net VOL_{DOWN}: now also U1.27 (GPIO16); no longer U1.28 (GPIO17)
- net VOL_{SW}: now also U1.28 (GPIO17); no longer U1.29 (GPIO18)
- net VOL_{UP}: now also U1.18 (GPIO15); no longer U1.27 (GPIO16)
- new net RF_{CLK}: U1.32 (GPIO21)
- no-connect marks 7 -> 6
Changed lines of the file:
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@@
   (no_connect (at 177.8 71.12))
   (no_connect (at 50.8 53.34))
-  (no_connect (at 177.8 86.36))
   (no_connect (at 177.8 53.34))
   (no_connect (at 177.8 109.22))
@@
     (effects (font (size 1.27 1.27)) (justify left bottom))
   )
-  (hierarchical_label "TFT_{LED}" (shape output) (at 228.6 88.9 0) (fields_autoplaced)
+  (hierarchical_label "TFT_{LED}" (shape output) (at 228.6 86.36 0) (fields_autoplaced)
     (effects (font (size 1.27 1.27)) (justify left))
   )
@@
     (effects (font (size 1.27 1.27)) (justify left))
   )
-  (hierarchical_label "BTN_{SELECT}" (shape input) (at 228.6 106.68 0) (fields_autoplaced)
+  (hierarchical_label "BTN_{SELECT}" (shape input) (at 228.6 104.14 0) (fields_autoplaced)
     (effects (font (size 1.27 1.27)) (justify left))
   )
@@
     (effects (font (size 1.27 1.27)) (justify left))
   )
-  (hierarchical_label "VOL_{UP}" (shape input) (at 228.6 93.98 0) (fields_autoplaced)
+  (hierarchical_label "VOL_{UP}" (shape input) (at 228.6 91.44 0) (fields_autoplaced)
     (effects (font (size 1.27 1.27)) (justify left))
   )
@@
     (effects (font (size 1.27 1.27)) (justify left))
   )
-  (hierarchical_label "BTN_{START}" (shape input) (at 228.6 104.14 0) (fields_autoplaced)
+  (hierarchical_label "BTN_{START}" (shape input) (at 228.6 101.6 0) (fields_autoplaced)
     (effects (font (size 1.27 1.27)) (justify left))
   )
@@
     (effects (font (size 1.27 1.27)) (justify left))
   )
-  (hierarchical_label "OFF" (shape output) (at 228.6 86.36 0) (fields_autoplaced)
-    (effects (font (size 1.27 1.27)) (justify left))
+  (hierarchical_label "OFF" (shape output) (at 177.8 86.36 180) (fields_autoplaced)
+    (effects (font (size 1.27 1.27)) (justify right))
   )
   (hierarchical_label "T_{SCK}" (shape output) (at 228.6 58.42 0) (fields_autoplaced)
@@
     (effects (font (size 1.27 1.27)) (justify left))
   )
-  (hierarchical_label "AMP_{EN}" (shape output) (at 228.6 91.44 0) (fields_autoplaced)
+  (hierarchical_label "AMP_{EN}" (shape output) (at 228.6 88.9 0) (fields_autoplaced)
     (effects (font (size 1.27 1.27)) (justify left))
   )
@@
     (effects (font (size 1.27 1.27)) (justify left))
   )
-  (hierarchical_label "VOL_{SW}" (shape input) (at 228.6 99.06 0) (fields_autoplaced)
+  (hierarchical_label "VOL_{SW}" (shape input) (at 228.6 96.52 0) (fields_autoplaced)
     (effects (font (size 1.27 1.27)) (justify left))
   )
@@
     (effects (font (size 1.27 1.27)) (justify left))
   )
+  (hierarchical_label "RF_{CLK}" (shape output) (at 228.6 106.68 0) (fields_autoplaced)
+    (effects (font (size 1.27 1.27)) (justify left))
+  )
   (hierarchical_label "TFT_{SCK}" (shape output) (at 101.6 58.42 0) (fields_autoplaced)
     (effects (font (size 1.27 1.27)) (justify left))
@@
     (effects (font (size 1.27 1.27)) (justify left))
   )
-  (hierarchical_label "JOY_{SW}" (shape input) (at 228.6 101.6 0) (fields_autoplaced)
+  (hierarchical_label "JOY_{SW}" (shape input) (at 228.6 99.06 0) (fields_autoplaced)
     (effects (font (size 1.27 1.27)) (justify left))
   )
@@
     (effects (font (size 1.27 1.27)) (justify left))
   )
-  (hierarchical_label "VOL_{DOWN}" (shape input) (at 228.6 96.52 0) (fields_autoplaced)
-    (effects (font (size 1.27 1.27)) (justify left))
-  )
+  (hierarchical_label "VOL_{DOWN}" (shape input) (at 228.6 93.98 0) (fields_autoplaced)
+    (effects (font (size 1.27 1.27)) (justify left))
+  )
