File: hw/krecek-0.9/rp2040.kicad_sch (KiCad schematic)
At the start: 37 parts, among them J1 DAP, J2 AUX, SW1 SW_Push, U1 RP2040, U2 W25Q128JVS, Y1 12MHz

Commit message: Add discrete antenna
Signed-off-by: Jan Hamal Dvořák <mordae@anilinux.org>
Parts:
- renumbered C3 to C23, C1 to C24, C1 to C25, R2 to R3, R3 to R4, R1 to R5, U1 to U2, U1 to U3, U2 to U4

Commit message: Further progress with the PCB layout
Signed-off-by: Jan Hamal Dvořák <mordae@anilinux.org>
Connections:
- net USB_{D+} renamed USB+
- net USB_{D-} renamed USB-
Changed lines of the file:
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@@
     (effects (font (size 1.27 1.27)) (justify left))
   )
-  (hierarchical_label "USB_{D-}" (shape bidirectional) (at 19.05 63.5 180) (fields_autoplaced)
+  (hierarchical_label "USB-" (shape bidirectional) (at 19.05 63.5 180) (fields_autoplaced)
     (effects (font (size 1.27 1.27)) (justify right))
   )
@@
     (effects (font (size 1.27 1.27)) (justify left))
   )
-  (hierarchical_label "USB_{D+}" (shape bidirectional) (at 19.05 60.96 180) (fields_autoplaced)
+  (hierarchical_label "USB+" (shape bidirectional) (at 19.05 60.96 180) (fields_autoplaced)
     (effects (font (size 1.27 1.27)) (justify right))
   )

Commit message: Progress on PCB
Signed-off-by: Jan Hamal Dvořák <mordae@anilinux.org>
Connections:
- net BRACK_{L}: now also U3.39 (GPIO27_ADC1); no longer U3.40 (GPIO28_ADC2)
- net BRACK_{R}: now also U3.38 (GPIO26_ADC0); no longer U3.41 (GPIO29_ADC3)
- net BTN_{X}: now also U3.37 (GPIO25); no longer U3.36 (GPIO24)
- net BTN_{Y}: now also U3.36 (GPIO24); no longer U3.37 (GPIO25)
- net JOY_{X}: now also U3.40 (GPIO28_ADC2); no longer U3.38 (GPIO26_ADC0)
- net JOY_{Y}: now also U3.41 (GPIO29_ADC3); no longer U3.39 (GPIO27_ADC1)
Changed lines of the file:
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@@
     (effects (font (size 1.27 1.27)) (justify left))
   )
-  (hierarchical_label "JOY_{Y}" (shape input) (at 228.6 124.46 0) (fields_autoplaced)
+  (hierarchical_label "JOY_{Y}" (shape input) (at 228.6 129.54 0) (fields_autoplaced)
     (effects (font (size 1.27 1.27)) (justify left))
   )
@@
     (effects (font (size 1.27 1.27)) (justify left))
   )
-  (hierarchical_label "BRACK_{L}" (shape input) (at 228.6 127 0) (fields_autoplaced)
+  (hierarchical_label "BRACK_{L}" (shape input) (at 228.6 124.46 0) (fields_autoplaced)
     (effects (font (size 1.27 1.27)) (justify left))
   )
@@
     (effects (font (size 1.27 1.27)) (justify left))
   )
-  (hierarchical_label "BTN_{Y}" (shape input) (at 228.6 116.84 0) (fields_autoplaced)
+  (hierarchical_label "BTN_{Y}" (shape input) (at 228.6 114.3 0) (fields_autoplaced)
     (effects (font (size 1.27 1.27)) (justify left))
   )
-  (hierarchical_label "JOY_{X}" (shape input) (at 228.6 121.92 0) (fields_autoplaced)
+  (hierarchical_label "JOY_{X}" (shape input) (at 228.6 127 0) (fields_autoplaced)
     (effects (font (size 1.27 1.27)) (justify left))
   )
@@
     (effects (font (size 1.27 1.27)) (justify left))
   )
-  (hierarchical_label "BTN_{X}" (shape input) (at 228.6 114.3 0) (fields_autoplaced)
+  (hierarchical_label "BTN_{X}" (shape input) (at 228.6 116.84 0) (fields_autoplaced)
     (effects (font (size 1.27 1.27)) (justify left))
   )
@@
     (effects (font (size 1.27 1.27)) (justify left))
   )
-  (hierarchical_label "BRACK_{R}" (shape input) (at 228.6 129.54 0) (fields_autoplaced)
+  (hierarchical_label "BRACK_{R}" (shape input) (at 228.6 121.92 0) (fields_autoplaced)
     (effects (font (size 1.27 1.27)) (justify left))
   )

Commit message: Hardware as sent for manufacturing
Parts:
- R3: footprint Capacitor_SMD:C_0402_1005Metric -> Resistor_SMD:R_0402_1005Metric
Changed lines of the file:
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@@
+    (stroke (width 0) (type default))
+  )
+  (wire (pts (xy 101.6 116.84) (xy 165.1 116.84))
     (stroke (width 0) (type default))
   )
@@
   )
   (wire (pts (xy 210.82 44.45) (xy 210.82 45.72))
-    (stroke (width 0) (type default))
-  )
-  (wire (pts (xy 101.6 116.84) (xy 165.1 116.84))
     (stroke (width 0) (type default))
   )
@@
       (effects (font (size 1.27 1.27)) (justify left))
     )
-    (property "Footprint" "Capacitor_SMD:C_0402_1005Metric" (at 152.4 156.21 0)
-      (effects (font (size 1.27 1.27)) hide)
-    )
+    (property "Footprint" "Resistor_SMD:R_0402_1005Metric" (at 152.4 156.21 0)
+      (effects (font (size 1.27 1.27)) hide)
+    )

Commit message: Partially resolve some of the design issues
Related to #3 and #4.
Parts:
- added R40: 1k, Resistor_SMD:R_0402_1005Metric, symbol Device:R_Small
Connections:
- net GND: now also R40.1
- net at U3.56 (QSPI_SS): now also R40.2
- no-connect marks 6 -> 5
Changed lines of the file:
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@@
   (junction (at 200.66 44.45) (diameter 0) (color 0 0 0 0)
   )
-  (no_connect (at 177.8 71.12))
   (no_connect (at 50.8 53.34))
   (no_connect (at 177.8 53.34))
@@
     (stroke (width 0) (type default))
   )
+  (wire (pts (xy 152.4 71.12) (xy 162.56 71.12))
+    (stroke (width 0) (type default))
+  )
   (wire (pts (xy 226.06 34.29) (xy 226.06 38.1))
     (stroke (width 0) (type default))
@@
     (stroke (width 0) (type default))
   )
+  (wire (pts (xy 167.64 71.12) (xy 177.8 71.12))
+    (stroke (width 0) (type default))
+  )
   (wire (pts (xy 99.06 25.4) (xy 99.06 29.21))
     (stroke (width 0) (type default))
@@
         )
       )
+    )
+  )
+  (symbol (lib_id "power:GND") (at 152.4 71.12 270) (unit 1)
+    (in_bom yes) (on_board yes) (dnp no) (fields_autoplaced)
+    (property "Reference" "#PWR0113" (at 146.05 71.12 0)
+      (effects (font (size 1.27 1.27)) hide)
+    )
+    (property "Value" "GND" (at 148.59 71.12 90)
+      (effects (font (size 1.27 1.27)) (justify right))
+    )
+    (property "Footprint" "" (at 152.4 71.12 0)
+      (effects (font (size 1.27 1.27)) hide)
+    )
+    (property "Datasheet" "" (at 152.4 71.12 0)
+      (effects (font (size 1.27 1.27)) hide)
+    )
+    (pin "1")
+    (instances
+      (project "krecek-0.9"
+        (path "/8888f37b-ecc2-47df-8824-4b4e1e726451/6537dbea-4e11-4137-b8a0-9ae6b128c4e4"
+          (reference "#PWR0113") (unit 1)
+        )
+      )
+    )
+  )
+  (symbol (lib_id "Device:R_Small") (at 165.1 71.12 90) (unit 1)
+    (in_bom yes) (on_board yes) (dnp no) (fields_autoplaced)
+    (property "Reference" "R40" (at 165.1 66.04 90)
+      (effects (font (size 1.27 1.27)))
+    )
+    (property "Value" "1k" (at 165.1 68.58 90)
+      (effects (font (size 1.27 1.27)))
+    )
+    (property "Footprint" "Resistor_SMD:R_0402_1005Metric" (at 165.1 71.12 0)
+      (effects (font (size 1.27 1.27)) hide)
+    )
+    (property "Datasheet" "~" (at 165.1 71.12 0)
+      (effects (font (size 1.27 1.27)) hide)
+    )
+    (property "LCSC Part" "C11702" (at 165.1 71.12 90)
+      (effects (font (size 1.27 1.27)) hide)
+    )
+    (pin "1")
+    (pin "2")
+    (instances
+      (project "krecek-0.9"
+        (path "/8888f37b-ecc2-47df-8824-4b4e1e726451/6537dbea-4e11-4137-b8a0-9ae6b128c4e4"
+          (reference "R40") (unit 1)
+        )
+      )

Commit message: Fix OFF issues, rename buttons
Resolves #4.
Parts:
- added R41: 1k, Resistor_SMD:R_0402_1005Metric, symbol Device:R_Small
Connections:
- net BTN_{B}: now also U3.36 (GPIO24); no longer U3.35 (GPIO23)
- net BTN_{X}: now also U3.35 (GPIO23); no longer U3.37 (GPIO25)
- net BTN_{Y}: now also U3.37 (GPIO25); no longer U3.36 (GPIO24)
- net OFF: now also U3.28 (GPIO17); no longer U3.52 (QSPI_SCLK)
- net VOL_{SW}: now also R41.1; no longer U3.28 (GPIO17)
- new net: R41.2, U3.52 (QSPI_SCLK)
Changed lines of the file:
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@@
+    (stroke (width 0) (type default))
+  )
+  (wire (pts (xy 167.64 86.36) (xy 177.8 86.36))
     (stroke (width 0) (type default))
   )
@@
     (stroke (width 0) (type default))
   )
+  (wire (pts (xy 152.4 86.36) (xy 162.56 86.36))
+    (stroke (width 0) (type default))
+  )
   (wire (pts (xy 53.34 38.1) (xy 62.23 38.1))
     (stroke (width 0) (type default))
@@
     (effects (font (size 1.27 1.27)) (justify left))
   )
-  (hierarchical_label "BTN_{Y}" (shape input) (at 228.6 114.3 0) (fields_autoplaced)
+  (hierarchical_label "BTN_{Y}" (shape input) (at 228.6 116.84 0) (fields_autoplaced)
     (effects (font (size 1.27 1.27)) (justify left))
   )
@@
     (effects (font (size 1.27 1.27)) (justify left))
   )
-  (hierarchical_label "OFF" (shape output) (at 177.8 86.36 180) (fields_autoplaced)
+  (hierarchical_label "OFF" (shape output) (at 228.6 96.52 0) (fields_autoplaced)
+    (effects (font (size 1.27 1.27)) (justify left))
+  )
+  (hierarchical_label "T_{SCK}" (shape output) (at 228.6 58.42 0) (fields_autoplaced)
+    (effects (font (size 1.27 1.27)) (justify left))
+  )
+  (hierarchical_label "TFT_{RST}" (shape output) (at 101.6 68.58 0) (fields_autoplaced)
+    (effects (font (size 1.27 1.27)) (justify left))
+  )
+  (hierarchical_label "TFT_{CS}" (shape output) (at 101.6 55.88 0) (fields_autoplaced)
+    (effects (font (size 1.27 1.27)) (justify left))
+  )
+  (hierarchical_label "AMP_{EN}" (shape output) (at 228.6 88.9 0) (fields_autoplaced)
+    (effects (font (size 1.27 1.27)) (justify left))
+  )
+  (hierarchical_label "SD_{CS}" (shape output) (at 101.6 76.2 0) (fields_autoplaced)
+    (effects (font (size 1.27 1.27)) (justify left))
+  )
+  (hierarchical_label "DSP_{ASDIN}" (shape output) (at 101.6 88.9 0) (fields_autoplaced)
+    (effects (font (size 1.27 1.27)) (justify left))
+  )
+  (hierarchical_label "BTN_{X}" (shape input) (at 228.6 111.76 0) (fields_autoplaced)
+    (effects (font (size 1.27 1.27)) (justify left))
+  )
+  (hierarchical_label "USB_{CC2}" (shape input) (at 101.6 124.46 0) (fields_autoplaced)
+    (effects (font (size 1.27 1.27)) (justify left))
+  )
+  (hierarchical_label "TFT_{MISO}" (shape input) (at 101.6 53.34 0) (fields_autoplaced)
+    (effects (font (size 1.27 1.27)) (justify left))
+  )
+  (hierarchical_label "TFT_{MOSI}" (shape output) (at 101.6 60.96 0) (fields_autoplaced)
+    (effects (font (size 1.27 1.27)) (justify left))
+  )
+  (hierarchical_label "VOL_{SW}" (shape input) (at 152.4 86.36 180) (fields_autoplaced)
     (effects (font (size 1.27 1.27)) (justify right))
   )
-  (hierarchical_label "T_{SCK}" (shape output) (at 228.6 58.42 0) (fields_autoplaced)
-    (effects (font (size 1.27 1.27)) (justify left))
-  )
-  (hierarchical_label "TFT_{RST}" (shape output) (at 101.6 68.58 0) (fields_autoplaced)
-    (effects (font (size 1.27 1.27)) (justify left))
-  )
-  (hierarchical_label "TFT_{CS}" (shape output) (at 101.6 55.88 0) (fields_autoplaced)
-    (effects (font (size 1.27 1.27)) (justify left))
-  )
-  (hierarchical_label "AMP_{EN}" (shape output) (at 228.6 88.9 0) (fields_autoplaced)
-    (effects (font (size 1.27 1.27)) (justify left))
-  )
-  (hierarchical_label "SD_{CS}" (shape output) (at 101.6 76.2 0) (fields_autoplaced)
-    (effects (font (size 1.27 1.27)) (justify left))
-  )
-  (hierarchical_label "DSP_{ASDIN}" (shape output) (at 101.6 88.9 0) (fields_autoplaced)
-    (effects (font (size 1.27 1.27)) (justify left))
-  )
-  (hierarchical_label "BTN_{X}" (shape input) (at 228.6 116.84 0) (fields_autoplaced)
-    (effects (font (size 1.27 1.27)) (justify left))
-  )
-  (hierarchical_label "USB_{CC2}" (shape input) (at 101.6 124.46 0) (fields_autoplaced)
-    (effects (font (size 1.27 1.27)) (justify left))
-  )
-  (hierarchical_label "TFT_{MISO}" (shape input) (at 101.6 53.34 0) (fields_autoplaced)
-    (effects (font (size 1.27 1.27)) (justify left))
-  )
-  (hierarchical_label "TFT_{MOSI}" (shape output) (at 101.6 60.96 0) (fields_autoplaced)
-    (effects (font (size 1.27 1.27)) (justify left))
-  )
-  (hierarchical_label "VOL_{SW}" (shape input) (at 228.6 96.52 0) (fields_autoplaced)
-    (effects (font (size 1.27 1.27)) (justify left))
-  )
   (hierarchical_label "T_{CS}" (shape output) (at 228.6 55.88 0) (fields_autoplaced)
     (effects (font (size 1.27 1.27)) (justify left))
@@
     (effects (font (size 1.27 1.27)) (justify left))
   )
-  (hierarchical_label "BTN_{B}" (shape input) (at 228.6 111.76 0) (fields_autoplaced)
+  (hierarchical_label "BTN_{B}" (shape input) (at 228.6 114.3 0) (fields_autoplaced)
     (effects (font (size 1.27 1.27)) (justify left))
   )
@@
         )
       )
+    )
+  )
+  (symbol (lib_id "Device:R_Small") (at 165.1 86.36 90) (unit 1)
+    (in_bom yes) (on_board yes) (dnp no) (fields_autoplaced)
+    (property "Reference" "R41" (at 165.1 88.9 90)
+      (effects (font (size 1.27 1.27)))
+    )
+    (property "Value" "1k" (at 165.1 91.44 90)
+      (effects (font (size 1.27 1.27)))
+    )
+    (property "Footprint" "Resistor_SMD:R_0402_1005Metric" (at 165.1 86.36 0)
+      (effects (font (size 1.27 1.27)) hide)
+    )
+    (property "Datasheet" "~" (at 165.1 86.36 0)
+      (effects (font (size 1.27 1.27)) hide)
+    )
+    (property "LCSC Part" "C11702" (at 165.1 86.36 90)
+      (effects (font (size 1.27 1.27)) hide)
+    )
+    (pin "1")
+    (pin "2")
+    (instances
+      (project "krecek-0.9"
+        (path "/8888f37b-ecc2-47df-8824-4b4e1e726451/6537dbea-4e11-4137-b8a0-9ae6b128c4e4"
+          (reference "R41") (unit 1)
+        )
+      )

Commit message: Use QSPI pins only for inputs
There is always a series resistor to prevent short-circuit during boot.

Resolves #12.
Parts:
- removed R41: 1k, Resistor_SMD:R_0402_1005Metric, symbol Device:R_Small
Connections:
- net AMP_{EN}: now also U3.29 (GPIO18); no longer U3.17 (GPIO14)
- net AUX4: now also U3.16 (GPIO13); no longer U3.53 (QSPI_SD0)
- net AUX5: now also U3.17 (GPIO14); no longer U3.55 (QSPI_SD1)
- net AUX6: now also U3.18 (GPIO15); no longer U3.54 (QSPI_SD2)
- net AUX7: now also U3.27 (GPIO16); no longer U3.51 (QSPI_SD3)
- net BTN_{SELECT}: now also U3.55 (QSPI_SD1); no longer U3.31 (GPIO20)
- net BTN_{START}: now also U3.31 (GPIO20); no longer U3.30 (GPIO19)
- net JOY_{SW}: now also U3.53 (QSPI_SD0); no longer U3.29 (GPIO18)
- net OFF: now also U3.30 (GPIO19); no longer U3.28 (GPIO17)
- net TFT_{LED}: now also U3.28 (GPIO17); no longer U3.16 (GPIO13)
- net VOL_{DOWN}: now also U3.51 (QSPI_SD3); no longer U3.27 (GPIO16)
- net VOL_{SW}: now also U3.52 (QSPI_SCLK)
- net VOL_{UP}: now also U3.54 (QSPI_SD2); no longer U3.18 (GPIO15)
Other:
- moved on the sheet: R40
Changed lines of the file:
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@@
     (stroke (width 0) (type default))
   )
-  (wire (pts (xy 152.4 71.12) (xy 162.56 71.12))
+  (wire (pts (xy 165.1 71.12) (xy 168.91 71.12))
     (stroke (width 0) (type default))
   )
@@
     (stroke (width 0) (type default))
   )
-  (wire (pts (xy 177.8 78.74) (xy 152.4 78.74))
+  (wire (pts (xy 228.6 88.9) (xy 254 88.9))
     (stroke (width 0) (type default))
   )
-  (wire (pts (xy 177.8 83.82) (xy 152.4 83.82))
+  (wire (pts (xy 228.6 93.98) (xy 254 93.98))
     (stroke (width 0) (type default))
   )
@@
     (stroke (width 0) (type default))
   )
-  (wire (pts (xy 177.8 76.2) (xy 152.4 76.2))
+  (wire (pts (xy 228.6 86.36) (xy 254 86.36))
     (stroke (width 0) (type default))
   )
@@
     (stroke (width 0) (type default))
   )
-  (wire (pts (xy 167.64 86.36) (xy 177.8 86.36))
-    (stroke (width 0) (type default))
-  )
   (wire (pts (xy 124.46 175.26) (xy 139.7 175.26))
     (stroke (width 0) (type default))
@@
     (stroke (width 0) (type default))
   )
-  (wire (pts (xy 152.4 86.36) (xy 162.56 86.36))
-    (stroke (width 0) (type default))
-  )
   (wire (pts (xy 53.34 38.1) (xy 62.23 38.1))
     (stroke (width 0) (type default))
@@
     (stroke (width 0) (type default))
   )
-  (wire (pts (xy 177.8 81.28) (xy 152.4 81.28))
+  (wire (pts (xy 228.6 91.44) (xy 254 91.44))
     (stroke (width 0) (type default))
   )
@@
     (stroke (width 0) (type default))
   )
-  (wire (pts (xy 167.64 71.12) (xy 177.8 71.12))
+  (wire (pts (xy 173.99 71.12) (xy 177.8 71.12))
     (stroke (width 0) (type default))
   )
@@
     (effects (font (size 1.27 1.27)) (justify right bottom))
   )
-  (label "AUX4" (at 152.4 76.2 0) (fields_autoplaced)
-    (effects (font (size 1.27 1.27)) (justify left bottom))
+  (label "AUX4" (at 254 86.36 180) (fields_autoplaced)
+    (effects (font (size 1.27 1.27)) (justify right bottom))
   )
   (label "QSPI_SD0" (at 38.1 76.2 0) (fields_autoplaced)
@@
     (effects (font (size 1.27 1.27)) (justify left bottom))
   )
-  (label "AUX7" (at 152.4 83.82 0) (fields_autoplaced)
-    (effects (font (size 1.27 1.27)) (justify left bottom))
+  (label "AUX7" (at 254 93.98 180) (fields_autoplaced)
+    (effects (font (size 1.27 1.27)) (justify right bottom))
   )
-  (label "AUX6" (at 152.4 81.28 0) (fields_autoplaced)
-    (effects (font (size 1.27 1.27)) (justify left bottom))
+  (label "AUX6" (at 254 91.44 180) (fields_autoplaced)
+    (effects (font (size 1.27 1.27)) (justify right bottom))
   )
   (label "BUS0" (at 127 101.6 180) (fields_autoplaced)
@@
     (effects (font (size 1.27 1.27)) (justify right bottom))
   )
-  (label "AUX5" (at 152.4 78.74 0) (fields_autoplaced)
-    (effects (font (size 1.27 1.27)) (justify left bottom))
+  (label "AUX5" (at 254 88.9 180) (fields_autoplaced)
+    (effects (font (size 1.27 1.27)) (justify right bottom))
   )
   (label "QSPI_SD2" (at 139.7 175.26 180) (fields_autoplaced)
@@
     (effects (font (size 1.27 1.27)) (justify left bottom))
   )
-  (hierarchical_label "TFT_{LED}" (shape output) (at 228.6 86.36 0) (fields_autoplaced)
+  (hierarchical_label "TFT_{LED}" (shape output) (at 228.6 96.52 0) (fields_autoplaced)
     (effects (font (size 1.27 1.27)) (justify left))
   )
@@
     (effects (font (size 1.27 1.27)) (justify left))
   )
-  (hierarchical_label "BTN_{SELECT}" (shape input) (at 228.6 104.14 0) (fields_autoplaced)
-    (effects (font (size 1.27 1.27)) (justify left))
+  (hierarchical_label "BTN_{SELECT}" (shape input) (at 177.8 78.74 180) (fields_autoplaced)
+    (effects (font (size 1.27 1.27)) (justify right))
   )
   (hierarchical_label "IR_{TX}" (shape output) (at 101.6 99.06 0) (fields_autoplaced)
@@
     (effects (font (size 1.27 1.27)) (justify left))
   )
-  (hierarchical_label "VOL_{UP}" (shape input) (at 228.6 91.44 0) (fields_autoplaced)
-    (effects (font (size 1.27 1.27)) (justify left))
+  (hierarchical_label "VOL_{UP}" (shape input) (at 177.8 81.28 180) (fields_autoplaced)
+    (effects (font (size 1.27 1.27)) (justify right))
   )
   (hierarchical_label "DSP_{ASDOUT}" (shape input) (at 101.6 91.44 0) (fields_autoplaced)
@@
     (effects (font (size 1.27 1.27)) (justify left))
   )
-  (hierarchical_label "BTN_{START}" (shape input) (at 228.6 101.6 0) (fields_autoplaced)
+  (hierarchical_label "BTN_{START}" (shape input) (at 228.6 104.14 0) (fields_autoplaced)
     (effects (font (size 1.27 1.27)) (justify left))
   )
@@
     (effects (font (size 1.27 1.27)) (justify left))
   )
-  (hierarchical_label "OFF" (shape output) (at 228.6 96.52 0) (fields_autoplaced)
+  (hierarchical_label "OFF" (shape output) (at 228.6 101.6 0) (fields_autoplaced)
     (effects (font (size 1.27 1.27)) (justify left))
   )
@@
     (effects (font (size 1.27 1.27)) (justify left))
   )
-  (hierarchical_label "AMP_{EN}" (shape output) (at 228.6 88.9 0) (fields_autoplaced)
+  (hierarchical_label "AMP_{EN}" (shape output) (at 228.6 99.06 0) (fields_autoplaced)
     (effects (font (size 1.27 1.27)) (justify left))
   )
@@
     (effects (font (size 1.27 1.27)) (justify left))
   )
-  (hierarchical_label "VOL_{SW}" (shape input) (at 152.4 86.36 180) (fields_autoplaced)
+  (hierarchical_label "VOL_{SW}" (shape input) (at 177.8 86.36 180) (fields_autoplaced)
     (effects (font (size 1.27 1.27)) (justify right))
   )
@@
     (effects (font (size 1.27 1.27)) (justify left))
   )
-  (hierarchical_label "JOY_{SW}" (shape input) (at 228.6 99.06 0) (fields_autoplaced)
-    (effects (font (size 1.27 1.27)) (justify left))
+  (hierarchical_label "JOY_{SW}" (shape input) (at 177.8 76.2 180) (fields_autoplaced)
+    (effects (font (size 1.27 1.27)) (justify right))
   )
   (hierarchical_label "TFT_{RS}" (shape output) (at 101.6 63.5 0) (fields_autoplaced)
@@
     (effects (font (size 1.27 1.27)) (justify left))
   )
-  (hierarchical_label "VOL_{DOWN}" (shape input) (at 228.6 93.98 0) (fields_autoplaced)
-    (effects (font (size 1.27 1.27)) (justify left))
+  (hierarchical_label "VOL_{DOWN}" (shape input) (at 177.8 83.82 180) (fields_autoplaced)
+    (effects (font (size 1.27 1.27)) (justify right))
   )
   (hierarchical_label "T_{IRQ}" (shape input) (at 228.6 63.5 0) (fields_autoplaced)
@@
     )
   )
-  (symbol (lib_id "Device:R_Small") (at 165.1 86.36 90) (unit 1)
-    (in_bom yes) (on_board yes) (dnp no) (fields_autoplaced)
-    (property "Reference" "R41" (at 165.1 88.9 90)
-      (effects (font (size 1.27 1.27)))
-    )
-    (property "Value" "1k" (at 165.1 91.44 90)
-      (effects (font (size 1.27 1.27)))
-    )
-    (property "Footprint" "Resistor_SMD:R_0402_1005Metric" (at 165.1 86.36 0)
-      (effects (font (size 1.27 1.27)) hide)
-    )
-    (property "Datasheet" "~" (at 165.1 86.36 0)
-      (effects (font (size 1.27 1.27)) hide)
-    )
-    (property "LCSC Part" "C11702" (at 165.1 86.36 90)
-      (effects (font (size 1.27 1.27)) hide)
-    )
-    (pin "1")
-    (pin "2")
-    (instances
-      (project "krecek-0.9"
-        (path "/8888f37b-ecc2-47df-8824-4b4e1e726451/6537dbea-4e11-4137-b8a0-9ae6b128c4e4"
-          (reference "R41") (unit 1)
-        )
-      )
-    )
-  )
   (symbol (lib_id "MCU_RaspberryPi:RP2040") (at 203.2 91.44 0) (unit 1)
     (in_bom yes) (on_board yes) (dnp no) (fields_autoplaced)
@@
     )
   )
-  (symbol (lib_id "power:GND") (at 152.4 71.12 270) (unit 1)
+  (symbol (lib_id "power:GND") (at 165.1 71.12 270) (unit 1)
     (in_bom yes) (on_board yes) (dnp no) (fields_autoplaced)
-    (property "Reference" "#PWR0113" (at 146.05 71.12 0)
+    (property "Reference" "#PWR0113" (at 158.75 71.12 0)
       (effects (font (size 1.27 1.27)) hide)
     )
-    (property "Value" "GND" (at 148.59 71.12 90)
+    (property "Value" "GND" (at 161.29 71.12 90)
       (effects (font (size 1.27 1.27)) (justify right))
     )
-    (property "Footprint" "" (at 152.4 71.12 0)
+    (property "Footprint" "" (at 165.1 71.12 0)
       (effects (font (size 1.27 1.27)) hide)
     )
-    (property "Datasheet" "" (at 152.4 71.12 0)
+    (property "Datasheet" "" (at 165.1 71.12 0)
       (effects (font (size 1.27 1.27)) hide)
     )
@@
     )
   )
-  (symbol (lib_id "Device:R_Small") (at 165.1 71.12 90) (unit 1)
+  (symbol (lib_id "Device:R_Small") (at 171.45 71.12 90) (unit 1)
     (in_bom yes) (on_board yes) (dnp no) (fields_autoplaced)
-    (property "Reference" "R40" (at 165.1 66.04 90)
+    (property "Reference" "R40" (at 171.45 66.04 90)
       (effects (font (size 1.27 1.27)))
     )
-    (property "Value" "1k" (at 165.1 68.58 90)
+    (property "Value" "1k" (at 171.45 68.58 90)
       (effects (font (size 1.27 1.27)))
     )
-    (property "Footprint" "Resistor_SMD:R_0402_1005Metric" (at 165.1 71.12 0)
+    (property "Footprint" "Resistor_SMD:R_0402_1005Metric" (at 171.45 71.12 0)
       (effects (font (size 1.27 1.27)) hide)
     )
-    (property "Datasheet" "~" (at 165.1 71.12 0)
+    (property "Datasheet" "~" (at 171.45 71.12 0)
       (effects (font (size 1.27 1.27)) hide)
     )
-    (property "LCSC Part" "C11702" (at 165.1 71.12 90)
+    (property "LCSC Part" "C11702" (at 171.45 71.12 90)
       (effects (font (size 1.27 1.27)) hide)
     )

Commit message: Fix input PMOS orientation (again)
Parts:
- renumbered R40 to R3, R3 to R4, R4 to R5, R5 to R6
