File: hw/krecek-0.9/rp2040.kicad_sch (KiCad schematic)
At the start: 39 parts, among them J1 DAP, J2 AUX, SW1 SW_Push, U1 RP2040, U2 RP2040, U3 W25Q128JVS, Y1 12MHz

Commit message: hw: work on new board revision
Parts:
- added R41: 1M, Resistor_SMD:R_0402_1005Metric, symbol Device:R_Small
Connections:
- net AUX0: now also R41.2; no longer R40.2
- net AUX1: now also J2.5 (Pin_5); no longer J2.8 (Pin_8)
- net AUX2: now also J2.8 (Pin_8); no longer J2.12 (Pin_12)
- net AUX3: now also J2.7 (Pin_7); no longer J2.14 (Pin_14)
- net AUX4: now also J2.12 (Pin_12); no longer J2.5 (Pin_5)
- net AUX5: now also J2.11 (Pin_11); no longer J2.7 (Pin_7)
- net AUX6: now also J2.14 (Pin_14); no longer J2.11 (Pin_11)
- new net: R40.2, R41.1
Changed lines of the file:
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@@
 	(wire
 		(pts
-			(xy 269.24 114.3) (xy 279.4 114.3)
+			(xy 281.94 114.3) (xy 292.1 114.3)
 		)
 		(stroke
@@
 	(wire
 		(pts
-			(xy 260.35 152.4) (xy 279.4 152.4)
+			(xy 247.65 149.86) (xy 228.6 149.86)
 		)
 		(stroke
@@
 	(wire
 		(pts
-			(xy 247.65 152.4) (xy 228.6 152.4)
+			(xy 247.65 157.48) (xy 228.6 157.48)
 		)
 		(stroke
@@
 	(wire
 		(pts
-			(xy 247.65 157.48) (xy 228.6 157.48)
+			(xy 260.35 160.02) (xy 279.4 160.02)
 		)
 		(stroke
@@
 	(wire
 		(pts
+			(xy 260.35 157.48) (xy 279.4 157.48)
+		)
+		(stroke
+			(width 0)
+			(type default)
+		)
+	)
+	(wire
+		(pts
 			(xy 125.73 38.1) (xy 134.62 38.1)
 		)
@@
 	(wire
 		(pts
-			(xy 260.35 160.02) (xy 279.4 160.02)
+			(xy 269.24 114.3) (xy 276.86 114.3)
 		)
 		(stroke
@@
 	(wire
 		(pts
-			(xy 38.1 71.12) (xy 50.8 71.12)
+			(xy 247.65 152.4) (xy 228.6 152.4)
 		)
 		(stroke
@@
 	(wire
 		(pts
-			(xy 189.23 25.4) (xy 198.12 25.4)
+			(xy 38.1 71.12) (xy 50.8 71.12)
 		)
 		(stroke
@@
 	(wire
 		(pts
-			(xy 167.64 114.3) (xy 167.64 119.38)
+			(xy 189.23 25.4) (xy 198.12 25.4)
 		)
 		(stroke
@@
 	(wire
 		(pts
-			(xy 260.35 157.48) (xy 279.4 157.48)
+			(xy 167.64 114.3) (xy 167.64 119.38)
 		)
 		(stroke
@@
 	(wire
 		(pts
-			(xy 134.62 25.4) (xy 143.51 25.4)
+			(xy 260.35 152.4) (xy 279.4 152.4)
 		)
 		(stroke
@@
 	(wire
 		(pts
-			(xy 38.1 76.2) (xy 50.8 76.2)
+			(xy 134.62 25.4) (xy 143.51 25.4)
 		)
 		(stroke
@@
 	(wire
 		(pts
-			(xy 173.99 71.12) (xy 177.8 71.12)
+			(xy 38.1 76.2) (xy 50.8 76.2)
 		)
 		(stroke
@@
 	(wire
 		(pts
-			(xy 99.06 25.4) (xy 99.06 29.21)
+			(xy 173.99 71.12) (xy 177.8 71.12)
 		)
 		(stroke
@@
 	(wire
 		(pts
-			(xy 247.65 149.86) (xy 228.6 149.86)
+			(xy 99.06 25.4) (xy 99.06 29.21)
 		)
 		(stroke
@@
 	)
 	(label "AUX0"
-		(at 279.4 114.3 180)
+		(at 292.1 114.3 180)
 		(fields_autoplaced yes)
 		(effects
@@
 	)
 	(label "AUX6"
-		(at 228.6 157.48 0)
+		(at 279.4 160.02 180)
 		(fields_autoplaced yes)
 		(effects
@@
 				(size 1.27 1.27)
 			)
-			(justify left bottom)
+			(justify right bottom)
 		)
 	)
@@
 	)
 	(label "AUX5"
-		(at 228.6 152.4 0)
+		(at 228.6 157.48 0)
 		(fields_autoplaced yes)
 		(effects
@@
 	)
 	(label "AUX2"
-		(at 279.4 157.48 180)
+		(at 279.4 152.4 180)
 		(fields_autoplaced yes)
 		(effects
@@
 	)
 	(label "AUX1"
-		(at 279.4 152.4 180)
+		(at 228.6 149.86 0)
 		(fields_autoplaced yes)
 		(effects
@@
 				(size 1.27 1.27)
 			)
-			(justify right bottom)
+			(justify left bottom)
 		)
 	)
 	(label "AUX3"
-		(at 279.4 160.02 180)
+		(at 228.6 152.4 0)
 		(fields_autoplaced yes)
 		(effects
@@
 				(size 1.27 1.27)
 			)
-			(justify right bottom)
+			(justify left bottom)
 		)
 	)
@@
 	)
 	(label "AUX4"
-		(at 228.6 149.86 0)
+		(at 279.4 157.48 180)
 		(fields_autoplaced yes)
 		(effects
@@
 				(size 1.27 1.27)
 			)
-			(justify left bottom)
+			(justify right bottom)
 		)
 	)
@@
 					(unit 1)
 				)
+			)
+		)
+	)
+	(symbol
+		(lib_id "Device:R_Small")
+		(at 279.4 114.3 90)
+		(mirror x)
+		(unit 1)
+		(exclude_from_sim no)
+		(in_bom yes)
+		(on_board yes)
+		(dnp no)
+		(fields_autoplaced yes)
+		(property "Reference" "R41"
+			(at 279.4 109.22 90)
+			(effects
+				(font
+					(size 1.27 1.27)
+				)
+			)
+		)
+		(property "Value" "1M"
+			(at 279.4 111.76 90)
+			(effects
+				(font
+					(size 1.27 1.27)
+				)
+			)
+		)
+		(property "Footprint" "Resistor_SMD:R_0402_1005Metric"
+			(at 279.4 114.3 0)
+			(effects
+				(font
+					(size 1.27 1.27)
+				)
+				(hide yes)
+			)
+		)
+		(property "Datasheet" "~"
+			(at 279.4 114.3 0)
+			(effects
+				(font
+					(size 1.27 1.27)
+				)
+				(hide yes)
+			)
+		)
+		(property "Description" "Resistor, small symbol"
+			(at 279.4 114.3 0)
+			(effects
+				(font
+					(size 1.27 1.27)
+				)
+				(hide yes)
+			)
+		)
+		(property "LCSC Part" "C26083"
+			(at 279.4 114.3 0)
+			(effects
+				(font
+					(size 1.27 1.27)
+				)
+				(hide yes)
+			)
+		)
+		(pin "1"
+		)
+		(pin "2"
+		)
+		(instances
+			(project "krecek-0.9"
+				(path "/8888f37b-ecc2-47df-8824-4b4e1e726451/6537dbea-4e11-4137-b8a0-9ae6b128c4e4"
+					(reference "R41")
+					(unit 1)
+				)

Commit message: hw: work on new board revision
Connections:
- net DSP_{ASDIN}: now also U1.18 (GPIO15); no longer U1.17 (GPIO14)
- net DSP_{ASDOUT}: now also U1.17 (GPIO14); no longer U1.18 (GPIO15)
Changed lines of the file:
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@@
 	(hierarchical_label "DSP_{ASDOUT}"
 		(shape input)
-		(at 101.6 91.44 0)
+		(at 101.6 88.9 0)
 		(fields_autoplaced yes)
 		(effects
@@
 	(hierarchical_label "DSP_{ASDIN}"
 		(shape output)
-		(at 101.6 88.9 0)
-		(fields_autoplaced yes)
-		(effects
+		(at 101.6 91.44 0)
+		(fields_autoplaced yes)
+		(effects
