File: hw/krecek-0.9/power.kicad_sch (KiCad schematic)
At the start: 1 part, among them U3 BQ24045DSQR

Commit message: More work on power supply section
Parts:
- added C10: 100uF, Capacitor_Tantalum_SMD:CP_EIA-3528-21_Kemet-B, symbol Device:C_Polarized_Small
- added C11, C12, C13, C14, C15, C16, C4, C5, C6: 1uF, Capacitor_SMD:C_0805_2012Metric, symbol Device:C_Small
- added C7: 100nF, Capacitor_SMD:C_0402_1005Metric, symbol Device:C_Small
- added C8: 4.7uF, Capacitor_SMD:C_0603_1608Metric, symbol Device:C_Small
- added C9: 10pF, Capacitor_SMD:C_0402_1005Metric, symbol Device:C_Small
- added D1: red, LED_SMD:LED_0603_1608Metric, symbol Device:LED_Small
- added D2: yellow, LED_SMD:LED_0603_1608Metric, symbol Device:LED_Small
- added D5: SS54, Diode_SMD:D_SMA, symbol Device:D_Small
- added J1: USB_C_Receptacle_USB2.0, LCSC:USB-C-SMD_TYPEC-304J-BCP16, symbol Connector:USB_C_Receptacle_USB2.0
- added L1: 2.2uH, Inductor_SMD:L_1008_2520Metric, symbol Device:L_Small
- added Q1, Q2, Q3: AO3400A, Package_TO_SOT_SMD:SOT-23, symbol Transistor_FET:AO3400A
- added Q4, Q5: AO3401A, Package_TO_SOT_SMD:SOT-23, symbol Transistor_FET:AO3401A
- added R10, R11, R13, R15, R20, R8, R9: 100k, Resistor_SMD:R_0402_1005Metric, symbol Device:R_Small
- added R12: 1M, Resistor_SMD:R_0402_1005Metric, symbol Device:R_Small
- added R14: 100, Resistor_SMD:R_0402_1005Metric, symbol Device:R_Small
- added R16, R17, R18, R19: 200k, Resistor_SMD:R_0402_1005Metric, symbol Device:R_Small
- added R4: 560, Resistor_SMD:R_0603_1608Metric, symbol Device:R_Small
- added R5: 2k, Resistor_SMD:R_0402_1005Metric, symbol Device:R_Small
- added R6, R7: 4.7k, Resistor_SMD:R_0402_1005Metric, symbol Device:R_Small
- added SW1: ON, symbol Switch:SW_Push
- added U5: S2B-PH-KL(LF)(SN), LCSC:CONN-TH-2P-P2.00_S2B-PH-KL-LF-SN, symbol LCSC:S2B-PH-KL(LF)(SN)
- added U6: TPS63000, Package_SON:Texas_DRC0010J_ThermalVias, symbol Regulator_Switching:TPS63000
- added U7, U8, U9: AMS1117-3.3, Package_TO_SOT_SMD:SOT-223-3_TabPin2, symbol Regulator_Linear:AMS1117-3.3
Connections:
- net VBUS: now reaches U3.1 (IN)
- net VBUS: now also C4.1, D5.2 (A), J1.A4 (VBUS), J1.A9 (VBUS), J1.B4 (VBUS), J1.B9 (VBUS), Q5.1 (G), R13.2
- net +BATT: now reaches U3.10 (OUT)
- net +BATT: now also C5.1, Q5.3 (D), R6.1, R7.1, U5.1 (+)
- net GND: now reaches U3.11 (VSS), U3.3 (VSS)
- net GND: now also C10.2, C11.2, C12.2, C13.2, C14.2, C15.2, C16.2, C4.2, C5.2, C6.2, C7.2, C8.1, J1.A1 (GND), J1.A12 (GND), J1.B1 (GND), J1.B12 (GND), Q1.2 (S), Q2.2 (S), Q3.2 (S), R12.1, R13.1, R15.2, R4.2, R5.1, SW1.1, U5.2 (-), U6.11 (PGND), U6.3 (PGND), U6.9 (GND), U7.1 (GND), U8.1 (GND), U9.1 (GND)
- net at U3.2 (ISET): now also R4.1
- net at U3.4 (PRETERM): now also R5.2
- net ~{PG}: now reaches U3.5 (~{PG})
- net ~{PG}: now also D1.1 (K)
- net ISET2: now reaches U3.7 (ISET2)
- net ~{CHG}: now reaches U3.8 (~{CHG})
- net ~{CHG}: now also D2.1 (K)
- new net: C9.1, R15.1, R16.1, U6.10 (FB)
- new net: Q1.1 (G), R11.2, SW1.2
- new net: R18.2, R19.1
- new net: R19.2, R20.1
- new net: L1.1, U6.2 (L2)
- new net: L1.2, U6.4 (L1)
- new net: Q2.1 (G), Q3.3 (D), R10.1, R12.2
- new net: Q1.3 (D), R10.2, R8.1
- new net: C8.2, Q4.3 (D), R14.1, U6.5 (VIN)
- new net: C7.1, R14.2, U6.6 (EN), U6.7 (PS/SYNC), U6.8 (VINA)
- new net: Q2.3 (D), Q4.1 (G), R11.1, R9.1
- new net: D2.2 (A), R7.2
- new net: R17.2, R18.1
- new net: R16.2, R17.1
- new net: D1.2 (A), R6.2
- new net +3.3V: C14.1, U8.2 (VO)
- new net +3.3VA: C12.1, U7.2 (VO)
- new net +3.3VSD: C16.1, U9.2 (VO)
- new net +5V: C10.1, C11.1, C13.1, C15.1, C9.2, R20.2, U6.1 (VOUT), U7.3 (VI), U8.3 (VI), U9.3 (VI)
- new net OFF: Q3.1 (G)
- new net V_{USB/BATT}: C6.1, D5.1 (K), Q4.2 (S), Q5.2 (S), R8.2, R9.2
- no-connect marks 0 -> 3
Other:
- note added: "TODO: Pozor na zpetne napajeni pri praci z baterie."
- moved on the sheet: U3

Commit message: Expand hardware design to cover more areas
Signed-off-by: Jan Hamal Dvořák <mordae@anilinux.org>
Connections:
- net USB_{CC1}: now reaches J1.A5 (CC1)
- net USB_{D-}: now reaches J1.A6 (D+)
- net USB_{D-}: now also J1.B6 (D+)
- net USB_{D+}: now reaches J1.A7 (D-)
- net USB_{D+}: now also J1.B7 (D-)
- net USB_{CC2}: now reaches J1.B5 (CC2)
Changed lines of the file:
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@@
   (junction (at 82.55 152.4) (diameter 0) (color 0 0 0 0)
   )
+  (junction (at 54.61 46.99) (diameter 0) (color 0 0 0 0)
+  )
   (junction (at 171.45 127) (diameter 0) (color 0 0 0 0)
   )
@@
   )
   (junction (at 256.54 120.65) (diameter 0) (color 0 0 0 0)
+  )
+  (junction (at 54.61 41.91) (diameter 0) (color 0 0 0 0)
   )
   (junction (at 184.15 69.85) (diameter 0) (color 0 0 0 0)
@@
     (stroke (width 0) (type default))
   )
+  (wire (pts (xy 50.8 45.72) (xy 54.61 45.72))
+    (stroke (width 0) (type default))
+  )
   (wire (pts (xy 40.64 107.95) (xy 44.45 107.95))
     (stroke (width 0) (type default))
@@
     (stroke (width 0) (type default))
   )
+  (wire (pts (xy 54.61 46.99) (xy 54.61 48.26))
+    (stroke (width 0) (type default))
+  )
   (wire (pts (xy 137.16 43.18) (xy 147.32 43.18))
     (stroke (width 0) (type default))
@@
     (stroke (width 0) (type default))
   )
+  (wire (pts (xy 57.15 46.99) (xy 54.61 46.99))
+    (stroke (width 0) (type default))
+  )
   (wire (pts (xy 114.3 152.4) (xy 133.35 152.4))
     (stroke (width 0) (type default))
@@
     (stroke (width 0) (type default))
   )
+  (wire (pts (xy 54.61 40.64) (xy 54.61 41.91))
+    (stroke (width 0) (type default))
+  )
   (wire (pts (xy 139.7 114.3) (xy 139.7 120.65))
     (stroke (width 0) (type default))
@@
     (stroke (width 0) (type default))
   )
+  (wire (pts (xy 50.8 33.02) (xy 54.61 33.02))
+    (stroke (width 0) (type default))
+  )
   (wire (pts (xy 260.35 57.15) (xy 260.35 60.96))
     (stroke (width 0) (type default))
@@
     (stroke (width 0) (type default))
   )
+  (wire (pts (xy 54.61 48.26) (xy 50.8 48.26))
+    (stroke (width 0) (type default))
+  )
+  (wire (pts (xy 50.8 35.56) (xy 54.61 35.56))
+    (stroke (width 0) (type default))
+  )
   (wire (pts (xy 171.45 125.73) (xy 177.165 125.73))
     (stroke (width 0) (type default))
@@
     (stroke (width 0) (type default))
   )
+  (wire (pts (xy 54.61 41.91) (xy 54.61 43.18))
+    (stroke (width 0) (type default))
+  )
   (wire (pts (xy 133.35 152.4) (xy 158.75 152.4))
     (stroke (width 0) (type default))
@@
     (stroke (width 0) (type default))
   )
+  (wire (pts (xy 54.61 43.18) (xy 50.8 43.18))
+    (stroke (width 0) (type default))
+  )
   (wire (pts (xy 247.65 101.6) (xy 260.35 101.6))
     (stroke (width 0) (type default))
@@
     (stroke (width 0) (type default))
   )
+  (wire (pts (xy 54.61 40.64) (xy 50.8 40.64))
+    (stroke (width 0) (type default))
+  )
   (wire (pts (xy 31.75 152.4) (xy 63.5 152.4))
     (stroke (width 0) (type default))
@@
     (stroke (width 0) (type default))
   )
+  (wire (pts (xy 54.61 45.72) (xy 54.61 46.99))
+    (stroke (width 0) (type default))
+  )
   (wire (pts (xy 152.4 107.95) (xy 152.4 109.22))
     (stroke (width 0) (type default))
@@
   )
   (wire (pts (xy 247.65 102.87) (xy 247.65 101.6))
+    (stroke (width 0) (type default))
+  )
+  (wire (pts (xy 57.15 41.91) (xy 54.61 41.91))
     (stroke (width 0) (type default))
   )
@@
     (effects (font (size 1.27 1.27)) (justify right))
   )
+  (hierarchical_label "USB_{CC1}" (shape output) (at 54.61 33.02 0) (fields_autoplaced)
+    (effects (font (size 1.27 1.27)) (justify left))
+  )
+  (hierarchical_label "USB_{CC2}" (shape output) (at 54.61 35.56 0) (fields_autoplaced)
+    (effects (font (size 1.27 1.27)) (justify left))
+  )
+  (hierarchical_label "USB_{D-}" (shape bidirectional) (at 57.15 46.99 0) (fields_autoplaced)
+    (effects (font (size 1.27 1.27)) (justify left))
+  )
+  (hierarchical_label "USB_{D+}" (shape bidirectional) (at 57.15 41.91 0) (fields_autoplaced)
+    (effects (font (size 1.27 1.27)) (justify left))
+  )
   (symbol (lib_id "Device:R_Small") (at 203.2 146.05 0) (mirror y) (unit 1)

Commit message: Update schematic
Signed-off-by: Jan Hamal Dvořák <mordae@anilinux.org>
Parts:
- added C24: 4.7uF, Capacitor_SMD:C_0603_1608Metric, symbol Device:C_Small
Connections:
- net +5V: now also C24.2
- net GND: now also C24.1
Changed lines of the file:
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@@
   (junction (at 203.2 128.27) (diameter 0) (color 0 0 0 0)
+  )
+  (junction (at 203.2 120.65) (diameter 0) (color 0 0 0 0)
   )
   (junction (at 82.55 50.8) (diameter 0) (color 0 0 0 0)
@@
     (stroke (width 0) (type default))
   )
+  (wire (pts (xy 203.2 107.95) (xy 203.2 111.76))
+    (stroke (width 0) (type default))
+  )
   (wire (pts (xy 203.2 57.15) (xy 196.85 57.15))
     (stroke (width 0) (type default))
@@
     (stroke (width 0) (type default))
   )
+  (wire (pts (xy 203.2 116.84) (xy 203.2 120.65))
+    (stroke (width 0) (type default))
+  )
   (wire (pts (xy 133.35 133.35) (xy 133.35 152.4))
     (stroke (width 0) (type default))
@@
     (stroke (width 0) (type default))
   )
-  (wire (pts (xy 197.485 120.65) (xy 256.54 120.65))
+  (wire (pts (xy 197.485 120.65) (xy 203.2 120.65))
     (stroke (width 0) (type default))
   )
@@
   )
   (wire (pts (xy 82.55 120.65) (xy 95.885 120.65))
+    (stroke (width 0) (type default))
+  )
+  (wire (pts (xy 203.2 120.65) (xy 256.54 120.65))
     (stroke (width 0) (type default))
   )
@@
         (path "/8888f37b-ecc2-47df-8824-4b4e1e726451/bd29cd8c-9207-416a-90c1-7bdf6b5cfb97"
           (reference "R15") (unit 1)
+        )
+      )
+    )
+  )
+  (symbol (lib_id "Device:C_Small") (at 203.2 114.3 0) (unit 1)
+    (in_bom yes) (on_board yes) (dnp no) (fields_autoplaced)
+    (property "Reference" "C24" (at 205.74 113.0363 0)
+      (effects (font (size 1.27 1.27)) (justify left))
+    )
+    (property "Value" "4.7uF" (at 205.74 115.5763 0)
+      (effects (font (size 1.27 1.27)) (justify left))
+    )
+    (property "Footprint" "Capacitor_SMD:C_0603_1608Metric" (at 203.2 114.3 0)
+      (effects (font (size 1.27 1.27)) hide)
+    )
+    (property "Datasheet" "~" (at 203.2 114.3 0)
+      (effects (font (size 1.27 1.27)) hide)
+    )
+    (property "LCSC Part" "C19666" (at 203.2 114.3 0)
+      (effects (font (size 1.27 1.27)) hide)
+    )
+    (pin "1")
+    (pin "2")
+    (instances
+      (project "krecek-0.9"
+        (path "/8888f37b-ecc2-47df-8824-4b4e1e726451/bd29cd8c-9207-416a-90c1-7bdf6b5cfb97"
+          (reference "C24") (unit 1)
         )
       )
@@
         )
       )
+    )
+  )
+  (symbol (lib_id "power:GND") (at 203.2 107.95 180) (unit 1)
+    (in_bom yes) (on_board yes) (dnp no) (fields_autoplaced)
+    (property "Reference" "#PWR046" (at 203.2 101.6 0)
+      (effects (font (size 1.27 1.27)) hide)
+    )
+    (property "Value" "GND" (at 203.2 103.505 0)
+      (effects (font (size 1.27 1.27)))
+    )
+    (property "Footprint" "" (at 203.2 107.95 0)
+      (effects (font (size 1.27 1.27)) hide)
+    )
+    (property "Datasheet" "" (at 203.2 107.95 0)
+      (effects (font (size 1.27 1.27)) hide)
+    )
+    (pin "1")
+    (instances
+      (project "krecek-0.9"
+        (path "/8888f37b-ecc2-47df-8824-4b4e1e726451/bd29cd8c-9207-416a-90c1-7bdf6b5cfb97"
+          (reference "#PWR046") (unit 1)
+        )
+      )

Commit message: Further tweaks and improvements
- Use a nicer schematic template
- Tie START button with power on
- Add ferrite to USB shield
- Add CC1/CC2 makeshift ADC
- Tidy up schematics a little bit

Signed-off-by: Jan Hamal Dvořák <mordae@anilinux.org>
Parts:
- added C26, C27: 100pF, Capacitor_SMD:C_0402_1005Metric, symbol Device:C_Small
- added D3: 3.3V, Diode_SMD:D_MiniMELF, symbol Device:D_Zener_Small
- added FB1: 600Ω @ 100 MHz, Inductor_SMD:L_0805_2012Metric, symbol Device:FerriteBead_Small
- added Q6: AO3400A, Package_TO_SOT_SMD:SOT-23, symbol Transistor_FET:AO3400A
- added R3 (x2): 100k, Resistor_SMD:R_0402_1005Metric, symbol Device:R_Small
- added R3 (x2): 5.1k, Resistor_SMD:R_0402_1005Metric, symbol Device:R_Small
- R10: value 100k -> 10k; LCSC Part C25741 -> C25744
- R11, R8, R9: value 100k -> 330k; footprint Resistor_SMD:R_0402_1005Metric -> Resistor_SMD:R_0603_1608Metric; LCSC Part C25741 -> C23137
- R12: value 1M -> 10M; footprint Resistor_SMD:R_0402_1005Metric -> Resistor_SMD:R_0603_1608Metric; LCSC Part C26083 -> C7250
- SW1: value ON -> START; footprint (none) -> Krecek:RubberButton
- U5: value S2B-PH-KL(LF)(SN) -> JST-PH-2P
Connections:
- net +BATT: now also R10.1
- net GND: now also R11.1, C26.1, C27.1, D3.2 (A), FB1.1, Q6.2 (S), R3.2, R3.2; no longer SW1.1
- net USB_{CC1}: now also C26.2, R3.1; no longer J1.A5 (CC1)
- net USB_{CC2}: now also C27.2, R3.1; no longer J1.B5 (CC2)
- net ON: now reaches R11.2, SW1.2
- net ON: now also D3.1 (K), Q6.1 (G); no longer Q1.1 (G)
- net at Q2.1 (G), Q3.3 (D), R12.2: now also Q1.3 (D), R8.1; no longer R10.1
- net at Q2.3 (D), Q4.1 (G), R9.1: now also Q1.1 (G), Q6.3 (D); no longer R11.1
- net at J1.S1 (SHIELD): now also FB1.2
- new net: R10.2, SW1.1
- new net CC1: J1.A5 (CC1), R3.1, R3.2
- new net CC2: J1.B5 (CC2), R3.1, R3.2
Other:
- company: (none) -> DDM Spirála
- title: (none) -> Křeček
- moved on the sheet: C10, C11, C12, C13, C14, C15, C16, C24, C4, C5, C6, C7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

Commit message: TRRS audio connector
Signed-off-by: Jan Hamal Dvořák <mordae@anilinux.org>
Changed lines of the file:
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@@
   )
   (symbol (lib_id "Switch:SW_Push") (at 82.55 76.2 0) (unit 1)
-    (in_bom yes) (on_board yes) (dnp no)
-    (property "Reference" "SW1" (at 101.6 68.58 0)
+    (in_bom yes) (on_board yes) (dnp no) (fields_autoplaced)
+    (property "Reference" "SW1" (at 82.55 68.58 0)
       (effects (font (size 1.27 1.27)))
     )
@@
       (effects (font (size 1.27 1.27)) hide)
     )
-    (pin "2")
-    (pin "1")
+    (pin "1")
+    (pin "2")
     (instances
       (project "krecek-0.9"
@@
       (effects (font (size 1.27 1.27)) hide)
     )
-    (pin "2")
-    (pin "1")
-    (instances
-      (project "krecek-0.9"
+    (pin "1")
+    (pin "2")
+    (instances
+      (project "krecek-0.9"

Commit message: Complete most of the design, except for RF
Signed-off-by: Jan Hamal Dvořák <mordae@anilinux.org>
Parts:
- removed D3: 3.3V, Diode_SMD:D_MiniMELF, symbol Device:D_Zener_Small
- added R16, R17, R18: 1M, Resistor_SMD:R_0402_1005Metric, symbol Device:R_Small
- R15: renamed from R11; value 330k -> 33k; LCSC Part C23137 -> C25779
- renumbered C5 to C26, C11 to C27, C12 to C28, C4 to C29, C13 to C30, C14 to C31, C15 to C32, C16 to C33, C26 to C34, C27 to C35, C8 to C36, C24 to C37, C6 to C38, C10 to C39, C7 to C40, C9 to C41, D2 to D1, D1 to D2, D5 to D3, Q4 to Q1, Q5 to Q2, Q1 to Q3, Q2 to Q4, Q6 to Q5, Q3 to Q6, R10 to R13, R8 to R19, R9 to R20, R13 to R21, R14 to R22, R16 to R23, R17 to R24, R18 to R25, R19 to R26, R20 to R27, R12 to R28, R15 to R29, R4 to R6, R5 to R7, R7 to R8, R6 to R9, SW1 to SW2, U6 to U10, U7 to U5, U5 to U6
Connections:
- net +BATT: now also R16.2
- net GND: now also R18.1
- new net: R17.1, R18.2
- new net BAT_{Vsense}: R16.1, R17.2
Other:
- note removed: "TODO: Pozor na zpetne napajeni pri praci z baterie."
- moved on the sheet: C29, C40, R13, R15, R22, R23, R26, R6, R7, SW2, U10, U3

Commit message: Fix design bugs
Signed-off-by: Jan Hamal Dvořák <mordae@anilinux.org>
Parts:
- removed C34, C35: 100pF, Capacitor_SMD:C_0402_1005Metric, symbol Device:C_Small
- removed R3 (x2): 100k, Resistor_SMD:R_0402_1005Metric, symbol Device:R_Small
Connections:
- net CC1 is gone; now on net USB_{CC1}: J1.A5 (CC1), R3.1
- net CC2 is gone; now on net USB_{CC2}: J1.B5 (CC2), R3.1

Commit message: Add missing LCSC part id
Signed-off-by: Jan Hamal Dvořák <mordae@anilinux.org>
Parts:
- U10: LCSC Part (none) -> C24966
Changed lines of the file:
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@@
+      (effects (font (size 1.27 1.27)) hide)
+    )
+    (property "LCSC Part" "C24966" (at 181.61 143.51 0)
       (effects (font (size 1.27 1.27)) hide)
     )
