File: hw/krecek-0.9/power.kicad_sch (KiCad schematic)
At the start: 55 parts, among them J1 USB_C_Receptacle_USB2.0, Q1 AO3401A, Q2 AO3401A, Q3 AO3400A, Q4 AO3400A, Q5 AO3400A, Q6 AO3400A, SW2 START, U10 TPS63000, U3 BQ24045DSQR, U5 AMS1117-3.3, U6 JST-PH-2P, U8 AMS1117-3.3, U9 AMS1117-3.3

Commit message: Add more missing LCSC part ids
Signed-off-by: Jan Hamal Dvořák <mordae@anilinux.org>
Parts:
- U5, U8, U9: LCSC Part (none) -> C6186
Changed lines of the file:
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@@
+      (effects (font (size 1.27 1.27)) hide)
+    )
+    (property "LCSC Part" "C6186" (at 254 50.8 0)
       (effects (font (size 1.27 1.27)) hide)
     )
@@
       (effects (font (size 1.27 1.27)) hide)
     )
+    (property "LCSC Part" "C6186" (at 254 76.2 0)
+      (effects (font (size 1.27 1.27)) hide)
+    )
     (pin "1")
     (pin "2")
@@
       (effects (font (size 1.27 1.27)) hide)
     )
+    (property "LCSC Part" "C6186" (at 254 25.4 0)
+      (effects (font (size 1.27 1.27)) hide)
+    )

Commit message: Add missing transistor LCSC part ids
Signed-off-by: Jan Hamal Dvořák <mordae@anilinux.org>
Parts:
- Q1, Q2: LCSC Part (none) -> C15127
Changed lines of the file:
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@@
       (effects (font (size 1.27 1.27)) (justify left) hide)
+    )
+    (property "LCSC Part" "C15127" (at 35.56 133.35 0)
+      (effects (font (size 1.27 1.27)) hide)
     )
     (pin "1")
@@
       (effects (font (size 1.27 1.27)) (justify left) hide)
     )
+    (property "LCSC Part" "C15127" (at 143.51 127 0)
+      (effects (font (size 1.27 1.27)) hide)
+    )
     (pin "1")

Commit message: Fix part numbers
Signed-off-by: Jan Hamal Dvořák <mordae@anilinux.org>
Parts:
- renumbered C36 to C34, C37 to C35, C38 to C36, C39 to C37, C40 to C38, C41 to C39, R13 to R11, R15 to R13, R16 to R14, R17 to R15, R18 to R16, R19 to R17, R20 to R18, R21 to R19, R22 to R20, R23 to R21, R24 to R22, R25 to R23, R26 to R24, R27 to R25, R28 to R26, R29 to R27

Commit message: Fix symbol/footprint mismatches
Signed-off-by: Jan Hamal Dvořák <mordae@anilinux.org>
Parts:
- removed SW2: START, Krecek:RubberButton, symbol Switch:SW_Push
- added SW2: ~, Krecek:RubberButton, symbol Krecek:RubberButton
- J1: symbol Connector:USB_C_Receptacle_USB2.0 -> LCSC:USB_C_Receptacle_USB2.0
Connections:
- net GND: now also J1.A1B12 (GND), J1.B1A12 (GND); no longer J1.A1 (GND), J1.A12 (GND), J1.B1 (GND), J1.B12 (GND)
- net ON: now also SW2.C
- net VBUS: now also J1.A4B9 (VBUS), J1.B4A9 (VBUS); no longer J1.A4 (VBUS), J1.A9 (VBUS), J1.B4 (VBUS), J1.B9 (VBUS)
- net at R11.2: now also SW2.1
Changed lines of the file:
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@@
     )
   )
-  (symbol (lib_id "Switch:SW_Push") (at 82.55 88.9 0) (unit 1)
-    (in_bom yes) (on_board yes) (dnp no) (fields_autoplaced)
-    (property "Reference" "SW2" (at 82.55 81.28 0)
-      (effects (font (size 1.27 1.27)))
-    )
-    (property "Value" "START" (at 82.55 83.82 0)
-      (effects (font (size 1.27 1.27)))
-    )
-    (property "Footprint" "Krecek:RubberButton" (at 82.55 83.82 0)
-      (effects (font (size 1.27 1.27)) hide)
-    )
-    (property "Datasheet" "~" (at 82.55 83.82 0)
-      (effects (font (size 1.27 1.27)) hide)
-    )
-    (pin "1")
-    (pin "2")
+  (symbol (lib_id "Device:R_Small") (at 233.68 140.97 90) (mirror x) (unit 1)
+    (in_bom yes) (on_board yes) (dnp no) (fields_autoplaced)
+    (property "Reference" "R24" (at 233.68 135.89 90)
+      (effects (font (size 1.27 1.27)))
+    )
+    (property "Value" "200k" (at 233.68 138.43 90)
+      (effects (font (size 1.27 1.27)))
+    )
+    (property "Footprint" "Resistor_SMD:R_0402_1005Metric" (at 233.68 140.97 0)
+      (effects (font (size 1.27 1.27)) hide)
+    )
+    (property "Datasheet" "~" (at 233.68 140.97 0)
+      (effects (font (size 1.27 1.27)) hide)
+    )
+    (property "LCSC Part" " C25764 " (at 233.68 140.97 0)
+      (effects (font (size 1.27 1.27)) hide)
+    )
+    (pin "1")
+    (pin "2")
+    (instances
+      (project "krecek-0.9"
+        (path "/8888f37b-ecc2-47df-8824-4b4e1e726451/bd29cd8c-9207-416a-90c1-7bdf6b5cfb97"
+          (reference "R24") (unit 1)
+        )
+      )
+    )
+  )
+  (symbol (lib_id "power:GND") (at 15.24 82.55 0) (unit 1)
+    (in_bom yes) (on_board yes) (dnp no) (fields_autoplaced)
+    (property "Reference" "#PWR044" (at 15.24 88.9 0)
+      (effects (font (size 1.27 1.27)) hide)
+    )
+    (property "Value" "GND" (at 15.24 87.63 0)
+      (effects (font (size 1.27 1.27)))
+    )
+    (property "Footprint" "" (at 15.24 82.55 0)
+      (effects (font (size 1.27 1.27)) hide)
+    )
+    (property "Datasheet" "" (at 15.24 82.55 0)
+      (effects (font (size 1.27 1.27)) hide)
+    )
+    (pin "1")
+    (instances
+      (project "krecek-0.9"
+        (path "/8888f37b-ecc2-47df-8824-4b4e1e726451/bd29cd8c-9207-416a-90c1-7bdf6b5cfb97"
+          (reference "#PWR044") (unit 1)
+        )
+      )
+    )
+  )
+  (symbol (lib_id "Device:R_Small") (at 243.84 140.97 90) (mirror x) (unit 1)
+    (in_bom yes) (on_board yes) (dnp no) (fields_autoplaced)
+    (property "Reference" "R25" (at 243.84 135.89 90)
+      (effects (font (size 1.27 1.27)))
+    )
+    (property "Value" "100k" (at 243.84 138.43 90)
+      (effects (font (size 1.27 1.27)))
+    )
+    (property "Footprint" "Resistor_SMD:R_0402_1005Metric" (at 243.84 140.97 0)
+      (effects (font (size 1.27 1.27)) hide)
+    )
+    (property "Datasheet" "~" (at 243.84 140.97 0)
+      (effects (font (size 1.27 1.27)) hide)
+    )
+    (property "LCSC Part" "C25741 " (at 243.84 140.97 0)
+      (effects (font (size 1.27 1.27)) hide)
+    )
+    (pin "1")
+    (pin "2")
+    (instances
+      (project "krecek-0.9"
+        (path "/8888f37b-ecc2-47df-8824-4b4e1e726451/bd29cd8c-9207-416a-90c1-7bdf6b5cfb97"
+          (reference "R25") (unit 1)
+        )
+      )
+    )
+  )
+  (symbol (lib_id "Device:R_Small") (at 234.95 114.3 270) (mirror x) (unit 1)
+    (in_bom yes) (on_board yes) (dnp no) (fields_autoplaced)
+    (property "Reference" "R14" (at 234.95 109.22 90)
+      (effects (font (size 1.27 1.27)))
+    )
+    (property "Value" "1M" (at 234.95 111.76 90)
+      (effects (font (size 1.27 1.27)))
+    )
+    (property "Footprint" "Resistor_SMD:R_0402_1005Metric" (at 234.95 114.3 0)
+      (effects (font (size 1.27 1.27)) hide)
+    )
+    (property "Datasheet" "~" (at 234.95 114.3 0)
+      (effects (font (size 1.27 1.27)) hide)
+    )
+    (property "LCSC Part" "C26083" (at 234.95 114.3 0)
+      (effects (font (size 1.27 1.27)) hide)
+    )
+    (pin "1")
+    (pin "2")
+    (instances
+      (project "krecek-0.9"
+        (path "/8888f37b-ecc2-47df-8824-4b4e1e726451/bd29cd8c-9207-416a-90c1-7bdf6b5cfb97"
+          (reference "R14") (unit 1)
+        )
+      )
+    )
+  )
+  (symbol (lib_id "Krecek:RubberButton") (at 82.55 88.9 0) (unit 1)
+    (in_bom yes) (on_board yes) (dnp no) (fields_autoplaced)
+    (property "Reference" "SW2" (at 82.55 83.82 0)
+      (effects (font (size 1.27 1.27)))
+    )
+    (property "Value" "~" (at 82.55 88.9 0)
+      (effects (font (size 1.27 1.27)))
+    )
+    (property "Footprint" "Krecek:RubberButton" (at 82.55 91.44 0)
+      (effects (font (size 1.27 1.27)) hide)
+    )
+    (property "Datasheet" "" (at 82.55 88.9 0)
+      (effects (font (size 1.27 1.27)) hide)
+    )
+    (pin "1")
+    (pin "C")
     (instances
       (project "krecek-0.9"
         (path "/8888f37b-ecc2-47df-8824-4b4e1e726451/bd29cd8c-9207-416a-90c1-7bdf6b5cfb97"
           (reference "SW2") (unit 1)
-        )
-      )
-    )
-  )
-  (symbol (lib_id "Device:R_Small") (at 233.68 140.97 90) (mirror x) (unit 1)
-    (in_bom yes) (on_board yes) (dnp no) (fields_autoplaced)
-    (property "Reference" "R24" (at 233.68 135.89 90)
-      (effects (font (size 1.27 1.27)))
-    )
-    (property "Value" "200k" (at 233.68 138.43 90)
-      (effects (font (size 1.27 1.27)))
-    )
-    (property "Footprint" "Resistor_SMD:R_0402_1005Metric" (at 233.68 140.97 0)
-      (effects (font (size 1.27 1.27)) hide)
-    )
-    (property "Datasheet" "~" (at 233.68 140.97 0)
-      (effects (font (size 1.27 1.27)) hide)
-    )
-    (property "LCSC Part" " C25764 " (at 233.68 140.97 0)
-      (effects (font (size 1.27 1.27)) hide)
-    )
-    (pin "1")
-    (pin "2")
-    (instances
-      (project "krecek-0.9"
-        (path "/8888f37b-ecc2-47df-8824-4b4e1e726451/bd29cd8c-9207-416a-90c1-7bdf6b5cfb97"
-          (reference "R24") (unit 1)
-        )
-      )
-    )
-  )
-  (symbol (lib_id "power:GND") (at 15.24 82.55 0) (unit 1)
-    (in_bom yes) (on_board yes) (dnp no) (fields_autoplaced)
-    (property "Reference" "#PWR044" (at 15.24 88.9 0)
-      (effects (font (size 1.27 1.27)) hide)
-    )
-    (property "Value" "GND" (at 15.24 87.63 0)
-      (effects (font (size 1.27 1.27)))
-    )
-    (property "Footprint" "" (at 15.24 82.55 0)
-      (effects (font (size 1.27 1.27)) hide)
-    )
-    (property "Datasheet" "" (at 15.24 82.55 0)
-      (effects (font (size 1.27 1.27)) hide)
-    )
-    (pin "1")
-    (instances
-      (project "krecek-0.9"
-        (path "/8888f37b-ecc2-47df-8824-4b4e1e726451/bd29cd8c-9207-416a-90c1-7bdf6b5cfb97"
-          (reference "#PWR044") (unit 1)
-        )
-      )
-    )
-  )
-  (symbol (lib_id "Device:R_Small") (at 243.84 140.97 90) (mirror x) (unit 1)
-    (in_bom yes) (on_board yes) (dnp no) (fields_autoplaced)
-    (property "Reference" "R25" (at 243.84 135.89 90)
-      (effects (font (size 1.27 1.27)))
-    )
-    (property "Value" "100k" (at 243.84 138.43 90)
-      (effects (font (size 1.27 1.27)))
-    )
-    (property "Footprint" "Resistor_SMD:R_0402_1005Metric" (at 243.84 140.97 0)
-      (effects (font (size 1.27 1.27)) hide)
-    )
-    (property "Datasheet" "~" (at 243.84 140.97 0)
-      (effects (font (size 1.27 1.27)) hide)
-    )
-    (property "LCSC Part" "C25741 " (at 243.84 140.97 0)
-      (effects (font (size 1.27 1.27)) hide)
-    )
-    (pin "1")
-    (pin "2")
-    (instances
-      (project "krecek-0.9"
-        (path "/8888f37b-ecc2-47df-8824-4b4e1e726451/bd29cd8c-9207-416a-90c1-7bdf6b5cfb97"
-          (reference "R25") (unit 1)
-        )
-      )
-    )
-  )
-  (symbol (lib_id "Device:R_Small") (at 234.95 114.3 270) (mirror x) (unit 1)
-    (in_bom yes) (on_board yes) (dnp no) (fields_autoplaced)
-    (property "Reference" "R14" (at 234.95 109.22 90)
-      (effects (font (size 1.27 1.27)))
-    )
-    (property "Value" "1M" (at 234.95 111.76 90)
-      (effects (font (size 1.27 1.27)))
-    )
-    (property "Footprint" "Resistor_SMD:R_0402_1005Metric" (at 234.95 114.3 0)
-      (effects (font (size 1.27 1.27)) hide)
-    )
-    (property "Datasheet" "~" (at 234.95 114.3 0)
-      (effects (font (size 1.27 1.27)) hide)
-    )
-    (property "LCSC Part" "C26083" (at 234.95 114.3 0)
-      (effects (font (size 1.27 1.27)) hide)
-    )
-    (pin "1")
-    (pin "2")
-    (instances
-      (project "krecek-0.9"
-        (path "/8888f37b-ecc2-47df-8824-4b4e1e726451/bd29cd8c-9207-416a-90c1-7bdf6b5cfb97"
-          (reference "R14") (unit 1)
         )
       )
@@
     )
   )
-  (symbol (lib_id "Connector:USB_C_Receptacle_USB2.0") (at 22.86 40.64 0) (unit 1)
+  (symbol (lib_id "LCSC:USB_C_Receptacle_USB2.0") (at 22.86 40.64 0) (unit 1)
     (in_bom yes) (on_board yes) (dnp no)
     (property "Reference" "J1" (at 35.56 17.78 0)
@@
       (effects (font (size 1.27 1.27)) hide)
     )
-    (property "Datasheet" "https://www.usb.org/sites/default/files/documents/usb_type-c.zip" (at 26.67 40.64 0)
+    (property "Datasheet" "https://www.usb.org/sites/default/files/documents/usb_type-c.zip" (at 22.86 74.93 0)
       (effects (font (size 1.27 1.27)) hide)
     )
@@
       (effects (font (size 1.27 1.27)) hide)
     )
-    (pin "A1")
-    (pin "A12")
-    (pin "A4")
+    (pin "A1B12")
+    (pin "A4B9")
     (pin "A5")
     (pin "A6")
     (pin "A7")
     (pin "A8")
-    (pin "A9")
-    (pin "B1")
-    (pin "B12")
-    (pin "B4")
+    (pin "B1A12")
+    (pin "B4A9")
     (pin "B5")
     (pin "B6")
     (pin "B7")
     (pin "B8")
-    (pin "B9")
     (pin "S1")
     (instances

Commit message: Add discrete antenna
Signed-off-by: Jan Hamal Dvořák <mordae@anilinux.org>
Parts:
- renumbered J1 to J3, U3 to U7
Changed lines of the file:
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@@
   (symbol (lib_id "LCSC:BQ24045DSQR") (at 130.81 30.48 0) (unit 1)
     (in_bom yes) (on_board yes) (dnp no) (fields_autoplaced)
-    (property "Reference" "U3" (at 130.81 17.78 0)
+    (property "Reference" "U7" (at 130.81 17.78 0)
       (effects (font (size 1.27 1.27)))
     )
@@
     (instances
       (project "krecek-0.9"
-        (path "/8888f37b-ecc2-47df-8824-4b4e1e726451"
-          (reference "U3") (unit 1)
-        )
         (path "/8888f37b-ecc2-47df-8824-4b4e1e726451/bd29cd8c-9207-416a-90c1-7bdf6b5cfb97"
           (reference "U7") (unit 1)
@@
   (symbol (lib_id "LCSC:USB_C_Receptacle_USB2.0") (at 22.86 40.64 0) (unit 1)
     (in_bom yes) (on_board yes) (dnp no)
-    (property "Reference" "J1" (at 35.56 17.78 0)
+    (property "Reference" "J3" (at 35.56 17.78 0)
       (effects (font (size 1.27 1.27)) (justify right))
     )
@@
     (instances
       (project "krecek-0.9"
-        (path "/8888f37b-ecc2-47df-8824-4b4e1e726451"
-          (reference "J1") (unit 1)
-        )
         (path "/8888f37b-ecc2-47df-8824-4b4e1e726451/bd29cd8c-9207-416a-90c1-7bdf6b5cfb97"
           (reference "J3") (unit 1)

Commit message: Further progress with the PCB layout
Signed-off-by: Jan Hamal Dvořák <mordae@anilinux.org>
Connections:
- net USB_{D+} renamed USB+
- net USB_{D-} renamed USB-
Changed lines of the file:
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@@
     (effects (font (size 1.27 1.27)) (justify right))
   )
-  (hierarchical_label "USB_{D-}" (shape bidirectional) (at 44.45 44.45 0) (fields_autoplaced)
+  (hierarchical_label "USB-" (shape bidirectional) (at 44.45 44.45 0) (fields_autoplaced)
     (effects (font (size 1.27 1.27)) (justify left))
   )
-  (hierarchical_label "USB_{D+}" (shape bidirectional) (at 44.45 39.37 0) (fields_autoplaced)
+  (hierarchical_label "USB+" (shape bidirectional) (at 44.45 39.37 0) (fields_autoplaced)
     (effects (font (size 1.27 1.27)) (justify left))
   )

Commit message: Further progress on routing the PCB
Signed-off-by: Jan Hamal Dvořák <mordae@anilinux.org>
Connections:
- net vin: now reaches C34.2, Q1.3 (D), R20.1, U10.5 (VIN)
- net vina: now reaches C38.1, R20.2, U10.6 (EN), U10.7 (PS/SYNC), U10.8 (VINA)
Changed lines of the file:
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@@
     (effects (font (size 1.27 1.27)) (justify right bottom))
+  )
+  (label "vina" (at 165.1 135.89 0) (fields_autoplaced)
+    (effects (font (size 1.27 1.27)) (justify left bottom))
   )
   (label "CC1" (at 165.1 76.2 0) (fields_autoplaced)
@@
     (effects (font (size 1.27 1.27)) (justify right bottom))
   )
+  (label "vin" (at 153.67 133.35 0) (fields_autoplaced)
+    (effects (font (size 1.27 1.27)) (justify left bottom))
+  )
   (label "CC1" (at 50.8 30.48 180) (fields_autoplaced)
