File: hw/krecek-0.9/power.kicad_sch (KiCad schematic)
At the start: 55 parts, among them J3 USB_C_Receptacle_USB2.0, Q1 AO3401A, Q2 AO3401A, Q3 AO3400A, Q4 AO3400A, Q5 AO3400A, Q6 AO3400A, U10 TPS63000, U5 AMS1117-3.3, U6 JST-PH-2P, U7 BQ24045DSQR, U8 AMS1117-3.3, U9 AMS1117-3.3

Commit message: Hardware as sent for manufacturing
Parts:
- added JP1: Jumper, Jumper:SolderJumper-2_P1.3mm_Bridged_RoundedPad1.0x1.5mm, symbol Jumper:SolderJumper_2_Bridged
- added JP2: Jumper_3_Bridged12, Jumper:SolderJumper-3_P1.3mm_Bridged12_RoundedPad1.0x1.5mm, symbol Jumper:Jumper_3_Bridged12
- C26, C27, C28, C29, C30, C31, C32, C33, C36: value 1uF -> 1u
- C34, C35: value 4.7uF -> 4.7u
- C37: value 100uF -> 100u
- C38: value 100nF -> 100n
- C39: value 10pF -> 10p
- D1: LCSC C72043 -> C72038
- L1: value 2.2uH -> 2.2u
- R13: footprint Resistor_SMD:R_0603_1608Metric -> Resistor_SMD:R_0402_1005Metric
Connections:
- net +5V: now also JP2.2 (C); no longer C35.2, C37.1, C39.2, R25.2, U10.1 (VOUT)
- net VBUS: now also JP1.1 (A), JP2.3 (B); no longer C29.1, U7.1 (IN)
- new net: C29.1, JP1.2 (B), U7.1 (IN)
- new net tps63000_vout: C35.2, C37.1, C39.2, JP2.1 (A), R25.2, U10.1 (VOUT)
Changed lines of the file:
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@@
     (stroke (width 0) (type default))
   )
-  (wire (pts (xy 41.91 25.4) (xy 76.2 25.4))
+  (wire (pts (xy 41.91 25.4) (xy 53.34 25.4))
     (stroke (width 0) (type default))
   )
@@
     (stroke (width 0) (type default))
   )
+  (wire (pts (xy 60.96 25.4) (xy 76.2 25.4))
+    (stroke (width 0) (type default))
+  )
   (wire (pts (xy 241.3 114.3) (xy 245.11 114.3))
     (stroke (width 0) (type default))
@@
   )
   (wire (pts (xy 38.1 120.65) (xy 57.15 120.65))
-    (stroke (width 0) (type default))
-  )
-  (wire (pts (xy 269.24 133.35) (xy 266.7 133.35))
     (stroke (width 0) (type default))
   )
@@
     (effects (font (size 1.27 1.27)) (justify left bottom))
   )
+  (label "tps63000_vout" (at 215.9 133.35 0) (fields_autoplaced)
+    (effects (font (size 1.27 1.27)) (justify left bottom))
+  )
   (label "V_{USB{slash}BATT}" (at 50.165 120.65 180) (fields_autoplaced)
     (effects (font (size 1.27 1.27)) (justify right bottom))
@@
       (effects (font (size 1.27 1.27)) (justify left))
     )
-    (property "Value" "4.7uF" (at 199.39 128.2763 0)
+    (property "Value" "4.7u" (at 199.39 128.2763 0)
       (effects (font (size 1.27 1.27)) (justify left))
     )
@@
       (effects (font (size 1.27 1.27)) (justify right))
     )
-    (property "Value" "2.2uH" (at 166.37 149.86 0)
+    (property "Value" "2.2u" (at 166.37 149.86 0)
       (effects (font (size 1.27 1.27)) (justify right))
     )
@@
       (effects (font (size 1.27 1.27)) (justify left))
     )
-    (property "Value" "1uF" (at 59.69 134.6263 0)
+    (property "Value" "1u" (at 59.69 134.6263 0)
       (effects (font (size 1.27 1.27)) (justify left))
     )
@@
       (effects (font (size 1.27 1.27)) (justify left))
     )
-    (property "Value" "1uF" (at 238.76 33.0263 0)
+    (property "Value" "1u" (at 238.76 33.0263 0)
       (effects (font (size 1.27 1.27)) (justify left))
     )
@@
       (effects (font (size 1.27 1.27)) (justify left))
     )
-    (property "Value" "1uF" (at 78.74 34.2963 0)
+    (property "Value" "1u" (at 78.74 34.2963 0)
       (effects (font (size 1.27 1.27)) (justify left))
     )
@@
       (effects (font (size 1.27 1.27)) hide)
     )
-    (property "LCSC" "C72043 " (at 171.45 53.34 0)
+    (property "LCSC" "C72038" (at 171.45 53.34 0)
       (effects (font (size 1.27 1.27)) hide)
     )
@@
       (effects (font (size 1.27 1.27)) (justify right))
     )
-    (property "Footprint" "Resistor_SMD:R_0603_1608Metric" (at 88.9 95.25 0)
+    (property "Footprint" "Resistor_SMD:R_0402_1005Metric" (at 88.9 95.25 0)
       (effects (font (size 1.27 1.27)) hide)
     )
@@
       (effects (font (size 1.27 1.27)) (justify left))
     )
-    (property "Value" "100nF" (at 151.13 151.1363 0)
+    (property "Value" "100n" (at 151.13 151.1363 0)
       (effects (font (size 1.27 1.27)) (justify left))
     )
@@
       (effects (font (size 1.27 1.27)) (justify left))
     )
-    (property "Value" "1uF" (at 238.76 83.8263 0)
+    (property "Value" "1u" (at 238.76 83.8263 0)
       (effects (font (size 1.27 1.27)) (justify left))
     )
@@
       (effects (font (size 1.27 1.27)) (justify left))
     )
-    (property "Value" "1uF" (at 269.24 33.0263 0)
+    (property "Value" "1u" (at 269.24 33.0263 0)
       (effects (font (size 1.27 1.27)) (justify left))
     )
@@
       (effects (font (size 1.27 1.27)))
     )
-    (property "Value" "10pF" (at 224.7963 148.59 90)
+    (property "Value" "10p" (at 224.7963 148.59 90)
       (effects (font (size 1.27 1.27)))
     )
@@
       (effects (font (size 1.27 1.27)) (justify left))
     )
-    (property "Value" "4.7uF" (at 167.64 128.2763 0)
+    (property "Value" "4.7u" (at 167.64 128.2763 0)
       (effects (font (size 1.27 1.27)) (justify left))
     )
@@
       (effects (font (size 1.27 1.27)) (justify left))
     )
-    (property "Value" "1uF" (at 238.76 58.4263 0)
+    (property "Value" "1u" (at 238.76 58.4263 0)
       (effects (font (size 1.27 1.27)) (justify left))
     )
@@
     )
   )
+  (symbol (lib_id "Jumper:Jumper_3_Bridged12") (at 266.7 127 90) (unit 1)
+    (in_bom yes) (on_board yes) (dnp no) (fields_autoplaced)
+    (property "Reference" "JP2" (at 264.16 125.73 90)
+      (effects (font (size 1.27 1.27)) (justify left))
+    )
+    (property "Value" "Jumper_3_Bridged12" (at 264.16 128.27 90)
+      (effects (font (size 1.27 1.27)) (justify left))
+    )
+    (property "Footprint" "Jumper:SolderJumper-3_P1.3mm_Bridged12_RoundedPad1.0x1.5mm" (at 266.7 127 0)
+      (effects (font (size 1.27 1.27)) hide)
+    )
+    (property "Datasheet" "~" (at 266.7 127 0)
+      (effects (font (size 1.27 1.27)) hide)
+    )
+    (pin "3")
+    (pin "2")
+    (pin "1")
+    (instances
+      (project "krecek-0.9"
+        (path "/8888f37b-ecc2-47df-8824-4b4e1e726451/bd29cd8c-9207-416a-90c1-7bdf6b5cfb97"
+          (reference "JP2") (unit 1)
+        )
+      )
+    )
+  )
   (symbol (lib_id "Device:C_Small") (at 266.7 82.55 0) (unit 1)
     (in_bom yes) (on_board yes) (dnp no) (fields_autoplaced)
@@
       (effects (font (size 1.27 1.27)) (justify left))
     )
-    (property "Value" "1uF" (at 269.24 83.8263 0)
+    (property "Value" "1u" (at 269.24 83.8263 0)
       (effects (font (size 1.27 1.27)) (justify left))
     )
@@
     )
   )
+  (symbol (lib_id "power:VBUS") (at 266.7 120.65 90) (unit 1)
+    (in_bom yes) (on_board yes) (dnp no) (fields_autoplaced)
+    (property "Reference" "#PWR0112" (at 270.51 120.65 0)
+      (effects (font (size 1.27 1.27)) hide)
+    )
+    (property "Value" "VBUS" (at 262.89 120.65 90)
+      (effects (font (size 1.27 1.27)) (justify left))
+    )
+    (property "Footprint" "" (at 266.7 120.65 0)
+      (effects (font (size 1.27 1.27)) hide)
+    )
+    (property "Datasheet" "" (at 266.7 120.65 0)
+      (effects (font (size 1.27 1.27)) hide)
+    )
+    (pin "1")
+    (instances
+      (project "krecek-0.9"
+        (path "/8888f37b-ecc2-47df-8824-4b4e1e726451/bd29cd8c-9207-416a-90c1-7bdf6b5cfb97"
+          (reference "#PWR0112") (unit 1)
+        )
+      )
+    )
+  )
+  (symbol (lib_id "Jumper:SolderJumper_2_Bridged") (at 57.15 25.4 0) (unit 1)
+    (in_bom yes) (on_board yes) (dnp no) (fields_autoplaced)
+    (property "Reference" "JP1" (at 57.15 19.05 0)
+      (effects (font (size 1.27 1.27)))
+    )
+    (property "Value" "Jumper" (at 57.15 21.59 0)
+      (effects (font (size 1.27 1.27)))
+    )
+    (property "Footprint" "Jumper:SolderJumper-2_P1.3mm_Bridged_RoundedPad1.0x1.5mm" (at 57.15 25.4 0)
+      (effects (font (size 1.27 1.27)) hide)
+    )
+    (property "Datasheet" "~" (at 57.15 25.4 0)
+      (effects (font (size 1.27 1.27)) hide)
+    )
+    (pin "1")
+    (pin "2")
+    (instances
+      (project "krecek-0.9"
+        (path "/8888f37b-ecc2-47df-8824-4b4e1e726451/bd29cd8c-9207-416a-90c1-7bdf6b5cfb97"
+          (reference "JP1") (unit 1)
+        )
+      )
+    )
+  )
   (symbol (lib_id "power:GND") (at 25.4 166.37 0) (unit 1)
     (in_bom yes) (on_board yes) (dnp no) (fields_autoplaced)
@@
       (effects (font (size 1.27 1.27)) (justify left))
     )
-    (property "Value" "1uF" (at 173.99 31.7563 0)
+    (property "Value" "1u" (at 173.99 31.7563 0)
       (effects (font (size 1.27 1.27)) (justify left))
     )
@@
       (effects (font (size 1.27 1.27)) (justify left))
     )
-    (property "Value" "1uF" (at 269.24 58.4263 0)
+    (property "Value" "1u" (at 269.24 58.4263 0)
       (effects (font (size 1.27 1.27)) (justify left))
     )
@@
     )
   )
-  (symbol (lib_id "power:+5V") (at 269.24 133.35 270) (unit 1)
-    (in_bom yes) (on_board yes) (dnp no) (fields_autoplaced)
-    (property "Reference" "#PWR054" (at 265.43 133.35 0)
-      (effects (font (size 1.27 1.27)) hide)
-    )
-    (property "Value" "+5V" (at 272.415 133.35 90)
-      (effects (font (size 1.27 1.27)) (justify left))
-    )
-    (property "Footprint" "" (at 269.24 133.35 0)
-      (effects (font (size 1.27 1.27)) hide)
-    )
-    (property "Datasheet" "" (at 269.24 133.35 0)
+  (symbol (lib_id "power:+5V") (at 270.51 127 270) (unit 1)
+    (in_bom yes) (on_board yes) (dnp no) (fields_autoplaced)
+    (property "Reference" "#PWR054" (at 266.7 127 0)
+      (effects (font (size 1.27 1.27)) hide)
+    )
+    (property "Value" "+5V" (at 273.685 127 90)
+      (effects (font (size 1.27 1.27)) (justify left))
+    )
+    (property "Footprint" "" (at 270.51 127 0)
+      (effects (font (size 1.27 1.27)) hide)
+    )
+    (property "Datasheet" "" (at 270.51 127 0)
       (effects (font (size 1.27 1.27)) hide)
     )
@@
   (symbol (lib_id "Device:C_Polarized_Small") (at 266.7 140.97 0) (unit 1)
     (in_bom yes) (on_board yes) (dnp no) (fields_autoplaced)
-    (property "Reference" "C37" (at 269.875 139.1539 0)
-      (effects (font (size 1.27 1.27)) (justify left))
-    )
-    (property "Value" "100uF" (at 269.875 141.6939 0)
-      (effects (font (size 1.27 1.27)) (justify left))
-    )
+    (property "Reference" "C37" (at 269.24 139.1539 0)
+      (effects (font (size 1.27 1.27)) (justify left))
+    )
+    (property "Value" "100u" (at 269.24 141.6939 0)
+      (effects (font (size 1.27 1.27)) (justify left))
+    )

Commit message: Partially resolve some of the design issues
Related to #3 and #4.
Connections:
- net USB+: now also J3.A6 (D+), J3.B6 (D+); no longer J3.A7 (D-), J3.B7 (D-)
- net USB-: now also J3.A7 (D-), J3.B7 (D-); no longer J3.A6 (D+), J3.B6 (D+)
Changed lines of the file:
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@@
     (effects (font (size 1.27 1.27)) (justify right))
   )
-  (hierarchical_label "USB-" (shape bidirectional) (at 44.45 44.45 0) (fields_autoplaced)
+  (hierarchical_label "USB-" (shape bidirectional) (at 44.45 39.37 0) (fields_autoplaced)
     (effects (font (size 1.27 1.27)) (justify left))
   )
-  (hierarchical_label "USB+" (shape bidirectional) (at 44.45 39.37 0) (fields_autoplaced)
+  (hierarchical_label "USB+" (shape bidirectional) (at 44.45 44.45 0) (fields_autoplaced)
     (effects (font (size 1.27 1.27)) (justify left))
   )

Commit message: Replace charger with correct one for our battery
Resolves #9.
Parts:
- removed U7: BQ24045DSQR, LCSC:WSON-10_L2.0-W2.0-P0.40-BL-EP, symbol LCSC:BQ24045DSQR
- added U7: BQ24040DSQR, LCSC:WSON-10_L2.0-W2.0-P0.40-BL-EP, symbol LCSC:BQ24040DSQR
Connections:
- net +BATT: now also U7.10 (OUT)
- net GND: now also U7.11 (VSS), U7.3 (VSS)
- net ISET2: now also U7.7 (ISET2)
- net ~{CHG}: now also U7.8 (~{CHG})
- net ~{PG}: now also U7.5 (~{PG})
- net at C29.1, JP1.2 (B): now also U7.1 (IN)
- net at R6.1: now also U7.2 (ISET)
- net at R7.2: now also U7.4 (PRETERM)
Changed lines of the file:
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@@
+    )
+  )
+  (symbol (lib_id "LCSC:BQ24040DSQR") (at 130.81 30.48 0) (unit 1)
+    (in_bom yes) (on_board yes) (dnp no) (fields_autoplaced)
+    (property "Reference" "U7" (at 130.81 17.78 0)
+      (effects (font (size 1.27 1.27)))
+    )
+    (property "Value" "BQ24040DSQR" (at 130.81 20.32 0)
+      (effects (font (size 1.27 1.27)))
+    )
+    (property "Footprint" "LCSC:WSON-10_L2.0-W2.0-P0.40-BL-EP" (at 130.81 45.72 0)
+      (effects (font (size 1.27 1.27)) hide)
+    )
+    (property "Datasheet" "https://lcsc.com/product-detail/PMIC-Battery-Management_TI_BQ24040DSQR_BQ24040DSQR_C81080.html" (at 130.81 48.26 0)
+      (effects (font (size 1.27 1.27)) hide)
+    )
+    (property "LCSC Part" "C81080" (at 130.81 50.8 0)
+      (effects (font (size 1.27 1.27)) hide)
+    )
+    (pin "6")
+    (pin "10")
+    (pin "4")
+    (pin "7")
+    (pin "3")
+    (pin "1")
+    (pin "2")
+    (pin "5")
+    (pin "11")
+    (pin "9")
+    (pin "8")
+    (instances
+      (project "krecek-0.9"
+        (path "/8888f37b-ecc2-47df-8824-4b4e1e726451/bd29cd8c-9207-416a-90c1-7bdf6b5cfb97"
+          (reference "U7") (unit 1)
+        )
+      )
     )
   )
@@
         )
       )
-    )
-  )
-  (symbol (lib_id "LCSC:BQ24045DSQR") (at 130.81 30.48 0) (unit 1)
-    (in_bom yes) (on_board yes) (dnp no) (fields_autoplaced)
-    (property "Reference" "U7" (at 130.81 17.78 0)
-      (effects (font (size 1.27 1.27)))
-    )
-    (property "Value" "BQ24045DSQR" (at 130.81 20.32 0)
-      (effects (font (size 1.27 1.27)))
-    )
-    (property "Footprint" "LCSC:WSON-10_L2.0-W2.0-P0.40-BL-EP" (at 130.81 55.88 0)
-      (effects (font (size 1.27 1.27)) hide)
-    )
-    (property "Datasheet" "https://lcsc.com/product-detail/PMIC-Battery-Management_TI_BQ24045DSQR_BQ24045DSQR_C148983.html" (at 130.81 58.42 0)
-      (effects (font (size 1.27 1.27)) hide)
-    )
-    (property "LCSC Part" "C148983" (at 130.81 60.96 0)
-      (effects (font (size 1.27 1.27)) hide)
-    )
-    (pin "1")
-    (pin "10")
-    (pin "11")
-    (pin "2")
-    (pin "3")
-    (pin "4")
-    (pin "5")
-    (pin "6")
-    (pin "7")
-    (pin "8")
-    (pin "9")
-    (instances
-      (project "krecek-0.9"
-        (path "/8888f37b-ecc2-47df-8824-4b4e1e726451/bd29cd8c-9207-416a-90c1-7bdf6b5cfb97"
-          (reference "U7") (unit 1)
-        )
-      )

Commit message: Fix OFF issues, rename buttons
Resolves #4.
Parts:
- removed JP1: Jumper, Jumper:SolderJumper-2_P1.3mm_Bridged_RoundedPad1.0x1.5mm, symbol Jumper:SolderJumper_2_Bridged
Connections:
- net VBUS: now also C29.1, U7.1 (IN)
Changed lines of the file:
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@@
-    (stroke (width 0) (type default))
-  )
-  (wire (pts (xy 41.91 25.4) (xy 53.34 25.4))
     (stroke (width 0) (type default))
   )
@@
     (stroke (width 0) (type default))
   )
-  (wire (pts (xy 60.96 25.4) (xy 76.2 25.4))
+  (wire (pts (xy 41.91 25.4) (xy 76.2 25.4))
     (stroke (width 0) (type default))
   )
   (wire (pts (xy 241.3 114.3) (xy 245.11 114.3))
-    (stroke (width 0) (type default))
-  )
-  (wire (pts (xy 76.2 22.86) (xy 76.2 25.4))
     (stroke (width 0) (type default))
   )
@@
         (path "/8888f37b-ecc2-47df-8824-4b4e1e726451/bd29cd8c-9207-416a-90c1-7bdf6b5cfb97"
           (reference "#PWR0112") (unit 1)
-        )
-      )
-    )
-  )
-  (symbol (lib_id "Jumper:SolderJumper_2_Bridged") (at 57.15 25.4 0) (unit 1)
-    (in_bom yes) (on_board yes) (dnp no) (fields_autoplaced)
-    (property "Reference" "JP1" (at 57.15 19.05 0)
-      (effects (font (size 1.27 1.27)))
-    )
-    (property "Value" "Jumper" (at 57.15 21.59 0)
-      (effects (font (size 1.27 1.27)))
-    )
-    (property "Footprint" "Jumper:SolderJumper-2_P1.3mm_Bridged_RoundedPad1.0x1.5mm" (at 57.15 25.4 0)
-      (effects (font (size 1.27 1.27)) hide)
-    )
-    (property "Datasheet" "~" (at 57.15 25.4 0)
-      (effects (font (size 1.27 1.27)) hide)
-    )
-    (pin "1")
-    (pin "2")
-    (instances
-      (project "krecek-0.9"
-        (path "/8888f37b-ecc2-47df-8824-4b4e1e726451/bd29cd8c-9207-416a-90c1-7bdf6b5cfb97"
-          (reference "JP1") (unit 1)
         )
       )
@@
         )
       )
-    )
-  )
-  (symbol (lib_id "power:PWR_FLAG") (at 76.2 22.86 0) (unit 1)
-    (in_bom yes) (on_board yes) (dnp no) (fields_autoplaced)
-    (property "Reference" "#FLG01" (at 76.2 20.955 0)
-      (effects (font (size 1.27 1.27)) hide)
-    )
-    (property "Value" "PWR_FLAG" (at 76.2 17.78 0)
-      (effects (font (size 1.27 1.27)))
-    )
-    (property "Footprint" "" (at 76.2 22.86 0)
-      (effects (font (size 1.27 1.27)) hide)
-    )
-    (property "Datasheet" "~" (at 76.2 22.86 0)
-      (effects (font (size 1.27 1.27)) hide)
-    )
-    (pin "1")
-    (instances
-      (project "krecek-0.9"
-        (path "/8888f37b-ecc2-47df-8824-4b4e1e726451/bd29cd8c-9207-416a-90c1-7bdf6b5cfb97"
-          (reference "#FLG01") (unit 1)
-        )
-      )

Commit message: Stabilizovat ISET2 na 100mA při bootu
Parts:
- added R42: 10k, Resistor_SMD:R_0402_1005Metric, symbol Device:R_Small
- added R43: 39k, Resistor_SMD:R_0603_1608Metric, symbol Device:R_Small
Connections:
- net GND: now also R42.1
- net ISET2: now also R42.2, R43.1
- net VBUS: now also R43.2
Changed lines of the file:
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@@
   (junction (at 254 63.5) (diameter 0) (color 0 0 0 0)
+  )
+  (junction (at 88.9 59.69) (diameter 0) (color 0 0 0 0)
   )
   (junction (at 266.7 76.2) (diameter 0) (color 0 0 0 0)
@@
     (stroke (width 0) (type default))
   )
+  (wire (pts (xy 85.09 59.69) (xy 88.9 59.69))
+    (stroke (width 0) (type default))
+  )
   (wire (pts (xy 88.9 88.9) (xy 101.6 88.9))
     (stroke (width 0) (type default))
@@
     (stroke (width 0) (type default))
   )
+  (wire (pts (xy 88.9 59.69) (xy 88.9 63.5))
+    (stroke (width 0) (type default))
+  )
   (wire (pts (xy 44.45 44.45) (xy 41.91 44.45))
     (stroke (width 0) (type default))
@@
     (stroke (width 0) (type default))
   )
+  (wire (pts (xy 88.9 68.58) (xy 88.9 72.39))
+    (stroke (width 0) (type default))
+  )
   (wire (pts (xy 273.05 76.2) (xy 266.7 76.2))
     (stroke (width 0) (type default))
@@
     (stroke (width 0) (type default))
   )
+  (wire (pts (xy 101.6 59.69) (xy 88.9 59.69))
+    (stroke (width 0) (type default))
+  )
   (wire (pts (xy 110.49 162.56) (xy 110.49 165.1))
     (stroke (width 0) (type default))
@@
   )
   (wire (pts (xy 127 129.54) (xy 127 133.35))
+    (stroke (width 0) (type default))
+  )
+  (wire (pts (xy 76.2 59.69) (xy 80.01 59.69))
     (stroke (width 0) (type default))
   )
@@
     (effects (font (size 1.27 1.27)) (justify right))
   )
+  (hierarchical_label "ISET2" (shape input) (at 101.6 59.69 0) (fields_autoplaced)
+    (effects (font (size 1.27 1.27)) (justify left))
+  )
   (hierarchical_label "ON" (shape output) (at 101.6 88.9 0) (fields_autoplaced)
     (effects (font (size 1.27 1.27)) (justify left))
@@
         (path "/8888f37b-ecc2-47df-8824-4b4e1e726451/bd29cd8c-9207-416a-90c1-7bdf6b5cfb97"
           (reference "#PWR048") (unit 1)
+        )
+      )
+    )
+  )
+  (symbol (lib_id "Device:R_Small") (at 88.9 66.04 0) (mirror x) (unit 1)
+    (in_bom yes) (on_board yes) (dnp no) (fields_autoplaced)
+    (property "Reference" "R42" (at 86.36 64.77 0)
+      (effects (font (size 1.27 1.27)) (justify right))
+    )
+    (property "Value" "10k" (at 86.36 67.31 0)
+      (effects (font (size 1.27 1.27)) (justify right))
+    )
+    (property "Footprint" "Resistor_SMD:R_0402_1005Metric" (at 88.9 66.04 0)
+      (effects (font (size 1.27 1.27)) hide)
+    )
+    (property "Datasheet" "~" (at 88.9 66.04 0)
+      (effects (font (size 1.27 1.27)) hide)
+    )
+    (property "LCSC Part" "C25744" (at 88.9 66.04 0)
+      (effects (font (size 1.27 1.27)) hide)
+    )
+    (pin "1")
+    (pin "2")
+    (instances
+      (project "krecek-0.9"
+        (path "/8888f37b-ecc2-47df-8824-4b4e1e726451/bd29cd8c-9207-416a-90c1-7bdf6b5cfb97"
+          (reference "R42") (unit 1)
         )
       )
@@
         (path "/8888f37b-ecc2-47df-8824-4b4e1e726451/bd29cd8c-9207-416a-90c1-7bdf6b5cfb97"
           (reference "R23") (unit 1)
+        )
+      )
+    )
+  )
+  (symbol (lib_id "power:VBUS") (at 76.2 59.69 90) (mirror x) (unit 1)
+    (in_bom yes) (on_board yes) (dnp no) (fields_autoplaced)
+    (property "Reference" "#PWR0114" (at 80.01 59.69 0)
+      (effects (font (size 1.27 1.27)) hide)
+    )
+    (property "Value" "VBUS" (at 72.39 59.69 90)
+      (effects (font (size 1.27 1.27)) (justify left))
+    )
+    (property "Footprint" "" (at 76.2 59.69 0)
+      (effects (font (size 1.27 1.27)) hide)
+    )
+    (property "Datasheet" "" (at 76.2 59.69 0)
+      (effects (font (size 1.27 1.27)) hide)
+    )
+    (pin "1")
+    (instances
+      (project "krecek-0.9"
+        (path "/8888f37b-ecc2-47df-8824-4b4e1e726451/bd29cd8c-9207-416a-90c1-7bdf6b5cfb97"
+          (reference "#PWR0114") (unit 1)
         )
       )
@@
     )
   )
+  (symbol (lib_id "Device:R_Small") (at 82.55 59.69 270) (mirror x) (unit 1)
+    (in_bom yes) (on_board yes) (dnp no) (fields_autoplaced)
+    (property "Reference" "R43" (at 82.55 54.61 90)
+      (effects (font (size 1.27 1.27)))
+    )
+    (property "Value" "39k" (at 82.55 57.15 90)
+      (effects (font (size 1.27 1.27)))
+    )
+    (property "Footprint" "Resistor_SMD:R_0603_1608Metric" (at 82.55 59.69 0)
+      (effects (font (size 1.27 1.27)) hide)
+    )
+    (property "Datasheet" "~" (at 82.55 59.69 0)
+      (effects (font (size 1.27 1.27)) hide)
+    )
+    (property "LCSC Part" "C23153" (at 82.55 59.69 0)
+      (effects (font (size 1.27 1.27)) hide)
+    )
+    (pin "1")
+    (pin "2")
+    (instances
+      (project "krecek-0.9"
+        (path "/8888f37b-ecc2-47df-8824-4b4e1e726451/bd29cd8c-9207-416a-90c1-7bdf6b5cfb97"
+          (reference "R43") (unit 1)
+        )
+      )
+    )
+  )
   (symbol (lib_id "power:GND") (at 191.77 27.94 270) (unit 1)
     (in_bom yes) (on_board yes) (dnp no) (fields_autoplaced)
@@
         )
       )
+    )
+  )
+  (symbol (lib_id "power:GND") (at 88.9 72.39 0) (mirror y) (unit 1)
+    (in_bom yes) (on_board yes) (dnp no) (fields_autoplaced)
+    (property "Reference" "#PWR0115" (at 88.9 78.74 0)
+      (effects (font (size 1.27 1.27)) hide)
+    )
+    (property "Value" "GND" (at 88.9 77.47 0)
+      (effects (font (size 1.27 1.27)))
+    )
+    (property "Footprint" "" (at 88.9 72.39 0)
+      (effects (font (size 1.27 1.27)) hide)
+    )
+    (property "Datasheet" "" (at 88.9 72.39 0)
+      (effects (font (size 1.27 1.27)) hide)
+    )
+    (pin "1")
+    (instances
+      (project "krecek-0.9"
+        (path "/8888f37b-ecc2-47df-8824-4b4e1e726451/bd29cd8c-9207-416a-90c1-7bdf6b5cfb97"
+          (reference "#PWR0115") (unit 1)
+        )
+      )

Commit message: Improve flip-flop design
Parts:
- added JP1: Jumper_2_Bridged, Jumper:SolderJumper-2_P1.3mm_Bridged_RoundedPad1.0x1.5mm, symbol Jumper:Jumper_2_Bridged
- R18: value 330k -> 100k; footprint Resistor_SMD:R_0603_1608Metric -> Resistor_SMD:R_0402_1005Metric; LCSC Part C23137 -> C25741
- R26: value 10M -> 330k; LCSC Part C7250 -> C23137
Connections:
- net GND: no longer R26.1
- net VBUS: now also JP1.1 (A); no longer C29.1, U7.1 (IN)
- net at Q3.1 (G), Q4.3 (D), Q5.3 (D)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: now also R26.2; no longer Q1.1 (G)
- net at Q3.3 (D), Q4.1 (G), Q6.3 (D)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: no longer R26.2
- new net: C29.1, JP1.2 (B), U7.1 (IN)
- new net: Q1.1 (G), R26.1
Other:
- moved on the sheet: C34, C35, C37, C38, C39, JP2, L1, Q1, R14, R15, R16, R20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
