File: hw/krecek-0.9/power.kicad_sch (KiCad schematic)
At the start: 59 parts, among them J3 USB_C_Receptacle_USB2.0, Q1 AO3401A, Q2 AO3401A, Q3 AO3400A, Q4 AO3400A, Q5 AO3400A, Q6 AO3400A, U10 TPS63000, U5 AMS1117-3.3, U6 JST-PH-2P, U7 BQ24040DSQR, U8 AMS1117-3.3, U9 AMS1117-3.3

Commit message: Fix battery PMOS orientation
Connections:
- net +BATT: now also Q2.2 (S); no longer Q2.3 (D)
- net V_{USB/BATT}: now also Q2.3 (D); no longer Q2.2 (S)
Changed lines of the file:
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@@
     )
   )
-  (symbol (lib_name "AO3401A_1") (lib_id "Transistor_FET:AO3401A") (at 35.56 133.35 0) (mirror x) (unit 1)
-    (in_bom yes) (on_board yes) (dnp no)
-    (property "Reference" "Q2" (at 41.91 134.62 0)
+  (symbol (lib_name "AO3401A_1") (lib_id "Transistor_FET:AO3401A") (at 35.56 133.35 0) (unit 1)
+    (in_bom yes) (on_board yes) (dnp no) (fields_autoplaced)
+    (property "Reference" "Q2" (at 41.91 132.08 0)
       (effects (font (size 1.27 1.27)) (justify left))
     )
-    (property "Value" "AO3401A" (at 41.91 132.08 0)
+    (property "Value" "AO3401A" (at 41.91 134.62 0)
       (effects (font (size 1.27 1.27)) (justify left))
     )
-    (property "Footprint" "Package_TO_SOT_SMD:SOT-23" (at 40.64 131.445 0)
+    (property "Footprint" "Package_TO_SOT_SMD:SOT-23" (at 40.64 135.255 0)
       (effects (font (size 1.27 1.27) italic) (justify left) hide)
     )

Commit message: Fix input PMOS orientation (again)
Parts:
- removed D3: SS54, Diode_SMD:D_SMA, symbol Device:D_Small
- added D3: SS54, symbol Device:D_Schottky_Small
- renumbered R43 to R10, R42 to R11, R9 to R12, R11 to R14, R13 to R16, R14 to R17, R15 to R18, R16 to R19, R17 to R20, R18 to R21, R26 to R22, R19 to R23, R20 to R24, R21 to R25, R22 to R26, R23 to R27, R24 to R28, R25 to R29, R27 to R30, R6 to R7, R7 to R8, R8 to R9
Connections:
- net +BATT: now also Q2.3 (D); no longer Q2.2 (S)
- net VBUS: now also D3.2 (A)
- net V_{USB/BATT}: now also Q2.2 (S), D3.1 (K); no longer Q2.3 (D)
