File: hw/krecek-0.9/audio.kicad_sch (KiCad schematic)
At the start: 6 parts, among them CN1 PJ-313B6-B, U10 TPA2028D1YZFT, U11 ES8312

Commit message: Fix amplifier/speaker connection
Signed-off-by: Jan Hamal Dvořák <mordae@anilinux.org>
Connections:
- net at SPK1.1 (+): now also U10.C1 (OUT-); no longer C5.2
- net at SPK1.2: now also U10.B1 (OUT+); no longer C5.2
- net at C5.1: no longer U10.B1 (OUT+)
- net at U10.B3 (IN+): now also C5.2
- net at C5.1: no longer U10.C1 (OUT-)
- net at U10.C3 (IN-): now also C5.2
Other:
- moved on the sheet: C5, SPK1, U10
Changed lines of the file:
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@@
 (kicad_sch (version 20230121) (generator eeschema)
   (paper "A4")
-  (wire (pts (xy 222.25 60.96) (xy 232.41 60.96))
+  (wire (pts (xy 205.74 55.88) (xy 220.98 55.88))
     (stroke (width 0) (type default))
   )
-  (wire (pts (xy 250.19 58.42) (xy 254 58.42))
+  (wire (pts (xy 205.74 53.34) (xy 220.98 53.34))
     (stroke (width 0) (type default))
   )
-  (wire (pts (xy 237.49 60.96) (xy 254 60.96))
-    (stroke (width 0) (type default))
-  )
-  (wire (pts (xy 222.25 58.42) (xy 245.11 58.42))
-    (stroke (width 0) (type default))
-  )
-  (symbol (lib_id "power:GND") (at 222.25 66.04 90) (unit 1)
-    (in_bom yes) (on_board yes) (dnp no) (fields_autoplaced)
-    (property "Reference" "#PWR031" (at 228.6 66.04 0)
-      (effects (font (size 1.27 1.27)) hide)
-    )
-    (property "Value" "GND" (at 226.06 66.04 90)
+  (symbol (lib_id "power:GND") (at 259.08 66.04 90) (unit 1)
+    (in_bom yes) (on_board yes) (dnp no) (fields_autoplaced)
+    (property "Reference" "#PWR031" (at 265.43 66.04 0)
+      (effects (font (size 1.27 1.27)) hide)
+    )
+    (property "Value" "GND" (at 262.89 66.04 90)
       (effects (font (size 1.27 1.27)) (justify right))
     )
-    (property "Footprint" "" (at 222.25 66.04 0)
-      (effects (font (size 1.27 1.27)) hide)
-    )
-    (property "Datasheet" "" (at 222.25 66.04 0)
+    (property "Footprint" "" (at 259.08 66.04 0)
+      (effects (font (size 1.27 1.27)) hide)
+    )
+    (property "Datasheet" "" (at 259.08 66.04 0)
       (effects (font (size 1.27 1.27)) hide)
     )
@@
     )
   )
-  (symbol (lib_id "LCSC:FS-1540") (at 257.81 59.69 0) (unit 1)
-    (in_bom yes) (on_board yes) (dnp no) (fields_autoplaced)
-    (property "Reference" "SPK1" (at 262.89 58.42 0)
+  (symbol (lib_id "LCSC:FS-1540") (at 262.89 59.69 0) (unit 1)
+    (in_bom yes) (on_board yes) (dnp no) (fields_autoplaced)
+    (property "Reference" "SPK1" (at 267.97 58.42 0)
       (effects (font (size 1.27 1.27)) (justify left))
     )
-    (property "Value" "FS-1540" (at 262.89 60.96 0)
+    (property "Value" "FS-1540" (at 267.97 60.96 0)
       (effects (font (size 1.27 1.27)) (justify left))
     )
-    (property "Footprint" "LCSC:BUZ-SMD_5P-L15.0-W15.0-P13.7-BL" (at 257.81 72.39 0)
-      (effects (font (size 1.27 1.27)) hide)
-    )
-    (property "Datasheet" "" (at 257.81 59.69 0)
-      (effects (font (size 1.27 1.27)) hide)
-    )
-    (property "LCSC Part" "C482341" (at 257.81 74.93 0)
+    (property "Footprint" "LCSC:BUZ-SMD_5P-L15.0-W15.0-P13.7-BL" (at 262.89 72.39 0)
+      (effects (font (size 1.27 1.27)) hide)
+    )
+    (property "Datasheet" "" (at 262.89 59.69 0)
+      (effects (font (size 1.27 1.27)) hide)
+    )
+    (property "LCSC Part" "C482341" (at 262.89 74.93 0)
       (effects (font (size 1.27 1.27)) hide)
     )
@@
     )
   )
-  (symbol (lib_id "LCSC:TPA2028D1YZFT") (at 203.2 60.96 0) (unit 1)
-    (in_bom yes) (on_board yes) (dnp no) (fields_autoplaced)
-    (property "Reference" "U10" (at 203.2 45.72 0)
+  (symbol (lib_id "LCSC:TPA2028D1YZFT") (at 240.03 60.96 0) (unit 1)
+    (in_bom yes) (on_board yes) (dnp no) (fields_autoplaced)
+    (property "Reference" "U10" (at 240.03 45.72 0)
       (effects (font (size 1.524 1.524)))
     )
-    (property "Value" "TPA2028D1YZFT" (at 203.2 48.26 0)
+    (property "Value" "TPA2028D1YZFT" (at 240.03 48.26 0)
       (effects (font (size 1.524 1.524)))
     )
-    (property "Footprint" "LCSC:TPA2028" (at 203.2 73.66 0)
+    (property "Footprint" "LCSC:TPA2028" (at 240.03 73.66 0)
       (effects (font (size 1.27 1.27) italic) hide)
     )
-    (property "Datasheet" "TPA2028D1YZFT" (at 203.2 76.2 0)
+    (property "Datasheet" "TPA2028D1YZFT" (at 240.03 76.2 0)
       (effects (font (size 1.27 1.27) italic) hide)
     )
@@
     )
   )
-  (symbol (lib_id "Device:C_Small") (at 234.95 60.96 90) (mirror x) (unit 1)
-    (in_bom yes) (on_board yes) (dnp no) (fields_autoplaced)
-    (property "Reference" "C5" (at 234.9563 64.77 90)
-      (effects (font (size 1.27 1.27)))
-    )
-    (property "Value" "10uF" (at 234.9563 67.31 90)
-      (effects (font (size 1.27 1.27)))
-    )
-    (property "Footprint" "Capacitor_SMD:C_0805_2012Metric" (at 234.95 60.96 0)
-      (effects (font (size 1.27 1.27)) hide)
-    )
-    (property "Datasheet" "~" (at 234.95 60.96 0)
-      (effects (font (size 1.27 1.27)) hide)
-    )
-    (property "LCSC Part" "C15850" (at 234.95 60.96 0)
+  (symbol (lib_id "Device:C_Small") (at 203.2 55.88 90) (mirror x) (unit 1)
+    (in_bom yes) (on_board yes) (dnp no) (fields_autoplaced)
+    (property "Reference" "C5" (at 203.2063 59.69 90)
+      (effects (font (size 1.27 1.27)))
+    )
+    (property "Value" "10uF" (at 203.2063 62.23 90)
+      (effects (font (size 1.27 1.27)))
+    )
+    (property "Footprint" "Capacitor_SMD:C_0805_2012Metric" (at 203.2 55.88 0)
+      (effects (font (size 1.27 1.27)) hide)
+    )
+    (property "Datasheet" "~" (at 203.2 55.88 0)
+      (effects (font (size 1.27 1.27)) hide)
+    )
+    (property "LCSC Part" "C15850" (at 203.2 55.88 0)
       (effects (font (size 1.27 1.27)) hide)
     )
@@
     )
   )
-  (symbol (lib_id "power:+3.3VA") (at 222.25 53.34 270) (unit 1)
-    (in_bom yes) (on_board yes) (dnp no) (fields_autoplaced)
-    (property "Reference" "#PWR032" (at 218.44 53.34 0)
-      (effects (font (size 1.27 1.27)) hide)
-    )
-    (property "Value" "+3.3VA" (at 226.06 53.34 90)
+  (symbol (lib_id "power:+3.3VA") (at 259.08 53.34 270) (unit 1)
+    (in_bom yes) (on_board yes) (dnp no) (fields_autoplaced)
+    (property "Reference" "#PWR032" (at 255.27 53.34 0)
+      (effects (font (size 1.27 1.27)) hide)
+    )
+    (property "Value" "+3.3VA" (at 262.89 53.34 90)
       (effects (font (size 1.27 1.27)) (justify left))
     )
-    (property "Footprint" "" (at 222.25 53.34 0)
-      (effects (font (size 1.27 1.27)) hide)
-    )
-    (property "Datasheet" "" (at 222.25 53.34 0)
+    (property "Footprint" "" (at 259.08 53.34 0)
+      (effects (font (size 1.27 1.27)) hide)
+    )
+    (property "Datasheet" "" (at 259.08 53.34 0)
       (effects (font (size 1.27 1.27)) hide)
     )
@@
     )
   )
-  (symbol (lib_id "Device:C_Small") (at 247.65 58.42 90) (unit 1)
-    (in_bom yes) (on_board yes) (dnp no) (fields_autoplaced)
-    (property "Reference" "C5" (at 247.6563 52.07 90)
-      (effects (font (size 1.27 1.27)))
-    )
-    (property "Value" "10uF" (at 247.6563 54.61 90)
-      (effects (font (size 1.27 1.27)))
-    )
-    (property "Footprint" "Capacitor_SMD:C_0805_2012Metric" (at 247.65 58.42 0)
-      (effects (font (size 1.27 1.27)) hide)
-    )
-    (property "Datasheet" "~" (at 247.65 58.42 0)
-      (effects (font (size 1.27 1.27)) hide)
-    )
-    (property "LCSC Part" "C15850" (at 247.65 58.42 0)
-      (effects (font (size 1.27 1.27)) hide)
-    )
+  (symbol (lib_id "Device:C_Small") (at 203.2 53.34 90) (unit 1)
+    (in_bom yes) (on_board yes) (dnp no) (fields_autoplaced)
+    (property "Reference" "C5" (at 203.2063 46.99 90)
+      (effects (font (size 1.27 1.27)))
+    )
+    (property "Value" "10uF" (at 203.2063 49.53 90)
+      (effects (font (size 1.27 1.27)))
+    )
+    (property "Footprint" "Capacitor_SMD:C_0805_2012Metric" (at 203.2 53.34 0)
+      (effects (font (size 1.27 1.27)) hide)
+    )
+    (property "Datasheet" "~" (at 203.2 53.34 0)
+      (effects (font (size 1.27 1.27)) hide)
+    )
+    (property "LCSC Part" "C15850" (at 203.2 53.34 0)
+      (effects (font (size 1.27 1.27)) hide)
+    )

Commit message: Further tweaks and improvements
- Use a nicer schematic template
- Tie START button with power on
- Add ferrite to USB shield
- Add CC1/CC2 makeshift ADC
- Tidy up schematics a little bit

Signed-off-by: Jan Hamal Dvořák <mordae@anilinux.org>
Other:
- company: (none) -> DDM Spirála
- title: (none) -> Křeček
Changed lines of the file:
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@@
 (kicad_sch (version 20230121) (generator eeschema)
   (paper "A4")
+  (title_block
+    (title "Křeček")
+    (date "2023-12-20")
+    (rev "v0.9-wip")
+    (company "DDM Spirála")
+  )
   (wire (pts (xy 205.74 55.88) (xy 220.98 55.88))
     (stroke (width 0) (type default))

Commit message: TRRS audio connector
Signed-off-by: Jan Hamal Dvořák <mordae@anilinux.org>
Parts:
- added C14: 1uF, Capacitor_SMD:C_0805_2012Metric, symbol Device:C_Small
- added R7: 3.3k, Resistor_SMD:R_0402_1005Metric, symbol Device:R_Small
Connections:
- net +3.3VA: now also C14.1, R7.2
- net GND: now also CN1.R2, C14.2
- new net HP_{LEFT}: CN1.T
- new net HP_{RIGHT}: CN1.R1
- new net HP_{SENSE}: CN1.S, R7.1
Other:
- moved on the sheet: CN1
Changed lines of the file:
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@@
     (company "DDM Spirála")
   )
+  (junction (at 184.15 133.35) (diameter 0) (color 0 0 0 0)
+  )
+  (junction (at 203.2 133.35) (diameter 0) (color 0 0 0 0)
+  )
   (wire (pts (xy 205.74 55.88) (xy 220.98 55.88))
     (stroke (width 0) (type default))
   )
+  (wire (pts (xy 177.8 133.35) (xy 184.15 133.35))
+    (stroke (width 0) (type default))
+  )
+  (wire (pts (xy 215.9 135.89) (xy 228.6 135.89))
+    (stroke (width 0) (type default))
+  )
+  (wire (pts (xy 184.15 142.24) (xy 184.15 146.05))
+    (stroke (width 0) (type default))
+  )
+  (wire (pts (xy 215.9 128.27) (xy 228.6 128.27))
+    (stroke (width 0) (type default))
+  )
+  (wire (pts (xy 203.2 133.35) (xy 203.2 120.65))
+    (stroke (width 0) (type default))
+  )
+  (wire (pts (xy 203.2 133.35) (xy 228.6 133.35))
+    (stroke (width 0) (type default))
+  )
+  (wire (pts (xy 198.12 133.35) (xy 203.2 133.35))
+    (stroke (width 0) (type default))
+  )
+  (wire (pts (xy 184.15 133.35) (xy 184.15 137.16))
+    (stroke (width 0) (type default))
+  )
+  (wire (pts (xy 177.8 120.65) (xy 203.2 120.65))
+    (stroke (width 0) (type default))
+  )
   (wire (pts (xy 205.74 53.34) (xy 220.98 53.34))
     (stroke (width 0) (type default))
+  )
+  (wire (pts (xy 215.9 130.81) (xy 228.6 130.81))
+    (stroke (width 0) (type default))
+  )
+  (wire (pts (xy 184.15 133.35) (xy 193.04 133.35))
+    (stroke (width 0) (type default))
+  )
+  (label "HP_{MIC}" (at 215.9 133.35 0) (fields_autoplaced)
+    (effects (font (size 1.27 1.27)) (justify left bottom))
+  )
+  (label "HP_{LEFT}" (at 215.9 128.27 0) (fields_autoplaced)
+    (effects (font (size 1.27 1.27)) (justify left bottom))
+  )
+  (label "HP_{RIGHT}" (at 215.9 135.89 0) (fields_autoplaced)
+    (effects (font (size 1.27 1.27)) (justify left bottom))
+  )
+  (hierarchical_label "HP_{SENSE}" (shape output) (at 177.8 120.65 180) (fields_autoplaced)
+    (effects (font (size 1.27 1.27)) (justify right))
+  )
+  (symbol (lib_id "Device:C_Small") (at 184.15 139.7 0) (unit 1)
+    (in_bom yes) (on_board yes) (dnp no) (fields_autoplaced)
+    (property "Reference" "C14" (at 186.69 138.4363 0)
+      (effects (font (size 1.27 1.27)) (justify left))
+    )
+    (property "Value" "1uF" (at 186.69 140.9763 0)
+      (effects (font (size 1.27 1.27)) (justify left))
+    )
+    (property "Footprint" "Capacitor_SMD:C_0805_2012Metric" (at 184.15 139.7 0)
+      (effects (font (size 1.27 1.27)) hide)
+    )
+    (property "Datasheet" "~" (at 184.15 139.7 0)
+      (effects (font (size 1.27 1.27)) hide)
+    )
+    (property "LCSC Part" "C28323" (at 184.15 139.7 0)
+      (effects (font (size 1.27 1.27)) hide)
+    )
+    (pin "1")
+    (pin "2")
+    (instances
+      (project "krecek-0.9"
+        (path "/8888f37b-ecc2-47df-8824-4b4e1e726451/bd29cd8c-9207-416a-90c1-7bdf6b5cfb97"
+          (reference "C14") (unit 1)
+        )
+        (path "/8888f37b-ecc2-47df-8824-4b4e1e726451/a7733ec7-68c7-444f-aac5-8a965be5cbce"
+          (reference "C28") (unit 1)
+        )
+      )
+    )
+  )
+  (symbol (lib_id "power:+3.3VA") (at 177.8 133.35 90) (unit 1)
+    (in_bom yes) (on_board yes) (dnp no) (fields_autoplaced)
+    (property "Reference" "#PWR057" (at 181.61 133.35 0)
+      (effects (font (size 1.27 1.27)) hide)
+    )
+    (property "Value" "+3.3VA" (at 173.99 133.35 90)
+      (effects (font (size 1.27 1.27)) (justify left))
+    )
+    (property "Footprint" "" (at 177.8 133.35 0)
+      (effects (font (size 1.27 1.27)) hide)
+    )
+    (property "Datasheet" "" (at 177.8 133.35 0)
+      (effects (font (size 1.27 1.27)) hide)
+    )
+    (pin "1")
+    (instances
+      (project "krecek-0.9"
+        (path "/8888f37b-ecc2-47df-8824-4b4e1e726451/a7733ec7-68c7-444f-aac5-8a965be5cbce"
+          (reference "#PWR057") (unit 1)
+        )
+      )
+    )
   )
   (symbol (lib_id "power:GND") (at 259.08 66.04 90) (unit 1)
@@
     )
   )
-  (symbol (lib_id "LCSC:PJ-313B6-B") (at 186.69 91.44 0) (mirror y) (unit 1)
-    (in_bom yes) (on_board yes) (dnp no) (fields_autoplaced)
-    (property "Reference" "CN1" (at 199.39 91.44 0)
+  (symbol (lib_id "LCSC:PJ-313B6-B") (at 231.14 130.81 0) (mirror y) (unit 1)
+    (in_bom yes) (on_board yes) (dnp no) (fields_autoplaced)
+    (property "Reference" "CN1" (at 243.84 130.81 0)
       (effects (font (size 1.27 1.27)) (justify right))
     )
-    (property "Value" "PJ-313B6-B" (at 199.39 93.98 0)
+    (property "Value" "PJ-313B6-B" (at 243.84 133.35 0)
       (effects (font (size 1.27 1.27)) (justify right))
     )
-    (property "Footprint" "LCSC:AUDIO-TH_PJ-313B6-B" (at 186.69 104.14 0)
-      (effects (font (size 1.27 1.27)) hide)
-    )
-    (property "Datasheet" "https://lcsc.com/product-detail/Audio-Video-Connectors_XKB-Connectivity-PJ-313B6-B_C500087.html" (at 186.69 106.68 0)
-      (effects (font (size 1.27 1.27)) hide)
-    )
-    (property "LCSC Part" "C500087" (at 186.69 109.22 0)
-      (effects (font (size 1.27 1.27)) hide)
-    )
-    (pin "1")
-    (pin "2")
-    (pin "3")
-    (pin "4")
+    (property "Footprint" "LCSC:AUDIO-TH_PJ-313B6-B" (at 231.14 143.51 0)
+      (effects (font (size 1.27 1.27)) hide)
+    )
+    (property "Datasheet" "https://lcsc.com/product-detail/Audio-Video-Connectors_XKB-Connectivity-PJ-313B6-B_C500087.html" (at 231.14 146.05 0)
+      (effects (font (size 1.27 1.27)) hide)
+    )
+    (property "LCSC Part" "C500087" (at 231.14 148.59 0)
+      (effects (font (size 1.27 1.27)) hide)
+    )
+    (pin "R1")
+    (pin "R2")
+    (pin "S")
+    (pin "T")
     (instances
       (project "krecek-0.9"
         (path "/8888f37b-ecc2-47df-8824-4b4e1e726451/a7733ec7-68c7-444f-aac5-8a965be5cbce"
           (reference "CN1") (unit 1)
+        )
+      )
+    )
+  )
+  (symbol (lib_id "power:GND") (at 184.15 146.05 0) (unit 1)
+    (in_bom yes) (on_board yes) (dnp no) (fields_autoplaced)
+    (property "Reference" "#PWR058" (at 184.15 152.4 0)
+      (effects (font (size 1.27 1.27)) hide)
+    )
+    (property "Value" "GND" (at 184.15 151.13 0)
+      (effects (font (size 1.27 1.27)))
+    )
+    (property "Footprint" "" (at 184.15 146.05 0)
+      (effects (font (size 1.27 1.27)) hide)
+    )
+    (property "Datasheet" "" (at 184.15 146.05 0)
+      (effects (font (size 1.27 1.27)) hide)
+    )
+    (pin "1")
+    (instances
+      (project "krecek-0.9"
+        (path "/8888f37b-ecc2-47df-8824-4b4e1e726451/a7733ec7-68c7-444f-aac5-8a965be5cbce"
+          (reference "#PWR058") (unit 1)
         )
       )
@@
         )
       )
+    )
+  )
+  (symbol (lib_id "power:GND") (at 215.9 130.81 270) (unit 1)
+    (in_bom yes) (on_board yes) (dnp no) (fields_autoplaced)
+    (property "Reference" "#PWR056" (at 209.55 130.81 0)
+      (effects (font (size 1.27 1.27)) hide)
+    )
+    (property "Value" "GND" (at 212.09 130.81 90)
+      (effects (font (size 1.27 1.27)) (justify right))
+    )
+    (property "Footprint" "" (at 215.9 130.81 0)
+      (effects (font (size 1.27 1.27)) hide)
+    )
+    (property "Datasheet" "" (at 215.9 130.81 0)
+      (effects (font (size 1.27 1.27)) hide)
+    )
+    (pin "1")
+    (instances
+      (project "krecek-0.9"
+        (path "/8888f37b-ecc2-47df-8824-4b4e1e726451/a7733ec7-68c7-444f-aac5-8a965be5cbce"
+          (reference "#PWR056") (unit 1)
+        )
+      )
+    )
+  )
+  (symbol (lib_id "Device:R_Small") (at 195.58 133.35 270) (mirror x) (unit 1)
+    (in_bom yes) (on_board yes) (dnp no) (fields_autoplaced)
+    (property "Reference" "R7" (at 195.58 128.27 90)
+      (effects (font (size 1.27 1.27)))
+    )
+    (property "Value" "3.3k" (at 195.58 130.81 90)
+      (effects (font (size 1.27 1.27)))
+    )
+    (property "Footprint" "Resistor_SMD:R_0402_1005Metric" (at 195.58 133.35 0)
+      (effects (font (size 1.27 1.27)) hide)
+    )
+    (property "Datasheet" "~" (at 195.58 133.35 0)
+      (effects (font (size 1.27 1.27)) hide)
+    )
+    (property "LCSC Part" "C25890" (at 195.58 133.35 0)
+      (effects (font (size 1.27 1.27)) hide)
+    )
+    (pin "1")
+    (pin "2")
+    (instances
+      (project "krecek-0.9"
+        (path "/8888f37b-ecc2-47df-8824-4b4e1e726451/bd29cd8c-9207-416a-90c1-7bdf6b5cfb97"
+          (reference "R7") (unit 1)
+        )
+        (path "/8888f37b-ecc2-47df-8824-4b4e1e726451/a7733ec7-68c7-444f-aac5-8a965be5cbce"
+          (reference "R31") (unit 1)
+        )
+      )

Commit message: Complete most of the design, except for RF
Signed-off-by: Jan Hamal Dvořák <mordae@anilinux.org>
Parts:
- removed C14: 1uF, Capacitor_SMD:C_0805_2012Metric, symbol Device:C_Small
- removed C5 (x2): 10uF, Capacitor_SMD:C_0805_2012Metric, symbol Device:C_Small
- added C6 (x9): 10u, Capacitor_SMD:C_0402_1005Metric, symbol Device:C_Small
- added C7 (x11): 1u, Capacitor_SMD:C_0402_1005Metric, symbol Device:C_Small
- added D1 (x2): IR333, LED_THT:LED_D5.0mm_Horizontal_O1.27mm_Z3.0mm_Clear, symbol Device:LED
- added Q1: PT334, LED_THT:LED_D5.0mm_Horizontal_O1.27mm_Z3.0mm_IRBlack, symbol Device:Q_Photo_NPN
- added Q2: AO3400A, Package_TO_SOT_SMD:SOT-23, symbol Transistor_FET:AO3400A
- added R3 (x3): 1, Resistor_SMD:R_1206_3216Metric, symbol Device:R_Small
- added R3: 1k, Resistor_SMD:R_0402_1005Metric, symbol Device:R_Small
- renumbered U10 to U12
Connections:
- net +3.3VA: now also U11.15 (AVDD), C6.1, C6.1, C6.1, C6.1, C6.1, C7.1, R3.1
- net GND: now also U11.1 (CE), U11.14 (AGND), U11.29 (PAD), U11.7 (DGND), C6.2, C6.2, C6.2, C6.2, C6.2, C6.2, C6.2, C6.2, C6.2, C7.1, C7.2, C7.2, C7.2, Q1.2 (E), Q2.2 (S)
- net HP_{LEFT}: now also C7.2
- net HP_{RIGHT}: now also C7.2
- net HP_{SENSE}: now also C7.1
- net LRCK: now reaches U11.10 (LRCK)
- net DAC: now reaches U11.11 (DSDIN)
- net at U11.13 (MONOOUT): now also C7.1, C7.1
- net at U11.16 (OUTP): now also C7.1
- net at U11.17 (OUTN): now also C7.1
- net at U11.18 (DACVREF): now also C7.1
- net at U11.19 (ADCVREF): now also C7.1
- net CDATA: now reaches U11.2 (CDATA)
- net CDATA: now also U12.A3 (SDA)
- net at U11.20 (VMID): now also C7.1
- net IR-: now reaches U11.22 (MIC2N)
- net IR-: now also C7.2
- net IR+: now reaches U11.23 (MIC2P)
- net IR+: now also C7.2
- net at U11.24 (MIC1N): now also C7.2
- net at U11.25 (MIC1P/DMIC_SDA): now also C7.2
- net CCLK: now reaches U11.3 (CCLK)
- net CCLK: now also U12.A2 (SCL)
- net +3.3V: now reaches U11.5 (PVDD)
- net +3.3V: now also U11.6 (DVDD), C6.1, C6.1, C6.1
- net SCLK: now reaches U11.8 (SCLK/DMIC_SCL)
- net ADC: now reaches U11.9 (ASDOUT)
- net at SPK1.3: no longer SPK1.4
- net AMP_{EN}: now reaches U12.B2 (EN)
- net at U12.B3 (IN+): now also C7.2
- net at U12.C3 (IN-): now also C7.2
- new net: Q2.3 (D), R3.2
- new net: C7.1, Q1.1 (C), R3.2
- new net: R3.1, R3.2 (x2)
- new net: D1.1 (K), R3.1
- new net: D1.1 (K), D1.2 (A)
- new net +5V: C6.1, D1.2 (A)
- new net IR_{TX}: Q2.1 (G)
- no-connect marks 0 -> 3
Other:
- moved on the sheet: CN1, R7, SPK1, U12

Commit message: Fix design bugs
Signed-off-by: Jan Hamal Dvořák <mordae@anilinux.org>
Connections:
- net +3.3V: now also U12.C2 (PVDD)
- net +3.3VA: no longer U12.C2 (PVDD)
Changed lines of the file:
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@@
+    )
+  )
+  (symbol (lib_id "power:+3.3V") (at 233.68 132.08 270) (unit 1)
+    (in_bom yes) (on_board yes) (dnp no) (fields_autoplaced)
+    (property "Reference" "#PWR04" (at 229.87 132.08 0)
+      (effects (font (size 1.27 1.27)) hide)
+    )
+    (property "Value" "+3.3V" (at 237.49 132.08 90)
+      (effects (font (size 1.27 1.27)) (justify left))
+    )
+    (property "Footprint" "" (at 233.68 132.08 0)
+      (effects (font (size 1.27 1.27)) hide)
+    )
+    (property "Datasheet" "" (at 233.68 132.08 0)
+      (effects (font (size 1.27 1.27)) hide)
+    )
+    (pin "1")
+    (instances
+      (project "krecek-0.9"
+        (path "/8888f37b-ecc2-47df-8824-4b4e1e726451"
+          (reference "#PWR04") (unit 1)
+        )
+        (path "/8888f37b-ecc2-47df-8824-4b4e1e726451/6537dbea-4e11-4137-b8a0-9ae6b128c4e4"
+          (reference "#PWR019") (unit 1)
+        )
+        (path "/8888f37b-ecc2-47df-8824-4b4e1e726451/a7733ec7-68c7-444f-aac5-8a965be5cbce"
+          (reference "#PWR031") (unit 1)
+        )
+      )
     )
   )
@@
         )
       )
-    )
-  )
-  (symbol (lib_id "power:+3.3VA") (at 233.68 132.08 270) (unit 1)
-    (in_bom yes) (on_board yes) (dnp no) (fields_autoplaced)
-    (property "Reference" "#PWR080" (at 229.87 132.08 0)
-      (effects (font (size 1.27 1.27)) hide)
-    )
-    (property "Value" "+3.3VA" (at 237.49 132.08 90)
-      (effects (font (size 1.27 1.27)) (justify left))
-    )
-    (property "Footprint" "" (at 233.68 132.08 0)
-      (effects (font (size 1.27 1.27)) hide)
-    )
-    (property "Datasheet" "" (at 233.68 132.08 0)
-      (effects (font (size 1.27 1.27)) hide)
-    )
-    (pin "1")
-    (instances
-      (project "krecek-0.9"
-        (path "/8888f37b-ecc2-47df-8824-4b4e1e726451/a7733ec7-68c7-444f-aac5-8a965be5cbce"
-          (reference "#PWR080") (unit 1)
-        )
-      )
