File: hw/krecek-0.9/audio.kicad_sch (KiCad schematic)
At the start: 33 parts, among them CN1 PJ-313B6-B, Q1 PT334, Q2 AO3400A, U11 ES8312, U12 TPA2028D1YZFT

Commit message: Add missing decoupling caps
Signed-off-by: Jan Hamal Dvořák <mordae@anilinux.org>
Parts:
- added C6: 10u, Capacitor_SMD:C_0402_1005Metric, symbol Device:C_Small
Connections:
- net +3.3V: now also C6.1
- net GND: now also C6.2
Other:
- moved on the sheet: C6
Changed lines of the file:
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@@
+    (stroke (width 0) (type default))
+  )
+  (wire (pts (xy 266.7 142.24) (xy 266.7 146.05))
     (stroke (width 0) (type default))
   )
@@
     (stroke (width 0) (type default))
   )
-  (wire (pts (xy 179.07 91.44) (xy 179.07 101.6))
+  (wire (pts (xy 177.8 91.44) (xy 177.8 101.6))
     (stroke (width 0) (type default))
   )
@@
     (stroke (width 0) (type default))
   )
-  (wire (pts (xy 179.07 101.6) (xy 165.1 101.6))
+  (wire (pts (xy 177.8 101.6) (xy 165.1 101.6))
     (stroke (width 0) (type default))
   )
@@
     (stroke (width 0) (type default))
   )
-  (wire (pts (xy 179.07 86.36) (xy 179.07 76.2))
+  (wire (pts (xy 177.8 86.36) (xy 177.8 76.2))
     (stroke (width 0) (type default))
   )
@@
     (stroke (width 0) (type default))
   )
-  (wire (pts (xy 179.07 76.2) (xy 165.1 76.2))
+  (wire (pts (xy 177.8 76.2) (xy 165.1 76.2))
     (stroke (width 0) (type default))
   )
@@
   )
   (wire (pts (xy 146.05 38.1) (xy 154.94 38.1))
+    (stroke (width 0) (type default))
+  )
+  (wire (pts (xy 266.7 133.35) (xy 266.7 137.16))
     (stroke (width 0) (type default))
   )
@@
         (path "/8888f37b-ecc2-47df-8824-4b4e1e726451/a7733ec7-68c7-444f-aac5-8a965be5cbce"
           (reference "#PWR065") (unit 1)
+        )
+      )
+    )
+  )
+  (symbol (lib_id "power:+3.3V") (at 266.7 133.35 0) (unit 1)
+    (in_bom yes) (on_board yes) (dnp no) (fields_autoplaced)
+    (property "Reference" "#PWR04" (at 266.7 137.16 0)
+      (effects (font (size 1.27 1.27)) hide)
+    )
+    (property "Value" "+3.3V" (at 266.7 128.27 0)
+      (effects (font (size 1.27 1.27)))
+    )
+    (property "Footprint" "" (at 266.7 133.35 0)
+      (effects (font (size 1.27 1.27)) hide)
+    )
+    (property "Datasheet" "" (at 266.7 133.35 0)
+      (effects (font (size 1.27 1.27)) hide)
+    )
+    (pin "1")
+    (instances
+      (project "krecek-0.9"
+        (path "/8888f37b-ecc2-47df-8824-4b4e1e726451"
+          (reference "#PWR04") (unit 1)
+        )
+        (path "/8888f37b-ecc2-47df-8824-4b4e1e726451/6537dbea-4e11-4137-b8a0-9ae6b128c4e4"
+          (reference "#PWR019") (unit 1)
+        )
+        (path "/8888f37b-ecc2-47df-8824-4b4e1e726451/a7733ec7-68c7-444f-aac5-8a965be5cbce"
+          (reference "#PWR056") (unit 1)
         )
       )
@@
     )
   )
-  (symbol (lib_id "Device:C_Small") (at 179.07 88.9 0) (mirror y) (unit 1)
-    (in_bom yes) (on_board yes) (dnp no) (fields_autoplaced)
-    (property "Reference" "C6" (at 181.61 87.6363 0)
-      (effects (font (size 1.27 1.27)) (justify right))
-    )
-    (property "Value" "10u" (at 181.61 90.1763 0)
-      (effects (font (size 1.27 1.27)) (justify right))
-    )
-    (property "Footprint" "Capacitor_SMD:C_0402_1005Metric" (at 179.07 88.9 0)
-      (effects (font (size 1.27 1.27)) hide)
-    )
-    (property "Datasheet" "~" (at 179.07 88.9 0)
-      (effects (font (size 1.27 1.27)) hide)
-    )
-    (property "LCSC Part" "C15525" (at 179.07 88.9 0)
+  (symbol (lib_id "Device:C_Small") (at 177.8 88.9 0) (mirror y) (unit 1)
+    (in_bom yes) (on_board yes) (dnp no) (fields_autoplaced)
+    (property "Reference" "C6" (at 180.34 87.6363 0)
+      (effects (font (size 1.27 1.27)) (justify right))
+    )
+    (property "Value" "10u" (at 180.34 90.1763 0)
+      (effects (font (size 1.27 1.27)) (justify right))
+    )
+    (property "Footprint" "Capacitor_SMD:C_0402_1005Metric" (at 177.8 88.9 0)
+      (effects (font (size 1.27 1.27)) hide)
+    )
+    (property "Datasheet" "~" (at 177.8 88.9 0)
+      (effects (font (size 1.27 1.27)) hide)
+    )
+    (property "LCSC Part" "C15525" (at 177.8 88.9 0)
       (effects (font (size 1.27 1.27)) hide)
     )
@@
     )
   )
+  (symbol (lib_id "power:GND") (at 266.7 146.05 0) (unit 1)
+    (in_bom yes) (on_board yes) (dnp no) (fields_autoplaced)
+    (property "Reference" "#PWR056" (at 266.7 152.4 0)
+      (effects (font (size 1.27 1.27)) hide)
+    )
+    (property "Value" "GND" (at 266.7 151.13 0)
+      (effects (font (size 1.27 1.27)))
+    )
+    (property "Footprint" "" (at 266.7 146.05 0)
+      (effects (font (size 1.27 1.27)) hide)
+    )
+    (property "Datasheet" "" (at 266.7 146.05 0)
+      (effects (font (size 1.27 1.27)) hide)
+    )
+    (pin "1")
+    (instances
+      (project "pipi"
+        (path "/73d1f64b-b6d8-45c3-ab75-e79bce2c5a38/94670045-b9e9-4921-8dd4-cc6059cd92ef"
+          (reference "#PWR056") (unit 1)
+        )
+      )
+      (project "krecek-0.9"
+        (path "/8888f37b-ecc2-47df-8824-4b4e1e726451/a7733ec7-68c7-444f-aac5-8a965be5cbce"
+          (reference "#PWR0109") (unit 1)
+        )
+      )
+    )
+  )
   (symbol (lib_id "Device:LED") (at 254 44.45 90) (unit 1)
     (in_bom yes) (on_board yes) (dnp no) (fields_autoplaced)
@@
         )
       )
+    )
+  )
+  (symbol (lib_id "Device:C_Small") (at 266.7 139.7 0) (mirror y) (unit 1)
+    (in_bom yes) (on_board yes) (dnp no) (fields_autoplaced)
+    (property "Reference" "C6" (at 269.24 138.4363 0)
+      (effects (font (size 1.27 1.27)) (justify right))
+    )
+    (property "Value" "10u" (at 269.24 140.9763 0)
+      (effects (font (size 1.27 1.27)) (justify right))
+    )
+    (property "Footprint" "Capacitor_SMD:C_0402_1005Metric" (at 266.7 139.7 0)
+      (effects (font (size 1.27 1.27)) hide)
+    )
+    (property "Datasheet" "~" (at 266.7 139.7 0)
+      (effects (font (size 1.27 1.27)) hide)
+    )
+    (property "LCSC Part" "C15525" (at 266.7 139.7 0)
+      (effects (font (size 1.27 1.27)) hide)
+    )
+    (pin "1")
+    (pin "2")
+    (instances
+      (project "barbecue"
+        (path "/12829710-d93a-4fa1-96c6-084c1af2e761"
+          (reference "C6") (unit 1)
+        )
+      )
+      (project "bento-vna"
+        (path "/36176a8e-13d1-429b-8815-63472bc0665c"
+          (reference "C2") (unit 1)
+        )
+      )
+      (project "pipi"
+        (path "/5de6f2b6-19be-45cf-b069-ee289a326d21"
+          (reference "C2") (unit 1)
+        )
+        (path "/5de6f2b6-19be-45cf-b069-ee289a326d21/5b1ff778-5e2f-4eb6-acb1-23bd0a5149e9"
+          (reference "C2") (unit 1)
+        )
+        (path "/5de6f2b6-19be-45cf-b069-ee289a326d21/882742c5-0484-4b86-b485-99790a82e2a9"
+          (reference "C2") (unit 1)
+        )
+      )
+      (project "pipi"
+        (path "/73d1f64b-b6d8-45c3-ab75-e79bce2c5a38/350168a7-ca84-4da6-868a-c5a486a494d0"
+          (reference "C2") (unit 1)
+        )
+      )
+      (project "krecek-0.9"
+        (path "/8888f37b-ecc2-47df-8824-4b4e1e726451/6537dbea-4e11-4137-b8a0-9ae6b128c4e4"
+          (reference "C12") (unit 1)
+        )
+        (path "/8888f37b-ecc2-47df-8824-4b4e1e726451/a7733ec7-68c7-444f-aac5-8a965be5cbce"
+          (reference "C79") (unit 1)
+        )
+      )

Commit message: Add more missing LCSC part ids
Signed-off-by: Jan Hamal Dvořák <mordae@anilinux.org>
Parts:
- U12: LCSC Part (none) -> C2869063
Changed lines of the file:
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@@
       (effects (font (size 1.27 1.27) italic) hide)
+    )
+    (property "LCSC Part" "C2869063" (at 214.63 139.7 0)
+      (effects (font (size 1.27 1.27)) hide)
     )
     (pin "A1")
