File: hw/krecek-0.9/audio.kicad_sch (KiCad schematic)
At the start: 30 parts, among them CN1 PJ-313B6-B, Q1 PT334, Q2 AO3400A, U10 ES8312, U11 PAM8302AASCR

Commit message: hw: work on new board revision
Parts:
- removed TP1, TP2: TestPoint, TestPoint:TestPoint_Pad_D1.0mm, symbol Connector:TestPoint
Connections:
- net at U11.8 (VO-): now also SPK1.2
Changed lines of the file:
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@@
-	)
-	(junction
-		(at 139.7 134.62)
-		(diameter 0)
-		(color 0 0 0 0)
-	)
-	(junction
-		(at 139.7 132.08)
-		(diameter 0)
-		(color 0 0 0 0)
 	)
 	(junction
@@
 	(wire
 		(pts
-			(xy 139.7 127) (xy 152.4 127)
-		)
-		(stroke
-			(width 0)
-			(type default)
-		)
-	)
-	(wire
-		(pts
 			(xy 50.8 34.29) (xy 50.8 39.37)
 		)
@@
 	(wire
 		(pts
-			(xy 139.7 134.62) (xy 139.7 139.7)
-		)
-		(stroke
-			(width 0)
-			(type default)
-		)
-	)
-	(wire
-		(pts
-			(xy 139.7 139.7) (xy 152.4 139.7)
-		)
-		(stroke
-			(width 0)
-			(type default)
-		)
-	)
-	(wire
-		(pts
 			(xy 266.7 142.24) (xy 266.7 146.05)
 		)
@@
 	(wire
 		(pts
-			(xy 129.54 134.62) (xy 139.7 134.62)
-		)
-		(stroke
-			(width 0)
-			(type default)
-		)
-	)
-	(wire
-		(pts
 			(xy 114.3 157.48) (xy 114.3 152.4)
 		)
@@
 	(wire
 		(pts
-			(xy 139.7 127) (xy 139.7 132.08)
-		)
-		(stroke
-			(width 0)
-			(type default)
-		)
-	)
-	(wire
-		(pts
 			(xy 25.4 147.32) (xy 29.21 147.32)
 		)
@@
 	(wire
 		(pts
-			(xy 139.7 132.08) (xy 205.74 132.08)
-		)
-		(stroke
-			(width 0)
-			(type default)
-		)
-	)
-	(wire
-		(pts
 			(xy 165.1 76.2) (xy 165.1 80.01)
 		)
@@
 	(wire
 		(pts
-			(xy 139.7 134.62) (xy 205.74 134.62)
+			(xy 129.54 134.62) (xy 205.74 134.62)
 		)
 		(stroke
@@
 	(wire
 		(pts
-			(xy 129.54 132.08) (xy 139.7 132.08)
+			(xy 129.54 132.08) (xy 205.74 132.08)
 		)
 		(stroke
@@
 	)
 	(label "HP_{LEFT}"
-		(at 152.4 127 180)
+		(at 152.4 132.08 180)
 		(fields_autoplaced yes)
 		(effects
@@
 	)
 	(label "HP_{RIGHT}"
-		(at 152.4 139.7 180)
+		(at 152.4 134.62 180)
 		(fields_autoplaced yes)
 		(effects
@@
 	)
 	(symbol
-		(lib_id "Connector:TestPoint")
-		(at 152.4 127 270)
-		(unit 1)
-		(exclude_from_sim no)
-		(in_bom yes)
-		(on_board yes)
-		(dnp no)
-		(fields_autoplaced yes)
-		(property "Reference" "TP1"
-			(at 157.48 125.73 90)
-			(effects
-				(font
-					(size 1.27 1.27)
-				)
-				(justify left)
-			)
-		)
-		(property "Value" "TestPoint"
-			(at 157.48 128.27 90)
-			(effects
-				(font
-					(size 1.27 1.27)
-				)
-				(justify left)
-			)
-		)
-		(property "Footprint" "TestPoint:TestPoint_Pad_D1.0mm"
-			(at 152.4 132.08 0)
-			(effects
-				(font
-					(size 1.27 1.27)
-				)
-				(hide yes)
-			)
-		)
-		(property "Datasheet" "~"
-			(at 152.4 132.08 0)
-			(effects
-				(font
-					(size 1.27 1.27)
-				)
-				(hide yes)
-			)
-		)
-		(property "Description" "test point"
-			(at 152.4 127 0)
-			(effects
-				(font
-					(size 1.27 1.27)
-				)
-				(hide yes)
-			)
-		)
-		(pin "1"
-		)
-		(instances
-			(project "krecek-0.9"
-				(path "/8888f37b-ecc2-47df-8824-4b4e1e726451/a7733ec7-68c7-444f-aac5-8a965be5cbce"
-					(reference "TP1")
-					(unit 1)
-				)
-			)
-		)
-	)
-	(symbol
 		(lib_id "power:GND")
 		(at 50.8 39.37 0)
@@
 	)
 	(symbol
-		(lib_name "LCSC:PAM8302AASCR")
 		(lib_id "LCSC:PAM8302AASCR")
 		(at 215.9 132.08 0)
@@
 					(unit 1)
 				)
-			)
-		)
-	)
-	(symbol
-		(lib_id "Connector:TestPoint")
-		(at 152.4 139.7 270)
-		(unit 1)
-		(exclude_from_sim no)
-		(in_bom yes)
-		(on_board yes)
-		(dnp no)
-		(fields_autoplaced yes)
-		(property "Reference" "TP2"
-			(at 157.48 138.43 90)
-			(effects
-				(font
-					(size 1.27 1.27)
-				)
-				(justify left)
-			)
-		)
-		(property "Value" "TestPoint"
-			(at 157.48 140.97 90)
-			(effects
-				(font
-					(size 1.27 1.27)
-				)
-				(justify left)
-			)
-		)
-		(property "Footprint" "TestPoint:TestPoint_Pad_D1.0mm"
-			(at 152.4 144.78 0)
-			(effects
-				(font
-					(size 1.27 1.27)
-				)
-				(hide yes)
-			)
-		)
-		(property "Datasheet" "~"
-			(at 152.4 144.78 0)
-			(effects
-				(font
-					(size 1.27 1.27)
-				)
-				(hide yes)
-			)
-		)
-		(property "Description" "test point"
-			(at 152.4 139.7 0)
-			(effects
-				(font
-					(size 1.27 1.27)
-				)
-				(hide yes)
-			)
-		)
-		(pin "1"
-		)
-		(instances
-			(project "krecek-0.9"
-				(path "/8888f37b-ecc2-47df-8824-4b4e1e726451/a7733ec7-68c7-444f-aac5-8a965be5cbce"
-					(reference "TP2")
-					(unit 1)
-				)

Commit message: Progress on HW design
Parts:
- removed C6: 10u, Capacitor_SMD:C_0402_1005Metric, symbol Device:C_Small
- removed C7 (x5): 1u, Capacitor_SMD:C_0402_1005Metric, symbol Device:C_Small
- removed U10: ES8312, LCSC:VQFN-28_L4.0-W4.0-P0.45-TL-EP2.6, symbol LCSC:ES8312
- removed U11: PAM8302AASCR, LCSC:MSOP-8_L3.0-W3.0-P0.65-LS5.0-BL, symbol LCSC:PAM8302AASCR
- added C48, C50: 47u, Capacitor_SMD:C_0805_2012Metric, symbol Device:C_Small
- added C52, C53: 4.7u, Capacitor_SMD:C_0402_1005Metric, symbol Device:C_Small
- added U10: NAU88C22YG, LCSC:QFN-32_L5.0-W5.0-P0.50-BL-EP2.7, symbol LCSC:NAU88C22YG_C914209
- R35: renamed from R29; value 3.3k -> 2.2k; LCSC Part C25890 -> C25879
Connections:
- net +3.3V: now also U10.13 (VDD), U10.14 (VDD); no longer C6.1
- net +3.3VA: now also U10.31 (VDDA); no longer R35.2
- net +5V: now also C6.1, U10.26 (VDDSPK)
- net ADC: now also U10.9 (ADCOUT)
- net CCLK: now also U10.16 (SCLK)
- net CDATA: now also U10.17 (SDIO)
- net DAC: now also U10.10 (DACIN)
- net GND: now also C52.1, C53.1, U10.12 (VSS), U10.18 (MODE), U10.24 (VSSSPK), U10.28 (VSS), U10.33 (EP)
- net HP_{LEFT}: now also C48.2
- net HP_{RIGHT}: now also C50.2
- net IR+: now also U10.1 (LMICP)
- net IR-: now also U10.2 (LMICN)
- net LRCK: now also U10.7 (FS)
- net SCLK: now also U10.11 (MCLK), U10.8 (BCLK)
- net at C7.2: now also U10.5 (RMICN)
- net at SPK1.1 (+): now also U10.25 (LSPKOUT)
- net at SPK1.2: now also U10.23 (RSPKOUT)
- net at C7.2: now also U10.4 (RMICP)
- new net: C53.2, R35.2, U10.32 (MICBIAS)
- new net: C50.1, U10.29 (RHP)
- new net: C52.2, U10.27 (VREF)
- new net: C48.1, U10.30 (LHP)
- no-connect marks 4 -> 7
Other:
- moved on the sheet: C6, C7, R35, SPK1
