File: hw/krecek-0.9/audio.kicad_sch (KiCad schematic)
At the start: 25 parts, among them CN1 PJ-313B6-B, Q1 PT334, Q2 AO3400A, U10 NAU88C22YG

Commit message: Work on board layout
Parts:
- removed C7: 1u, Capacitor_SMD:C_0402_1005Metric, symbol Device:C_Small
Connections:
- net +3.3VA: no longer C7.1
- net at Q1.1 (C), R3.2: now also C7.1
- net IR: now reaches U10.19 (LAUXIN)
- net IR: now also C7.2
- net IR+: no longer names the net of U10.1 (LMICP)
- net IR+: no longer C7.2
- net IR-: no longer names the net of U10.2 (LMICN)
- no-connect marks 7 -> 8
Other:
- moved on the sheet: C7
Changed lines of the file:
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@@
 	)
 	(no_connect
-		(at 76.2 114.3)
+		(at 76.2 121.92)
 	)
 	(no_connect
@@
 	)
 	(no_connect
+		(at 76.2 119.38)
+	)
+	(no_connect
 		(at 76.2 124.46)
 	)
@@
 	(wire
 		(pts
-			(xy 127 88.9) (xy 144.78 88.9)
-		)
-		(stroke
-			(width 0)
-			(type default)
-		)
-	)
-	(wire
-		(pts
-			(xy 64.77 121.92) (xy 76.2 121.92)
-		)
-		(stroke
-			(width 0)
-			(type default)
-		)
-	)
-	(wire
-		(pts
 			(xy 88.9 78.74) (xy 88.9 83.82)
 		)
@@
 	(wire
 		(pts
-			(xy 165.1 85.09) (xy 165.1 88.9)
-		)
-		(stroke
-			(width 0)
-			(type default)
-		)
-	)
-	(wire
-		(pts
 			(xy 177.8 140.97) (xy 177.8 144.78)
 		)
@@
 	(wire
 		(pts
-			(xy 165.1 88.9) (xy 149.86 88.9)
-		)
-		(stroke
-			(width 0)
-			(type default)
-		)
-	)
-	(wire
-		(pts
 			(xy 34.29 132.08) (xy 38.1 132.08)
 		)
@@
 	(wire
 		(pts
-			(xy 165.1 76.2) (xy 149.86 76.2)
+			(xy 165.1 88.9) (xy 149.86 88.9)
 		)
 		(stroke
@@
 	(wire
 		(pts
+			(xy 165.1 88.9) (xy 165.1 90.17)
+		)
+		(stroke
+			(width 0)
+			(type default)
+		)
+	)
+	(wire
+		(pts
 			(xy 254 35.56) (xy 254 40.64)
 		)
@@
 	(wire
 		(pts
-			(xy 64.77 119.38) (xy 76.2 119.38)
+			(xy 64.77 114.3) (xy 76.2 114.3)
 		)
 		(stroke
@@
 	(wire
 		(pts
-			(xy 165.1 88.9) (xy 165.1 90.17)
+			(xy 165.1 85.09) (xy 165.1 88.9)
 		)
 		(stroke
@@
 	(wire
 		(pts
-			(xy 127 76.2) (xy 144.78 76.2)
+			(xy 127 88.9) (xy 144.78 88.9)
 		)
 		(stroke
@@
 		)
 	)
-	(label "IR+"
-		(at 64.77 121.92 0)
-		(fields_autoplaced yes)
-		(effects
-			(font
-				(size 1.27 1.27)
-			)
-			(justify left bottom)
-		)
-	)
-	(label "IR-"
-		(at 64.77 119.38 0)
+	(label "IR"
+		(at 64.77 114.3 0)
 		(fields_autoplaced yes)
 		(effects
@@
 		)
 	)
-	(label "IR+"
-		(at 127 76.2 0)
-		(fields_autoplaced yes)
-		(effects
-			(font
-				(size 1.27 1.27)
-			)
-			(justify left bottom)
-		)
-	)
-	(label "IR-"
+	(label "IR"
 		(at 127 88.9 0)
 		(fields_autoplaced yes)
@@
 		(instances
 			(project "pipi"
-				(path "/73d1f64b-b6d8-45c3-ab75-e79bce2c5a38/94670045-b9e9-4921-8dd4-cc6059cd92ef"
+				(path "/73d1f64b-b6d8-45c3-ab75-e79bce2c5a38/350168a7-ca84-4da6-868a-c5a486a494d0"
 					(reference "Q2")
 					(unit 1)
 				)
-				(path "/73d1f64b-b6d8-45c3-ab75-e79bce2c5a38/350168a7-ca84-4da6-868a-c5a486a494d0"
+				(path "/73d1f64b-b6d8-45c3-ab75-e79bce2c5a38/94670045-b9e9-4921-8dd4-cc6059cd92ef"
 					(reference "Q2")
 					(unit 1)
@@
 	(symbol
 		(lib_id "Device:C_Small")
-		(at 147.32 76.2 270)
+		(at 147.32 88.9 270)
 		(unit 1)
 		(exclude_from_sim no)
@@
 		(fields_autoplaced yes)
 		(property "Reference" "C7"
-			(at 147.3136 69.85 90)
+			(at 147.3136 82.55 90)
 			(effects
 				(font
@@
 		)
 		(property "Value" "1u"
-			(at 147.3136 72.39 90)
+			(at 147.3136 85.09 90)
 			(effects
 				(font
@@
 		)
 		(property "Footprint" "Capacitor_SMD:C_0402_1005Metric"
-			(at 147.32 76.2 0)
+			(at 147.32 88.9 0)
 			(effects
 				(font
@@
 		)
 		(property "Datasheet" "~"
-			(at 147.32 76.2 0)
+			(at 147.32 88.9 0)
 			(effects
 				(font
@@
 		)
 		(property "Description" "Unpolarized capacitor, small symbol"
-			(at 147.32 76.2 0)
+			(at 147.32 88.9 0)
 			(effects
 				(font
@@
 		)
 		(property "LCSC Part" "C52923"
-			(at 147.32 76.2 0)
+			(at 147.32 88.9 0)
 			(effects
 				(font
@@
 		(dnp no)
 		(fields_autoplaced yes)
-		(property "Reference" "#PWR042"
+		(property "Reference" "#PWR036"
 			(at 254 109.22 0)
 			(effects
@@
 		(instances
 			(project "pipi"
-				(path "/73d1f64b-b6d8-45c3-ab75-e79bce2c5a38/94670045-b9e9-4921-8dd4-cc6059cd92ef"
-					(reference "#PWR042")
-					(unit 1)
-				)
 				(path "/73d1f64b-b6d8-45c3-ab75-e79bce2c5a38/350168a7-ca84-4da6-868a-c5a486a494d0"
 					(reference "#PWR036")
 					(unit 1)
 				)
+				(path "/73d1f64b-b6d8-45c3-ab75-e79bce2c5a38/94670045-b9e9-4921-8dd4-cc6059cd92ef"
+					(reference "#PWR042")
+					(unit 1)
+				)
 			)
 			(project "krecek-0.9"
@@
 		(dnp no)
 		(fields_autoplaced yes)
-		(property "Reference" "#PWR042"
+		(property "Reference" "#PWR036"
 			(at 266.7 44.45 0)
 			(effects
@@
 		(instances
 			(project "pipi"
-				(path "/73d1f64b-b6d8-45c3-ab75-e79bce2c5a38/94670045-b9e9-4921-8dd4-cc6059cd92ef"
-					(reference "#PWR042")
-					(unit 1)
-				)
 				(path "/73d1f64b-b6d8-45c3-ab75-e79bce2c5a38/350168a7-ca84-4da6-868a-c5a486a494d0"
 					(reference "#PWR036")
 					(unit 1)
 				)
+				(path "/73d1f64b-b6d8-45c3-ab75-e79bce2c5a38/94670045-b9e9-4921-8dd4-cc6059cd92ef"
+					(reference "#PWR042")
+					(unit 1)
+				)
 			)
 			(project "krecek-0.9"
@@
 	)
 	(symbol
-		(lib_id "Device:C_Small")
-		(at 147.32 88.9 270)
-		(mirror x)
-		(unit 1)
-		(exclude_from_sim no)
-		(in_bom yes)
-		(on_board yes)
-		(dnp no)
-		(fields_autoplaced yes)
-		(property "Reference" "C7"
-			(at 147.3136 82.55 90)
-			(effects
-				(font
-					(size 1.27 1.27)
-				)
-			)
-		)
-		(property "Value" "1u"
-			(at 147.3136 85.09 90)
-			(effects
-				(font
-					(size 1.27 1.27)
-				)
-			)
-		)
-		(property "Footprint" "Capacitor_SMD:C_0402_1005Metric"
-			(at 147.32 88.9 0)
-			(effects
-				(font
-					(size 1.27 1.27)
-				)
-				(hide yes)
-			)
-		)
-		(property "Datasheet" "~"
-			(at 147.32 88.9 0)
-			(effects
-				(font
-					(size 1.27 1.27)
-				)
-				(hide yes)
-			)
-		)
-		(property "Description" "Unpolarized capacitor, small symbol"
-			(at 147.32 88.9 0)
-			(effects
-				(font
-					(size 1.27 1.27)
-				)
-				(hide yes)
-			)
-		)
-		(property "LCSC Part" "C52923"
-			(at 147.32 88.9 0)
-			(effects
-				(font
-					(size 1.27 1.27)
-				)
-				(hide yes)
-			)
-		)
-		(pin "1"
-		)
-		(pin "2"
-		)
-		(instances
-			(project "barbecue"
-				(path "/12829710-d93a-4fa1-96c6-084c1af2e761"
-					(reference "C7")
-					(unit 1)
-				)
-			)
-			(project "bento-vna"
-				(path "/36176a8e-13d1-429b-8815-63472bc0665c"
-					(reference "C3")
-					(unit 1)
-				)
-			)
-			(project "pipi"
-				(path "/5de6f2b6-19be-45cf-b069-ee289a326d21"
-					(reference "C3")
-					(unit 1)
-				)
-				(path "/5de6f2b6-19be-45cf-b069-ee289a326d21/5b1ff778-5e2f-4eb6-acb1-23bd0a5149e9"
-					(reference "C3")
-					(unit 1)
-				)
-				(path "/5de6f2b6-19be-45cf-b069-ee289a326d21/882742c5-0484-4b86-b485-99790a82e2a9"
-					(reference "C3")
-					(unit 1)
-				)
-			)
-			(project "pipi"
-				(path "/73d1f64b-b6d8-45c3-ab75-e79bce2c5a38/350168a7-ca84-4da6-868a-c5a486a494d0"
-					(reference "C3")
-					(unit 1)
-				)
-				(path "/73d1f64b-b6d8-45c3-ab75-e79bce2c5a38/94670045-b9e9-4921-8dd4-cc6059cd92ef"
-					(reference "C38")
-					(unit 1)
-				)
-			)
-			(project "krecek-0.9"
-				(path "/8888f37b-ecc2-47df-8824-4b4e1e726451/a7733ec7-68c7-444f-aac5-8a965be5cbce"
-					(reference "C45")
-					(unit 1)
-				)
-			)
-		)
-	)
-	(symbol
 		(lib_id "Device:R_Small")
 		(at 254 57.15 0)
@@
 					(unit 1)
 				)
-				(path "/73d1f64b-b6d8-45c3-ab75-e79bce2c5a38/94670045-b9e9-4921-8dd4-cc6059cd92ef"
-					(reference "D1")
-					(unit 1)
-				)
 				(path "/73d1f64b-b6d8-45c3-ab75-e79bce2c5a38/350168a7-ca84-4da6-868a-c5a486a494d0"
 					(reference "D14")
 					(unit 1)
 				)
+				(path "/73d1f64b-b6d8-45c3-ab75-e79bce2c5a38/94670045-b9e9-4921-8dd4-cc6059cd92ef"
+					(reference "D1")
+					(unit 1)
+				)
 			)
 			(project "krecek-0.9"
@@
 					(unit 1)
 				)
-				(path "/73d1f64b-b6d8-45c3-ab75-e79bce2c5a38/94670045-b9e9-4921-8dd4-cc6059cd92ef"
-					(reference "D1")
-					(unit 1)
-				)
 				(path "/73d1f64b-b6d8-45c3-ab75-e79bce2c5a38/350168a7-ca84-4da6-868a-c5a486a494d0"
 					(reference "D14")
 					(unit 1)
 				)
+				(path "/73d1f64b-b6d8-45c3-ab75-e79bce2c5a38/94670045-b9e9-4921-8dd4-cc6059cd92ef"
+					(reference "D1")
+					(unit 1)
+				)

Commit message: Work on board layout
Connections:
- net at SPK1.1 (+): now also U10.23 (RSPKOUT); no longer U10.25 (LSPKOUT)
- net at SPK1.2: now also U10.25 (LSPKOUT); no longer U10.23 (RSPKOUT)
Changed lines of the file:
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@@
 		(lib_id "LCSC:FS-1540")
 		(at 156.21 171.45 0)
+		(mirror x)
 		(unit 1)
 		(exclude_from_sim no)
@@
 		(fields_autoplaced yes)
 		(property "Reference" "SPK1"
-			(at 161.29 170.18 0)
+			(at 157.355 162.56 0)
 			(effects
 				(font
 					(size 1.27 1.27)
 				)
-				(justify left)
 			)
 		)
 		(property "Value" "FS-1540"
-			(at 161.29 172.72 0)
+			(at 157.355 165.1 0)
 			(effects
 				(font
 					(size 1.27 1.27)
 				)
-				(justify left)
 			)
 		)
 		(property "Footprint" "LCSC:BUZ-SMD_5P-L15.0-W15.0-P13.7-BL"
-			(at 156.21 184.15 0)
+			(at 156.21 158.75 0)
 			(effects
 				(font
@@
 		)
 		(property "LCSC Part" "C482341"
-			(at 156.21 186.69 0)
+			(at 156.21 156.21 0)
 			(effects
 				(font

Commit message: Route more parts of the board
Parts:
- removed C6: 10u, Capacitor_SMD:C_0402_1005Metric, symbol Device:C_Small
Changed lines of the file:
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@@
-	)
-	(junction
-		(at 165.1 76.2)
-		(diameter 0)
-		(color 0 0 0 0)
 	)
 	(junction
@@
 	)
 	(junction
-		(at 165.1 101.6)
-		(diameter 0)
-		(color 0 0 0 0)
-	)
-	(junction
 		(at 50.8 152.4)
 		(diameter 0)
@@
 	(wire
 		(pts
-			(xy 165.1 102.87) (xy 165.1 101.6)
+			(xy 165.1 100.33) (xy 165.1 102.87)
 		)
 		(stroke
@@
 	(wire
 		(pts
-			(xy 177.8 91.44) (xy 177.8 101.6)
-		)
-		(stroke
-			(width 0)
-			(type default)
-		)
-	)
-	(wire
-		(pts
 			(xy 101.6 78.74) (xy 101.6 83.82)
 		)
@@
 	(wire
 		(pts
-			(xy 165.1 100.33) (xy 165.1 101.6)
-		)
-		(stroke
-			(width 0)
-			(type default)
-		)
-	)
-	(wire
-		(pts
 			(xy 66.04 170.18) (xy 66.04 157.48)
 		)
@@
 	(wire
 		(pts
-			(xy 177.8 101.6) (xy 165.1 101.6)
-		)
-		(stroke
-			(width 0)
-			(type default)
-		)
-	)
-	(wire
-		(pts
 			(xy 66.04 157.48) (xy 76.2 157.48)
 		)
@@
 	(wire
 		(pts
-			(xy 165.1 76.2) (xy 165.1 80.01)
+			(xy 165.1 74.93) (xy 165.1 80.01)
 		)
 		(stroke
@@
 	(wire
 		(pts
-			(xy 177.8 86.36) (xy 177.8 76.2)
-		)
-		(stroke
-			(width 0)
-			(type default)
-		)
-	)
-	(wire
-		(pts
 			(xy 127 170.18) (xy 152.4 170.18)
 		)
@@
 	(wire
 		(pts
-			(xy 177.8 76.2) (xy 165.1 76.2)
-		)
-		(stroke
-			(width 0)
-			(type default)
-		)
-	)
-	(wire
-		(pts
 			(xy 266.7 34.29) (xy 266.7 38.1)
 		)
@@
 		(pts
 			(xy 177.8 132.08) (xy 177.8 135.89)
-		)
-		(stroke
-			(width 0)
-			(type default)
-		)
-	)
-	(wire
-		(pts
-			(xy 165.1 74.93) (xy 165.1 76.2)
 		)
 		(stroke
@@
 					(unit 1)
 				)
-			)
-		)
-	)
-	(symbol
-		(lib_id "Device:C_Small")
-		(at 177.8 88.9 0)
-		(mirror y)
-		(unit 1)
-		(exclude_from_sim no)
-		(in_bom yes)
-		(on_board yes)
-		(dnp no)
-		(fields_autoplaced yes)
-		(property "Reference" "C6"
-			(at 180.34 87.6363 0)
-			(effects
-				(font
-					(size 1.27 1.27)
-				)
-				(justify right)
-			)
-		)
-		(property "Value" "10u"
-			(at 180.34 90.1763 0)
-			(effects
-				(font
-					(size 1.27 1.27)
-				)
-				(justify right)
-			)
-		)
-		(property "Footprint" "Capacitor_SMD:C_0402_1005Metric"
-			(at 177.8 88.9 0)
-			(effects
-				(font
-					(size 1.27 1.27)
-				)
-				(hide yes)
-			)
-		)
-		(property "Datasheet" "~"
-			(at 177.8 88.9 0)
-			(effects
-				(font
-					(size 1.27 1.27)
-				)
-				(hide yes)
-			)
-		)
-		(property "Description" "Unpolarized capacitor, small symbol"
-			(at 177.8 88.9 0)
-			(effects
-				(font
-					(size 1.27 1.27)
-				)
-				(hide yes)
-			)
-		)
-		(property "LCSC Part" "C15525"
-			(at 177.8 88.9 0)
-			(effects
-				(font
-					(size 1.27 1.27)
-				)
-				(hide yes)
-			)
-		)
-		(pin "1"
-		)
-		(pin "2"
-		)
-		(instances
-			(project "barbecue"
-				(path "/12829710-d93a-4fa1-96c6-084c1af2e761"
-					(reference "C6")
-					(unit 1)
-				)
-			)
-			(project "bento-vna"
-				(path "/36176a8e-13d1-429b-8815-63472bc0665c"
-					(reference "C2")
-					(unit 1)
-				)
-			)
-			(project "pipi"
-				(path "/5de6f2b6-19be-45cf-b069-ee289a326d21"
-					(reference "C2")
-					(unit 1)
-				)
-				(path "/5de6f2b6-19be-45cf-b069-ee289a326d21/5b1ff778-5e2f-4eb6-acb1-23bd0a5149e9"
-					(reference "C2")
-					(unit 1)
-				)
-				(path "/5de6f2b6-19be-45cf-b069-ee289a326d21/882742c5-0484-4b86-b485-99790a82e2a9"
-					(reference "C2")
-					(unit 1)
-				)
-			)
-			(project "pipi"
-				(path "/73d1f64b-b6d8-45c3-ab75-e79bce2c5a38/350168a7-ca84-4da6-868a-c5a486a494d0"
-					(reference "C2")
-					(unit 1)
-				)
-			)
-			(project "krecek-0.9"
-				(path "/8888f37b-ecc2-47df-8824-4b4e1e726451/a7733ec7-68c7-444f-aac5-8a965be5cbce"
-					(reference "C46")
-					(unit 1)
-				)

Commit message: Sent to manufacturing
Parts:
- D1: LCSC Part (none) -> C841525
- Q1: LCSC Part (none) -> C390047
Changed lines of the file:
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@@
+			)
+		)
+		(property "LCSC Part" "C390047"
+			(at 162.56 95.25 0)
+			(effects
+				(font
+					(size 1.27 1.27)
+				)
+				(hide yes)
 			)
 		)
@@
 			)
 		)
+		(property "LCSC Part" "C841525"
+			(at 254 44.45 90)
+			(effects
+				(font
+					(size 1.27 1.27)
+				)
+				(hide yes)
+			)
+		)
 		(pin "1"
 		)
@@
 			(effects
 				(font
+					(size 1.27 1.27)
+				)
+				(hide yes)
+			)
+		)
+		(property "LCSC Part" "C841525"
+			(at 254 31.75 90)
+			(effects
+				(font
