File: hw/krecek-0.9/radio.kicad_sch (KiCad schematic)
At the start: 1 part, among them U12 CC1101RGPR

Commit message: Further tweaks and improvements
- Use a nicer schematic template
- Tie START button with power on
- Add ferrite to USB shield
- Add CC1/CC2 makeshift ADC
- Tidy up schematics a little bit

Signed-off-by: Jan Hamal Dvořák <mordae@anilinux.org>
Other:
- company: (none) -> DDM Spirála
- title: (none) -> Křeček
Changed lines of the file:
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@@
 (kicad_sch (version 20230121) (generator eeschema)
   (paper "A4")
+  (title_block
+    (title "Křeček")
+    (date "2023-12-20")
+    (rev "v0.9-wip")
+    (company "DDM Spirála")
+  )
   (hierarchical_label "RF_{MOSI}" (shape input) (at 121.92 105.41 180) (fields_autoplaced)
     (effects (font (size 1.27 1.27)) (justify right))

Commit message: Complete most of the design, except for RF
Signed-off-by: Jan Hamal Dvořák <mordae@anilinux.org>
Parts:
- renumbered U12 to U13
Connections:
- net AVDD: now reaches U13.11 (AVDD)
- net AVDD: now also U13.14 (AVDD), U13.15 (AVDD), U13.9 (AVDD)
- net GND: now reaches U13.16 (GND)
- net GND: now also U13.19 (GND), U13.21 (EP)
- no-connect marks 0 -> 11
Changed lines of the file:
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@@
     (company "DDM Spirála")
   )
-  (hierarchical_label "RF_{MOSI}" (shape input) (at 121.92 105.41 180) (fields_autoplaced)
+  (junction (at 140.97 106.68) (diameter 0) (color 0 0 0 0)
+  )
+  (no_connect (at 157.48 85.09))
+  (no_connect (at 157.48 80.01))
+  (no_connect (at 121.92 95.25))
+  (no_connect (at 157.48 97.79))
+  (no_connect (at 121.92 87.63))
+  (no_connect (at 157.48 95.25))
+  (no_connect (at 157.48 90.17))
+  (no_connect (at 121.92 97.79))
+  (no_connect (at 121.92 90.17))
+  (no_connect (at 157.48 77.47))
+  (no_connect (at 157.48 87.63))
+  (wire (pts (xy 140.97 106.68) (xy 139.7 106.68))
+    (stroke (width 0) (type default))
+  )
+  (wire (pts (xy 142.24 106.68) (xy 140.97 106.68))
+    (stroke (width 0) (type default))
+  )
+  (wire (pts (xy 140.97 106.68) (xy 140.97 107.95))
+    (stroke (width 0) (type default))
+  )
+  (wire (pts (xy 142.24 105.41) (xy 142.24 106.68))
+    (stroke (width 0) (type default))
+  )
+  (wire (pts (xy 139.7 106.68) (xy 139.7 105.41))
+    (stroke (width 0) (type default))
+  )
+  (hierarchical_label "RF_{MOSI}" (shape input) (at 121.92 82.55 180) (fields_autoplaced)
     (effects (font (size 1.27 1.27)) (justify right))
   )
-  (hierarchical_label "RF_{CS}" (shape input) (at 121.92 97.79 180) (fields_autoplaced)
+  (hierarchical_label "RF_{CS}" (shape input) (at 121.92 77.47 180) (fields_autoplaced)
     (effects (font (size 1.27 1.27)) (justify right))
   )
-  (hierarchical_label "RF_{SCLK}" (shape input) (at 121.92 100.33 180) (fields_autoplaced)
+  (hierarchical_label "RF_{SCLK}" (shape input) (at 121.92 80.01 180) (fields_autoplaced)
     (effects (font (size 1.27 1.27)) (justify right))
   )
-  (hierarchical_label "RF_{MISO}" (shape input) (at 121.92 102.87 180) (fields_autoplaced)
+  (hierarchical_label "RF_{MISO}" (shape output) (at 121.92 85.09 180) (fields_autoplaced)
     (effects (font (size 1.27 1.27)) (justify right))
+  )
+  (symbol (lib_id "power:GND") (at 140.97 107.95 0) (unit 1)
+    (in_bom yes) (on_board yes) (dnp no) (fields_autoplaced)
+    (property "Reference" "#PWR0106" (at 140.97 114.3 0)
+      (effects (font (size 1.27 1.27)) hide)
+    )
+    (property "Value" "GND" (at 140.97 113.03 0)
+      (effects (font (size 1.27 1.27)))
+    )
+    (property "Footprint" "" (at 140.97 107.95 0)
+      (effects (font (size 1.27 1.27)) hide)
+    )
+    (property "Datasheet" "" (at 140.97 107.95 0)
+      (effects (font (size 1.27 1.27)) hide)
+    )
+    (pin "1")
+    (instances
+      (project "krecek-0.9"
+        (path "/8888f37b-ecc2-47df-8824-4b4e1e726451/40971852-55ba-4d75-a9d8-2b5de9b08cbd"
+          (reference "#PWR0106") (unit 1)
+        )
+      )
+    )
   )
   (symbol (lib_id "LCSC:CC1101RGPR") (at 139.7 92.71 0) (unit 1)
     (in_bom yes) (on_board yes) (dnp no) (fields_autoplaced)
-    (property "Reference" "U12" (at 139.7 71.12 0)
+    (property "Reference" "U13" (at 139.7 71.12 0)
       (effects (font (size 1.27 1.27)))
     )
@@
       (project "krecek-0.9"
         (path "/8888f37b-ecc2-47df-8824-4b4e1e726451/40971852-55ba-4d75-a9d8-2b5de9b08cbd"
-          (reference "U12") (unit 1)
+          (reference "U13") (unit 1)
         )
       )

Commit message: Complete the RF section
Parts:
- added C6 (x3): 10u, Capacitor_SMD:C_0402_1005Metric, symbol Device:C_Small
- added C7 (x2): 4.7p, Capacitor_SMD:C_0402_1005Metric, symbol Device:C_Small
- added C7: 10p, Capacitor_SMD:C_0402_1005Metric, symbol Device:C_Small
- added C7: 3.3p, Capacitor_SMD:C_0402_1005Metric, symbol Device:C_Small
- added C7: 100nF, Capacitor_SMD:C_0402_1005Metric, symbol Device:C_Small
- added C7 (x2): 220p, Capacitor_SMD:C_0402_1005Metric, symbol Device:C_Small
- added J5: SMA, LCSC:CONN-SMD_KH-SMA-KE8-G, symbol Connector:Conn_Coaxial
- added L2, L3, L4, L5: 27n, Inductor_SMD:L_0402_1005Metric, symbol Device:L_Small
- added R11: 56k, Resistor_SMD:R_0603_1608Metric, symbol Device:R_Small
Connections:
- net AVDD is gone; now on net +3.3V: U13.11 (AVDD), U13.14 (AVDD), U13.15 (AVDD), U13.9 (AVDD)
- net GND: now also C6.2, C6.2, C6.2, C7.1, C7.2, C7.2, C7.2, C7.2, J5.2 (Ext), R11.2
- net at U13.12 (RF_P): now also C7.2, L3.1
- net at U13.13 (RF_N): now also C7.1, L2.1
- net at U13.17 (RBIAS): now also R11.1
- net +3.3V: now reaches U13.18 (DGUARD)
- net +3.3V: now also U13.4 (DVDD), C6.1, C6.1, C6.1
- net at U13.5 (DCOUPL): now also C7.1
- net RF_{CLK}: now reaches U13.8 (XOSC_Q1)
- new net: C7.2, L3.2, L4.1
- new net: C7.1, L4.2, L5.1
- new net: C7.1, C7.2, L5.2
- new net: C7.1, L2.2
- new net: C7.1, J5.1 (In)
- no-connect marks 11 -> 3
Other:
- moved on the sheet: U13

Commit message: Fix part numbers
Signed-off-by: Jan Hamal Dvořák <mordae@anilinux.org>
Parts:
- renumbered J5 to J4, L3 to L2, L4 to L3, L5 to L4, L2 to L5, R11 to R33

Commit message: Work in progress on board layout
Signed-off-by: Jan Hamal Dvořák <mordae@anilinux.org>
Parts:
- J4: value SMA -> U.FL; footprint LCSC:CONN-SMD_KH-SMA-KE8-G -> Connector_Coaxial:U.FL_Hirose_U.FL-R-SMT-1_Vertical; LCSC Part (none) -> C5137195
Changed lines of the file:
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@@
   (symbol (lib_id "Connector:Conn_Coaxial") (at 203.2 77.47 0) (unit 1)
     (in_bom yes) (on_board yes) (dnp no) (fields_autoplaced)
-    (property "Reference" "J4" (at 207.01 76.4932 0)
+    (property "Reference" "J4" (at 205.74 76.4932 0)
       (effects (font (size 1.27 1.27)) (justify left))
     )
-    (property "Value" "SMA" (at 207.01 79.0332 0)
+    (property "Value" "U.FL" (at 205.74 79.0332 0)
       (effects (font (size 1.27 1.27)) (justify left))
     )
-    (property "Footprint" "LCSC:CONN-SMD_KH-SMA-KE8-G" (at 203.2 77.47 0)
+    (property "Footprint" "Connector_Coaxial:U.FL_Hirose_U.FL-R-SMT-1_Vertical" (at 203.2 77.47 0)
       (effects (font (size 1.27 1.27)) hide)
     )
@@
       (effects (font (size 1.27 1.27)) hide)
     )
+    (property "LCSC Part" "C5137195" (at 203.2 77.47 0)
+      (effects (font (size 1.27 1.27)) hide)
+    )

Commit message: Add discrete antenna
Signed-off-by: Jan Hamal Dvořák <mordae@anilinux.org>
Parts:
- added AE1: Antenna, LCSC:ANT-TH_T14-433M, symbol Device:Antenna
- renumbered C7 to C64, C7 to C65, C7 to C66, C7 to C67, C7 to C68, C7 to C69, C7 to C70
Connections:
- net at C65.1, J4.1 (In): now also AE1.1 (A)
Other:
- moved on the sheet: J4

Commit message: PCB layout progress
Signed-off-by: Jan Hamal Dvořák <mordae@anilinux.org>
Parts:
- added C82: 10u, Capacitor_SMD:C_0402_1005Metric, symbol Device:C_Small
Connections:
- net +3.3V: now also C82.1
- net GND: now also C82.2
Changed lines of the file:
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@@
     (company "DDM Spirála")
   )
+  (junction (at 88.9 50.8) (diameter 0) (color 0 0 0 0)
+  )
   (junction (at 127 80.01) (diameter 0) (color 0 0 0 0)
   )
@@
   )
   (junction (at 77.47 106.68) (diameter 0) (color 0 0 0 0)
+  )
+  (junction (at 88.9 38.1) (diameter 0) (color 0 0 0 0)
   )
   (junction (at 165.1 77.47) (diameter 0) (color 0 0 0 0)
@@
     (stroke (width 0) (type default))
   )
+  (wire (pts (xy 88.9 38.1) (xy 101.6 38.1))
+    (stroke (width 0) (type default))
+  )
   (wire (pts (xy 186.69 77.47) (xy 203.2 77.47))
     (stroke (width 0) (type default))
@@
     (stroke (width 0) (type default))
   )
+  (wire (pts (xy 101.6 46.99) (xy 101.6 50.8))
+    (stroke (width 0) (type default))
+  )
   (wire (pts (xy 152.4 77.47) (xy 156.21 77.47))
+    (stroke (width 0) (type default))
+  )
+  (wire (pts (xy 101.6 38.1) (xy 101.6 41.91))
+    (stroke (width 0) (type default))
+  )
+  (wire (pts (xy 88.9 50.8) (xy 101.6 50.8))
     (stroke (width 0) (type default))
   )
@@
         )
       )
+    )
+  )
+  (symbol (lib_id "Device:C_Small") (at 101.6 44.45 0) (mirror y) (unit 1)
+    (in_bom yes) (on_board yes) (dnp no) (fields_autoplaced)
+    (property "Reference" "C82" (at 104.14 43.1863 0)
+      (effects (font (size 1.27 1.27)) (justify right))
+    )
+    (property "Value" "10u" (at 104.14 45.7263 0)
+      (effects (font (size 1.27 1.27)) (justify right))
+    )
+    (property "Footprint" "Capacitor_SMD:C_0402_1005Metric" (at 101.6 44.45 0)
+      (effects (font (size 1.27 1.27)) hide)
+    )
+    (property "Datasheet" "~" (at 101.6 44.45 0)
+      (effects (font (size 1.27 1.27)) hide)
+    )
+    (property "LCSC Part" "C15525" (at 101.6 44.45 0)
+      (effects (font (size 1.27 1.27)) hide)
+    )
+    (pin "1")
+    (pin "2")
+    (instances
+      (project "krecek-0.9"
+        (path "/8888f37b-ecc2-47df-8824-4b4e1e726451/40971852-55ba-4d75-a9d8-2b5de9b08cbd"
+          (reference "C82") (unit 1)
+        )
+      )
