File: hw/krecek-0.9/radio.kicad_sch (KiCad schematic)
At the start: 19 parts, among them J4 U.FL, U13 CC1101RGPR

Commit message: Hardware as sent for manufacturing
Parts:
- C69: value 100nF -> 100n
Changed lines of the file:
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@@
       (effects (font (size 1.27 1.27)) (justify right))
     )
-    (property "Value" "100nF" (at 116.84 104.1463 0)
+    (property "Value" "100n" (at 116.84 104.1463 0)
       (effects (font (size 1.27 1.27)) (justify right))
     )

Commit message: Fix input PMOS orientation (again)
Parts:
- renumbered C82 to C60, C64 to C61, C65 to C62, C66 to C63, C67 to C64, C68 to C65, C69 to C66, C70 to C67, R33 to R36

Commit message: Add display components to library
Also move CC1101 communication to second chip.
Resolves #13.
Connections:
- net RF_{CLK} renamed RF_{XOSC}
Changed lines of the file:
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@@
     (effects (font (size 1.27 1.27)) (justify right))
   )
-  (hierarchical_label "RF_{CLK}" (shape input) (at 58.42 95.25 180) (fields_autoplaced)
+  (hierarchical_label "RF_{XOSC}" (shape input) (at 58.42 95.25 180) (fields_autoplaced)
     (effects (font (size 1.27 1.27)) (justify right))
   )

Commit message: Fix ERC-indicated issues
Parts:
- renumbered C60 to C59, C61 to C60, C62 to C61, C63 to C62, C64 to C63, C65 to C64, C66 to C65, C67 to C66, R36 to R34, U13 to U12

Commit message: Progress on HW design
Parts:
- renumbered C59 to C57, C60 to C58, C61 to C59, C62 to C60, C63 to C61, C64 to C62, C65 to C63, C66 to C64, R34 to R36, U12 to U11
Changed lines of the file:
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@@
 		(dnp no)
 		(fields_autoplaced yes)
-		(property "Reference" "#PWR082"
+		(property "Reference" "#PWR081"
 			(at 76.2 39.37 0)
 			(effects
@@
 			(project "krecek-0.9"
 				(path "/8888f37b-ecc2-47df-8824-4b4e1e726451/40971852-55ba-4d75-a9d8-2b5de9b08cbd"
-					(reference "#PWR082")
+					(reference "#PWR081")
 					(unit 1)
 				)
@@
 		(dnp no)
 		(fields_autoplaced yes)
-		(property "Reference" "#PWR092"
+		(property "Reference" "#PWR091"
 			(at 127 114.3 0)
 			(effects
@@
 			(project "krecek-0.9"
 				(path "/8888f37b-ecc2-47df-8824-4b4e1e726451/40971852-55ba-4d75-a9d8-2b5de9b08cbd"
-					(reference "#PWR092")
+					(reference "#PWR091")
 					(unit 1)
 				)
@@
 		(dnp no)
 		(fields_autoplaced yes)
-		(property "Reference" "#PWR091"
+		(property "Reference" "#PWR090"
 			(at 114.3 114.3 0)
 			(effects
@@
 			(project "krecek-0.9"
 				(path "/8888f37b-ecc2-47df-8824-4b4e1e726451/40971852-55ba-4d75-a9d8-2b5de9b08cbd"
-					(reference "#PWR091")
+					(reference "#PWR090")
 					(unit 1)
 				)
@@
 			(project "krecek-0.9"
 				(path "/8888f37b-ecc2-47df-8824-4b4e1e726451/40971852-55ba-4d75-a9d8-2b5de9b08cbd"
-					(reference "C56")
+					(reference "C54")
 					(unit 1)
 				)
@@
 		(dnp no)
 		(fields_autoplaced yes)
-		(property "Reference" "#PWR089"
+		(property "Reference" "#PWR088"
 			(at 77.47 114.3 0)
 			(effects
@@
 			(project "krecek-0.9"
 				(path "/8888f37b-ecc2-47df-8824-4b4e1e726451/40971852-55ba-4d75-a9d8-2b5de9b08cbd"
-					(reference "#PWR089")
+					(reference "#PWR088")
 					(unit 1)
 				)
@@
 		(dnp no)
 		(fields_autoplaced yes)
-		(property "Reference" "#PWR088"
+		(property "Reference" "#PWR087"
 			(at 215.9 95.25 0)
 			(effects
@@
 			(project "krecek-0.9"
 				(path "/8888f37b-ecc2-47df-8824-4b4e1e726451/40971852-55ba-4d75-a9d8-2b5de9b08cbd"
-					(reference "#PWR088")
+					(reference "#PWR087")
 					(unit 1)
 				)
@@
 		(dnp no)
 		(fields_autoplaced yes)
-		(property "Reference" "C64"
+		(property "Reference" "C62"
 			(at 180.34 82.5563 0)
 			(effects
@@
 			(project "krecek-0.9"
 				(path "/8888f37b-ecc2-47df-8824-4b4e1e726451/40971852-55ba-4d75-a9d8-2b5de9b08cbd"
-					(reference "C64")
+					(reference "C62")
 					(unit 1)
 				)
@@
 		(dnp no)
 		(fields_autoplaced yes)
-		(property "Reference" "#PWR085"
+		(property "Reference" "#PWR084"
 			(at 92.71 87.63 0)
 			(effects
@@
 			(project "krecek-0.9"
 				(path "/8888f37b-ecc2-47df-8824-4b4e1e726451/40971852-55ba-4d75-a9d8-2b5de9b08cbd"
-					(reference "#PWR085")
+					(reference "#PWR084")
 					(unit 1)
 				)
@@
 		(dnp no)
 		(fields_autoplaced yes)
-		(property "Reference" "#PWR086"
+		(property "Reference" "#PWR085"
 			(at 165.1 95.25 0)
 			(effects
@@
 			(project "krecek-0.9"
 				(path "/8888f37b-ecc2-47df-8824-4b4e1e726451/40971852-55ba-4d75-a9d8-2b5de9b08cbd"
-					(reference "#PWR086")
+					(reference "#PWR085")
 					(unit 1)
 				)
@@
 		(dnp no)
 		(fields_autoplaced yes)
-		(property "Reference" "#PWR090"
+		(property "Reference" "#PWR089"
 			(at 96.52 114.3 0)
 			(effects
@@
 			(project "krecek-0.9"
 				(path "/8888f37b-ecc2-47df-8824-4b4e1e726451/40971852-55ba-4d75-a9d8-2b5de9b08cbd"
-					(reference "#PWR090")
+					(reference "#PWR089")
 					(unit 1)
 				)
@@
 			(project "krecek-0.9"
 				(path "/8888f37b-ecc2-47df-8824-4b4e1e726451/40971852-55ba-4d75-a9d8-2b5de9b08cbd"
-					(reference "C58")
+					(reference "C56")
 					(unit 1)
 				)
@@
 			(project "krecek-0.9"
 				(path "/8888f37b-ecc2-47df-8824-4b4e1e726451/40971852-55ba-4d75-a9d8-2b5de9b08cbd"
-					(reference "#PWR083")
+					(reference "#PWR082")
 					(unit 1)
 				)
@@
 		(dnp no)
 		(fields_autoplaced yes)
-		(property "Reference" "C63"
+		(property "Reference" "C61"
 			(at 167.64 82.5563 0)
 			(effects
@@
 			(project "krecek-0.9"
 				(path "/8888f37b-ecc2-47df-8824-4b4e1e726451/40971852-55ba-4d75-a9d8-2b5de9b08cbd"
-					(reference "C63")
+					(reference "C61")
 					(unit 1)
 				)
@@
 		(dnp no)
 		(fields_autoplaced yes)
-		(property "Reference" "C60"
+		(property "Reference" "C58"
 			(at 129.54 68.5863 0)
 			(effects
@@
 			(project "krecek-0.9"
 				(path "/8888f37b-ecc2-47df-8824-4b4e1e726451/40971852-55ba-4d75-a9d8-2b5de9b08cbd"
-					(reference "C60")
+					(reference "C58")
 					(unit 1)
 				)
@@
 		(dnp no)
 		(fields_autoplaced yes)
-		(property "Reference" "U12"
+		(property "Reference" "U11"
 			(at 76.2 69.85 0)
 			(effects
@@
 			(project "krecek-0.9"
 				(path "/8888f37b-ecc2-47df-8824-4b4e1e726451/40971852-55ba-4d75-a9d8-2b5de9b08cbd"
-					(reference "U12")
+					(reference "U11")
 					(unit 1)
 				)
@@
 		(dnp no)
 		(fields_autoplaced yes)
-		(property "Reference" "C65"
+		(property "Reference" "C63"
 			(at 116.84 101.6063 0)
 			(effects
@@
 			(project "krecek-0.9"
 				(path "/8888f37b-ecc2-47df-8824-4b4e1e726451/40971852-55ba-4d75-a9d8-2b5de9b08cbd"
-					(reference "C65")
+					(reference "C63")
 					(unit 1)
 				)
@@
 		(dnp no)
 		(fields_autoplaced yes)
-		(property "Reference" "#PWR087"
+		(property "Reference" "#PWR086"
 			(at 177.8 95.25 0)
 			(effects
@@
 			(project "krecek-0.9"
 				(path "/8888f37b-ecc2-47df-8824-4b4e1e726451/40971852-55ba-4d75-a9d8-2b5de9b08cbd"
-					(reference "#PWR087")
+					(reference "#PWR086")
 					(unit 1)
 				)
@@
 			(project "krecek-0.9"
 				(path "/8888f37b-ecc2-47df-8824-4b4e1e726451/40971852-55ba-4d75-a9d8-2b5de9b08cbd"
-					(reference "C57")
+					(reference "C55")
 					(unit 1)
 				)
@@
 		(dnp no)
 		(fields_autoplaced yes)
-		(property "Reference" "C59"
+		(property "Reference" "C57"
 			(at 104.14 43.1863 0)
 			(effects
@@
 			(project "krecek-0.9"
 				(path "/8888f37b-ecc2-47df-8824-4b4e1e726451/40971852-55ba-4d75-a9d8-2b5de9b08cbd"
-					(reference "C59")
+					(reference "C57")
 					(unit 1)
 				)
@@
 		(dnp no)
 		(fields_autoplaced yes)
-		(property "Reference" "C66"
+		(property "Reference" "C64"
 			(at 129.54 101.6063 0)
 			(effects
@@
 			(project "krecek-0.9"
 				(path "/8888f37b-ecc2-47df-8824-4b4e1e726451/40971852-55ba-4d75-a9d8-2b5de9b08cbd"
-					(reference "C66")
+					(reference "C64")
 					(unit 1)
 				)
@@
 		(dnp no)
 		(fields_autoplaced yes)
-		(property "Reference" "#PWR084"
+		(property "Reference" "#PWR083"
 			(at 127 57.15 0)
 			(effects
@@
 			(project "krecek-0.9"
 				(path "/8888f37b-ecc2-47df-8824-4b4e1e726451/40971852-55ba-4d75-a9d8-2b5de9b08cbd"
-					(reference "#PWR084")
+					(reference "#PWR083")
 					(unit 1)
 				)
@@
 		(dnp no)
 		(fields_autoplaced yes)
-		(property "Reference" "C61"
+		(property "Reference" "C59"
 			(at 184.1436 71.12 90)
 			(effects
@@
 			(project "krecek-0.9"
 				(path "/8888f37b-ecc2-47df-8824-4b4e1e726451/40971852-55ba-4d75-a9d8-2b5de9b08cbd"
-					(reference "C61")
+					(reference "C59")
 					(unit 1)
 				)
@@
 		(dnp no)
 		(fields_autoplaced yes)
-		(property "Reference" "R34"
+		(property "Reference" "R36"
 			(at 99.06 101.6 0)
 			(effects
@@
 			(project "krecek-0.9"
 				(path "/8888f37b-ecc2-47df-8824-4b4e1e726451/40971852-55ba-4d75-a9d8-2b5de9b08cbd"
-					(reference "R34")
+					(reference "R36")
 					(unit 1)
 				)
@@
 		(dnp no)
 		(fields_autoplaced yes)
-		(property "Reference" "C62"
+		(property "Reference" "C60"
 			(at 146.0563 83.82 90)
 			(effects
@@
 			(project "krecek-0.9"
 				(path "/8888f37b-ecc2-47df-8824-4b4e1e726451/40971852-55ba-4d75-a9d8-2b5de9b08cbd"
-					(reference "C62")
-					(unit 1)
-				)
+					(reference "C60")
+					(unit 1)
+				)

Commit message: Work on board layout
Parts:
- removed C58: 3.3p, Capacitor_SMD:C_0402_1005Metric, symbol Device:C_Small
- removed C59, C64: 220p, Capacitor_SMD:C_0402_1005Metric, symbol Device:C_Small
- removed C60, C62: 4.7p, Capacitor_SMD:C_0402_1005Metric, symbol Device:C_Small
- removed C61: 10p, Capacitor_SMD:C_0402_1005Metric, symbol Device:C_Small
- removed L2, L3, L4, L5: 27n, Inductor_SMD:L_0402_1005Metric, symbol Device:L_Small
- added U14: BW21S5011A01TF, LCSC:FILTER-SMD_4P-L2.0-W1.2-BL-1, symbol LCSC:BW21S5011A01TF
Connections:
- net GND: now also U14.1
- net at U11.12 (RF_P): now also U14.3
- net at AE1.1 (A), J4.1 (In): now also U14.4
- net at U11.13 (RF_N): now also U14.2
Other:
- moved on the sheet: AE1, J4
