File: hw/krecek-0.9/krecek-0.9.kicad_pcb (KiCad board)
At the start: 2 copper layers, 0 parts

Commit message: Complete the RF section
Other:
- copper layers 2 -> 4
Changed lines of the file:
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@@
   (layers
     (0 "F.Cu" signal)
+    (1 "In1.Cu" signal)
+    (2 "In2.Cu" signal)
     (31 "B.Cu" signal)
     (32 "B.Adhes" user "B.Adhesive")
@@
   )
   (setup
+    (stackup
+      (layer "F.SilkS" (type "Top Silk Screen") (color "White"))
+      (layer "F.Paste" (type "Top Solder Paste"))
+      (layer "F.Mask" (type "Top Solder Mask") (color "Green") (thickness 0.01))
+      (layer "F.Cu" (type "copper") (thickness 0.035))
+      (layer "dielectric 1" (type "prepreg") (color "FR4 natural") (thickness 0.1) (material "FR4") (epsilon_r 4.5) (loss_tangent 0.02))
+      (layer "In1.Cu" (type "copper") (thickness 0.035))
+      (layer "dielectric 2" (type "core") (color "FR4 natural") (thickness 1.24) (material "FR4") (epsilon_r 4.5) (loss_tangent 0.02))
+      (layer "In2.Cu" (type "copper") (thickness 0.035))
+      (layer "dielectric 3" (type "prepreg") (color "FR4 natural") (thickness 0.1) (material "FR4") (epsilon_r 4.5) (loss_tangent 0.02))
+      (layer "B.Cu" (type "copper") (thickness 0.035))
+      (layer "B.Mask" (type "Bottom Solder Mask") (color "Green") (thickness 0.01))
+      (layer "B.Paste" (type "Bottom Solder Paste"))
+      (layer "B.SilkS" (type "Bottom Silk Screen") (color "White"))
+      (copper_finish "None")
+      (dielectric_constraints no)
+    )
     (pad_to_mask_clearance 0)
     (pcbplotparams

Commit message: Work in progress on board layout
Signed-off-by: Jan Hamal Dvořák <mordae@anilinux.org>
Parts:
- added C1: 10u, Capacitor_SMD:C_0402_1005Metric, F.Cu at (-33.8, 68.9)
- added C10: 10u, Capacitor_SMD:C_0402_1005Metric, F.Cu at (-31.0, 72.8)
- added C11: 10u, Capacitor_SMD:C_0402_1005Metric, F.Cu at (-31.0, 74.8)
- added C12: 10u, Capacitor_SMD:C_0402_1005Metric, F.Cu at (-31.0, 76.8)
- added C13: 10u, Capacitor_SMD:C_0402_1005Metric, F.Cu at (-31.0, 78.7)
- added C14: 10u, Capacitor_SMD:C_0402_1005Metric, F.Cu at (-31.0, 80.7)
- added C15: 10u, Capacitor_SMD:C_0402_1005Metric, F.Cu at (-28.1, 68.9)
- added C16: 10u, Capacitor_SMD:C_0402_1005Metric, F.Cu at (-28.1, 70.9)
- added C17: 10u, Capacitor_SMD:C_0402_1005Metric, F.Cu at (-28.1, 72.8)
- added C18: 10u, Capacitor_SMD:C_0402_1005Metric, F.Cu at (-28.1, 74.8)
- added C19: 10u, Capacitor_SMD:C_0402_1005Metric, F.Cu at (-28.1, 76.8)
- added C2: 10u, Capacitor_SMD:C_0402_1005Metric, F.Cu at (-33.8, 70.9)
- added C20: 10u, Capacitor_SMD:C_0402_1005Metric, F.Cu at (-28.1, 78.7)
- added C21: 10u, Capacitor_SMD:C_0402_1005Metric, F.Cu at (-28.1, 80.7)
- added C22: 10u, Capacitor_SMD:C_0402_1005Metric, F.Cu at (-25.2, 68.9)
- added C23: 100n, Capacitor_SMD:C_0402_1005Metric, F.Cu at (-25.2, 70.9)
- added C24: 33p, Capacitor_SMD:C_0402_1005Metric, F.Cu at (-25.2, 72.8)
- added C25: 33p, Capacitor_SMD:C_0402_1005Metric, F.Cu at (-25.2, 74.8)
- added C26: 1uF, Capacitor_SMD:C_0805_2012Metric, F.Cu at (139.8, 118.5)
- added C27: 1uF, Capacitor_SMD:C_0805_2012Metric, F.Cu at (186.4, 102.9)
- added C28: 1uF, Capacitor_SMD:C_0805_2012Metric, F.Cu at (186.4, 99.9)
- added C29: 1uF, Capacitor_SMD:C_0805_2012Metric, F.Cu at (160.0, 47.9)
- added C3: 10u, Capacitor_SMD:C_0402_1005Metric, F.Cu at (-33.8, 72.8)
- added C30: 1uF, Capacitor_SMD:C_0805_2012Metric, F.Cu at (64.7, 119.9)
- added C31: 1uF, Capacitor_SMD:C_0805_2012Metric, F.Cu at (64.6, 117.6)
- added C32: 1uF, Capacitor_SMD:C_0805_2012Metric, F.Cu at (80.7, 118.4)
- added C33: 1uF, Capacitor_SMD:C_0805_2012Metric, F.Cu at (94.0, 114.6)
- added C34: 4.7uF, Capacitor_SMD:C_0603_1608Metric, F.Cu at (58.2, 113.8)
- added C35: 4.7uF, Capacitor_SMD:C_0603_1608Metric, F.Cu at (58.2, 108.2)
- added C36: 1uF, Capacitor_SMD:C_0805_2012Metric, F.Cu at (61.2, 97.5)
- added C37: 100uF, Capacitor_Tantalum_SMD:CP_EIA-3528-21_Kemet-B, F.Cu at (58.9, 119.8)
- added C38: 100nF, Capacitor_SMD:C_0402_1005Metric, F.Cu at (64.3, 111.2)
- added C39: 10pF, Capacitor_SMD:C_0402_1005Metric, F.Cu at (55.3, 117.2)
- added C4: 10u, Capacitor_SMD:C_0402_1005Metric, F.Cu at (-33.8, 74.8)
- added C40: 10u, Capacitor_SMD:C_0402_1005Metric, F.Cu at (171.3, 123.2)
- added C41: 10u, Capacitor_SMD:C_0402_1005Metric, F.Cu at (173.3, 123.2)
- added C42: 10u, Capacitor_SMD:C_0402_1005Metric, F.Cu at (175.2, 123.2)
- added C43: 10u, Capacitor_SMD:C_0402_1005Metric, F.Cu at (177.2, 123.2)
- added C44: 10u, Capacitor_SMD:C_0402_1005Metric, F.Cu at (179.2, 123.2)
- added C45: 10u, Capacitor_SMD:C_0402_1005Metric, F.Cu at (181.2, 123.2)
- added C46: 10u, Capacitor_SMD:C_0402_1005Metric, F.Cu at (183.1, 123.2)
- added C47: 10u, Capacitor_SMD:C_0402_1005Metric, F.Cu at (171.3, 120.3)
- added C48: 1u, Capacitor_SMD:C_0402_1005Metric, F.Cu at (173.3, 120.3)
- added C49: 1u, Capacitor_SMD:C_0402_1005Metric, F.Cu at (175.2, 120.3)
- added C5: 10u, Capacitor_SMD:C_0402_1005Metric, F.Cu at (-33.8, 76.8)
- added C50: 10u, Capacitor_SMD:C_0402_1005Metric, F.Cu at (177.2, 120.3)
- added C51: 1u, Capacitor_SMD:C_0402_1005Metric, F.Cu at (179.2, 120.3)
- added C52: 1u, Capacitor_SMD:C_0402_1005Metric, F.Cu at (181.2, 120.3)
- added C53: 10u, Capacitor_SMD:C_0402_1005Metric, F.Cu at (183.1, 120.3)
- added C54: 1u, Capacitor_SMD:C_0402_1005Metric, F.Cu at (171.3, 117.5)
- added C55: 1u, Capacitor_SMD:C_0402_1005Metric, F.Cu at (173.3, 117.5)
- added C56: 1u, Capacitor_SMD:C_0402_1005Metric, F.Cu at (175.2, 117.5)
- added C57: 1u, Capacitor_SMD:C_0402_1005Metric, F.Cu at (177.2, 117.5)
- added C58: 1u, Capacitor_SMD:C_0402_1005Metric, F.Cu at (179.2, 117.5)
- added C59: 1u, Capacitor_SMD:C_0402_1005Metric, F.Cu at (181.2, 117.5)
- added C6: 10u, Capacitor_SMD:C_0402_1005Metric, F.Cu at (-33.8, 78.7)
- added C60: 1u, Capacitor_SMD:C_0402_1005Metric, F.Cu at (183.1, 117.5)
- added C61: 10u, Capacitor_SMD:C_0402_1005Metric, F.Cu at (63.7, 60.7)
- added C62: 10u, Capacitor_SMD:C_0402_1005Metric, F.Cu at (65.6, 60.7)
- added C63: 10u, Capacitor_SMD:C_0402_1005Metric, F.Cu at (67.6, 60.7)
- added C64: 3.3p, Capacitor_SMD:C_0402_1005Metric, F.Cu at (69.6, 60.7)
- added C65: 220p, Capacitor_SMD:C_0402_1005Metric, F.Cu at (71.5, 60.7)
- added C66: 4.7p, Capacitor_SMD:C_0402_1005Metric, F.Cu at (63.7, 57.8)
- added C67: 10p, Capacitor_SMD:C_0402_1005Metric, F.Cu at (65.6, 57.8)
- added C68: 4.7p, Capacitor_SMD:C_0402_1005Metric, F.Cu at (67.6, 57.8)
- added C69: 100nF, Capacitor_SMD:C_0402_1005Metric, F.Cu at (69.6, 57.8)
- added C7: 10u, Capacitor_SMD:C_0402_1005Metric, F.Cu at (-33.8, 80.7)
- added C70: 220p, Capacitor_SMD:C_0402_1005Metric, F.Cu at (71.5, 57.8)
- added C71: 100nF, Capacitor_SMD:C_0402_1005Metric, F.Cu at (127.5, 102.9)
- added C72: 100nF, Capacitor_SMD:C_0402_1005Metric, F.Cu at (215.1, 91.4)
- added C73: 100nF, Capacitor_SMD:C_0402_1005Metric, F.Cu at (215.1, 96.5)
- added C74: 100nF, Capacitor_SMD:C_0402_1005Metric, F.Cu at (215.1, 88.9)
- added C75: 100nF, Capacitor_SMD:C_0402_1005Metric, F.Cu at (215.1, 94.0)
- added C76: 100nF, Capacitor_SMD:C_0402_1005Metric, F.Cu at (193.0, 124.9)
- added C77: 100nF, Capacitor_SMD:C_0402_1005Metric, F.Cu at (85.9, 86.4)
- added C78: 100nF, Capacitor_SMD:C_0402_1005Metric, F.Cu at (190.5, 124.9)
- added C79: 100nF, Capacitor_SMD:C_0402_1005Metric, F.Cu at (188.0, 124.9)
- added C8: 10u, Capacitor_SMD:C_0402_1005Metric, F.Cu at (-31.0, 68.9)
- added C80: 100uF, Capacitor_Tantalum_SMD:CP_EIA-3528-21_Kemet-B, F.Cu at (94.0, 119.6)
- added C81: 10u, Capacitor_SMD:C_0402_1005Metric, F.Cu at (95.9, 115.1)
- added C9: 10u, Capacitor_SMD:C_0402_1005Metric, F.Cu at (-31.0, 70.9)
- added CN1: PJ-313B6-B, LCSC:AUDIO-TH_PJ-313B6-B, F.Cu at (151.1, 44.9)
- added D1: yellow, LED_SMD:LED_0603_1608Metric, F.Cu at (147.3, 118.5)
- added D2: red, LED_SMD:LED_0603_1608Metric, F.Cu at (147.3, 120.1)
- added D3: SS54, Diode_SMD:D_SMA, F.Cu at (160.0, 41.9)
- added D4: IR333, LED_THT:LED_D5.0mm_Horizontal_O1.27mm_Z3.0mm_Clear, F.Cu at (142.0, 48.3)
- added D5: IR333, LED_THT:LED_D5.0mm_Horizontal_O1.27mm_Z3.0mm_Clear, F.Cu at (134.5, 48.3)
- added FB1: 600Ω @ 100 MHz, Inductor_SMD:L_0805_2012Metric, F.Cu at (177.1, 25.0)
- added J1: DAP, Connector_PinHeader_2.54mm:PinHeader_1x03_P2.54mm_Vertical, F.Cu at (-18.3, 96.8)
- added J2: AUX, Connector_PinHeader_2.54mm:PinHeader_2x08_P2.54mm_Vertical, F.Cu at (120.7, 40.6)
- added J3: USB_C_Receptacle_USB2.0, LCSC:USB-C-SMD_TYPEC-304J-BCP16, F.Cu at (167.6, 43.2)
- added J4: U.FL, Connector_Coaxial:U.FL_Hirose_U.FL-R-SMT-1_Vertical, F.Cu at (96.5, 48.3)
- added J5: Micro_SD_Card_Det1, LCSC:TF-SMD_TF-012, F.Cu at (106.7, 117.1)
- added JOY1: RKJXV1224005, LCSC:SW-TH_RKJXV1224005, F.Cu at (76.2, 76.2)
- added L1: 2.2uH, Inductor_SMD:L_1008_2520Metric, F.Cu at (58.3, 111.0)
- added L2: 27n, Inductor_SMD:L_0402_1005Metric, F.Cu at (63.7, 54.9)
- added L3: 27n, Inductor_SMD:L_0402_1005Metric, F.Cu at (65.7, 54.9)
- added L4: 27n, Inductor_SMD:L_0402_1005Metric, F.Cu at (67.7, 54.9)
- added L5: 27n, Inductor_SMD:L_0402_1005Metric, F.Cu at (69.6, 54.9)
- added Q1: AO3401A, Package_TO_SOT_SMD:SOT-23, F.Cu at (66.8, 97.3)
- added Q2: AO3401A, Package_TO_SOT_SMD:SOT-23, F.Cu at (62.2, 93.1)
- added Q3: AO3400A, Package_TO_SOT_SMD:SOT-23, F.Cu at (66.9, 101.1)
- added Q4: AO3400A, Package_TO_SOT_SMD:SOT-23, F.Cu at (57.4, 101.7)
- added Q5: AO3400A, Package_TO_SOT_SMD:SOT-23, F.Cu at (66.6, 93.2)
- added Q6: AO3400A, Package_TO_SOT_SMD:SOT-23, F.Cu at (56.1, 95.1)
- added Q7: PT334, LED_THT:LED_D5.0mm_Horizontal_O1.27mm_Z3.0mm_IRBlack, F.Cu at (127.0, 48.3)
- added Q8: AO3400A, Package_TO_SOT_SMD:SOT-23, F.Cu at (180.0, 97.7)
- added R1: 27, Resistor_SMD:R_0603_1608Metric, F.Cu at (-37.8, 96.8)
- added R10: 5.1k, Resistor_SMD:R_0402_1005Metric, F.Cu at (-36.2, 57.3)
- added R11: 10k, Resistor_SMD:R_0402_1005Metric, F.Cu at (154.1, 101.8)
- added R12: 5.1k, Resistor_SMD:R_0402_1005Metric, F.Cu at (-32.9, 57.0)
- added R13: 33k, Resistor_SMD:R_0603_1608Metric, F.Cu at (150.7, 101.6)
- added R14: 1M, Resistor_SMD:R_0402_1005Metric, F.Cu at (61.1, 88.6)
- added R15: 1M, Resistor_SMD:R_0402_1005Metric, F.Cu at (58.7, 88.6)
- added R16: 1M, Resistor_SMD:R_0402_1005Metric, F.Cu at (56.5, 88.8)
- added R17: 330k, Resistor_SMD:R_0603_1608Metric, F.Cu at (57.2, 92.6)
- added R18: 330k, Resistor_SMD:R_0603_1608Metric, F.Cu at (62.3, 101.3)
- added R19: 100k, Resistor_SMD:R_0402_1005Metric, F.Cu at (137.4, 122.8)
- added R2: 27, Resistor_SMD:R_0603_1608Metric, F.Cu at (-37.8, 99.3)
- added R20: 100, Resistor_SMD:R_0402_1005Metric, F.Cu at (60.3, 114.3)
- added R21: 200k, Resistor_SMD:R_0402_1005Metric, F.Cu at (67.9, 109.3)
- added R22: 200k, Resistor_SMD:R_0402_1005Metric, F.Cu at (71.1, 109.5)
- added R23: 200k, Resistor_SMD:R_0402_1005Metric, F.Cu at (74.5, 109.6)
- added R24: 200k, Resistor_SMD:R_0402_1005Metric, F.Cu at (77.2, 109.6)
- added R25: 100k, Resistor_SMD:R_0402_1005Metric, F.Cu at (79.5, 109.6)
- added R26: 10M, Resistor_SMD:R_0603_1608Metric, F.Cu at (56.3, 97.9)
- added R27: 100k, Resistor_SMD:R_0402_1005Metric, F.Cu at (68.2, 112.4)
- added R28: 3.3k, Resistor_SMD:R_0402_1005Metric, F.Cu at (178.8, 93.8)
- added R29: 1, Resistor_SMD:R_1206_3216Metric, F.Cu at (172.0, 113.2)
- added R3: 33k, Capacitor_SMD:C_0402_1005Metric, F.Cu at (-25.2, 76.8)
- added R30: 1, Resistor_SMD:R_1206_3216Metric, F.Cu at (175.3, 113.2)
- added R31: 1k, Resistor_SMD:R_0402_1005Metric, F.Cu at (180.8, 93.8)
- added R32: 1, Resistor_SMD:R_1206_3216Metric, F.Cu at (178.6, 113.2)
- added R33: 56k, Resistor_SMD:R_0603_1608Metric, F.Cu at (73.8, 54.1)
- added R34: 3.3k, Resistor_SMD:R_0402_1005Metric, F.Cu at (193.0, 122.4)
- added R35: 3.3k, Resistor_SMD:R_0402_1005Metric, F.Cu at (85.8, 83.8)
- added R36: RDC506002A, LCSC:RES-ADJ-SMD_RDC506002A, F.Cu at (88.9, 61.0)
- added R37: 3.3k, Resistor_SMD:R_0402_1005Metric, F.Cu at (190.5, 122.4)
- added R38: RDC506002A, LCSC:RES-ADJ-SMD_RDC506002A, F.Cu at (180.3, 61.0)
- added R39: 3.3k, Resistor_SMD:R_0402_1005Metric, F.Cu at (188.0, 122.4)
- added R4: 1k, Resistor_SMD:R_0402_1005Metric, F.Cu at (-38.3, 101.6)
- added R5: 1k, Resistor_SMD:R_0402_1005Metric, F.Cu at (-38.3, 103.6)
- added R6: 560, Resistor_SMD:R_0603_1608Metric, F.Cu at (135.9, 119.7)
- added R7: 2k, Resistor_SMD:R_0402_1005Metric, F.Cu at (134.6, 120.3)
- added R8: 4.7k, Resistor_SMD:R_0402_1005Metric, F.Cu at (144.5, 118.5)
- added R9: 4.7k, Resistor_SMD:R_0402_1005Metric, F.Cu at (144.5, 120.1)
- added SPK1: FS-1540, LCSC:BUZ-SMD_5P-L15.0-W15.0-P13.7-BL, F.Cu at (200.7, 109.2)
- added SW1: SW_Push, LCSC:SW-SMD_4P-L5.1-W5.1-P3.70-LS6.5-TL-2, F.Cu at (-8.10, 81.6)
- added SW2: ~, Krecek:RubberButton, F.Cu at (152.4, 111.8)
- added SW3: ~, Krecek:RubberButton, F.Cu at (127.0, 111.8)
- added SW4: ~, Krecek:ABXY, F.Cu at (200.7, 76.2)
- added SW5: TM-2023, LCSC:SW-SMD_TM-2023-1, F.Cu at (200.0, 123.4)
- added U1: Display, Krecek:TftDisplay, F.Cu at (134.6, 76.2)
- added U10: TPS63000, Package_SON:Texas_DRC0010J_ThermalVias, F.Cu at (61.7, 111.0)
- added U11: ES8312, LCSC:VQFN-28_L4.0-W4.0-P0.45-TL-EP2.6, F.Cu at (180.6, 102.9)
- added U12: TPA2028D1YZFT, LCSC:TPA2028, F.Cu at (171.8, 108.9)
- added U13: CC1101RGPR, LCSC:QFN-20_L4.0-W4.0-P0.5-TL-EP, F.Cu at (75.4, 59.0)
- added U2: RP2040, Package_DFN_QFN:QFN-56-1EP_7x7mm_P0.4mm_EP3.2x3.2mm, F.Cu at (-39.9, 72.5)
- added U3: RP2040, Package_DFN_QFN:QFN-56-1EP_7x7mm_P0.4mm_EP3.2x3.2mm, F.Cu at (-39.9, 81.8)
- added U4: W25Q128JVS, Package_SO:SOIC-8_5.23x5.23mm_P1.27mm, F.Cu at (-28.4, 91.8)
- added U5: AMS1117-3.3, Package_TO_SOT_SMD:SOT-223-3_TabPin2, F.Cu at (185.4, 110.5)
- added U6: JST-PH-2P, LCSC:CONN-TH-2P-P2.00_S2B-PH-KL-LF-SN, B.Cu at (139.7, 115.3)
- added U7: BQ24045DSQR, LCSC:WSON-10_L2.0-W2.0-P0.40-BL-EP, F.Cu at (135.5, 123.1)
- added U8: AMS1117-3.3, Package_TO_SOT_SMD:SOT-223-3_TabPin2, F.Cu at (73.5, 118.1)
- added U9: AMS1117-3.3, Package_TO_SOT_SMD:SOT-223-3_TabPin2, F.Cu at (87.0, 118.1)
- added Y1: 12MHz, LCSC:OSC-SMD_4P-L3.2-W2.5-BL, F.Cu at (-48.9, 92.5)
Routing:
- net Net-(J4-In): track 0.00 -> 142.8 mm
- net /Power/~{PG}: track 0.00 -> 22.8 mm
- net +BATT: track 0.00 -> 19.6 mm
- net /Power/~{CHG}: track 0.00 -> 19.0 mm
- net GND: track 0.00 -> 8.93 mm, vias 0 -> 2
- net Net-(U7-ISET): track 0.00 -> 1.70 mm
- net Net-(U7-PRETERM): track 0.00 -> 1.63 mm
- net Net-(D1-A): track 0.00 -> 1.47 mm
- net Net-(D2-A): track 0.00 -> 1.47 mm
- net VBUS: track 0.00 -> 1.18 mm
Other:
- board outline added: 177.8 x 88.9 mm

Commit message: Continue with layout
Signed-off-by: Jan Hamal Dvořák <mordae@anilinux.org>
Parts:
- moved J1 244.2 mm to (223.0, 59.3)
- moved SW1 227.5 mm to (217.4, 51.4)
- moved R4 205.3 mm to (166.5, 87.4)
- moved R1 205.3 mm to (167.0, 82.7)
- moved R2 205.3 mm to (167.0, 85.2)
- moved C15 170.2 mm to (142.1, 69.1)
- moved C16 170.2 mm to (142.1, 71.1)
- moved C17 170.2 mm to (142.1, 73.0)
- moved C22 170.2 mm to (145.0, 69.1)
- moved C23 170.2 mm to (145.0, 71.1)
- moved R10 166.3 mm to (126.0, 94.0)
- moved R12 166.3 mm to (129.3, 93.7)
- moved U3 164.4 mm to (124.5, 86.4)
- moved C12 161.8 mm to (130.6, 85.1)
- moved C13 161.8 mm to (130.6, 87.1)
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Routing:
- net Net-(U2-VREG_VOUT): track 0.00 -> 15.8 mm
- net +3.3V: track 0.00 -> 11.0 mm, vias 0 -> 10
- net Net-(U3-VREG_VOUT): track 0.00 -> 10.8 mm
- net GND: vias 2 -> 20
- added copper zone on F.Cu, net +3.3V

Commit message: Add discrete antenna
Signed-off-by: Jan Hamal Dvořák <mordae@anilinux.org>
Parts:
- added AE1: Antenna, LCSC:ANT-TH_T14-433M, F.Cu at (55.9, 52.6)
- moved J4 40.7 mm to (55.9, 48.5), turned to 90 degrees
- moved C65 13.5 mm to (60.8, 52.6), turned to 0 degrees
- moved C39 1.78 mm to (55.4, 115.4)
- moved C37 1.52 mm to (59.9, 118.6)
Routing:
- net Net-(AE1-A): track 142.8 -> 0.00 mm
- added copper zone on B.Cu, net GND
- added copper zone on In1.Cu, net GND
Changed lines of the file:
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@@
   (net 31 "Net-(U11-DACVREF)")
   (net 32 "Net-(U13-RF_P)")
-  (net 33 "Net-(J4-In)")
+  (net 33 "Net-(AE1-A)")
   (net 34 "Net-(C65-Pad2)")
   (net 35 "Net-(U13-RF_N)")
@@
   )
   (footprint "Connector_Coaxial:U.FL_Hirose_U.FL-R-SMT-1_Vertical" (layer "F.Cu")
-    (at 96.52 48.26 180)
+    (at 55.86 48.548 90)
     (descr "Hirose U.FL Coaxial https://www.hirose.com/product/en/products/U.FL/U.FL-R-SMT-1%2810%29/")
     (tags "Hirose U.FL Coaxial")
@@
     (property "ki_keywords" "BNC SMA SMB SMC LEMO coaxial connector CINCH RCA")
     (attr smd)
-    (fp_text reference "J4" (at 0.475 4.015) (layer "F.SilkS")
+    (fp_text reference "J4" (at 0.475 3.175 90) (layer "F.SilkS")
         (effects (font (size 1 1) (thickness 0.15)))
     )
-    (fp_text value "U.FL" (at 0.475 3.2) (layer "F.Fab") hide
+    (fp_text value "U.FL" (at 0.475 3.2 90) (layer "F.Fab") hide
         (effects (font (size 1 1) (thickness 0.15)))
     )
-    (fp_text user "${REFERENCE}" (at 0.475 0 90) (layer "F.Fab")
+    (fp_text user "${REFERENCE}" (at 0.475 0) (layer "F.Fab")
         (effects (font (size 0.6 0.6) (thickness 0.09)))
     )
@@
     (fp_line (start 1.775 1.3) (end 1.375 1.3)
       (stroke (width 0.1) (type solid)) (layer "F.Fab"))
-    (pad "1" smd rect (at -1.05 0 180) (size 1.05 1) (layers "F.Cu" "F.Paste" "F.Mask")
-      (net 33 "Net-(J4-In)") (pinfunction "In") (pintype "passive"))
-    (pad "2" smd rect (at 0.475 -1.475 180) (size 2.2 1.05) (layers "F.Cu" "F.Paste" "F.Mask")
+    (pad "1" smd rect (at -1.05 0 90) (size 1.05 1) (layers "F.Cu" "F.Paste" "F.Mask")
+      (net 33 "Net-(AE1-A)") (pinfunction "In") (pintype "passive"))
+    (pad "2" smd rect (at 0.475 -1.475 90) (size 2.2 1.05) (layers "F.Cu" "F.Paste" "F.Mask")
       (net 2 "GND") (pinfunction "Ext") (pintype "passive"))
-    (pad "2" smd rect (at 0.475 1.475 180) (size 2.2 1.05) (layers "F.Cu" "F.Paste" "F.Mask")
+    (pad "2" smd rect (at 0.475 1.475 90) (size 2.2 1.05) (layers "F.Cu" "F.Paste" "F.Mask")
       (net 2 "GND") (pinfunction "Ext") (pintype "passive"))
     (model "${KICAD6_3DMODEL_DIR}/Connector_Coaxial.3dshapes/U.FL_Hirose_U.FL-R-SMT-1_Vertical.wrl"
@@
   )
   (footprint "Capacitor_SMD:C_0402_1005Metric" (layer "F.Cu")
-    (at 55.273 117.221)
+    (at 55.38 115.443)
     (descr "Capacitor SMD 0402 (1005 Metric), square (rectangular) end terminal, IPC_7351 nominal, (Body size source: IPC-SM-782 page 76, https://www.pcb-3d.com/wordpress/wp-content/uploads/ipc-sm-782a_amendment_1_and_2.pdf), generated with kicad-footprint-generator")
     (tags "capacitor")
@@
     )
   )
+  (footprint "LCSC:ANT-TH_T14-433M" (layer "F.Cu")
+    (at 55.86 52.578)
+    (property "LCSC Part" "C381188")
+    (property "Sheetfile" "radio.kicad_sch")
+    (property "Sheetname" "Radio")
+    (property "ki_description" "Antenna")
+    (property "ki_keywords" "antenna")
+    (attr through_hole)
+    (fp_text reference "AE1" (at 0 17.0665 90) (layer "F.SilkS")
+        (effects (font (size 1 1) (thickness 0.15)))
+    )
+    (fp_text value "Antenna" (at 0 4) (layer "F.Fab") hide
+        (effects (font (size 1 1) (thickness 0.15)))
+    )
+    (fp_text user "${REFERENCE}" (at 0 0) (layer "F.Fab")
+        (effects (font (size 1 1) (thickness 0.15)))
+    )
+    (fp_line (start -2.7 4.6) (end 2.7 4.6)
+      (stroke (width 0.25) (type solid)) (layer "F.SilkS"))
+    (fp_line (start -2.7 28.4) (end -2.7 4.6)
+      (stroke (width 0.25) (type solid)) (layer "F.SilkS"))
+    (fp_line (start 2.7 4.6) (end 2.7 4.7)
+      (stroke (width 0.25) (type solid)) (layer "F.SilkS"))
+    (fp_line (start 2.7 4.7) (end 2.7 28.4)
+      (stroke (width 0.25) (type solid)) (layer "F.SilkS"))
+    (fp_line (start 2.7 28.4) (end -2.7 28.4)
+      (stroke (width 0.25) (type solid)) (layer "F.SilkS"))
+    (fp_circle (center 0 0) (end 0.25 0)
+      (stroke (width 0.5) (type solid)) (fill none) (layer "F.Fab"))
+    (fp_circle (center 2.3 -0.5) (end 2.33 -0.5)
+      (stroke (width 0.06) (type solid)) (fill none) (layer "F.Fab"))
+    (pad "1" thru_hole circle (at 0 0 270) (size 2.5 2.5) (drill 1.599997) (layers "*.Cu" "*.Mask")
+      (net 33 "Net-(AE1-A)") (pinfunction "A") (pintype "input"))
+    (model "${KIPRJMOD}/LCSC.3dshapes/ANT-TH_BD4.6-L27.9.wrl"
+      (offset (xyz 0 0 3))
+      (scale (xyz 1 1 1))
+      (rotate (xyz 0 0 0))
+    )
+  )
   (footprint "Package_TO_SOT_SMD:SOT-23" (layer "F.Cu")
     (at 62.1815 93.091)
@@
   )
   (footprint "Capacitor_Tantalum_SMD:CP_EIA-3528-21_Kemet-B" (layer "F.Cu")
-    (at 58.9395 119.761)
+    (at 59.9375 118.618)
     (descr "Tantalum Capacitor SMD Kemet-B (3528-21 Metric), IPC_7351 nominal, (Body size from: http://www.kemet.com/Lists/ProductCatalog/Attachments/253/KEM_TC101_STD.pdf), generated with kicad-footprint-generator")
     (tags "capacitor tantalum")
@@
   )
   (footprint "Capacitor_SMD:C_0402_1005Metric" (layer "F.Cu")
-    (at 71.545 60.695001 90)
+    (at 60.785 52.578)
     (descr "Capacitor SMD 0402 (1005 Metric), square (rectangular) end terminal, IPC_7351 nominal, (Body size source: IPC-SM-782 page 76, https://www.pcb-3d.com/wordpress/wp-content/uploads/ipc-sm-782a_amendment_1_and_2.pdf), generated with kicad-footprint-generator")
     (tags "capacitor")
@@
     (property "ki_keywords" "capacitor cap")
     (attr smd)
-    (fp_text reference "C65" (at 0 -1.16 90) (layer "F.SilkS")
+    (fp_text reference "C65" (at 0 -1.16) (layer "F.SilkS")
         (effects (font (size 0.8 0.8) (thickness 0.15)))
     )
-    (fp_text value "220p" (at 0 1.16 90) (layer "F.Fab") hide
+    (fp_text value "220p" (at 0 1.16) (layer "F.Fab") hide
         (effects (font (size 1 1) (thickness 0.15)))
     )
-    (fp_text user "${REFERENCE}" (at 0 0 90) (layer "F.Fab")
+    (fp_text user "${REFERENCE}" (at 0 0) (layer "F.Fab")
         (effects (font (size 0.8 0.8) (thickness 0.15)))
     )
@@
     (fp_line (start 0.5 0.25) (end -0.5 0.25)
       (stroke (width 0.1) (type solid)) (layer "F.Fab"))
-    (pad "1" smd roundrect (at -0.48 0 90) (size 0.56 0.62) (layers "F.Cu" "F.Paste" "F.Mask") (roundrect_rratio 0.25)
-      (net 33 "Net-(J4-In)") (pintype "passive"))
-    (pad "2" smd roundrect (at 0.48 0 90) (size 0.56 0.62) (layers "F.Cu" "F.Paste" "F.Mask") (roundrect_rratio 0.25)
+    (pad "1" smd roundrect (at -0.48 0) (size 0.56 0.62) (layers "F.Cu" "F.Paste" "F.Mask") (roundrect_rratio 0.25)
+      (net 33 "Net-(AE1-A)") (pintype "passive"))
+    (pad "2" smd roundrect (at 0.48 0) (size 0.56 0.62) (layers "F.Cu" "F.Paste" "F.Mask") (roundrect_rratio 0.25)
       (net 34 "Net-(C65-Pad2)") (pintype "passive"))
     (model "${KICAD6_3DMODEL_DIR}/Capacitor_SMD.3dshapes/C_0402_1005Metric.wrl"
@@
     )
   )
-  (gr_arc (start 63.5 125.73) (mid 55.417769 122.382231) (end 52.07 114.3)
-    (stroke (width 1) (type default)) (layer "F.Cu"))
-  (gr_arc (start 52.07 50.8) (mid 55.417769 42.717769) (end 63.5 39.37)
-    (stroke (width 1) (type default)) (layer "F.Cu"))
   (gr_arc (start 215.9 38.1) (mid 224.880256 41.819744) (end 228.6 50.8)
     (stroke (width 0.1) (type default)) (layer "Edge.Cuts"))
@@
   (segment (start 137.332 122.219) (end 137.414 122.301) (width 0.127) (layer "F.Cu") (net 10))
   (segment (start 136.271 122.219) (end 137.332 122.219) (width 0.25) (layer "F.Cu") (net 10))
-  (segment (start 62.23 39.37) (end 97.79 39.37) (width 1) (layer "F.Cu") (net 33))
-  (segment (start 100.33 46.99) (end 99.06 48.26) (width 1) (layer "F.Cu") (net 33))
-  (segment (start 100.33 41.91) (end 100.33 46.99) (width 1) (layer "F.Cu") (net 33))
-  (segment (start 97.79 39.37) (end 100.33 41.91) (width 1) (layer "F.Cu") (net 33))
-  (segment (start 62.23 125.73) (end 91.44 125.73) (width 1) (layer "F.Cu") (net 33))
-  (segment (start 52.07 49.53) (end 52.07 115.57) (width 1) (layer "F.Cu") (net 33))
-  (segment (start 99.06 48.26) (end 97.57 48.26) (width 1) (layer "F.Cu") (net 33))
   (segment (start 135.471 125.184) (end 136.017 125.73) (width 0.127) (layer "F.Cu") (net 49))
   (segment (start 147.32 122.809) (end 147.32 119.253) (width 0.127) (layer "F.Cu") (net 49))
@@
       )
     )
+  )
+  (zone (net 0) (net_name "") (layers "F.Cu" "In1.Cu" "In2.Cu" "B.Cu") (name "antenna") (hatch edge 0.5)
+    (connect_pads (clearance 0))
+    (min_thickness 0.25) (filled_areas_thickness no)
+    (keepout (tracks allowed) (vias allowed) (pads allowed) (copperpour not_allowed) (footprints allowed))
+    (fill (thermal_gap 0.5) (thermal_bridge_width 0.5))
+    (polygon
+      (pts
+        (xy 50.78 86.233)
+        (xy 60.94 86.233)
+        (xy 60.94 54.483)
+        (xy 50.78 54.483)
+      )
+    )
+  )
+  (zone (net 2) (net_name "GND") (layers "In1.Cu" "B.Cu") (name "GND") (hatch edge 0.5)
+    (priority 2)
+    (connect_pads (clearance 0.128))
+    (min_thickness 0.128) (filled_areas_thickness no)
+    (fill yes (thermal_gap 0.5) (thermal_bridge_width 0.5))
+    (polygon
+      (pts
+        (xy 48.875 37.338)
+        (xy 229.215 37.338)
+        (xy 229.215 128.143)
+        (xy 48.875 128.143)
+      )
+    )

Commit message: PCB layout progress
Signed-off-by: Jan Hamal Dvořák <mordae@anilinux.org>
Parts:
- added C82: 10u, Capacitor_SMD:C_0402_1005Metric, F.Cu at (75.5, 106.1)
- moved Q6 102.6 mm to (158.4, 87.8), turned to 180 degrees
- moved R26 100.7 mm to (157.0, 95.8)
- moved Q4 97.6 mm to (154.0, 87.8), turned to 180 degrees
- moved R17 96.7 mm to (153.8, 95.8), turned to 180 degrees
- moved C36 92.8 mm to (154.0, 98.9)
- moved Q5 91.8 mm to (158.4, 92.6), turned to 180 degrees
- moved R18 88.1 mm to (149.4, 88.1), turned to 180 degrees
- moved R20 88.0 mm to (147.3, 101.1)
- moved R16 87.9 mm to (144.1, 95.9)
- moved Q3 87.5 mm to (154.0, 92.6)
- moved R15 87.0 mm to (145.4, 95.9), turned to 90 degrees
- moved C35 86.7 mm to (144.8, 112.1), turned to -90 degrees
- moved R14 85.9 mm to (146.7, 95.9)
- moved C38 83.4 mm to (147.3, 103.9), turned to -90 degrees
- moved Q1 82.9 mm to (149.5, 92.6)
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Connections:
- SPK1 pad 2: Net-(U12-OUT+) -> Net-(U12-OUT-)
- U12 pad B1: Net-(U12-OUT+) -> Net-(SPK1-+)
- U12 pad C1: Net-(SPK1-+) -> Net-(U12-OUT-)
Routing:
- net GND: vias 20 -> 29

Commit message: Further progress with the PCB layout
Signed-off-by: Jan Hamal Dvořák <mordae@anilinux.org>
Parts:
- moved R10 62.8 mm to (168.9, 48.1), turned to -90 degrees
- moved R12 58.4 mm to (165.8, 48.1), turned to -90 degrees
- moved R2 53.6 mm to (115.0, 72.3), turned to 180 degrees
- moved R1 52.8 mm to (115.0, 73.8), turned to 180 degrees
- moved R14 34.3 mm to (117.6, 77.7), turned to 90 degrees
- moved R15 32.4 mm to (118.6, 77.7), turned to -90 degrees
- moved C23 31.3 mm to (114.1, 66.2)
- moved R16 30.5 mm to (119.6, 77.7), turned to 90 degrees
- moved C16 29.6 mm to (120.8, 91.5), turned to -90 degrees
- moved C22 29.1 mm to (119.3, 82.7), turned to 180 degrees
- moved R3 25.7 mm to (104.8, 64.0), turned to -90 degrees
- moved C19 22.1 mm to (119.7, 91.5), turned to -90 degrees
- moved C17 21.1 mm to (129.6, 90.0)
- moved C15 20.1 mm to (125.2, 79.9), turned to 90 degrees
- moved C8 20.1 mm to (105.5, 85.2), turned to -90 degrees
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Connections:
- net /Power/USB_{D+} renamed /Power/USB+
- net /Power/USB_{D-} renamed /Power/USB-
Routing:
- net /Power/CC1: track 0.00 -> 71.6 mm, vias 0 -> 2
- net /Power/CC2: track 0.00 -> 68.5 mm, vias 0 -> 2
- net /Audio/HP_{SENSE}: track 0.00 -> 53.9 mm
- net /RP2040/T_{MOSI}: track 0.00 -> 30.4 mm, vias 0 -> 1
- net /RP2040/T_{SCK}: track 0.00 -> 28.8 mm, vias 0 -> 1
- net /RP2040/T_{MISO}: track 0.00 -> 25.0 mm, vias 0 -> 1
- net /RP2040/T_{IRQ}: track 0.00 -> 25.0 mm, vias 0 -> 1
- net /RP2040/TFT_{CS}: track 0.00 -> 23.3 mm
- net /RP2040/T_{CS}: track 0.00 -> 23.2 mm, vias 0 -> 1
- net /RP2040/TFT_{RS}: track 0.00 -> 22.0 mm
- net /RP2040/TFT_{RST}: track 0.00 -> 18.6 mm, vias 0 -> 1
- net /RP2040/TFT_{MOSI}: track 0.00 -> 18.5 mm
- net /RP2040/QSPI_SD0: track 0.00 -> 16.0 mm
- net /RP2040/TFT_{MISO}: track 0.00 -> 16.0 mm
- net /RP2040/QSPI_SD3: track 0.00 -> 15.4 mm
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