File: hw/krecek-0.9/krecek-0.9.kicad_pcb (KiCad board)
At the start: 4 copper layers, 177.8 x 88.9 mm, 168 parts, among them CN1 PJ-313B6-B, J1 DAP, J2 AUX, J3 USB_C_Receptacle_USB2.0, J4 U.FL, J5 Micro_SD_Card_Det1, Q1 AO3401A, Q2 AO3401A, Q3 AO3400A, Q4 AO3400A, Q5 AO3400A, Q6 AO3400A, Q7 PT334, Q8 AO3400A, SW1 SW_Push, SW5 TM-2023, U1 Display, U10 TPS63000, U11 ES8312, U12 TPA2028D1YZFT, U13 CC1101RGPR, U2 RP2040, U3 RP2040, U4 W25Q128JVS, U5 AMS1117-3.3, U6 JST-PH-2P, U7 BQ24045DSQR, U8 AMS1117-3.3, U9 AMS1117-3.3, Y1 12MHz

Commit message: Progress on PCB
Signed-off-by: Jan Hamal Dvořák <mordae@anilinux.org>
Parts:
- removed C40, C42, C44, C45: 10u, Capacitor_SMD:C_0402_1005Metric
- moved SW1 160.9 mm to (56.5, 53.5)
- moved J1 116.9 mm to (125.2, 123.4), turned to -90 degrees
- moved C50 87.4 mm to (124.1, 51.7), turned to 180 degrees
- moved C46 84.9 mm to (132.0, 50.6), turned to -90 degrees
- moved R31 84.2 mm to (126.5, 51.7), turned to 0 degrees
- moved R30 81.0 mm to (140.2, 53.3)
- moved R32 81.0 mm to (143.5, 53.3), turned to -90 degrees
- moved R29 81.0 mm to (136.9, 53.3), turned to -90 degrees
- moved Q8 69.6 mm to (142.9, 57.7)
- moved R4 64.5 mm to (106.4, 64.0), turned to 90 degrees
- moved C73 42.8 mm to (191.7, 60.7), turned to 180 degrees
- moved C31 40.5 mm to (70.0, 117.1)
- moved U8 40.5 mm to (63.0, 117.5)
- moved C30 40.5 mm to (70.2, 119.4)
- moved C70 40.4 mm to (91.3, 84.1)
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Connections:
- D4 pad 2: +5V -> Net-(D4-A)
- D5 pad 1: Net-(D5-K) -> Net-(D4-A)
- D5 pad 2: Net-(D4-K) -> +5V
- R29 pad 1: Net-(D5-K) -> Net-(D4-K)
- U1 pad 7: /RP2040/TFT_{MISO} -> /RP2040/TFT_{SCK}
- U13 pad 1: /RP2040/TFT_{MISO} -> /RP2040/TFT_{SCK}
- U2 pad 4: /RP2040/TFT_{MISO} -> /RP2040/TFT_{SCK}
- U3 pad 36: /Inputs/BTN_{X} -> /Inputs/BTN_{Y}
- U3 pad 37: /Inputs/BTN_{Y} -> /Inputs/BTN_{X}
- U3 pad 38: /Inputs/JOY_{X} -> /Inputs/BRACK_{R}
- U3 pad 39: /Inputs/JOY_{Y} -> /Inputs/BRACK_{L}
- U3 pad 40: /Inputs/BRACK_{L} -> /Inputs/JOY_{X}
- U3 pad 41: /Inputs/BRACK_{R} -> /Inputs/JOY_{Y}
Routing:
- net /Audio/CDATA: track 0.00 -> 116.5 mm, vias 0 -> 2
- net /Audio/CCLK: track 0.00 -> 109.0 mm, vias 0 -> 2
- net /Inputs/BTN_{Y}: track 0.00 -> 108.5 mm, vias 0 -> 2
- net /Inputs/VOL_{UP}: track 0.00 -> 103.5 mm
- net /Inputs/JOY_{Y}: track 0.00 -> 101.8 mm
- net GND: track 16.0 -> 114.4 mm, vias 33 -> 121
- net Net-(Q7-C): track 0.00 -> 98.4 mm, vias 0 -> 2
- net /Audio/ADC: track 0.00 -> 96.5 mm, vias 0 -> 2
- net /Audio/HP_{SENSE}: track 53.9 -> 148.9 mm, vias 0 -> 5
- net /Inputs/JOY_{X}: track 0.00 -> 94.3 mm
- net /Audio/HP_{LEFT}: track 0.00 -> 94.0 mm, vias 0 -> 2
- net /Audio/DAC: track 0.00 -> 93.7 mm, vias 0 -> 2
- net /Audio/SCLK: track 0.00 -> 93.6 mm, vias 0 -> 2
- net /Inputs/VOL_{SW}: track 0.00 -> 93.4 mm, vias 0 -> 4
- net /Audio/LRCK: track 0.00 -> 92.8 mm, vias 0 -> 2
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- added copper zone on F.Cu, net +3.3VA
- added copper zone on F.Cu, net +3.3VSD

Commit message: Further progress on routing the PCB
Signed-off-by: Jan Hamal Dvořák <mordae@anilinux.org>
Parts:
- moved C58 11.8 mm to (178.2, 102.8), turned to 90 degrees
- moved C59 10.1 mm to (179.2, 102.8), turned to 90 degrees
- moved C60 10.0 mm to (180.2, 102.8), turned to 90 degrees
- moved C31 8.46 mm to (63.2, 112.1), turned to 180 degrees
- moved R20 7.38 mm to (144.9, 108.1), turned to 180 degrees
- moved C38 5.72 mm to (144.9, 109.1), turned to 0 degrees
- moved R27 3.32 mm to (144.4, 105.3)
- moved C30 3.04 mm to (68.8, 122.1), turned to -90 degrees
- moved U8 1.22 mm to (64.1, 118.0), turned to 90 degrees
- moved C35 0.61 mm to (144.4, 111.6), turned to 180 degrees
- moved R13 0.50 mm to (156.0, 118.3)
- moved C41 0.25 mm to (181.7, 105.6)
Connections:
- net Net-(Q1-D) renamed /Power/vin
- net Net-(U10-EN) renamed /Power/vina
Routing:
- net /RP2040/AUX0: track 0.00 -> 147.6 mm, vias 0 -> 1
- net /RP2040/AUX1: track 0.00 -> 146.5 mm, vias 0 -> 1
- net /RP2040/AUX2: track 0.00 -> 142.2 mm, vias 0 -> 1
- net /RP2040/AUX3: track 6.48 -> 141.4 mm, vias 0 -> 1
- net /RP2040/TFT_{LED}: track 7.36 -> 74.8 mm, vias 0 -> 3
- net /RP2040/AUX7: track 0.00 -> 63.6 mm
- net /Power/OFF: track 0.00 -> 57.1 mm, vias 0 -> 2
- net /RP2040/AUX6: track 0.00 -> 55.5 mm
- net /RP2040/AUX4: track 0.00 -> 52.0 mm
- net /RP2040/AUX5: track 0.00 -> 50.9 mm, vias 0 -> 1
- net GND: track 114.4 -> 162.3 mm, vias 121 -> 156
- net /Power/ON: track 0.00 -> 26.6 mm
- net Net-(U2-GPIO24): track 45.0 -> 26.2 mm
- net Net-(U2-GPIO25): track 41.5 -> 23.6 mm
- net Net-(U11-OUTN): track 0.00 -> 17.9 mm, vias 0 -> 2
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- added copper zone on F.Cu, net +5V
- added copper zone on F.Cu, net /Power/vin
- added copper zone on F.Cu, net /Power/vina
