File: hw/krecek-0.9/krecek-0.9.kicad_pcb (KiCad board)
At the start: 4 copper layers, 152.4 x 63.5 mm, 178 parts, among them CN1 PJ-313B6-B, J1 DAP, J2 AUX, J3 USB_C_Receptacle_USB2.0, J4 U.FL, J5 Micro_SD_Card_Det1, Q1 AO3401A, Q2 AO3401A, Q3 AO3400A, Q4 PT334, Q5 AO3400A, Q6 AO3400A, SW1 SW_Push, SW5 TM-2023, U1 RP2040, U10 ES8312, U11 PAM8302AASCR, U12 CC1101RGPR, U13 FlatJoyCon, U14 TSC2046EIRGVR, U2 RP2040, U3 W25Q128JVS, U4 AMS1117-3.3, U5 JST-PH-2P, U6 BQ24040DSQR, U7 AMS1117-3.3, U8 AMS1117-3.3, U9 TPS63000, Y1 12MHz

Commit message: hw: work on new board revision
Parts:
- added R41: 1M, Resistor_SMD:R_0402_1005Metric, F.Cu at (115.9, 45.2)
- added REF**: Panel, Krecek:Panel, B.Cu at (131.4, 71.1)
- U5: moved to F.Cu
- moved D3 125.1 mm to (356.5, 26.5), turned to 180 degrees
- moved C77 123.6 mm to (121.9, 70.0), turned to -90 degrees
- moved C34 113.7 mm to (339.8, 17.4)
- moved C37 113.7 mm to (363.1, 60.6)
- moved JP2 113.7 mm to (345.7, 58.8)
- moved Q1 113.7 mm to (358.6, 54.3)
- moved Q2 113.7 mm to (354.2, 54.3)
- moved Q3 113.7 mm to (363.1, 54.3)
- moved R16 113.7 mm to (361.4, 40.3)
- moved R21 113.7 mm to (336.0, 34.7)
- moved R28 113.7 mm to (362.9, 57.4)
- moved U9 113.7 mm to (331.3, 34.5)
- moved C35 113.7 mm to (325.9, 37.5)
- moved C36 113.7 mm to (335.5, 38.2)
- moved C38 113.7 mm to (330.9, 38.2)
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Connections:
- J2 pad 11: /RP2040/AUX6 -> /RP2040/AUX5
- J2 pad 12: /RP2040/AUX2 -> /RP2040/AUX4
- J2 pad 14: /RP2040/AUX3 -> /RP2040/AUX6
- J2 pad 5: /RP2040/AUX4 -> /RP2040/AUX1
- J2 pad 7: /RP2040/AUX5 -> /RP2040/AUX3
- J2 pad 8: /RP2040/AUX1 -> /RP2040/AUX2
- R40 pad 2: /RP2040/AUX0 -> Net-(R40-Pad2)
Routing:
- net Net-(Q4-C): track 1.91 -> 62.0 mm
- net /Power/USB-: track 85.1 -> 115.8 mm
- net /Display/TOUCH_{CS}: track 0.94 -> 29.5 mm, vias 1 -> 2
- net /Power/USB+: track 86.0 -> 112.4 mm
- net /Display/TOUCH_{MOSI}: track 0.86 -> 27.1 mm, vias 1 -> 2
- net /Display/TOUCH_{SCLK}: track 0.86 -> 26.6 mm, vias 1 -> 2
- net +3.3VSD: track 1.69 -> 24.4 mm
- net /RP2040/AUX5: track 2.57 -> 21.7 mm, vias 1 -> 0
- net /RP2040/AUX3: track 2.67 -> 19.5 mm, vias 1 -> 0
- net /RP2040/AUX1: track 5.00 -> 21.5 mm, vias 1 -> 0
- net /RP2040/AUX4: track 2.39 -> 18.8 mm, vias 1 -> 0
- net /RP2040/AUX0: track 5.46 -> 20.5 mm, vias 1 -> 0
- net /RP2040/AUX2: track 2.56 -> 16.6 mm, vias 1 -> 0
- net /RP2040/AUX7: track 2.50 -> 14.5 mm, vias 1 -> 0
- net GND: track 88.4 -> 99.4 mm, vias 95 -> 109
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- added copper zone on F.Cu, net Net-(R40-Pad2)

Commit message: hw: work on new board revision
Parts:
- moved JP1 83.2 mm to (81.9, 46.4), turned to 180 degrees
- moved C44 77.1 mm to (162.7, 41.9)
- moved R29 76.1 mm to (162.2, 40.4), turned to 0 degrees
- moved R14 66.8 mm to (88.6, 49.0)
- moved FB1 66.8 mm to (97.0, 41.8)
- moved R13 66.8 mm to (91.9, 49.0)
- moved J3 66.8 mm to (90.7, 43.2)
- moved CN1 64.9 mm to (156.3, 44.9)
- moved C70 2.73 mm to (86.9, 72.4)
- moved C42 1.11 mm to (149.1, 86.8), turned to 135 degrees
- moved REF** 0.64 mm to (132.1, 71.1)
Connections:
- U1 pad 17: /Audio/DAC -> /Audio/ADC
- U1 pad 18: /Audio/ADC -> /Audio/DAC
Routing:
- net /Power/USB-: track 115.8 -> 38.2 mm, vias 2 -> 0
- net /Power/USB+: track 112.4 -> 40.3 mm, vias 2 -> 0
- net /Audio/HP_{RIGHT}: track 1.89 -> 73.2 mm
- net /Audio/LRCK: track 3.25 -> 73.4 mm, vias 1 -> 2
- net /Audio/HP_{LEFT}: track 1.89 -> 68.4 mm
- net /Audio/SCLK: track 3.42 -> 66.3 mm, vias 1 -> 2
- net /Audio/DAC: track 3.62 -> 61.9 mm, vias 1 -> 2
- net /Audio/ADC: track 3.81 -> 58.4 mm, vias 1 -> 2
- net /Power/USB_{CC1}: track 81.4 -> 30.7 mm, vias 2 -> 0
- net /Power/USB_{CC2}: track 82.0 -> 31.9 mm
- net /Audio/CCLK: track 3.52 -> 51.2 mm, vias 1 -> 2
- net /Audio/CDATA: track 3.42 -> 49.4 mm, vias 1 -> 2
- net Net-(J1-Pin_1): track 3.94 -> 5.73 mm
- net GND: track 99.4 -> 98.0 mm, vias 109 -> 118
- net /Audio/HP_{SENSE}: track 8.21 -> 9.39 mm
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
Commit message: Progress on HW design
Parts:
- removed the C44 at (162.7, 41.9)
- removed C49: 1u, Capacitor_SMD:C_0402_1005Metric
- removed the C51 at (151.6, 82.7)
- removed the C54 at (157.5, 85.7)
- removed the C55 at (157.5, 86.8)
- removed REF**: Panel, Krecek:Panel
- removed the U11 at (150.2, 91.9)
- added C50: 47u, Capacitor_SMD:C_0805_2012Metric, F.Cu at (159.6, 88.9)
- added TFT1: Panel, Krecek:Panel, B.Cu at (132.1, 71.1)
- C48: value 1u -> 47u; footprint Capacitor_SMD:C_0402_1005Metric -> Capacitor_SMD:C_0805_2012Metric
- C52, C53: value 1u -> 4.7u
- R35: renamed from R29; value 3.3k -> 2.2k
- U10: value ES8312 -> NAU88C22YG; footprint LCSC:VQFN-28_L4.0-W4.0-P0.45-TL-EP2.6 -> LCSC:QFN-32_L5.0-W5.0-P0.50-BL-EP2.7
- moved C43 11.1 mm to (146.4, 76.0)
- moved C52 9.90 mm to (158.8, 90.4), turned to 180 degrees
- moved C48 6.67 mm to (159.6, 86.9), turned to 0 degrees
- moved U10 1.06 mm to (153.0, 87.7), turned to 180 degrees
- moved C53 0.88 mm to (156.6, 84.6), turned to -90 degrees
- renumbered C43 to C41, C41 to C42, C42 to C43, C45 to C44, C46 to C45, C47 to C46, C50 to C51, C56 to C54, C57 to C55, C58 to C56, C59 to C57, C60 to C58, C61 to C59, C62 to C60, C63 to C61, C64 to C62, C65 to C63, C66 to C64, C67 to C65, C68 to C66, C69 to C67, C70 to C68, C71 to C69, C72 to C70, C73 to C71, C74 to C72, C75 to C73, C76 to C74, C77 to C75, C78 to C76, C79 to C77, C80 to C78, H1 to H2, H2 to H3, H3 to H4, H4 to H5, H5 to H6, H6 to H7, H7 to H8, H8 to H9, R8 to R10, R9 to R11, R10 to R12, R11 to R13, R12 to R14, R13 to R15, R14 to R16, R15 to R17, R16 to R18, R17 to R19, R18 to R20, R19 to R21, R20 to R22, R21 to R23, R22 to R24, R23 to R25, R24 to R26, R25 to R27, R26 to R28, R27 to R29, R28 to R30, R30 to R31, R31 to R32, R32 to R33, R33 to R34, R34 to R36, R35 to R37, R36 to R38, R37 to R39, R40 to R4, R38 to R40, R39 to R41, R41 to R5, R4 to R6, R5 to R7, R6 to R8, R7 to R9, U12 to U11, U13 to U12, U14 to U13
Connections:
- C48 pad 1: Net-(U10-OUTP) -> Net-(U10-LHP)
- C51 pad 1: +3.3V -> +5V
- C52 pad 2: Net-(U10-MIC1N) -> Net-(U10-VREF)
- C53 pad 1: Net-(U10-VMID) -> GND
- C53 pad 2: GND -> Net-(U10-MICBIAS)
- R35 pad 2: +3.3VA -> Net-(U10-MICBIAS)
- SPK1 pad 2: Net-(U11-VO-) -> Net-(U10-RSPKOUT)
- U10 pad 1: GND -> /Audio/IR+
- U10 pad 10: /Audio/LRCK -> /Audio/DAC
- U10 pad 11: /Audio/DAC -> /Audio/SCLK
- U10 pad 12: unconnected-(U10-NC-Pad12) -> GND
- U10 pad 13: unconnected-(U10-MONOOUT-Pad13) -> +3.3V
- U10 pad 14: GND -> +3.3V
- U10 pad 15: +3.3VA -> unconnected-(U10-CSB/GPIO1-Pad15)
- U10 pad 16: Net-(U10-OUTP) -> /Audio/CCLK
- U10 pad 17: Net-(U10-OUTN) -> /Audio/CDATA
- U10 pad 18: Net-(U10-DACVREF) -> GND
- U10 pad 19: Net-(U10-ADCVREF) -> unconnected-(U10-LAUXIN-Pad19)
- U10 pad 2: /Audio/CDATA -> /Audio/IR-
- U10 pad 20: Net-(U10-VMID) -> unconnected-(U10-RAUXIN-Pad20)
- U10 pad 22: /Audio/IR- -> unconnected-(U10-AUXOUT2-Pad22)
- U10 pad 23: /Audio/IR+ -> Net-(U10-RSPKOUT)
- U10 pad 24: Net-(U10-MIC1N) -> GND
- U10 pad 25: Net-(U10-MIC1P/DMIC_SDA) -> Net-(SPK1-+)
- U10 pad 26: unconnected-(U10-MUTE/DMIC_SCL-Pad26) -> +5V
- U10 pad 27: unconnected-(U10-NC-Pad27) -> Net-(U10-VREF)
- U10 pad 28: unconnected-(U10-NC-Pad28) -> GND
- U10 pad 29: GND -> Net-(U10-RHP)
- U10 pad 3: /Audio/CCLK -> unconnected-(U10-LLIN/GPIO2-Pad3)
- U10 pad 4: unconnected-(U10-MCLK-Pad4) -> Net-(U10-RMICP)
- U10 pad 5: +3.3V -> Net-(U10-RMICN)
- U10 pad 6: +3.3V -> unconnected-(U10-RLIN/GPIO3-Pad6)
- U10 pad 7: GND -> /Audio/LRCK
- U2 pad 29: /Audio/AMP_{EN} -> unconnected-(U2-GPIO18-Pad29)
Routing:
- net /Audio/HP_{LEFT}: track 68.4 -> 11.6 mm
- net /Audio/HP_{RIGHT}: track 73.2 -> 24.4 mm
- net /Audio/DAC: track 61.9 -> 17.4 mm
- net /Audio/SCLK: track 66.3 -> 23.3 mm
- net /Audio/ADC: track 58.4 -> 16.1 mm
- net /Audio/LRCK: track 73.4 -> 32.6 mm
- net /Audio/CCLK: track 51.2 -> 11.6 mm
- net /Audio/CDATA: track 49.4 -> 11.6 mm
- net Net-(U11-VO-): track 18.0 -> 0.00 mm
- net GND: track 98.0 -> 83.0 mm, vias 118 -> 108
- net Net-(U10-RSPKOUT): track 0.00 -> 10.4 mm
- net Net-(U10-OUTN): track 8.69 -> 0.00 mm
- net Net-(U10-OUTP): track 6.48 -> 0.00 mm
- net Net-(SPK1-+): track 4.83 -> 0.00 mm
- net Net-(U10-VMID): track 3.00 -> 0.00 mm
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
Commit message: Work on board layout
Parts:
- removed C45: 1u, Capacitor_SMD:C_0402_1005Metric
- removed C58: 3.3p, Capacitor_SMD:C_0402_1005Metric
- removed C59, C64: 220p, Capacitor_SMD:C_0402_1005Metric
- removed C60, C62: 4.7p, Capacitor_SMD:C_0402_1005Metric
- removed C61: 10p, Capacitor_SMD:C_0402_1005Metric
- removed FB1: 600Ω @ 100 MHz, Inductor_SMD:L_0805_2012Metric
- removed JP1: Jumper_2_Bridged, Jumper:SolderJumper-2_P1.3mm_Bridged_RoundedPad1.0x1.5mm
- removed JP2: Jumper_3_Bridged12, Jumper:SolderJumper-3_P1.3mm_Bridged12_RoundedPad1.0x1.5mm
- removed L2, L3, L4, L5: 27n, Inductor_SMD:L_0402_1005Metric
- added C47: 1u, Capacitor_SMD:C_0402_1005Metric, F.Cu at (155.4, 83.5)
- added C49: 1u, Capacitor_SMD:C_0402_1005Metric, F.Cu at (156.5, 83.5)
- added U14: BW21S5011A01TF, LCSC:FILTER-SMD_4P-L2.0-W1.2-BL-1, F.Cu at (63.1, 79.6)
- moved C37 76.8 mm to (286.3, 61.2)
- moved D3 76.8 mm to (279.8, 27.1)
- moved Q1 76.8 mm to (281.9, 54.9)
- moved Q2 76.8 mm to (277.4, 54.9)
- moved Q3 76.8 mm to (286.3, 54.9)
- moved R18 76.8 mm to (284.6, 41.0)
- moved R23 76.8 mm to (259.2, 35.3)
- moved R30 76.8 mm to (286.2, 58.1)
- moved U9 76.8 mm to (254.5, 35.2)
- moved C35 76.8 mm to (249.1, 38.1)
- moved C36 76.8 mm to (258.7, 38.9)
- moved C38 76.8 mm to (254.1, 38.9)
- moved C39 76.8 mm to (259.2, 36.3)
- moved C40 76.8 mm to (264.6, 40.0)
- moved L1 76.8 mm to (251.1, 35.2)
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- renumbered H2 to H1, H3 to H2, H4 to H3, H5 to H4, H6 to H5, H7 to H6, H8 to H7, H9 to H8
Connections:
- C29 pad 1: Net-(JP1-B) -> VBUS
- C36 pad 2: /Power/tps63000_vout -> +5V
- C38 pad 1: /Power/tps63000_vout -> +5V
- C40 pad 2: /Power/tps63000_vout -> +5V
- C44 pad 1: +3.3VA -> Net-(Q4-C)
- C44 pad 2: /Audio/IR+ -> /Audio/IR
- J3 pad S1: Net-(J3-SHIELD) -> GND
- R28 pad 2: /Power/tps63000_vout -> +5V
- U10 pad 1: /Audio/IR+ -> unconnected-(U10-LMICP-Pad1)
- U10 pad 19: unconnected-(U10-LAUXIN-Pad19) -> /Audio/IR
- U10 pad 2: /Audio/IR- -> unconnected-(U10-LMICN-Pad2)
- U6 pad 1: Net-(JP1-B) -> VBUS
- U9 pad 1: /Power/tps63000_vout -> +5V
Routing:
- net /Audio/HP_{SENSE}: track 9.39 -> 137.3 mm, vias 0 -> 1
- net /Display/TOUCH_{MOSI}: track 27.1 -> 88.6 mm, vias 2 -> 3
- net /RP2040/RF_{CS}: track 1.05 -> 56.2 mm, vias 1 -> 2
- net /Display/TOUCH_{SCLK}: track 26.6 -> 74.4 mm, vias 2 -> 3
- net /Display/TOUCH_{MISO}: track 1.45 -> 48.4 mm, vias 1 -> 2
- net /Audio/SCLK: track 23.3 -> 67.9 mm
- net /Audio/DAC: track 17.4 -> 58.7 mm
- net /Audio/LRCK: track 32.6 -> 72.9 mm
- net /Audio/ADC: track 16.1 -> 56.1 mm
- net +3.3VA: track 1.14 -> 34.4 mm, vias 0 -> 2
- net /Audio/HP_{RIGHT}: track 24.4 -> 0.00 mm
- net /Audio/IR: track 0.00 -> 15.8 mm, vias 0 -> 2
- net /RP2040/RF_{XOSC}: track 55.1 -> 65.0 mm
- net GND: track 83.0 -> 90.6 mm, vias 108 -> 115
- net Net-(Q4-C): track 62.0 -> 55.5 mm
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- added copper zone on F.Cu, net GND
