File: hw/krecek-0.9/krecek-0.9.kicad_pcb (KiCad board)
At the start: 4 copper layers, 152.4 x 63.5 mm, 164 parts, among them CN1 PJ-313B6-B, J1 DAP, J2 AUX, J3 USB_C_Receptacle_USB2.0, J4 U.FL, J5 Micro_SD_Card_Det1, Q1 AO3401A, Q2 AO3401A, Q3 AO3400A, Q4 PT334, Q5 AO3400A, Q6 AO3400A, SW1 SW_Push, SW5 TM-2023, U1 RP2040, U10 NAU88C22YG, U11 CC1101RGPR, U12 FlatJoyCon, U13 TSC2046EIRGVR, U14 BW21S5011A01TF, U2 RP2040, U3 W25Q128JVS, U4 AMS1117-3.3, U5 JST-PH-2P, U6 BQ24040DSQR, U7 AMS1117-3.3, U8 AMS1117-3.3, U9 TPS63000, Y1 12MHz

Commit message: Work on board layout
Parts:
- moved R30 53.4 mm to (258.4, 12.5)
- moved C37 53.4 mm to (258.5, 15.7)
- moved Q1 53.4 mm to (254.0, 9.34)
- moved Q2 53.4 mm to (249.6, 9.34)
- moved Q3 53.4 mm to (258.5, 9.34)
- moved R22 53.4 mm to (250.3, 4.28)
- moved C36 43.7 mm to (229.0, 6.92)
- moved C38 43.7 mm to (224.3, 6.92)
- moved C39 43.7 mm to (229.4, 4.38)
- moved C40 43.7 mm to (234.8, 8.10)
- moved L1 43.7 mm to (221.3, 3.24)
- moved R20 43.7 mm to (244.8, -7.33)
- moved U9 43.7 mm to (224.8, 3.24)
- moved C34 43.7 mm to (239.9, -7.69)
- moved C35 43.7 mm to (219.4, 6.16)
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Connections:
- SPK1 pad 2: Net-(U10-RSPKOUT) -> Net-(U10-LSPKOUT)
- U10 pad 23: Net-(U10-RSPKOUT) -> Net-(SPK1-+)
- U10 pad 25: Net-(SPK1-+) -> Net-(U10-LSPKOUT)
Routing:
- net /Audio/LRCK: track 72.9 -> 14.9 mm, vias 2 -> 1
- net /Audio/HP_{RIGHT}: track 0.00 -> 55.5 mm
- net /Audio/SCLK: track 67.9 -> 12.5 mm, vias 2 -> 1
- net /Audio/DAC: track 58.7 -> 6.08 mm, vias 2 -> 1
- net /Audio/ADC: track 56.1 -> 5.29 mm, vias 2 -> 1
- net /Audio/HP_{LEFT}: track 7.30 -> 56.6 mm
- net Net-(U10-LSPKOUT): track 0.00 -> 35.6 mm
- net +5V: track 25.3 -> 56.2 mm
- net +3.3VA: track 34.4 -> 58.3 mm, vias 2 -> 4
- net Net-(SPK1-+): track 0.00 -> 18.5 mm
- net Net-(U10-RSPKOUT): track 10.4 -> 0.00 mm
- net /Audio/IR: track 15.8 -> 5.59 mm, vias 2 -> 0
- net Net-(Q4-C): track 55.5 -> 64.6 mm
- net /Audio/CDATA: track 11.6 -> 4.38 mm, vias 2 -> 1
- net /Audio/CCLK: track 11.6 -> 4.64 mm, vias 2 -> 1
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- removed copper zone on F.Cu, net GND

Commit message: Route more parts of the board
Parts:
- removed C46: 10u, Capacitor_SMD:C_0402_1005Metric
- removed Q6: AO3400A, Package_TO_SOT_SMD:SOT-23
- moved D3 164.6 mm to (89.9, 33.4)
- moved SW2 125.3 mm to (177.8, 91.4)
- moved R29 105.7 mm to (159.8, 75.9), turned to 0 degrees
- moved R24 103.2 mm to (159.8, 69.8), turned to 0 degrees
- moved R25 102.6 mm to (159.8, 70.9), turned to 180 degrees
- moved R26 102.0 mm to (159.8, 71.9), turned to 0 degrees
- moved R27 101.5 mm to (159.8, 72.9), turned to 180 degrees
- moved R28 101.0 mm to (159.8, 73.9), turned to 0 degrees
- moved C40 100.5 mm to (159.7, 74.9), turned to 0 degrees
- moved R19 97.6 mm to (197.0, 81.8), turned to 180 degrees
- moved R18 97.1 mm to (197.0, 82.8), turned to 0 degrees
- moved R17 96.7 mm to (197.0, 83.8), turned to 180 degrees
- moved SW3 93.3 mm to (84.5, 91.4)
- moved C36 90.9 mm to (163.8, 70.4)
- moved C39 90.3 mm to (161.2, 63.5), turned to -90 degrees
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Connections:
- net Net-(U1-GPIO24) renamed /RP2040/SWCLK
- net Net-(U1-GPIO25) renamed /RP2040/SWD
- FPC1 pad 11: Net-(Q6-S) -> GND
- FPC1 pad 12: Net-(Q6-S) -> GND
- FPC1 pad 13: Net-(Q6-S) -> GND
- FPC1 pad 14: Net-(Q6-S) -> GND
- SW2 pad C: Net-(D4-Pad3) -> /Inputs/BTN_{SELECT}
- SW3 pad 1: /Inputs/BTN_{SELECT} -> Net-(D4-Pad3)
- U1 pad 17: /Audio/ADC -> /Audio/DAC
- U1 pad 18: /Audio/DAC -> /Audio/ADC
- U1 pad 29: /Audio/IR_{TX} -> /RP2040/BUS0
- U1 pad 3: /MicroSD Card/SD_{CS} -> /Audio/IR_{TX}
- U1 pad 30: /RP2040/BUS0 -> /RP2040/BUS1
- U1 pad 31: /RP2040/BUS1 -> /RP2040/BUS2
- U1 pad 32: /RP2040/BUS2 -> /RP2040/BUS3
- U1 pad 34: /RP2040/BUS3 -> unconnected-(U1-GPIO22-Pad34)
- U1 pad 35: Net-(U1-GPIO23) -> /RP2040/XIN
- U1 pad 40: /Power/BAT_{Vsense} -> /Audio/HP_{SENSE}
- U1 pad 41: /Audio/HP_{SENSE} -> /Power/BAT_{Vsense}
- U1 pad 7: /Display/TFT_{LED} -> /MicroSD Card/SD_{CS}
- U2 pad 20: Net-(U1-GPIO23) -> /RP2040/XIN
- U2 pad 34: /Inputs/BTN_{A} -> /Inputs/BTN_{Y}
- U2 pad 35: /Inputs/BTN_{X} -> /Inputs/BTN_{B}
- U2 pad 36: /Inputs/BTN_{B} -> /Inputs/BTN_{A}
- U2 pad 37: /Inputs/BTN_{Y} -> /Inputs/BTN_{X}
- U2 pad 40: /Inputs/JOY_{X} -> /Inputs/JOY_{Y}
- U2 pad 41: /Inputs/JOY_{Y} -> /Inputs/JOY_{X}
- Y1 pad 1: /RP2040/XIN -> Net-(C25-Pad2)
- Y1 pad 3: Net-(C25-Pad2) -> /RP2040/XIN
Routing:
- net /Power/BAT_{Vsense}: track 5.94 -> 184.8 mm, vias 1 -> 2
- net /Inputs/JOY_{X}: track 7.20 -> 175.4 mm, vias 1 -> 3
- net /Inputs/JOY_{Y}: track 7.73 -> 149.6 mm, vias 1 -> 3
- net /Inputs/BTN_{SELECT}: track 3.24 -> 139.6 mm, vias 1 -> 3
- net /Inputs/BRACK_{R}: track 7.03 -> 111.9 mm, vias 1 -> 2
- net /Audio/IR_{TX}: track 2.17 -> 89.5 mm, vias 1 -> 2
- net /Inputs/BTN_{A}: track 3.82 -> 73.4 mm
- net /Inputs/BTN_{B}: track 5.01 -> 64.5 mm
- net /Audio/CDATA: track 4.38 -> 58.4 mm, vias 1 -> 2
- net /Audio/SCLK: track 12.5 -> 66.0 mm, vias 1 -> 2
- net /Audio/CCLK: track 4.64 -> 56.2 mm, vias 1 -> 2
- net /Audio/ADC: track 5.29 -> 55.1 mm, vias 1 -> 2
- net /Audio/DAC: track 6.08 -> 54.8 mm, vias 1 -> 2
- net /Inputs/BTN_{X}: track 4.42 -> 52.7 mm
- net /Audio/LRCK: track 14.9 -> 62.7 mm, vias 1 -> 2
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- added copper zone on F.Cu, net +5V
- added copper zone on F.Cu, net /Power/vin
- added copper zone on F.Cu, net /Power/vina
- added copper zone on F.Cu, net GND
- removed copper zone on F.Cu, net Net-(Q6-S)

Commit message: Show JoyCon 3D model
Connections:
- U2 pad 34: /Inputs/BTN_{Y} -> /Inputs/BTN_{A}
- U2 pad 35: /Inputs/BTN_{B} -> unconnected-(U2-GPIO23-Pad35)
- U2 pad 36: /Inputs/BTN_{A} -> /Inputs/BTN_{B}
- U2 pad 37: /Inputs/BTN_{X} -> /Inputs/BTN_{Y}

Commit message: Further progress on PCB
Parts:
- C26, C27, C28, C29, C30, C31, C32, C33, C37: footprint Capacitor_SMD:C_0805_2012Metric -> Capacitor_SMD:C_0603_1608Metric
- moved R22 161.6 mm to (94.5, 47.1), turned to 180 degrees
- moved D4 135.8 mm to (119.4, 51.3), turned to 90 degrees
- moved D3 100.4 mm to (183.9, 68.9), turned to 90 degrees
- moved C37 93.0 mm to (182.2, 68.9), turned to 90 degrees
- moved Q3 88.9 mm to (186.8, 61.8)
- moved Q1 87.5 mm to (186.8, 65.4)
- moved Q2 86.6 mm to (186.8, 69.0)
- moved R30 83.0 mm to (190.4, 60.1)
- moved R21 82.4 mm to (184.0, 60.1), turned to -90 degrees
- moved R20 78.7 mm to (189.4, 69.4), turned to -90 degrees
- moved D5 73.6 mm to (186.8, 58.3)
- moved C34 70.9 mm to (189.4, 62.3), turned to 90 degrees
- moved R13 51.3 mm to (192.8, 76.5)
- moved R12 48.8 mm to (192.5, 77.7), turned to 180 degrees
- moved C26 44.0 mm to (196.5, 75.5), turned to 0 degrees
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Connections:
- Q3 pad 2: Net-(Q1-G) -> GND
- Q3 pad 3: GND -> Net-(Q1-G)
- SW3 pad 1: Net-(D4-Pad3) -> GND
- SW3 pad C: GND -> Net-(D4-Pad3)
- U2 pad 29: unconnected-(U2-GPIO18-Pad29) -> /Power/ON
- U2 pad 31: /Power/ON -> unconnected-(U2-GPIO20-Pad31)
Routing:
- net +BATT: track 3.43 -> 83.9 mm, vias 0 -> 1
- net Net-(D4-Pad3): track 0.00 -> 62.9 mm, vias 0 -> 2
- net /Power/~{CHG}: track 0.00 -> 51.6 mm
- net /Power/~{PG}: track 0.00 -> 49.8 mm, vias 0 -> 2
- net /Inputs/JOY_{X}: track 175.4 -> 128.9 mm
- net /Inputs/JOY_{Y}: track 149.6 -> 128.3 mm
- net VBUS: track 6.38 -> 22.3 mm, vias 0 -> 2
- net /Power/ON: track 3.09 -> 17.3 mm, vias 1 -> 2
- net +3.3VSD: track 24.3 -> 30.4 mm
- net /Power/BAT_{Vsense}: track 184.8 -> 181.8 mm
- net unconnected-(U2-GPIO18-Pad29): track 2.89 -> 0.00 mm, vias 1 -> 0
- net GND: track 107.0 -> 109.4 mm, vias 152 -> 155
- net /Power/ISET2: track 8.65 -> 10.9 mm
- net Net-(U6-ISET): track 0.00 -> 2.11 mm
- net Net-(U10-LSPKOUT): track 35.6 -> 34.0 mm
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
Commit message: Route more power
Parts:
- moved Q1 24.3 mm to (163.1, 60.1), turned to -90 degrees
- moved SW1 23.3 mm to (41.4, 88.8), turned to 90 degrees
- moved C30 13.2 mm to (76.6, 97.6)
- moved C34 10.9 mm to (180.8, 69.2)
- moved R20 9.53 mm to (179.8, 69.1)
- moved C31 8.42 mm to (76.6, 92.8), turned to -90 degrees
- moved U7 3.84 mm to (71.8, 95.2)
- moved R30 1.78 mm to (190.3, 58.3)
- moved C55 0.22 mm to (62.5, 76.3)
- moved R21 0.14 mm to (183.9, 60.1)
Connections:
- U1 pad 35: /RP2040/XIN -> /RP2040/XIN2
- U2 pad 20: /RP2040/XIN -> /RP2040/XIN2
Routing:
- net +5V: track 55.6 -> 209.9 mm, vias 0 -> 4
- net VBUS: track 22.3 -> 152.6 mm, vias 2 -> 5
- net /Power/OFF: track 3.45 -> 96.4 mm, vias 1 -> 2
- net Net-(Q1-G): track 0.00 -> 88.1 mm, vias 0 -> 4
- net +3.3V: track 37.0 -> 91.2 mm, vias 0 -> 5
- net /Power/V_{USB/BATT}: track 0.00 -> 33.5 mm
- net /RP2040/XIN2: track 0.00 -> 22.9 mm, vias 0 -> 2
- net /RP2040/XIN: track 33.8 -> 10.8 mm, vias 2 -> 0
- net Net-(D4-Pad3): track 62.9 -> 79.3 mm, vias 2 -> 3
- net GND: track 109.4 -> 118.9 mm, vias 155 -> 179
- net Net-(Q3-G): track 0.00 -> 5.99 mm
- net /Display/TOUCH_{MOSI}: track 95.7 -> 98.0 mm
- net /Inputs/JOY_{X}: track 128.9 -> 131.1 mm, vias 3 -> 4
- net Net-(D5-Pad2): track 0.00 -> 2.01 mm
- net /Power/BAT_{Vsense}: track 181.8 -> 180.3 mm
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- added copper zone on F.Cu, net +BATT
- added copper zone on F.Cu, net /Power/V_{USB/BATT}
- added copper zone on F.Cu, net VBUS

Commit message: Continue routing
Parts:
- moved SW1 46.2 mm to (84.7, 72.8), turned to 180 degrees
- moved C6 14.1 mm to (112.7, 73.9), turned to 0 degrees
- moved R7 0.98 mm to (84.8, 77.3), turned to 0 degrees
- moved R6 0.98 mm to (84.8, 78.4), turned to 180 degrees
- moved C3 0.85 mm to (99.6, 74.9)
Routing:
- net +3.3V: track 91.2 -> 171.5 mm, vias 5 -> 7
- net GND: track 118.9 -> 131.3 mm, vias 179 -> 186
- net Net-(R7-Pad2): track 0.00 -> 11.7 mm, vias 0 -> 2
- net /Power/BAT_{Vsense}: track 180.3 -> 181.9 mm
- net Net-(D4-Pad3): vias 3 -> 5

Commit message: Finalize routing
Connections:
- U2 pad 34: /Inputs/BTN_{A} -> /Inputs/BTN_{Y}
- U2 pad 35: unconnected-(U2-GPIO23-Pad35) -> /Inputs/BTN_{B}
- U2 pad 36: /Inputs/BTN_{B} -> /Inputs/BTN_{A}
- U2 pad 37: /Inputs/BTN_{Y} -> /Inputs/BTN_{X}
Routing:
- net +3.3V: track 171.5 -> 424.0 mm, vias 7 -> 19
- net /Power/ISET2: track 10.9 -> 103.8 mm, vias 1 -> 2
- net GND: track 131.3 -> 140.9 mm, vias 186 -> 204
- net Net-(U9-FB): track 3.41 -> 10.3 mm
- net /Audio/IR_{TX}: track 89.5 -> 90.6 mm
- net /RP2040/XIN2: track 22.9 -> 23.6 mm
- net Net-(U13-X+): track 19.3 -> 19.8 mm
- net /Display/TOUCH_{SCLK}: track 84.8 -> 84.6 mm, vias 4 -> 3
- added copper zone on F.Cu, net +3.3VSD

Commit message: Sent to manufacturing
Parts:
- added R42: 10k, Resistor_SMD:R_0402_1005Metric, F.Cu at (195.8, 78.0)
- D3: footprint LED_SMD:LED_0603_1608Metric -> Diode_SMD:D_SMA
- moved D3 4.63 mm to (182.6, 64.4), turned to 135 degrees
Connections:
- U6 pad 9: unconnected-(U6-TS-Pad9) -> /Power/TS
Routing:
- net /Power/V_{USB/BATT}: track 33.5 -> 37.8 mm
- net /Power/TS: track 0.00 -> 3.02 mm
- net /Power/~{CHG}: track 52.1 -> 54.1 mm
- net VBUS: track 152.6 -> 154.1 mm
- net GND: track 140.9 -> 141.8 mm
- net Net-(Q1-G): track 88.1 -> 87.4 mm
- net +BATT: track 83.9 -> 84.4 mm
Other:
- board text added: "Kreček v0.11 2025-02-26 Elektrotechnika & Hry DDM Spirála, Praha 8"
- board text removed: "Kreček v0.9 2024-03-06 Elektrotechnika & Hry DDM Spirála, Praha 8"
