File: hw/krecek-0.9/inputs.kicad_sch (KiCad schematic)
At the start: 13 parts

Commit message: Further tweaks and improvements
- Use a nicer schematic template
- Tie START button with power on
- Add ferrite to USB shield
- Add CC1/CC2 makeshift ADC
- Tidy up schematics a little bit

Signed-off-by: Jan Hamal Dvořák <mordae@anilinux.org>
Other:
- company: (none) -> DDM Spirála
- title: (none) -> Křeček
Changed lines of the file:
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@@
 (kicad_sch (version 20230121) (generator eeschema)
   (paper "A4")
+  (title_block
+    (title "Křeček")
+    (date "2023-12-20")
+    (rev "v0.9-wip")
+    (company "DDM Spirála")
+  )
   (junction (at 139.7 152.4) (diameter 0) (color 0 0 0 0)
   )

Commit message: Complete most of the design, except for RF
Signed-off-by: Jan Hamal Dvořák <mordae@anilinux.org>
Parts:
- removed R11 (x2): 100k, Resistor_SMD:R_0402_1005Metric, symbol Device:R_Small
- removed R14: 33k, Resistor_SMD:R_0402_1005Metric, symbol Device:R_Small
- removed SW3: ~, Krecek:RubberButton, symbol Krecek:RubberButton
- added C7 (x4): 100nF, Capacitor_SMD:C_0402_1005Metric, symbol Device:C_Small
- added R14 (x3): 3.3k, Resistor_SMD:R_0402_1005Metric, symbol Device:R_Small
- added R37, R39: RDC506002A, LCSC:RES-ADJ-SMD_RDC506002A, symbol LCSC:RDC506002A
- added SW5: TM-2023, LCSC:SW-SMD_TM-2023-1, symbol LCSC:TM-2023
- R14: value 33k -> 3.3k; LCSC Part C25779 -> C25890
- renumbered SW4 to SW3, SW2 to SW4
Connections:
- net +3.3V: now also R37.1 (1T), R39.1 (1T)
- net BTN_{SELECT}: now also C7.1
- net GND: now also C7.2, C7.2, C7.2, C7.2, R37.3 (3T), R39.3 (3T), SW5.C (COM), SW5.SH
- new net BRACK_{L}: R37.2 (2T)
- new net BRACK_{R}: R39.2 (2T)
- new net VOL_{DOWN}: C7.1, R14.1
- new net VOL_{SW}: C7.1, R14.1
- new net VOL_{UP}: C7.1, R14.1
- new net vol_ccw: R14.2, SW5.1 (CCW)
- new net vol_cw: R14.2, SW5.2 (CW)
- new net vol_push: R14.2, SW5.T (PUSH)
Other:
- moved on the sheet: C7, JOY1, R14, SW3, SW4A, SW4B, SW4C, SW4D

Commit message: Fix part numbers
Signed-off-by: Jan Hamal Dvořák <mordae@anilinux.org>
Parts:
- renumbered R37 to R36, R39 to R38

Commit message: Fix symbol/footprint mismatches
Signed-off-by: Jan Hamal Dvořák <mordae@anilinux.org>
Connections:
- net GND: now also JOY1.SH
Changed lines of the file:
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@@
   (symbol (lib_id "power:GND") (at 50.8 88.9 0) (unit 1)
     (in_bom yes) (on_board yes) (dnp no) (fields_autoplaced)
-    (property "Reference" "#PWR099" (at 50.8 95.25 0)
+    (property "Reference" "#PWR0100" (at 50.8 95.25 0)
       (effects (font (size 1.27 1.27)) hide)
     )
@@
       (project "krecek-0.9"
         (path "/8888f37b-ecc2-47df-8824-4b4e1e726451/11c64485-27fc-47ac-864e-0b013ddf7d3c"
-          (reference "#PWR099") (unit 1)
+          (reference "#PWR0100") (unit 1)
         )
       )
@@
   (symbol (lib_id "power:GND") (at 129.54 88.9 90) (unit 1)
     (in_bom yes) (on_board yes) (dnp no) (fields_autoplaced)
-    (property "Reference" "#PWR0101" (at 135.89 88.9 0)
+    (property "Reference" "#PWR0102" (at 135.89 88.9 0)
       (effects (font (size 1.27 1.27)) hide)
     )
@@
       (project "krecek-0.9"
         (path "/8888f37b-ecc2-47df-8824-4b4e1e726451/11c64485-27fc-47ac-864e-0b013ddf7d3c"
+          (reference "#PWR0102") (unit 1)
+        )
+      )
+    )
+  )
+  (symbol (lib_id "power:GND") (at 146.05 52.07 0) (mirror y) (unit 1)
+    (in_bom yes) (on_board yes) (dnp no) (fields_autoplaced)
+    (property "Reference" "#PWR094" (at 146.05 58.42 0)
+      (effects (font (size 1.27 1.27)) hide)
+    )
+    (property "Value" "GND" (at 146.05 57.15 0)
+      (effects (font (size 1.27 1.27)))
+    )
+    (property "Footprint" "" (at 146.05 52.07 0)
+      (effects (font (size 1.27 1.27)) hide)
+    )
+    (property "Datasheet" "" (at 146.05 52.07 0)
+      (effects (font (size 1.27 1.27)) hide)
+    )
+    (pin "1")
+    (instances
+      (project "krecek-0.9"
+        (path "/8888f37b-ecc2-47df-8824-4b4e1e726451/11c64485-27fc-47ac-864e-0b013ddf7d3c"
+          (reference "#PWR094") (unit 1)
+        )
+      )
+    )
+  )
+  (symbol (lib_id "power:+3.3V") (at 111.76 88.9 90) (unit 1)
+    (in_bom yes) (on_board yes) (dnp no) (fields_autoplaced)
+    (property "Reference" "#PWR0101" (at 115.57 88.9 0)
+      (effects (font (size 1.27 1.27)) hide)
+    )
+    (property "Value" "+3.3V" (at 107.95 88.9 90)
+      (effects (font (size 1.27 1.27)) (justify left))
+    )
+    (property "Footprint" "" (at 111.76 88.9 0)
+      (effects (font (size 1.27 1.27)) hide)
+    )
+    (property "Datasheet" "" (at 111.76 88.9 0)
+      (effects (font (size 1.27 1.27)) hide)
+    )
+    (pin "1")
+    (instances
+      (project "krecek-0.9"
+        (path "/8888f37b-ecc2-47df-8824-4b4e1e726451/11c64485-27fc-47ac-864e-0b013ddf7d3c"
           (reference "#PWR0101") (unit 1)
         )
@@
     )
   )
-  (symbol (lib_id "power:GND") (at 146.05 52.07 0) (mirror y) (unit 1)
-    (in_bom yes) (on_board yes) (dnp no) (fields_autoplaced)
-    (property "Reference" "#PWR094" (at 146.05 58.42 0)
-      (effects (font (size 1.27 1.27)) hide)
-    )
-    (property "Value" "GND" (at 146.05 57.15 0)
-      (effects (font (size 1.27 1.27)))
-    )
-    (property "Footprint" "" (at 146.05 52.07 0)
-      (effects (font (size 1.27 1.27)) hide)
-    )
-    (property "Datasheet" "" (at 146.05 52.07 0)
-      (effects (font (size 1.27 1.27)) hide)
-    )
-    (pin "1")
-    (instances
-      (project "krecek-0.9"
-        (path "/8888f37b-ecc2-47df-8824-4b4e1e726451/11c64485-27fc-47ac-864e-0b013ddf7d3c"
-          (reference "#PWR094") (unit 1)
-        )
-      )
-    )
-  )
-  (symbol (lib_id "power:+3.3V") (at 111.76 88.9 90) (unit 1)
-    (in_bom yes) (on_board yes) (dnp no) (fields_autoplaced)
-    (property "Reference" "#PWR0100" (at 115.57 88.9 0)
-      (effects (font (size 1.27 1.27)) hide)
-    )
-    (property "Value" "+3.3V" (at 107.95 88.9 90)
-      (effects (font (size 1.27 1.27)) (justify left))
-    )
-    (property "Footprint" "" (at 111.76 88.9 0)
-      (effects (font (size 1.27 1.27)) hide)
-    )
-    (property "Datasheet" "" (at 111.76 88.9 0)
-      (effects (font (size 1.27 1.27)) hide)
-    )
-    (pin "1")
-    (instances
-      (project "krecek-0.9"
-        (path "/8888f37b-ecc2-47df-8824-4b4e1e726451/11c64485-27fc-47ac-864e-0b013ddf7d3c"
-          (reference "#PWR0100") (unit 1)
-        )
-      )
-    )
-  )
   (symbol (lib_id "power:GND") (at 107.95 52.07 0) (mirror y) (unit 1)
     (in_bom yes) (on_board yes) (dnp no) (fields_autoplaced)
@@
   (symbol (lib_id "power:GND") (at 50.8 127 0) (unit 1)
     (in_bom yes) (on_board yes) (dnp no) (fields_autoplaced)
-    (property "Reference" "#PWR0106" (at 50.8 133.35 0)
+    (property "Reference" "#PWR0107" (at 50.8 133.35 0)
       (effects (font (size 1.27 1.27)) hide)
     )
@@
       (project "krecek-0.9"
         (path "/8888f37b-ecc2-47df-8824-4b4e1e726451/11c64485-27fc-47ac-864e-0b013ddf7d3c"
-          (reference "#PWR0106") (unit 1)
+          (reference "#PWR0107") (unit 1)
         )
       )
@@
     )
     (pin "GND")
+    (pin "SH")
     (pin "SW")
     (pin "VCC")
@@
     )
   )
+  (symbol (lib_id "power:GND") (at 176.53 86.36 270) (unit 1)
+    (in_bom yes) (on_board yes) (dnp no) (fields_autoplaced)
+    (property "Reference" "#PWR099" (at 170.18 86.36 0)
+      (effects (font (size 1.27 1.27)) hide)
+    )
+    (property "Value" "GND" (at 172.72 86.36 90)
+      (effects (font (size 1.27 1.27)) (justify right))
+    )
+    (property "Footprint" "" (at 176.53 86.36 0)
+      (effects (font (size 1.27 1.27)) hide)
+    )
+    (property "Datasheet" "" (at 176.53 86.36 0)
+      (effects (font (size 1.27 1.27)) hide)
+    )
+    (pin "1")
+    (instances
+      (project "krecek-0.9"
+        (path "/8888f37b-ecc2-47df-8824-4b4e1e726451/11c64485-27fc-47ac-864e-0b013ddf7d3c"
+          (reference "#PWR099") (unit 1)
+        )
+      )
+    )
+  )
   (symbol (lib_id "Krecek:ABXY") (at 184.15 38.1 0) (mirror y) (unit 3)
     (in_bom yes) (on_board yes) (dnp no) (fields_autoplaced)
@@
   (symbol (lib_id "power:GND") (at 50.8 165.1 0) (unit 1)
     (in_bom yes) (on_board yes) (dnp no) (fields_autoplaced)
-    (property "Reference" "#PWR0107" (at 50.8 171.45 0)
+    (property "Reference" "#PWR0108" (at 50.8 171.45 0)
       (effects (font (size 1.27 1.27)) hide)
     )
@@
       (project "krecek-0.9"
         (path "/8888f37b-ecc2-47df-8824-4b4e1e726451/11c64485-27fc-47ac-864e-0b013ddf7d3c"
-          (reference "#PWR0107") (unit 1)
+          (reference "#PWR0108") (unit 1)
         )
       )
@@
   (symbol (lib_id "power:GND") (at 129.54 114.3 90) (unit 1)
     (in_bom yes) (on_board yes) (dnp no) (fields_autoplaced)
-    (property "Reference" "#PWR0105" (at 135.89 114.3 0)
+    (property "Reference" "#PWR0106" (at 135.89 114.3 0)
       (effects (font (size 1.27 1.27)) hide)
     )
@@
       (project "krecek-0.9"
         (path "/8888f37b-ecc2-47df-8824-4b4e1e726451/11c64485-27fc-47ac-864e-0b013ddf7d3c"
-          (reference "#PWR0105") (unit 1)
+          (reference "#PWR0106") (unit 1)
         )
       )
@@
   (symbol (lib_id "power:GND") (at 176.53 88.9 270) (unit 1)
     (in_bom yes) (on_board yes) (dnp no) (fields_autoplaced)
-    (property "Reference" "#PWR0102" (at 170.18 88.9 0)
+    (property "Reference" "#PWR0103" (at 170.18 88.9 0)
       (effects (font (size 1.27 1.27)) hide)
     )
@@
       (project "krecek-0.9"
         (path "/8888f37b-ecc2-47df-8824-4b4e1e726451/11c64485-27fc-47ac-864e-0b013ddf7d3c"
-          (reference "#PWR0102") (unit 1)
+          (reference "#PWR0103") (unit 1)
         )
       )
@@
   (symbol (lib_id "power:+3.3V") (at 111.76 114.3 90) (unit 1)
     (in_bom yes) (on_board yes) (dnp no) (fields_autoplaced)
-    (property "Reference" "#PWR0104" (at 115.57 114.3 0)
+    (property "Reference" "#PWR0105" (at 115.57 114.3 0)
       (effects (font (size 1.27 1.27)) hide)
     )
@@
       (project "krecek-0.9"
         (path "/8888f37b-ecc2-47df-8824-4b4e1e726451/11c64485-27fc-47ac-864e-0b013ddf7d3c"
-          (reference "#PWR0104") (unit 1)
+          (reference "#PWR0105") (unit 1)
         )
       )
@@
   (symbol (lib_id "power:GND") (at 215.9 101.6 0) (unit 1)
     (in_bom yes) (on_board yes) (dnp no) (fields_autoplaced)
-    (property "Reference" "#PWR0103" (at 215.9 107.95 0)
+    (property "Reference" "#PWR0104" (at 215.9 107.95 0)
       (effects (font (size 1.27 1.27)) hide)
     )
@@
       (project "krecek-0.9"
         (path "/8888f37b-ecc2-47df-8824-4b4e1e726451/11c64485-27fc-47ac-864e-0b013ddf7d3c"
-          (reference "#PWR0103") (unit 1)
-        )
-      )
+          (reference "#PWR0104") (unit 1)
+        )
+      )

Commit message: Add discrete antenna
Signed-off-by: Jan Hamal Dvořák <mordae@anilinux.org>
Parts:
- renumbered C7 to C71, C7 to C72, C7 to C73, C7 to C74, C7 to C75, C7 to C76, C7 to C77, C7 to C78, C7 to C79, R14 to R34, R14 to R35, R14 to R37, R14 to R39
Changed lines of the file:
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@@
   (symbol (lib_id "Device:C_Small") (at 50.8 82.55 0) (mirror y) (unit 1)
     (in_bom yes) (on_board yes) (dnp no) (fields_autoplaced)
-    (property "Reference" "C7" (at 53.34 81.2863 0)
+    (property "Reference" "C76" (at 53.34 81.2863 0)
       (effects (font (size 1.27 1.27)) (justify right))
     )
@@
     (instances
       (project "krecek-0.9"
-        (path "/8888f37b-ecc2-47df-8824-4b4e1e726451/bd29cd8c-9207-416a-90c1-7bdf6b5cfb97"
-          (reference "C7") (unit 1)
-        )
         (path "/8888f37b-ecc2-47df-8824-4b4e1e726451/11c64485-27fc-47ac-864e-0b013ddf7d3c"
           (reference "C76") (unit 1)
@@
   (symbol (lib_id "Device:R_Small") (at 44.45 76.2 270) (unit 1)
     (in_bom yes) (on_board yes) (dnp no) (fields_autoplaced)
-    (property "Reference" "R14" (at 44.45 71.12 90)
+    (property "Reference" "R34" (at 44.45 71.12 90)
       (effects (font (size 1.27 1.27)))
     )
@@
     (instances
       (project "krecek-0.9"
-        (path "/8888f37b-ecc2-47df-8824-4b4e1e726451/bd29cd8c-9207-416a-90c1-7bdf6b5cfb97"
-          (reference "R14") (unit 1)
-        )
         (path "/8888f37b-ecc2-47df-8824-4b4e1e726451/11c64485-27fc-47ac-864e-0b013ddf7d3c"
           (reference "R34") (unit 1)
@@
   (symbol (lib_id "Device:R_Small") (at 209.55 88.9 270) (unit 1)
     (in_bom yes) (on_board yes) (dnp no) (fields_autoplaced)
-    (property "Reference" "R14" (at 209.55 83.82 90)
+    (property "Reference" "R35" (at 209.55 83.82 90)
       (effects (font (size 1.27 1.27)))
     )
@@
     (instances
       (project "krecek-0.9"
-        (path "/8888f37b-ecc2-47df-8824-4b4e1e726451/bd29cd8c-9207-416a-90c1-7bdf6b5cfb97"
-          (reference "R14") (unit 1)
-        )
         (path "/8888f37b-ecc2-47df-8824-4b4e1e726451/11c64485-27fc-47ac-864e-0b013ddf7d3c"
           (reference "R35") (unit 1)
@@
   (symbol (lib_id "Device:R_Small") (at 44.45 114.3 270) (unit 1)
     (in_bom yes) (on_board yes) (dnp no) (fields_autoplaced)
-    (property "Reference" "R14" (at 44.45 109.22 90)
+    (property "Reference" "R37" (at 44.45 109.22 90)
       (effects (font (size 1.27 1.27)))
     )
@@
     (instances
       (project "krecek-0.9"
-        (path "/8888f37b-ecc2-47df-8824-4b4e1e726451/bd29cd8c-9207-416a-90c1-7bdf6b5cfb97"
-          (reference "R14") (unit 1)
-        )
         (path "/8888f37b-ecc2-47df-8824-4b4e1e726451/11c64485-27fc-47ac-864e-0b013ddf7d3c"
           (reference "R37") (unit 1)
@@
   (symbol (lib_id "Device:R_Small") (at 44.45 152.4 270) (unit 1)
     (in_bom yes) (on_board yes) (dnp no) (fields_autoplaced)
-    (property "Reference" "R14" (at 44.45 147.32 90)
+    (property "Reference" "R39" (at 44.45 147.32 90)
       (effects (font (size 1.27 1.27)))
     )
@@
     (instances
       (project "krecek-0.9"
-        (path "/8888f37b-ecc2-47df-8824-4b4e1e726451/bd29cd8c-9207-416a-90c1-7bdf6b5cfb97"
-          (reference "R14") (unit 1)
-        )
         (path "/8888f37b-ecc2-47df-8824-4b4e1e726451/11c64485-27fc-47ac-864e-0b013ddf7d3c"
           (reference "R39") (unit 1)
@@
   (symbol (lib_id "Device:C_Small") (at 50.8 120.65 0) (mirror y) (unit 1)
     (in_bom yes) (on_board yes) (dnp no) (fields_autoplaced)
-    (property "Reference" "C7" (at 53.34 119.3863 0)
+    (property "Reference" "C78" (at 53.34 119.3863 0)
       (effects (font (size 1.27 1.27)) (justify right))
     )
@@
     (instances
       (project "krecek-0.9"
-        (path "/8888f37b-ecc2-47df-8824-4b4e1e726451/bd29cd8c-9207-416a-90c1-7bdf6b5cfb97"
-          (reference "C7") (unit 1)
-        )
         (path "/8888f37b-ecc2-47df-8824-4b4e1e726451/11c64485-27fc-47ac-864e-0b013ddf7d3c"
           (reference "C78") (unit 1)
@@
   (symbol (lib_id "Device:C_Small") (at 152.4 44.45 0) (mirror y) (unit 1)
     (in_bom yes) (on_board yes) (dnp no)
-    (property "Reference" "C7" (at 149.86 43.1863 0)
+    (property "Reference" "C72" (at 149.86 43.1863 0)
       (effects (font (size 1.27 1.27)) (justify left))
     )
@@
     (instances
       (project "krecek-0.9"
-        (path "/8888f37b-ecc2-47df-8824-4b4e1e726451/bd29cd8c-9207-416a-90c1-7bdf6b5cfb97"
-          (reference "C7") (unit 1)
-        )
         (path "/8888f37b-ecc2-47df-8824-4b4e1e726451/11c64485-27fc-47ac-864e-0b013ddf7d3c"
           (reference "C72") (unit 1)
@@
   (symbol (lib_id "Device:C_Small") (at 228.6 44.45 0) (mirror y) (unit 1)
     (in_bom yes) (on_board yes) (dnp no)
-    (property "Reference" "C7" (at 226.06 43.1863 0)
+    (property "Reference" "C74" (at 226.06 43.1863 0)
       (effects (font (size 1.27 1.27)) (justify left))
     )
@@
     (instances
       (project "krecek-0.9"
-        (path "/8888f37b-ecc2-47df-8824-4b4e1e726451/bd29cd8c-9207-416a-90c1-7bdf6b5cfb97"
-          (reference "C7") (unit 1)
-        )
         (path "/8888f37b-ecc2-47df-8824-4b4e1e726451/11c64485-27fc-47ac-864e-0b013ddf7d3c"
           (reference "C74") (unit 1)
@@
   (symbol (lib_id "Device:C_Small") (at 266.7 44.45 0) (mirror y) (unit 1)
     (in_bom yes) (on_board yes) (dnp no)
-    (property "Reference" "C7" (at 264.16 43.1863 0)
+    (property "Reference" "C75" (at 264.16 43.1863 0)
       (effects (font (size 1.27 1.27)) (justify left))
     )
@@
     (instances
       (project "krecek-0.9"
-        (path "/8888f37b-ecc2-47df-8824-4b4e1e726451/bd29cd8c-9207-416a-90c1-7bdf6b5cfb97"
-          (reference "C7") (unit 1)
-        )
         (path "/8888f37b-ecc2-47df-8824-4b4e1e726451/11c64485-27fc-47ac-864e-0b013ddf7d3c"
           (reference "C75") (unit 1)
@@
   (symbol (lib_id "Device:C_Small") (at 190.5 44.45 0) (mirror y) (unit 1)
     (in_bom yes) (on_board yes) (dnp no)
-    (property "Reference" "C7" (at 187.96 43.1863 0)
+    (property "Reference" "C73" (at 187.96 43.1863 0)
       (effects (font (size 1.27 1.27)) (justify left))
     )
@@
     (instances
       (project "krecek-0.9"
-        (path "/8888f37b-ecc2-47df-8824-4b4e1e726451/bd29cd8c-9207-416a-90c1-7bdf6b5cfb97"
-          (reference "C7") (unit 1)
-        )
         (path "/8888f37b-ecc2-47df-8824-4b4e1e726451/11c64485-27fc-47ac-864e-0b013ddf7d3c"
           (reference "C73") (unit 1)
@@
   (symbol (lib_id "Device:C_Small") (at 215.9 95.25 0) (mirror y) (unit 1)
     (in_bom yes) (on_board yes) (dnp no) (fields_autoplaced)
-    (property "Reference" "C7" (at 218.44 93.9863 0)
+    (property "Reference" "C77" (at 218.44 93.9863 0)
       (effects (font (size 1.27 1.27)) (justify right))
     )
@@
     (instances
       (project "krecek-0.9"
-        (path "/8888f37b-ecc2-47df-8824-4b4e1e726451/bd29cd8c-9207-416a-90c1-7bdf6b5cfb97"
-          (reference "C7") (unit 1)
-        )
         (path "/8888f37b-ecc2-47df-8824-4b4e1e726451/11c64485-27fc-47ac-864e-0b013ddf7d3c"
           (reference "C77") (unit 1)
@@
   (symbol (lib_id "Device:C_Small") (at 114.3 44.45 0) (mirror y) (unit 1)
     (in_bom yes) (on_board yes) (dnp no)
-    (property "Reference" "C7" (at 111.76 43.1863 0)
+    (property "Reference" "C71" (at 111.76 43.1863 0)
       (effects (font (size 1.27 1.27)) (justify left))
     )
@@
     (instances
       (project "krecek-0.9"
-        (path "/8888f37b-ecc2-47df-8824-4b4e1e726451/bd29cd8c-9207-416a-90c1-7bdf6b5cfb97"
-          (reference "C7") (unit 1)
-        )
         (path "/8888f37b-ecc2-47df-8824-4b4e1e726451/11c64485-27fc-47ac-864e-0b013ddf7d3c"
           (reference "C71") (unit 1)
@@
   (symbol (lib_id "Device:C_Small") (at 50.8 158.75 0) (mirror y) (unit 1)
     (in_bom yes) (on_board yes) (dnp no) (fields_autoplaced)
-    (property "Reference" "C7" (at 53.34 157.4863 0)
+    (property "Reference" "C79" (at 53.34 157.4863 0)
       (effects (font (size 1.27 1.27)) (justify right))
     )
@@
     (instances
       (project "krecek-0.9"
-        (path "/8888f37b-ecc2-47df-8824-4b4e1e726451/bd29cd8c-9207-416a-90c1-7bdf6b5cfb97"
-          (reference "C7") (unit 1)
-        )
         (path "/8888f37b-ecc2-47df-8824-4b4e1e726451/11c64485-27fc-47ac-864e-0b013ddf7d3c"
           (reference "C79") (unit 1)

Commit message: Hardware as sent for manufacturing
Parts:
- C71, C72, C73, C74, C75, C76, C77, C78, C79: value 100nF -> 100n
Changed lines of the file:
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@@
       (effects (font (size 1.27 1.27)) (justify right))
     )
-    (property "Value" "100nF" (at 53.34 83.8263 0)
+    (property "Value" "100n" (at 53.34 83.8263 0)
       (effects (font (size 1.27 1.27)) (justify right))
     )
@@
       (effects (font (size 1.27 1.27)) (justify right))
     )
-    (property "Value" "100nF" (at 53.34 121.9263 0)
+    (property "Value" "100n" (at 53.34 121.9263 0)
       (effects (font (size 1.27 1.27)) (justify right))
     )
@@
       (effects (font (size 1.27 1.27)) (justify left))
     )
-    (property "Value" "100nF" (at 149.86 45.7263 0)
+    (property "Value" "100n" (at 149.86 45.7263 0)
       (effects (font (size 1.27 1.27)) (justify left))
     )
@@
       (effects (font (size 1.27 1.27)) (justify left))
     )
-    (property "Value" "100nF" (at 226.06 45.7263 0)
+    (property "Value" "100n" (at 226.06 45.7263 0)
       (effects (font (size 1.27 1.27)) (justify left))
     )
@@
       (effects (font (size 1.27 1.27)) (justify left))
     )
-    (property "Value" "100nF" (at 264.16 45.7263 0)
+    (property "Value" "100n" (at 264.16 45.7263 0)
       (effects (font (size 1.27 1.27)) (justify left))
     )
@@
       (effects (font (size 1.27 1.27)) (justify left))
     )
-    (property "Value" "100nF" (at 187.96 45.7263 0)
+    (property "Value" "100n" (at 187.96 45.7263 0)
       (effects (font (size 1.27 1.27)) (justify left))
     )
@@
       (effects (font (size 1.27 1.27)) (justify right))
     )
-    (property "Value" "100nF" (at 218.44 96.5263 0)
+    (property "Value" "100n" (at 218.44 96.5263 0)
       (effects (font (size 1.27 1.27)) (justify right))
     )
@@
       (effects (font (size 1.27 1.27)) (justify left))
     )
-    (property "Value" "100nF" (at 111.76 45.7263 0)
+    (property "Value" "100n" (at 111.76 45.7263 0)
       (effects (font (size 1.27 1.27)) (justify left))
     )
@@
       (effects (font (size 1.27 1.27)) (justify right))
     )
-    (property "Value" "100nF" (at 53.34 160.0263 0)
-      (effects (font (size 1.27 1.27)) (justify right))
-    )
+    (property "Value" "100n" (at 53.34 160.0263 0)
+      (effects (font (size 1.27 1.27)) (justify right))
+    )

Commit message: Fix OFF issues, rename buttons
Resolves #4.
Connections:
- net BTN_{B}: now also C75.1, SW4.4; no longer C74.1, SW4.2
- net BTN_{X}: now also C74.1, SW4.2; no longer C73.1, SW4.3
- net BTN_{Y}: now also C73.1, SW4.3; no longer C75.1, SW4.4
Changed lines of the file:
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@@
     (effects (font (size 1.27 1.27)) (justify left))
   )
-  (hierarchical_label "BTN_{B}" (shape output) (at 232.41 38.1 0) (fields_autoplaced)
+  (hierarchical_label "BTN_{Y}" (shape output) (at 194.31 38.1 0) (fields_autoplaced)
     (effects (font (size 1.27 1.27)) (justify left))
   )
@@
     (effects (font (size 1.27 1.27)) (justify left))
   )
-  (hierarchical_label "BTN_{Y}" (shape output) (at 270.51 38.1 0) (fields_autoplaced)
+  (hierarchical_label "BTN_{B}" (shape output) (at 270.51 38.1 0) (fields_autoplaced)
     (effects (font (size 1.27 1.27)) (justify left))
   )
@@
     (effects (font (size 1.27 1.27)) (justify left))
   )
-  (hierarchical_label "BTN_{X}" (shape output) (at 194.31 38.1 0) (fields_autoplaced)
+  (hierarchical_label "BTN_{X}" (shape output) (at 232.41 38.1 0) (fields_autoplaced)
     (effects (font (size 1.27 1.27)) (justify left))
   )
