File: hw/krecek-0.9/sdcard.kicad_sch (KiCad schematic)
At the start: 3 parts, among them J4 Micro_SD_Card_Det1

Commit message: Add more missing LCSC part ids
Signed-off-by: Jan Hamal Dvořák <mordae@anilinux.org>
Parts:
- J4: LCSC Part (none) -> C5333937
Changed lines of the file:
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@@
+      (effects (font (size 1.27 1.27)) hide)
+    )
+    (property "LCSC Part" "C5333937" (at 171.45 66.04 0)
       (effects (font (size 1.27 1.27)) hide)
     )

Commit message: Fix part numbers
Signed-off-by: Jan Hamal Dvořák <mordae@anilinux.org>
Parts:
- renumbered J4 to J5
Changed lines of the file:
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@@
   (symbol (lib_id "Krecek:+3.3VSD") (at 88.9 63.5 90) (unit 1)
     (in_bom no) (on_board no) (dnp no) (fields_autoplaced)
-    (property "Reference" "#+3.3VSD03" (at 85.09 63.5 0)
+    (property "Reference" "#+3.3VSD02" (at 85.09 63.5 0)
       (effects (font (size 1.27 1.27)) hide)
     )
@@
       (project "krecek-0.9"
         (path "/8888f37b-ecc2-47df-8824-4b4e1e726451/a9ff151a-3813-42b7-837e-58004a43f525"
-          (reference "#+3.3VSD03") (unit 1)
+          (reference "#+3.3VSD02") (unit 1)
         )
       )
@@
         )
         (path "/8888f37b-ecc2-47df-8824-4b4e1e726451/a9ff151a-3813-42b7-837e-58004a43f525"
-          (reference "C72") (unit 1)
+          (reference "C81") (unit 1)
         )
       )
@@
         )
         (path "/8888f37b-ecc2-47df-8824-4b4e1e726451/a9ff151a-3813-42b7-837e-58004a43f525"
-          (reference "#PWR0105") (unit 1)
+          (reference "#PWR0110") (unit 1)
         )
       )
@@
         )
         (path "/8888f37b-ecc2-47df-8824-4b4e1e726451/a9ff151a-3813-42b7-837e-58004a43f525"
-          (reference "#PWR0104") (unit 1)
+          (reference "#PWR0109") (unit 1)
         )
       )
@@
         )
         (path "/8888f37b-ecc2-47df-8824-4b4e1e726451/a9ff151a-3813-42b7-837e-58004a43f525"
-          (reference "C71") (unit 1)
+          (reference "C80") (unit 1)
         )
       )
@@
         )
         (path "/8888f37b-ecc2-47df-8824-4b4e1e726451/a9ff151a-3813-42b7-837e-58004a43f525"
-          (reference "#PWR0103") (unit 1)
+          (reference "#PWR0108") (unit 1)
         )
       )
@@
   (symbol (lib_id "Connector:Micro_SD_Card_Det1") (at 171.45 66.04 0) (unit 1)
     (in_bom yes) (on_board yes) (dnp no) (fields_autoplaced)
-    (property "Reference" "J4" (at 172.085 44.45 0)
+    (property "Reference" "J5" (at 172.085 44.45 0)
       (effects (font (size 1.27 1.27)))
     )
@@
       (project "krecek-0.9"
         (path "/8888f37b-ecc2-47df-8824-4b4e1e726451/a9ff151a-3813-42b7-837e-58004a43f525"
-          (reference "J4") (unit 1)
-        )
-      )
+          (reference "J5") (unit 1)
+        )
+      )

Commit message: Add discrete antenna
Signed-off-by: Jan Hamal Dvořák <mordae@anilinux.org>
Parts:
- renumbered C29 to C80
Changed lines of the file:
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@@
       )
       (project "krecek-0.9"
-        (path "/8888f37b-ecc2-47df-8824-4b4e1e726451/6537dbea-4e11-4137-b8a0-9ae6b128c4e4"
-          (reference "C12") (unit 1)
-        )
-        (path "/8888f37b-ecc2-47df-8824-4b4e1e726451/a7733ec7-68c7-444f-aac5-8a965be5cbce"
-          (reference "C69") (unit 1)
-        )
         (path "/8888f37b-ecc2-47df-8824-4b4e1e726451/a9ff151a-3813-42b7-837e-58004a43f525"
           (reference "C81") (unit 1)
@@
   (symbol (lib_id "power:GND") (at 191.77 78.74 90) (unit 1)
     (in_bom yes) (on_board yes) (dnp no) (fields_autoplaced)
-    (property "Reference" "#PWR060" (at 198.12 78.74 0)
+    (property "Reference" "#PWR0111" (at 198.12 78.74 0)
       (effects (font (size 1.27 1.27)) hide)
     )
@@
     (instances
       (project "krecek-0.9"
-        (path "/8888f37b-ecc2-47df-8824-4b4e1e726451"
-          (reference "#PWR060") (unit 1)
-        )
         (path "/8888f37b-ecc2-47df-8824-4b4e1e726451/a9ff151a-3813-42b7-837e-58004a43f525"
           (reference "#PWR0111") (unit 1)
@@
   (symbol (lib_id "power:GND") (at 107.95 77.47 0) (unit 1)
     (in_bom yes) (on_board yes) (dnp no) (fields_autoplaced)
-    (property "Reference" "#PWR060" (at 107.95 83.82 0)
+    (property "Reference" "#PWR0110" (at 107.95 83.82 0)
       (effects (font (size 1.27 1.27)) hide)
     )
@@
     (instances
       (project "krecek-0.9"
-        (path "/8888f37b-ecc2-47df-8824-4b4e1e726451"
-          (reference "#PWR060") (unit 1)
-        )
         (path "/8888f37b-ecc2-47df-8824-4b4e1e726451/a9ff151a-3813-42b7-837e-58004a43f525"
           (reference "#PWR0110") (unit 1)
@@
   (symbol (lib_id "Device:C_Polarized_Small") (at 101.6 69.85 0) (unit 1)
     (in_bom yes) (on_board yes) (dnp no) (fields_autoplaced)
-    (property "Reference" "C29" (at 104.775 68.0339 0)
+    (property "Reference" "C80" (at 104.775 68.0339 0)
       (effects (font (size 1.27 1.27)) (justify left))
     )
@@
     (instances
       (project "krecek-0.9"
-        (path "/8888f37b-ecc2-47df-8824-4b4e1e726451/bd29cd8c-9207-416a-90c1-7bdf6b5cfb97"
-          (reference "C29") (unit 1)
-        )
         (path "/8888f37b-ecc2-47df-8824-4b4e1e726451/a9ff151a-3813-42b7-837e-58004a43f525"
           (reference "C80") (unit 1)
@@
   (symbol (lib_id "power:GND") (at 148.59 68.58 270) (unit 1)
     (in_bom yes) (on_board yes) (dnp no) (fields_autoplaced)
-    (property "Reference" "#PWR060" (at 142.24 68.58 0)
+    (property "Reference" "#PWR0109" (at 142.24 68.58 0)
       (effects (font (size 1.27 1.27)) hide)
     )
@@
     (instances
       (project "krecek-0.9"
-        (path "/8888f37b-ecc2-47df-8824-4b4e1e726451"
-          (reference "#PWR060") (unit 1)
-        )
         (path "/8888f37b-ecc2-47df-8824-4b4e1e726451/a9ff151a-3813-42b7-837e-58004a43f525"
           (reference "#PWR0109") (unit 1)

Commit message: Hardware as sent for manufacturing
Parts:
- C80: value 100uF -> 100u
Changed lines of the file:
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@@
   (symbol (lib_id "Device:C_Polarized_Small") (at 101.6 69.85 0) (unit 1)
     (in_bom yes) (on_board yes) (dnp no) (fields_autoplaced)
-    (property "Reference" "C80" (at 104.775 68.0339 0)
+    (property "Reference" "C80" (at 104.14 68.0339 0)
       (effects (font (size 1.27 1.27)) (justify left))
     )
-    (property "Value" "100uF" (at 104.775 70.5739 0)
+    (property "Value" "100u" (at 104.14 70.5739 0)
       (effects (font (size 1.27 1.27)) (justify left))
     )

Commit message: Fix input PMOS orientation (again)
Parts:
- renumbered C80 to C77
Changed lines of the file:
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@@
       (project "krecek-0.9"
         (path "/8888f37b-ecc2-47df-8824-4b4e1e726451/a9ff151a-3813-42b7-837e-58004a43f525"
-          (reference "C81") (unit 1)
+          (reference "C78") (unit 1)
         )
       )
@@
   (symbol (lib_id "power:GND") (at 191.77 78.74 90) (unit 1)
     (in_bom yes) (on_board yes) (dnp no) (fields_autoplaced)
-    (property "Reference" "#PWR0111" (at 198.12 78.74 0)
+    (property "Reference" "#PWR0115" (at 198.12 78.74 0)
       (effects (font (size 1.27 1.27)) hide)
     )
@@
       (project "krecek-0.9"
         (path "/8888f37b-ecc2-47df-8824-4b4e1e726451/a9ff151a-3813-42b7-837e-58004a43f525"
-          (reference "#PWR0111") (unit 1)
+          (reference "#PWR0115") (unit 1)
         )
       )
@@
   (symbol (lib_id "power:GND") (at 107.95 77.47 0) (unit 1)
     (in_bom yes) (on_board yes) (dnp no) (fields_autoplaced)
-    (property "Reference" "#PWR0110" (at 107.95 83.82 0)
+    (property "Reference" "#PWR0114" (at 107.95 83.82 0)
       (effects (font (size 1.27 1.27)) hide)
     )
@@
       (project "krecek-0.9"
         (path "/8888f37b-ecc2-47df-8824-4b4e1e726451/a9ff151a-3813-42b7-837e-58004a43f525"
-          (reference "#PWR0110") (unit 1)
+          (reference "#PWR0114") (unit 1)
         )
       )
@@
   (symbol (lib_id "Device:C_Polarized_Small") (at 101.6 69.85 0) (unit 1)
     (in_bom yes) (on_board yes) (dnp no) (fields_autoplaced)
-    (property "Reference" "C80" (at 104.14 68.0339 0)
+    (property "Reference" "C77" (at 104.14 68.0339 0)
       (effects (font (size 1.27 1.27)) (justify left))
     )
@@
       (project "krecek-0.9"
         (path "/8888f37b-ecc2-47df-8824-4b4e1e726451/a9ff151a-3813-42b7-837e-58004a43f525"
-          (reference "C80") (unit 1)
+          (reference "C77") (unit 1)
         )
       )
@@
   (symbol (lib_id "power:GND") (at 148.59 68.58 270) (unit 1)
     (in_bom yes) (on_board yes) (dnp no) (fields_autoplaced)
-    (property "Reference" "#PWR0109" (at 142.24 68.58 0)
+    (property "Reference" "#PWR0113" (at 142.24 68.58 0)
       (effects (font (size 1.27 1.27)) hide)
     )
@@
       (project "krecek-0.9"
         (path "/8888f37b-ecc2-47df-8824-4b4e1e726451/a9ff151a-3813-42b7-837e-58004a43f525"
-          (reference "#PWR0109") (unit 1)
+          (reference "#PWR0113") (unit 1)
         )
       )
