File: hw/krecek-0.9/sdcard.kicad_sch (KiCad schematic)
At the start: 3 parts, among them J5 Micro_SD_Card_Det1

Commit message: Fix ERC-indicated issues
Parts:
- renumbered C77 to C75
Changed lines of the file:
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@@
 			)
 		)
-		(property "Description" ""
+		(property "Description" "Unpolarized capacitor, small symbol"
 			(at 114.3 69.85 0)
 			(effects
@@
 			(project "krecek-0.9"
 				(path "/8888f37b-ecc2-47df-8824-4b4e1e726451/a9ff151a-3813-42b7-837e-58004a43f525"
-					(reference "C78")
+					(reference "C76")
 					(unit 1)
 				)
@@
 		(dnp no)
 		(fields_autoplaced yes)
-		(property "Reference" "#PWR0115"
+		(property "Reference" "#PWR0110"
 			(at 198.12 78.74 0)
 			(effects
@@
 			)
 		)
-		(property "Description" ""
+		(property "Description" "Power symbol creates a global label with name \"GND\" , ground"
 			(at 191.77 78.74 0)
 			(effects
@@
 			(project "krecek-0.9"
 				(path "/8888f37b-ecc2-47df-8824-4b4e1e726451/a9ff151a-3813-42b7-837e-58004a43f525"
-					(reference "#PWR0115")
+					(reference "#PWR0110")
 					(unit 1)
 				)
@@
 		(dnp no)
 		(fields_autoplaced yes)
-		(property "Reference" "#PWR0114"
+		(property "Reference" "#PWR0109"
 			(at 107.95 83.82 0)
 			(effects
@@
 			)
 		)
-		(property "Description" ""
+		(property "Description" "Power symbol creates a global label with name \"GND\" , ground"
 			(at 107.95 77.47 0)
 			(effects
@@
 			(project "krecek-0.9"
 				(path "/8888f37b-ecc2-47df-8824-4b4e1e726451/a9ff151a-3813-42b7-837e-58004a43f525"
-					(reference "#PWR0114")
+					(reference "#PWR0109")
 					(unit 1)
 				)
@@
 		(dnp no)
 		(fields_autoplaced yes)
-		(property "Reference" "C77"
+		(property "Reference" "C75"
 			(at 104.14 68.0339 0)
 			(effects
@@
 			)
 		)
-		(property "Description" ""
+		(property "Description" "Polarized capacitor, small symbol"
 			(at 101.6 69.85 0)
 			(effects
@@
 			(project "krecek-0.9"
 				(path "/8888f37b-ecc2-47df-8824-4b4e1e726451/a9ff151a-3813-42b7-837e-58004a43f525"
-					(reference "C77")
+					(reference "C75")
 					(unit 1)
 				)
@@
 		(dnp no)
 		(fields_autoplaced yes)
-		(property "Reference" "#PWR0113"
+		(property "Reference" "#PWR0108"
 			(at 142.24 68.58 0)
 			(effects
@@
 			)
 		)
-		(property "Description" ""
+		(property "Description" "Power symbol creates a global label with name \"GND\" , ground"
 			(at 148.59 68.58 0)
 			(effects
@@
 			(project "krecek-0.9"
 				(path "/8888f37b-ecc2-47df-8824-4b4e1e726451/a9ff151a-3813-42b7-837e-58004a43f525"
-					(reference "#PWR0113")
+					(reference "#PWR0108")
 					(unit 1)
 				)
@@
 			)
 		)
-		(property "Description" ""
+		(property "Description" "Micro SD Card Socket with one card detection pin"
 			(at 171.45 66.04 0)
 			(effects

Commit message: Progress on HW design
Parts:
- renumbered C75 to C73
Changed lines of the file:
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@@
 			(project "krecek-0.9"
 				(path "/8888f37b-ecc2-47df-8824-4b4e1e726451/a9ff151a-3813-42b7-837e-58004a43f525"
-					(reference "C76")
+					(reference "C74")
 					(unit 1)
 				)
@@
 		(dnp no)
 		(fields_autoplaced yes)
-		(property "Reference" "#PWR0110"
+		(property "Reference" "#PWR0109"
 			(at 198.12 78.74 0)
 			(effects
@@
 			(project "krecek-0.9"
 				(path "/8888f37b-ecc2-47df-8824-4b4e1e726451/a9ff151a-3813-42b7-837e-58004a43f525"
-					(reference "#PWR0110")
+					(reference "#PWR0109")
 					(unit 1)
 				)
@@
 		(dnp no)
 		(fields_autoplaced yes)
-		(property "Reference" "#PWR0109"
+		(property "Reference" "#PWR0108"
 			(at 107.95 83.82 0)
 			(effects
@@
 			(project "krecek-0.9"
 				(path "/8888f37b-ecc2-47df-8824-4b4e1e726451/a9ff151a-3813-42b7-837e-58004a43f525"
-					(reference "#PWR0109")
+					(reference "#PWR0108")
 					(unit 1)
 				)
@@
 		(dnp no)
 		(fields_autoplaced yes)
-		(property "Reference" "C75"
+		(property "Reference" "C73"
 			(at 104.14 68.0339 0)
 			(effects
@@
 			(project "krecek-0.9"
 				(path "/8888f37b-ecc2-47df-8824-4b4e1e726451/a9ff151a-3813-42b7-837e-58004a43f525"
-					(reference "C75")
+					(reference "C73")
 					(unit 1)
 				)
@@
 		(dnp no)
 		(fields_autoplaced yes)
-		(property "Reference" "#PWR0108"
+		(property "Reference" "#PWR0107"
 			(at 142.24 68.58 0)
 			(effects
@@
 			(project "krecek-0.9"
 				(path "/8888f37b-ecc2-47df-8824-4b4e1e726451/a9ff151a-3813-42b7-837e-58004a43f525"
-					(reference "#PWR0108")
-					(unit 1)
-				)
+					(reference "#PWR0107")
+					(unit 1)
+				)
