File: hw/krecek-0.9/display.kicad_sch (KiCad schematic)
At the start: 7 parts, among them Q4 AO3400A, U14 TSC2046EIRGVR

Commit message: Fix ERC-indicated issues
Parts:
- renumbered C81 to C77, C80 to C78, C51 to C79, C79 to C80, Q4 to Q6

Commit message: Progress on HW design
Parts:
- renumbered C77 to C75, C78 to C76, C79 to C77, C80 to C78, U14 to U13
Changed lines of the file:
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@@
 		(dnp no)
 		(fields_autoplaced yes)
-		(property "Reference" "#PWR0123"
+		(property "Reference" "#PWR0122"
 			(at 76.2 130.81 0)
 			(effects
@@
 			(project "krecek-0.9"
 				(path "/8888f37b-ecc2-47df-8824-4b4e1e726451/1e7e68f1-c5d4-4ff3-9e0f-8d242f7f0b14"
-					(reference "#PWR0123")
+					(reference "#PWR0122")
 					(unit 1)
 				)
@@
 		(dnp no)
 		(fields_autoplaced yes)
-		(property "Reference" "#PWR0124"
+		(property "Reference" "#PWR0123"
 			(at 88.9 130.81 0)
 			(effects
@@
 			(project "krecek-0.9"
 				(path "/8888f37b-ecc2-47df-8824-4b4e1e726451/1e7e68f1-c5d4-4ff3-9e0f-8d242f7f0b14"
-					(reference "#PWR0124")
+					(reference "#PWR0123")
 					(unit 1)
 				)
@@
 		(dnp no)
 		(fields_autoplaced yes)
-		(property "Reference" "C80"
+		(property "Reference" "C78"
 			(at 91.44 132.0863 0)
 			(effects
@@
 			(project "krecek-0.9"
 				(path "/8888f37b-ecc2-47df-8824-4b4e1e726451/1e7e68f1-c5d4-4ff3-9e0f-8d242f7f0b14"
-					(reference "C80")
+					(reference "C78")
 					(unit 1)
 				)
@@
 		(dnp no)
 		(fields_autoplaced yes)
-		(property "Reference" "C78"
+		(property "Reference" "C76"
 			(at 66.04 132.0863 0)
 			(effects
@@
 			(project "krecek-0.9"
 				(path "/8888f37b-ecc2-47df-8824-4b4e1e726451/1e7e68f1-c5d4-4ff3-9e0f-8d242f7f0b14"
-					(reference "C78")
+					(reference "C76")
 					(unit 1)
 				)
@@
 		(dnp no)
 		(fields_autoplaced yes)
-		(property "Reference" "#PWR0116"
+		(property "Reference" "#PWR0115"
 			(at 168.91 90.17 0)
 			(effects
@@
 			(project "krecek-0.9"
 				(path "/8888f37b-ecc2-47df-8824-4b4e1e726451/1e7e68f1-c5d4-4ff3-9e0f-8d242f7f0b14"
-					(reference "#PWR0116")
+					(reference "#PWR0115")
 					(unit 1)
 				)
@@
 		(dnp no)
 		(fields_autoplaced yes)
-		(property "Reference" "#PWR0122"
+		(property "Reference" "#PWR0121"
 			(at 63.5 130.81 0)
 			(effects
@@
 			(project "krecek-0.9"
 				(path "/8888f37b-ecc2-47df-8824-4b4e1e726451/1e7e68f1-c5d4-4ff3-9e0f-8d242f7f0b14"
-					(reference "#PWR0122")
+					(reference "#PWR0121")
 					(unit 1)
 				)
@@
 		(dnp no)
 		(fields_autoplaced yes)
-		(property "Reference" "#PWR0126"
+		(property "Reference" "#PWR0125"
 			(at 63.5 146.05 0)
 			(effects
@@
 			(project "krecek-0.9"
 				(path "/8888f37b-ecc2-47df-8824-4b4e1e726451/1e7e68f1-c5d4-4ff3-9e0f-8d242f7f0b14"
-					(reference "#PWR0126")
+					(reference "#PWR0125")
 					(unit 1)
 				)
@@
 		(dnp no)
 		(fields_autoplaced yes)
-		(property "Reference" "#PWR0119"
+		(property "Reference" "#PWR0118"
 			(at 118.11 102.87 0)
 			(effects
@@
 			(project "krecek-0.9"
 				(path "/8888f37b-ecc2-47df-8824-4b4e1e726451/1e7e68f1-c5d4-4ff3-9e0f-8d242f7f0b14"
-					(reference "#PWR0119")
+					(reference "#PWR0118")
 					(unit 1)
 				)
@@
 		(dnp no)
 		(fields_autoplaced yes)
-		(property "Reference" "#PWR0118"
+		(property "Reference" "#PWR0117"
 			(at 76.2 107.95 0)
 			(effects
@@
 			(project "krecek-0.9"
 				(path "/8888f37b-ecc2-47df-8824-4b4e1e726451/1e7e68f1-c5d4-4ff3-9e0f-8d242f7f0b14"
-					(reference "#PWR0118")
+					(reference "#PWR0117")
 					(unit 1)
 				)
@@
 		(dnp no)
 		(fields_autoplaced yes)
-		(property "Reference" "C77"
+		(property "Reference" "C75"
 			(at 205.74 68.5863 0)
 			(effects
@@
 			(project "krecek-0.9"
 				(path "/8888f37b-ecc2-47df-8824-4b4e1e726451/1e7e68f1-c5d4-4ff3-9e0f-8d242f7f0b14"
-					(reference "C77")
+					(reference "C75")
 					(unit 1)
 				)
@@
 		(dnp no)
 		(fields_autoplaced yes)
-		(property "Reference" "U14"
+		(property "Reference" "U13"
 			(at 129.1941 95.25 0)
 			(effects
@@
 			(project "krecek-0.9"
 				(path "/8888f37b-ecc2-47df-8824-4b4e1e726451/1e7e68f1-c5d4-4ff3-9e0f-8d242f7f0b14"
-					(reference "U14")
+					(reference "U13")
 					(unit 1)
 				)
@@
 		(dnp no)
 		(fields_autoplaced yes)
-		(property "Reference" "#PWR0120"
+		(property "Reference" "#PWR0119"
 			(at 173.99 121.92 0)
 			(effects
@@
 			(project "krecek-0.9"
 				(path "/8888f37b-ecc2-47df-8824-4b4e1e726451/1e7e68f1-c5d4-4ff3-9e0f-8d242f7f0b14"
-					(reference "#PWR0120")
+					(reference "#PWR0119")
 					(unit 1)
 				)
@@
 		(dnp no)
 		(fields_autoplaced yes)
-		(property "Reference" "#PWR0112"
+		(property "Reference" "#PWR0111"
 			(at 158.75 67.31 0)
 			(effects
@@
 			(project "krecek-0.9"
 				(path "/8888f37b-ecc2-47df-8824-4b4e1e726451/1e7e68f1-c5d4-4ff3-9e0f-8d242f7f0b14"
-					(reference "#PWR0112")
+					(reference "#PWR0111")
 					(unit 1)
 				)
@@
 		(dnp no)
 		(fields_autoplaced yes)
-		(property "Reference" "#PWR0128"
+		(property "Reference" "#PWR0127"
 			(at 88.9 146.05 0)
 			(effects
@@
 			(project "krecek-0.9"
 				(path "/8888f37b-ecc2-47df-8824-4b4e1e726451/1e7e68f1-c5d4-4ff3-9e0f-8d242f7f0b14"
-					(reference "#PWR0128")
+					(reference "#PWR0127")
 					(unit 1)
 				)
@@
 		(dnp no)
 		(fields_autoplaced yes)
-		(property "Reference" "#PWR0113"
+		(property "Reference" "#PWR0112"
 			(at 203.2 82.55 0)
 			(effects
@@
 			(project "krecek-0.9"
 				(path "/8888f37b-ecc2-47df-8824-4b4e1e726451/1e7e68f1-c5d4-4ff3-9e0f-8d242f7f0b14"
-					(reference "#PWR0113")
+					(reference "#PWR0112")
 					(unit 1)
 				)
@@
 		(dnp no)
 		(fields_autoplaced yes)
-		(property "Reference" "#PWR0127"
+		(property "Reference" "#PWR0126"
 			(at 76.2 146.05 0)
 			(effects
@@
 			(project "krecek-0.9"
 				(path "/8888f37b-ecc2-47df-8824-4b4e1e726451/1e7e68f1-c5d4-4ff3-9e0f-8d242f7f0b14"
-					(reference "#PWR0127")
+					(reference "#PWR0126")
 					(unit 1)
 				)
@@
 		(dnp no)
 		(fields_autoplaced yes)
-		(property "Reference" "#PWR0115"
+		(property "Reference" "#PWR0114"
 			(at 168.91 87.63 0)
 			(effects
@@
 			(project "krecek-0.9"
 				(path "/8888f37b-ecc2-47df-8824-4b4e1e726451/1e7e68f1-c5d4-4ff3-9e0f-8d242f7f0b14"
-					(reference "#PWR0115")
+					(reference "#PWR0114")
 					(unit 1)
 				)
@@
 		(dnp no)
 		(fields_autoplaced yes)
-		(property "Reference" "#PWR0111"
+		(property "Reference" "#PWR0110"
 			(at 203.2 67.31 0)
 			(effects
@@
 			(project "krecek-0.9"
 				(path "/8888f37b-ecc2-47df-8824-4b4e1e726451/1e7e68f1-c5d4-4ff3-9e0f-8d242f7f0b14"
-					(reference "#PWR0111")
+					(reference "#PWR0110")
 					(unit 1)
 				)
@@
 		(dnp no)
 		(fields_autoplaced yes)
-		(property "Reference" "C79"
+		(property "Reference" "C77"
 			(at 78.74 132.0863 0)
 			(effects
@@
 			(project "krecek-0.9"
 				(path "/8888f37b-ecc2-47df-8824-4b4e1e726451/1e7e68f1-c5d4-4ff3-9e0f-8d242f7f0b14"
-					(reference "C79")
+					(reference "C77")
 					(unit 1)
 				)
@@
 		(dnp no)
 		(fields_autoplaced yes)
-		(property "Reference" "#PWR0125"
+		(property "Reference" "#PWR0124"
 			(at 128.27 142.24 0)
 			(effects
@@
 			(project "krecek-0.9"
 				(path "/8888f37b-ecc2-47df-8824-4b4e1e726451/1e7e68f1-c5d4-4ff3-9e0f-8d242f7f0b14"
-					(reference "#PWR0125")
+					(reference "#PWR0124")
 					(unit 1)
 				)
@@
 		(dnp no)
 		(fields_autoplaced yes)
-		(property "Reference" "#PWR0117"
+		(property "Reference" "#PWR0116"
 			(at 127 101.6 0)
 			(effects
@@
 			(project "krecek-0.9"
 				(path "/8888f37b-ecc2-47df-8824-4b4e1e726451/1e7e68f1-c5d4-4ff3-9e0f-8d242f7f0b14"
-					(reference "#PWR0117")
+					(reference "#PWR0116")
 					(unit 1)
 				)
@@
 		(dnp no)
 		(fields_autoplaced yes)
-		(property "Reference" "#PWR0114"
+		(property "Reference" "#PWR0113"
 			(at 158.75 85.09 0)
 			(effects
@@
 			(project "krecek-0.9"
 				(path "/8888f37b-ecc2-47df-8824-4b4e1e726451/1e7e68f1-c5d4-4ff3-9e0f-8d242f7f0b14"
-					(reference "#PWR0114")
+					(reference "#PWR0113")
 					(unit 1)
 				)
@@
 		(dnp no)
 		(fields_autoplaced yes)
-		(property "Reference" "#PWR0121"
+		(property "Reference" "#PWR0120"
 			(at 118.11 125.73 0)
 			(effects
@@
 			(project "krecek-0.9"
 				(path "/8888f37b-ecc2-47df-8824-4b4e1e726451/1e7e68f1-c5d4-4ff3-9e0f-8d242f7f0b14"
-					(reference "#PWR0121")
-					(unit 1)
-				)
+					(reference "#PWR0120")
+					(unit 1)
+				)

Commit message: Route more parts of the board
Parts:
- removed Q6: AO3400A, Package_TO_SOT_SMD:SOT-23, symbol Transistor_FET:AO3400A
Connections:
- net GND: now also FPC1.11, FPC1.12, FPC1.13, FPC1.14
