File: hw/krecek/power.kicad_sch (KiCad schematic)
At the start: 57 parts, among them J3 USB_C_Receptacle_USB2.0, Q1 AO3401A, Q2 AO3401A, Q3 AO3400A, U4 AMS1117-3.3, U5 JST-PH-2P, U6 BQ24040DSQR, U7 AMS1117-3.3, U8 AMS1117-3.3, U9 TPS63000

Commit message: Rename hw/krecek-0.9 to just hw/krecek
Parts:
- C45, C46: value 100n -> 100p; LCSC Part C307331 -> C1546
- renumbered R3 to R15, R3 to R16
