File: hw/krecek/radio.kicad_sch (KiCad schematic)
At the start: 10 parts, among them J4 U.FL, U11 CC1101RGPR, U14 BW21S5011A01TF

Commit message: Rename hw/krecek-0.9 to just hw/krecek
Parts:
- renumbered C6 to C54, C6 to C55, C6 to C56
Changed lines of the file:
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@@
 (kicad_sch
-	(version 20231120)
+	(version 20250114)
 	(generator "eeschema")
-	(generator_version "8.0")
+	(generator_version "9.0")
 	(paper "A4")
 	(title_block
@@
 		(shape input)
 		(at 58.42 82.55 180)
-		(fields_autoplaced yes)
 		(effects
 			(font
@@
 		(shape input)
 		(at 58.42 77.47 180)
-		(fields_autoplaced yes)
 		(effects
 			(font
@@
 		(shape input)
 		(at 58.42 80.01 180)
-		(fields_autoplaced yes)
 		(effects
 			(font
@@
 		(shape input)
 		(at 58.42 95.25 180)
-		(fields_autoplaced yes)
 		(effects
 			(font
@@
 		(shape output)
 		(at 58.42 85.09 180)
-		(fields_autoplaced yes)
 		(effects
 			(font
@@
 		)
 		(instances
-			(project "krecek-0.9"
+			(project "krecek"
 				(path "/8888f37b-ecc2-47df-8824-4b4e1e726451/40971852-55ba-4d75-a9d8-2b5de9b08cbd"
 					(reference "#PWR081")
@@
 		)
 		(instances
-			(project "krecek-0.9"
+			(project "krecek"
 				(path "/8888f37b-ecc2-47df-8824-4b4e1e726451/40971852-55ba-4d75-a9d8-2b5de9b08cbd"
 					(reference "#PWR090")
@@
 		(dnp no)
 		(fields_autoplaced yes)
-		(property "Reference" "C6"
+		(property "Reference" "C54"
 			(at 66.04 43.1863 0)
 			(effects
@@
 				)
 			)
-			(project "krecek-0.9"
+			(project "krecek"
 				(path "/8888f37b-ecc2-47df-8824-4b4e1e726451/40971852-55ba-4d75-a9d8-2b5de9b08cbd"
 					(reference "C54")
@@
 		)
 		(instances
-			(project "krecek-0.9"
+			(project "krecek"
 				(path "/8888f37b-ecc2-47df-8824-4b4e1e726451/40971852-55ba-4d75-a9d8-2b5de9b08cbd"
 					(reference "#PWR088")
@@
 		)
 		(instances
-			(project "krecek-0.9"
+			(project "krecek"
 				(path "/8888f37b-ecc2-47df-8824-4b4e1e726451/40971852-55ba-4d75-a9d8-2b5de9b08cbd"
 					(reference "#PWR087")
@@
 		)
 		(instances
-			(project "krecek-0.9"
+			(project "krecek"
 				(path "/8888f37b-ecc2-47df-8824-4b4e1e726451/40971852-55ba-4d75-a9d8-2b5de9b08cbd"
 					(reference "#PWR084")
@@
 		)
 		(instances
-			(project "krecek-0.9"
+			(project "krecek"
 				(path "/8888f37b-ecc2-47df-8824-4b4e1e726451/40971852-55ba-4d75-a9d8-2b5de9b08cbd"
 					(reference "AE1")
@@
 		)
 		(instances
-			(project "krecek-0.9"
+			(project "krecek"
 				(path "/8888f37b-ecc2-47df-8824-4b4e1e726451/40971852-55ba-4d75-a9d8-2b5de9b08cbd"
 					(reference "#PWR089")
@@
 		(dnp no)
 		(fields_autoplaced yes)
-		(property "Reference" "C6"
+		(property "Reference" "C56"
 			(at 91.44 43.1863 0)
 			(effects
@@
 				)
 			)
-			(project "krecek-0.9"
+			(project "krecek"
 				(path "/8888f37b-ecc2-47df-8824-4b4e1e726451/40971852-55ba-4d75-a9d8-2b5de9b08cbd"
 					(reference "C56")
@@
 		(dnp no)
 		(fields_autoplaced yes)
-		(property "Reference" "#PWR056"
+		(property "Reference" "#PWR082"
 			(at 76.2 58.42 0)
 			(effects
@@
 				)
 			)
-			(project "krecek-0.9"
+			(project "krecek"
 				(path "/8888f37b-ecc2-47df-8824-4b4e1e726451/40971852-55ba-4d75-a9d8-2b5de9b08cbd"
 					(reference "#PWR082")
@@
 		)
 		(instances
-			(project "krecek-0.9"
+			(project "krecek"
 				(path "/8888f37b-ecc2-47df-8824-4b4e1e726451/40971852-55ba-4d75-a9d8-2b5de9b08cbd"
 					(reference "U11")
@@
 		)
 		(instances
-			(project "krecek-0.9"
+			(project "krecek"
 				(path "/8888f37b-ecc2-47df-8824-4b4e1e726451/40971852-55ba-4d75-a9d8-2b5de9b08cbd"
 					(reference "C63")
@@
 		(dnp no)
 		(fields_autoplaced yes)
-		(property "Reference" "C6"
+		(property "Reference" "C55"
 			(at 78.74 43.1863 0)
 			(effects
@@
 				)
 			)
-			(project "krecek-0.9"
+			(project "krecek"
 				(path "/8888f37b-ecc2-47df-8824-4b4e1e726451/40971852-55ba-4d75-a9d8-2b5de9b08cbd"
 					(reference "C55")
@@
 		)
 		(instances
-			(project "krecek-0.9"
+			(project "krecek"
 				(path "/8888f37b-ecc2-47df-8824-4b4e1e726451/40971852-55ba-4d75-a9d8-2b5de9b08cbd"
 					(reference "C57")
@@
 		)
 		(instances
-			(project "krecek-0.9"
+			(project "krecek"
 				(path "/8888f37b-ecc2-47df-8824-4b4e1e726451/40971852-55ba-4d75-a9d8-2b5de9b08cbd"
 					(reference "J4")
@@
 		)
 		(instances
-			(project "krecek-0.9"
+			(project "krecek"
 				(path "/8888f37b-ecc2-47df-8824-4b4e1e726451/40971852-55ba-4d75-a9d8-2b5de9b08cbd"
 					(reference "R36")
