File: hw/krecek/krecek.kicad_sch (KiCad schematic)
At the start: 9 parts

Commit message: Audio-related HW fixes
Other:
- sheet Audio ports: added MCLK; removed none
- sheet RP2040 ports: added DSP_{MCLK}; removed none
