File: hw/krecek/rp2040.kicad_sch (KiCad schematic)
At the start: 40 parts, among them J1 DAP, J2 AUX, SW1 SW_Push, U1 RP2040, U2 RP2040, U3 W25Q128JVS, Y1 12MHz

Commit message: Rename hw/krecek-0.9 to just hw/krecek
Parts:
- renumbered C6 to C1, C6 to C10, C6 to C11, C6 to C12, C6 to C13, C6 to C14, C6 to C15, C6 to C16, C6 to C17, C6 to C18, C6 to C19, C6 to C2, C6 to C20, C6 to C21, C6 to C22, C6 to C3, C6 to C4, C6 to C5, C6 to C7, C6 to C8, C6 to C9

Commit message: Audio-related HW fixes
Connections:
- net DSP_{MCLK}: now reaches U1.34 (GPIO22)
- no-connect marks 9 -> 8
Changed lines of the file:
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@@
-	)
-	(no_connect
-		(at 101.6 109.22)
 	)
 	(no_connect
@@
 		)
 	)
+	(hierarchical_label "DSP_{MCLK}"
+		(shape output)
+		(at 101.6 109.22 0)
+		(effects
+			(font
+				(size 1.27 1.27)
+			)
+			(justify left)
+		)
+	)
