File: hw/krecek/audio.kicad_sch (KiCad schematic)
At the start: 23 parts, among them CN1 PJ-313B6-B, Q1 PT334, Q2 AO3400A, U10 NAU88C22YG

Commit message: Rename hw/krecek-0.9 to just hw/krecek
Parts:
- renumbered C6 to C41, C6 to C42, C6 to C43, C7 to C44, C7 to C47, C7 to C49, C6 to C51, D1 to D6, D1 to D7, Q1 to Q4, Q2 to Q5, R3 to R31, R3 to R32, R3 to R33, R3 to R34

Commit message: Audio-related HW fixes
Parts:
- added C58: 1u, Capacitor_SMD:C_0402_1005Metric, symbol Device:C_Small
Connections:
- net GND: now also C58.2
- net IR: now also U10.2 (LMICN); no longer U10.19 (LAUXIN)
- net SCLK: no longer U10.11 (MCLK)
- net at U10.1 (LMICP): now also C58.1
- new net MCLK: U10.11 (MCLK)
- no-connect marks 8 -> 7
Changed lines of the file:
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@@
 	)
 	(junction
-		(at 66.04 157.48)
-		(diameter 0)
-		(color 0 0 0 0)
-	)
-	(junction
 		(at 50.8 152.4)
 		(diameter 0)
@@
 	)
 	(no_connect
-		(at 76.2 121.92)
-	)
-	(no_connect
 		(at 76.2 137.16)
 	)
@@
 	)
 	(no_connect
-		(at 76.2 119.38)
+		(at 76.2 114.3)
 	)
 	(no_connect
@@
 	(wire
 		(pts
-			(xy 63.5 157.48) (xy 66.04 157.48)
-		)
-		(stroke
-			(width 0)
-			(type default)
-		)
-	)
-	(wire
-		(pts
 			(xy 138.43 132.08) (xy 152.4 132.08)
 		)
@@
 	(wire
 		(pts
-			(xy 76.2 170.18) (xy 66.04 170.18)
-		)
-		(stroke
-			(width 0)
-			(type default)
-		)
-	)
-	(wire
-		(pts
-			(xy 66.04 170.18) (xy 66.04 157.48)
+			(xy 76.2 170.18) (xy 63.5 170.18)
 		)
 		(stroke
@@
 	(wire
 		(pts
-			(xy 66.04 157.48) (xy 76.2 157.48)
+			(xy 63.5 157.48) (xy 76.2 157.48)
 		)
 		(stroke
@@
 	(wire
 		(pts
-			(xy 64.77 114.3) (xy 76.2 114.3)
+			(xy 64.77 119.38) (xy 76.2 119.38)
 		)
 		(stroke
@@
 	(wire
 		(pts
+			(xy 72.39 121.92) (xy 76.2 121.92)
+		)
+		(stroke
+			(width 0)
+			(type default)
+		)
+	)
+	(wire
+		(pts
 			(xy 152.4 38.1) (xy 190.5 38.1)
 		)
@@
 	)
 	(label "IR"
-		(at 64.77 114.3 0)
+		(at 64.77 119.38 0)
 		(effects
 			(font
@@
 		)
 	)
+	(hierarchical_label "MCLK"
+		(shape input)
+		(at 63.5 170.18 180)
+		(effects
+			(font
+				(size 1.27 1.27)
+			)
+			(justify right)
+		)
+	)
 	(hierarchical_label "LRCK"
 		(shape input)
@@
 		(on_board yes)
 		(dnp no)
-		(fields_autoplaced yes)
 		(property "Reference" "#PWR065"
 			(at 165.1 78.74 0)
@@
 	)
 	(symbol
+		(lib_id "power:GND")
+		(at 67.31 121.92 270)
+		(unit 1)
+		(exclude_from_sim no)
+		(in_bom yes)
+		(on_board yes)
+		(dnp no)
+		(fields_autoplaced yes)
+		(property "Reference" "#PWR0129"
+			(at 60.96 121.92 0)
+			(effects
+				(font
+					(size 1.27 1.27)
+				)
+				(hide yes)
+			)
+		)
+		(property "Value" "GND"
+			(at 63.5 121.9199 90)
+			(effects
+				(font
+					(size 1.27 1.27)
+				)
+				(justify right)
+			)
+		)
+		(property "Footprint" ""
+			(at 67.31 121.92 0)
+			(effects
+				(font
+					(size 1.27 1.27)
+				)
+				(hide yes)
+			)
+		)
+		(property "Datasheet" ""
+			(at 67.31 121.92 0)
+			(effects
+				(font
+					(size 1.27 1.27)
+				)
+				(hide yes)
+			)
+		)
+		(property "Description" "Power symbol creates a global label with name \"GND\" , ground"
+			(at 67.31 121.92 0)
+			(effects
+				(font
+					(size 1.27 1.27)
+				)
+				(hide yes)
+			)
+		)
+		(pin "1"
+		)
+		(instances
+			(project "krecek"
+				(path "/8888f37b-ecc2-47df-8824-4b4e1e726451/a7733ec7-68c7-444f-aac5-8a965be5cbce"
+					(reference "#PWR0129")
+					(unit 1)
+				)
+			)
+		)
+	)
+	(symbol
 		(lib_id "Device:C_Small")
 		(at 101.6 76.2 0)
@@
 					(unit 1)
 				)
+			)
+		)
+	)
+	(symbol
+		(lib_id "Device:C_Small")
+		(at 69.85 121.92 270)
+		(unit 1)
+		(exclude_from_sim no)
+		(in_bom yes)
+		(on_board yes)
+		(dnp no)
+		(fields_autoplaced yes)
+		(property "Reference" "C58"
+			(at 69.8436 115.57 90)
+			(effects
+				(font
+					(size 1.27 1.27)
+				)
+			)
+		)
+		(property "Value" "1u"
+			(at 69.8436 118.11 90)
+			(effects
+				(font
+					(size 1.27 1.27)
+				)
+			)
+		)
+		(property "Footprint" "Capacitor_SMD:C_0402_1005Metric"
+			(at 69.85 121.92 0)
+			(effects
+				(font
+					(size 1.27 1.27)
+				)
+				(hide yes)
+			)
+		)
+		(property "Datasheet" "~"
+			(at 69.85 121.92 0)
+			(effects
+				(font
+					(size 1.27 1.27)
+				)
+				(hide yes)
+			)
+		)
+		(property "Description" "Unpolarized capacitor, small symbol"
+			(at 69.85 121.92 0)
+			(effects
+				(font
+					(size 1.27 1.27)
+				)
+				(hide yes)
+			)
+		)
+		(property "LCSC Part" "C52923"
+			(at 69.85 121.92 0)
+			(effects
+				(font
+					(size 1.27 1.27)
+				)
+				(hide yes)
+			)
+		)
+		(pin "1"
+		)
+		(pin "2"
+		)
+		(instances
+			(project "krecek"
+				(path "/8888f37b-ecc2-47df-8824-4b4e1e726451/a7733ec7-68c7-444f-aac5-8a965be5cbce"
+					(reference "C58")
+					(unit 1)
+				)

Commit message: Use audio socket with correct depth
Parts:
- removed CN1: PJ-313B6-B, LCSC:AUDIO-TH_PJ-313B6-B, symbol LCSC:PJ-313B6-B
- added CN1: PJ-320D, LCSC:AUDIO-SMD_PJ-320D, symbol LCSC:PJ-320D
Connections:
- net GND: now also CN1.3
- net HP_{LEFT}: now also CN1.1
- net HP_{RIGHT}: now also CN1.2
- net HP_{SENSE}: now also CN1.4
