File: hw/krecek/krecek.kicad_pcb (KiCad board)
At the start: 4 copper layers, 152.4 x 63.5 mm, 163 parts, among them CN1 PJ-313B6-B, J1 DAP, J2 AUX, J3 USB_C_Receptacle_USB2.0, J4 U.FL, J5 Micro_SD_Card_Det1, Q1 AO3401A, Q2 AO3401A, Q3 AO3400A, Q4 PT334, Q5 AO3400A, SW1 SW_Push, SW5 TM-2023, U1 RP2040, U10 NAU88C22YG, U11 CC1101RGPR, U12 FlatJoyCon, U13 TSC2046EIRGVR, U14 BW21S5011A01TF, U2 RP2040, U3 W25Q128JVS, U4 AMS1117-3.3, U5 JST-PH-2P, U6 BQ24040DSQR, U7 AMS1117-3.3, U8 AMS1117-3.3, U9 TPS63000, Y1 12MHz

Commit message: Use audio socket with correct depth
Parts:
- added C45: 100p, Capacitor_SMD:C_0402_1005Metric, F.Cu at (91.9, 48.5)
- added C46: 100p, Capacitor_SMD:C_0402_1005Metric, F.Cu at (88.6, 48.0)
- added C58: 1u, Capacitor_SMD:C_0402_1005Metric, F.Cu at (162.5, 85.4)
- CN1: value PJ-313B6-B -> PJ-320D; footprint LCSC:AUDIO-TH_PJ-313B6-B -> LCSC:AUDIO-SMD_PJ-320D
- moved CN1 32.4 mm to (165.4, 13.8), turned to 0 degrees
- moved R33 8.58 mm to (151.9, 82.8)
- moved C44 6.56 mm to (151.9, 83.8)
- moved R15 0.51 mm to (91.9, 49.5)
Connections:
- U1 pad 34: unconnected-(U1-GPIO22-Pad34) -> /Audio/MCLK
- U10 pad 1: unconnected-(U10-LMICP-Pad1) -> Net-(U10-LMICP)
- U10 pad 11: /Audio/SCLK -> /Audio/MCLK
- U10 pad 19: /Audio/IR -> unconnected-(U10-LAUXIN-Pad19)
- U10 pad 2: unconnected-(U10-LMICN-Pad2) -> /Audio/IR
Routing:
- net /Audio/MCLK: track 0.00 -> 67.6 mm, vias 0 -> 2
- net +3.3VA: track 58.7 -> 30.7 mm
- net Net-(Q4-C): track 72.1 -> 63.5 mm, vias 2 -> 1
- net Net-(U10-LMICP): track 0.00 -> 5.84 mm, vias 0 -> 2
- net GND: track 141.8 -> 146.2 mm, vias 204 -> 208
- net /Audio/SCLK: track 66.0 -> 63.7 mm
- net /Audio/DAC: track 54.8 -> 53.6 mm
- net /RP2040/XIN2: track 23.6 -> 24.4 mm
- net /Audio/ADC: track 55.1 -> 54.3 mm
- net /Audio/IR: track 5.82 -> 6.35 mm, vias 0 -> 2
